Commit message: better sim performance

File: src/robot_description/dual_arm_description/urdf/links/dual_arm_links.xacro (robot description, xacro)
@@ -22,5 +22,5 @@
       <origin xyz="-0.00277529 -0.000698397 -0.432554" rpy="0 0 -1.5708"/>
       <geometry>
-        <mesh filename="package://dual_arm_description/meshes/visual/b_base.stl"/>
+        <mesh filename="package://dual_arm_description/meshes/collision/b_base.stl"/>
       </geometry>
     </collision>
@@ -37,5 +37,5 @@
       <origin xyz="0.070373 -0.000705351 -0.431099" rpy="0 0 -1.5708"/>
       <geometry>
-        <mesh filename="package://dual_arm_description/meshes/visual/f_base.stl"/>
+        <mesh filename="package://dual_arm_description/meshes/collision/f_base.stl"/>
       </geometry>
     </collision>
@@ -62,5 +62,5 @@
       <origin xyz="3.95689e-06 -0.151502 0.42041" rpy="0 0 -1.5708"/>
       <geometry>
-        <mesh filename="package://dual_arm_description/meshes/visual/urdf_r_shoulder_plate.stl"/>
+        <mesh filename="package://dual_arm_description/meshes/collision/urdf_r_shoulder_plate.stl"/>
       </geometry>
     </collision>
@@ -77,5 +77,5 @@
       <origin xyz="3.95689e-06 0.153498 0.42041" rpy="0 0 -1.5708"/>
       <geometry>
-        <mesh filename="package://dual_arm_description/meshes/visual/urdf_l_shoulder_plate.stl"/>
+        <mesh filename="package://dual_arm_description/meshes/collision/urdf_l_shoulder_plate.stl"/>
       </geometry>
     </collision>
@@ -92,5 +92,5 @@
       <origin xyz="3.95689e-06 -1.69581e-06 -0.171" rpy="0 0 -1.5708"/>
       <geometry>
-        <mesh filename="package://dual_arm_description/meshes/visual/simplified_torso.stl"/>
+        <mesh filename="package://dual_arm_description/meshes/collision/simplified_torso.stl"/>
       </geometry>
     </collision>
@@ -107,5 +107,5 @@
       <origin xyz="0.00657135 -1.69581e-06 0.631" rpy="0 0 -1.5708"/>
       <geometry>
-        <mesh filename="package://dual_arm_description/meshes/visual/head.stl"/>
+        <mesh filename="package://dual_arm_description/meshes/collision/head.stl"/>
       </geometry>
     </collision>
@@ -132,5 +132,5 @@
       <origin xyz="-0.00130076 0.0502746 -6.96176e-06" rpy="0 0 -1.5708"/>
       <geometry>
-        <mesh filename="package://dual_arm_description/meshes/visual/l_shoulder.stl"/>
+        <mesh filename="package://dual_arm_description/meshes/collision/l_shoulder.stl"/>
       </geometry>
     </collision>
@@ -154,5 +154,5 @@
       <origin xyz="-0.0256703 0.015852 -0.0899016" rpy="0 0.174533 -1.5708"/>
       <geometry>
-        <mesh filename="package://dual_arm_description/meshes/visual/l_upper_arm.stl"/>
+        <mesh filename="package://dual_arm_description/meshes/collision/l_upper_arm.stl"/>
       </geometry>
     </collision>
@@ -176,5 +176,5 @@
       <origin xyz="1.15439e-05 0.000331628 -0.0512953" rpy="0 0 -1.57079"/>
       <geometry>
-        <mesh filename="package://dual_arm_description/meshes/visual/l_elbow.stl"/>
+        <mesh filename="package://dual_arm_description/meshes/collision/l_elbow.stl"/>
       </geometry>
     </collision>
@@ -198,5 +198,5 @@
       <origin xyz="0.00466961 -0.0254855 -0.0842108" rpy="0 0 -1.5708"/>
       <geometry>
-        <mesh filename="package://dual_arm_description/meshes/visual/l_upper_forearm.stl"/>
+        <mesh filename="package://dual_arm_description/meshes/collision/l_upper_forearm.stl"/>
       </geometry>
     </collision>
@@ -220,5 +220,5 @@
       <origin xyz="0.00198299 4.28405e-08 -0.0340631" rpy="0 0 -1.57079"/>
       <geometry>
-        <mesh filename="package://dual_arm_description/meshes/visual/l_lower_forearm.stl"/>
+        <mesh filename="package://dual_arm_description/meshes/collision/l_lower_forearm.stl"/>
       </geometry>
     </collision>
@@ -242,5 +242,5 @@
       <origin xyz="-0.0219314 4.45962e-06 -0.0434653" rpy="0 0 -1.5708"/>
       <geometry>
-        <mesh filename="package://dual_arm_description/meshes/visual/l_wrist.stl"/>
+        <mesh filename="package://dual_arm_description/meshes/collision/l_wrist.stl"/>
       </geometry>
     </collision>
@@ -267,5 +267,5 @@
       <origin xyz="-0.00130076 -0.0502746 -6.95902e-06" rpy="0 0 -1.5708"/>
       <geometry>
-        <mesh filename="package://dual_arm_description/meshes/visual/r_shoulder.stl"/>
+        <mesh filename="package://dual_arm_description/meshes/collision/r_shoulder.stl"/>
       </geometry>
     </collision>
@@ -289,5 +289,5 @@
       <origin xyz="-0.0256704 -0.0158521 -0.0899019" rpy="0 -0.174533 -1.5708"/>
       <geometry>
-        <mesh filename="package://dual_arm_description/meshes/visual/r_upper_arm.stl"/>
+        <mesh filename="package://dual_arm_description/meshes/collision/r_upper_arm.stl"/>
       </geometry>
     </collision>
@@ -311,5 +311,5 @@
       <origin xyz="1.16036e-05 -0.000331582 -0.0512953" rpy="0 0 -1.57079"/>
       <geometry>
-        <mesh filename="package://dual_arm_description/meshes/visual/r_elbow.stl"/>
+        <mesh filename="package://dual_arm_description/meshes/collision/r_elbow.stl"/>
       </geometry>
     </collision>
@@ -333,5 +333,5 @@
       <origin xyz="0.00466989 0.0254856 -0.0842107" rpy="0 0 -1.5708"/>
       <geometry>
-        <mesh filename="package://dual_arm_description/meshes/visual/r_upper_forearm.stl"/>
+        <mesh filename="package://dual_arm_description/meshes/collision/r_upper_forearm.stl"/>
       </geometry>
     </collision>
@@ -355,5 +355,5 @@
       <origin xyz="0.00198295 -9.2499e-09 -0.0340632" rpy="0 0 -1.57079"/>
       <geometry>
-        <mesh filename="package://dual_arm_description/meshes/visual/r_lower_forearm.stl"/>
+        <mesh filename="package://dual_arm_description/meshes/collision/r_lower_forearm.stl"/>
       </geometry>
     </collision>
@@ -377,5 +377,5 @@
       <origin xyz="-0.0219316 -4.59044e-06 -0.0434653" rpy="0 0 -1.5708"/>
       <geometry>
-        <mesh filename="package://dual_arm_description/meshes/visual/r_wrist.stl"/>
+        <mesh filename="package://dual_arm_description/meshes/collision/r_wrist.stl"/>
       </geometry>
     </collision>
@@ -402,5 +402,5 @@
       <origin xyz="0.0019136 0.053458 -9.14342e-09" rpy="0 0 -1.5708"/>
       <geometry>
-        <mesh filename="package://dual_arm_description/meshes/visual/hip.stl"/>
+        <mesh filename="package://dual_arm_description/meshes/collision/hip.stl"/>
       </geometry>
     </collision>
@@ -424,5 +424,5 @@
       <origin xyz="-0.0258673 0.0015371 -0.113387" rpy="0 0 -1.5708"/>
       <geometry>
-        <mesh filename="package://dual_arm_description/meshes/visual/l_upper_femur.stl"/>
+        <mesh filename="package://dual_arm_description/meshes/collision/l_upper_femur.stl"/>
       </geometry>
     </collision>
@@ -446,5 +446,5 @@
       <origin xyz="5.81796e-09 0.00391138 -0.0715537" rpy="0 0 -1.5708"/>
       <geometry>
-        <mesh filename="package://dual_arm_description/meshes/visual/lower_femur.stl"/>
+        <mesh filename="package://dual_arm_description/meshes/collision/lower_femur.stl"/>
       </geometry>
     </collision>
@@ -468,5 +468,5 @@
       <origin xyz="0.0302813 -0.054 -0.44863" rpy="0 0 -1.5708"/>
       <geometry>
-        <mesh filename="package://dual_arm_description/meshes/visual/shoe.stl"/>
+        <mesh filename="package://dual_arm_description/meshes/collision/shoe.stl"/>
       </geometry>
     </collision>
@@ -483,5 +483,5 @@
       <origin xyz="0.0301364 -0.054 -0.444982" rpy="0 0 -1.5708"/>
       <geometry>
-        <mesh filename="package://dual_arm_description/meshes/visual/foot.stl"/>
+        <mesh filename="package://dual_arm_description/meshes/collision/foot.stl"/>
       </geometry>
     </collision>
@@ -498,5 +498,5 @@
       <origin xyz="0.000699427 -0.042918 -0.182556" rpy="0 0 -1.5708"/>
       <geometry>
-        <mesh filename="package://dual_arm_description/meshes/visual/l_tibia.stl"/>
+        <mesh filename="package://dual_arm_description/meshes/collision/l_tibia.stl"/>
       </geometry>
     </collision>
@@ -530,5 +530,5 @@
       <origin xyz="0.00191336 -0.058458 3.03756e-05" rpy="3.12572 0 1.5708"/>
       <geometry>
-        <mesh filename="package://dual_arm_description/meshes/visual/hip.stl"/>
+        <mesh filename="package://dual_arm_description/meshes/collision/hip.stl"/>
       </geometry>
     </collision>
@@ -552,5 +552,5 @@
       <origin xyz="-0.0258608 -0.00171122 -0.11336" rpy="0 -0.00155 -1.5708"/>
       <geometry>
-        <mesh filename="package://dual_arm_description/meshes/visual/r_upper_femur.stl"/>
+        <mesh filename="package://dual_arm_description/meshes/collision/r_upper_femur.stl"/>
       </geometry>
     </collision>
@@ -574,5 +574,5 @@
       <origin xyz="1.00366e-08 -0.00391138 -0.0715537" rpy="0 0 1.5708"/>
       <geometry>
-        <mesh filename="package://dual_arm_description/meshes/visual/lower_femur.stl"/>
+        <mesh filename="package://dual_arm_description/meshes/collision/lower_femur.stl"/>
       </geometry>
     </collision>
@@ -596,5 +596,5 @@
       <origin xyz="0.000426339 0.0429179 -0.182557" rpy="-0.00149587 0 -1.5708"/>
       <geometry>
-        <mesh filename="package://dual_arm_description/meshes/visual/r_tibia.stl"/>
+        <mesh filename="package://dual_arm_description/meshes/collision/r_tibia.stl"/>
       </geometry>
     </collision>
@@ -611,5 +611,5 @@
       <origin xyz="0.0296101 0.056 -0.448675" rpy="-0.00149587 0 -1.5708"/>
       <geometry>
-        <mesh filename="package://dual_arm_description/meshes/visual/shoe.stl"/>
+        <mesh filename="package://dual_arm_description/meshes/collision/shoe.stl"/>
       </geometry>
     </collision>
@@ -626,5 +626,5 @@
       <origin xyz="0.0294707 0.056 -0.445027" rpy="-0.00149587 0 -1.5708"/>
       <geometry>
-        <mesh filename="package://dual_arm_description/meshes/visual/foot.stl"/>
+        <mesh filename="package://dual_arm_description/meshes/collision/foot.stl"/>
       </geometry>
     </collision>
