Commit message: Simplify urdf for gazebo

File: src/robot_description/dual_arm_description/urdf/joints/dual_arm_joints.xacro (robot description, xacro)
@@ -92,87 +92,15 @@
     <limit effort="10" velocity="10" lower="-1.5708" upper="1.5708"/>
   </joint>
-<joint name="left_ankle_pitch_joint_2" type="fixed">
-    <origin xyz="-3.747e-16 -0.395 0.03" rpy="-3.14159 3.08616e-14 2.63855e-14"/>
-    <parent link="urdf_l_tibia_assembly"/>
-    <child link="ankle_assembly"/>
-    <axis xyz="0 0 1"/>
-    <limit effort="10" velocity="10" lower="-0.785398" upper="0.785398"/>
+  <!-- Left leg: single box replacing 6 links + 12 joints -->
+  <joint name="left_leg_joint" type="fixed">
+    <origin xyz="-0.175 0.055 -0.858" rpy="0 0 0"/>
+    <parent link="urdf_base"/>
+    <child link="left_leg_link"/>
   </joint>
-<joint name="left_ankle_pitch_joint" type="fixed">
-    <origin xyz="-3.747e-16 -0.395 0.03" rpy="-3.14159 3.08616e-14 2.63855e-14"/>
-    <parent link="urdf_l_tibia_assembly"/>
-    <child link="ankle_assembly_2"/>
-    <axis xyz="0 0 1"/>
-    <limit effort="10" velocity="10" lower="-0.785398" upper="0.785398"/>
-  </joint>
-<joint name="left_knee_joint" type="fixed">
-    <origin xyz="-0.055 8.60423e-16 -0.113" rpy="1.5708 1.15516e-14 1.5708"/>
-    <parent link="urdf_lower_femur_assembly"/>
-    <child link="urdf_l_tibia_assembly"/>
-    <axis xyz="0 0 1"/>
-    <limit effort="10" velocity="10" lower="0" upper="1.5708"/>
-  </joint>
-<joint name="left_hip_yaw_joint" type="fixed">
-    <origin xyz="2.77556e-17 -0.217 0.0551145" rpy="-1.5708 -2.56711e-31 -1.62214e-31"/>
-    <parent link="urdf_l_upper_femur_assembly"/>
-    <child link="urdf_lower_femur_assembly"/>
-    <axis xyz="0 0 1"/>
-    <limit effort="10" velocity="10" lower="-1.5708" upper="1.5708"/>
-  </joint>
-<joint name="left_hip_roll_joint" type="fixed">
-    <origin xyz="0.055 3.33067e-16 -0.073" rpy="-1.43744e-16 -1.5708 0"/>
-    <parent link="urdf_hip_assembly"/>
-    <child link="urdf_l_upper_femur_assembly"/>
-    <axis xyz="0 0 1"/>
-    <limit effort="10" velocity="10" lower="-3.14159" upper="0.349066"/>
-  </joint>
-<joint name="left_hip_pitch_joint" type="fixed">
-    <origin xyz="-0.111301 0.0333466 -0.46826" rpy="1.5708 4.63554e-15 1.5708"/>
+  <!-- Right leg: single box replacing 6 links + 12 joints -->
+  <joint name="right_leg_joint" type="fixed">
+    <origin xyz="0.177 0.058 -0.858" rpy="0 0 0"/>
     <parent link="urdf_base"/>
-    <child link="urdf_hip_assembly"/>
-    <axis xyz="0 0 1"/>
-    <limit effort="10" velocity="10" lower="-1.5708" upper="2.53073"/>
-  </joint>
-<joint name="right_ankle_pitch_joint_2" type="fixed">
-    <origin xyz="0.025 0.423 0.056" rpy="-3.14159 1.5708 0"/>
-    <parent link="urdf_r_tibia_assembly"/>
-    <child link="ankle_assembly_3"/>
-    <axis xyz="0 0 1"/>
-    <limit effort="10" velocity="10" lower="-0.785398" upper="0.785398"/>
-  </joint>
-<joint name="right_ankle_pitch_joint" type="fixed">
-    <origin xyz="0.025 0.423 0.056" rpy="-3.14159 1.5708 0"/>
-    <parent link="urdf_r_tibia_assembly"/>
-    <child link="ankle_assembly_4"/>
-    <axis xyz="0 0 1"/>
-    <limit effort="10" velocity="10" lower="-0.785398" upper="0.785398"/>
-  </joint>
-<joint name="right_knee_joint" type="fixed">
-    <origin xyz="0.055 1.37102e-06 -0.113" rpy="-1.5708 0.0173732 1.57082"/>
-    <parent link="urdf_lower_femur_assembly_2"/>
-    <child link="urdf_r_tibia_assembly"/>
-    <axis xyz="0 0 1"/>
-    <limit effort="10" velocity="10" lower="-0.191906" upper="2.33882"/>
-  </joint>
-<joint name="right_hip_yaw_joint" type="fixed">
-    <origin xyz="-2.77556e-17 -0.217 0.053" rpy="-1.5708 1.68892e-21 -1.05152e-19"/>
-    <parent link="urdf_r_upper_femur_assemby"/>
-    <child link="urdf_lower_femur_assembly_2"/>
-    <axis xyz="0 0 1"/>
-    <limit effort="10" velocity="10" lower="-1.57082" upper="1.57077"/>
-  </joint>
-<joint name="right_hip_roll_joint" type="fixed">
-    <origin xyz="0.0549931 -0.000872784 -0.078" rpy="1.5708 1.56925 -1.58667"/>
-    <parent link="urdf_hip_assembly_2"/>
-    <child link="urdf_r_upper_femur_assemby"/>
-    <axis xyz="0 0 1"/>
-    <limit effort="10" velocity="10" lower="-0.35061" upper="3.14005"/>
-  </joint>
-<joint name="right_hip_pitch_joint" type="fixed">
-    <origin xyz="0.107699 0.0333466 -0.46826" rpy="-1.5708 -1.41455e-17 1.5708"/>
-    <parent link="urdf_base"/>
-    <child link="urdf_hip_assembly_2"/>
-    <axis xyz="0 0 1"/>
-    <limit effort="10" velocity="10" lower="-2.51486" upper="1.58667"/>
+    <child link="right_leg_link"/>
   </joint>
 </robot>

File: src/robot_description/dual_arm_description/urdf/links/dual_arm_links.xacro (robot description, xacro)
@@ -1235,1621 +1235,47 @@
     </collision>
   </link>
-  <link name="urdf_hip_assembly">
-    <inertial>
-      <origin xyz="-0.00347422 1.43176e-08 -0.0692724" rpy="0 0 0"/>
-      <mass value="1.73"/>
-      <inertia ixx="0.00300557" ixy="-4.29793e-10" ixz="-5.85797e-07" iyy="0.00262683" iyz="-8.7286e-08" izz="0.00228193"/>
-    </inertial>
-    <!-- Part hip -->
-    <visual>
-      <origin xyz="0.0019136 -9.14342e-09 -0.053458" rpy="-1.5708 -1.5708 0"/>
-      <geometry>
-        <mesh filename="package://dual_arm_description/meshes/visual/hip.stl"/>
-      </geometry>
-      <material name="hip_material">
-        <color rgba="0.615686 0.811765 0.929412 1"/>
-      </material>
-    </visual>
-    <collision>
-      <origin xyz="0.0019136 -9.14342e-09 -0.053458" rpy="-1.5708 -1.5708 0"/>
-      <geometry>
-        <mesh filename="package://dual_arm_description/meshes/visual/hip.stl"/>
-      </geometry>
-    </collision>
-    <!-- Part rotor_x8_p20_120_4 -->
-    <visual>
-      <origin xyz="-0.043 0 -0.073" rpy="3.14159 -1.5708 0"/>
-      <geometry>
-        <mesh filename="package://dual_arm_description/meshes/visual/rotor_x8_p20_120.stl"/>
-      </geometry>
-      <material name="rotor_x8_p20_120_4_material">
-        <color rgba="0.596078 0.176471 0.0509804 1"/>
-      </material>
-    </visual>
-    <collision>
-      <origin xyz="-0.043 0 -0.073" rpy="3.14159 -1.5708 0"/>
-      <geometry>
-        <mesh filename="package://dual_arm_description/meshes/visual/rotor_x8_p20_120.stl"/>
-      </geometry>
-    </collision>
-    <!-- Part stator_x8_p20_120_4 -->
-    <visual>
-      <origin xyz="-0.043 0 -0.073" rpy="3.14159 -1.5708 0"/>
-      <geometry>
-        <mesh filename="package://dual_arm_description/meshes/visual/stator_x8_p20_120.stl"/>
-      </geometry>
-      <material name="stator_x8_p20_120_4_material">
-        <color rgba="0.882353 0.572549 0.478431 1"/>
-      </material>
-    </visual>
-    <collision>
-      <origin xyz="-0.043 0 -0.073" rpy="3.14159 -1.5708 0"/>
-      <geometry>
-        <mesh filename="package://dual_arm_description/meshes/visual/stator_x8_p20_120.stl"/>
-      </geometry>
-    </collision>
-  </link>
-  <link name="urdf_l_upper_femur_assembly">
-    <inertial>
-      <origin xyz="-0.0004115 -0.14917 0.0457344" rpy="0 0 0"/>
-      <mass value="1.912"/>
-      <inertia ixx="0.00560175" ixy="5.00339e-05" ixz="1.30384e-06" iyy="0.00337012" iyz="0.000930873" izz="0.0051703"/>
-    </inertial>
-    <!-- Part l_upper_femur -->
-    <visual>
-      <origin xyz="-0.00153668 -0.113387 0.0258673" rpy="-1.5708 -2.56711e-31 -1.62214e-31"/>
-      <geometry>
-        <mesh filename="package://dual_arm_description/meshes/visual/l_upper_femur.stl"/>
-      </geometry>
-      <material name="l_upper_femur_material">
-        <color rgba="0.615686 0.811765 0.929412 1"/>
-      </material>
-    </visual>
-    <collision>
-      <origin xyz="-0.00153668 -0.113387 0.0258673" rpy="-1.5708 -2.56711e-31 -1.62214e-31"/>
-      <geometry>
-        <mesh filename="package://dual_arm_description/meshes/visual/l_upper_femur.stl"/>
-      </geometry>
-    </collision>
-    <!-- Part rotor_x8_p20_120_5 -->
-    <visual>
-      <origin xyz="-5.55112e-17 -0.124 0.053" rpy="-1.5708 -0.420575 -3.14159"/>
-      <geometry>
-        <mesh filename="package://dual_arm_description/meshes/visual/rotor_x8_p20_120.stl"/>
-      </geometry>
-      <material name="rotor_x8_p20_120_5_material">
-        <color rgba="0.596078 0.176471 0.0509804 1"/>
-      </material>
-    </visual>
-    <collision>
-      <origin xyz="-5.55112e-17 -0.124 0.053" rpy="-1.5708 -0.420575 -3.14159"/>
-      <geometry>
-        <mesh filename="package://dual_arm_description/meshes/visual/rotor_x8_p20_120.stl"/>
-      </geometry>
-    </collision>
-    <!-- Part stator_x8_p20_120_5 -->
-    <visual>
-      <origin xyz="-8.32667e-17 -0.124 0.053" rpy="1.5708 -4.16331e-17 -5.56644e-31"/>
-      <geometry>
-        <mesh filename="package://dual_arm_description/meshes/visual/stator_x8_p20_120.stl"/>
-      </geometry>
-      <material name="stator_x8_p20_120_5_material">
-        <color rgba="0.882353 0.572549 0.478431 1"/>
-      </material>
-    </visual>
-    <collision>
-      <origin xyz="-8.32667e-17 -0.124 0.053" rpy="1.5708 -4.16331e-17 -5.56644e-31"/>
-      <geometry>
-        <mesh filename="package://dual_arm_description/meshes/visual/stator_x8_p20_120.stl"/>
-      </geometry>
-    </collision>
-  </link>
-  <link name="urdf_lower_femur_assembly">
-    <inertial>
-      <origin xyz="0.0027578 -1.05084e-08 -0.103488" rpy="0 0 0"/>
-      <mass value="1.817"/>
-      <inertia ixx="0.00418793" ixy="4.05713e-11" ixz="0.000182166" iyy="0.00382704" iyz="-3.93771e-08" izz="0.00258518"/>
-    </inertial>
-    <!-- Part lower_femur -->
-    <visual>
-      <origin xyz="-0.00391138 5.81796e-09 -0.0715537" rpy="2.19187e-14 -1.92346e-14 -1.90185e-15"/>
-      <geometry>
-        <mesh filename="package://dual_arm_description/meshes/visual/lower_femur.stl"/>
-      </geometry>
-      <material name="lower_femur_material">
-        <color rgba="0.615686 0.811765 0.929412 1"/>
-      </material>
-    </visual>
-    <collision>
-      <origin xyz="-0.00391138 5.81796e-09 -0.0715537" rpy="2.19187e-14 -1.92346e-14 -1.90185e-15"/>
-      <geometry>
-        <mesh filename="package://dual_arm_description/meshes/visual/lower_femur.stl"/>
-      </geometry>
-    </collision>
-    <!-- Part rotor_x8_p20_120_6 -->
-    <visual>
-      <origin xyz="0.043 7.91034e-16 -0.113" rpy="1.5708 -0.359962 -1.5708"/>
-      <geometry>
-        <mesh filename="package://dual_arm_description/meshes/visual/rotor_x8_p20_120.stl"/>
-      </geometry>
-      <material name="rotor_x8_p20_120_6_material">
-        <color rgba="0.596078 0.176471 0.0509804 1"/>
-      </material>
-    </visual>
-    <collision>
-      <origin xyz="0.043 7.91034e-16 -0.113" rpy="1.5708 -0.359962 -1.5708"/>
-      <geometry>
-        <mesh filename="package://dual_arm_description/meshes/visual/rotor_x8_p20_120.stl"/>
-      </geometry>
-    </collision>
-    <!-- Part stator_x8_p20_120_6 -->
-    <visual>
-      <origin xyz="0.043 7.14706e-16 -0.113" rpy="-1.87437e-15 -1.5708 0"/>
-      <geometry>
-        <mesh filename="package://dual_arm_description/meshes/visual/stator_x8_p20_120.stl"/>
-      </geometry>
-      <material name="stator_x8_p20_120_6_material">
-        <color rgba="0.882353 0.572549 0.478431 1"/>
-      </material>
-    </visual>
-    <collision>
-      <origin xyz="0.043 7.14706e-16 -0.113" rpy="-1.87437e-15 -1.5708 0"/>
-      <geometry>
-        <mesh filename="package://dual_arm_description/meshes/visual/stator_x8_p20_120.stl"/>
-      </geometry>
-    </collision>
-  </link>
-  <link name="urdf_l_tibia_assembly">
-    <inertial>
-      <origin xyz="0.0148171 -0.248943 0.0518904" rpy="0 0 0"/>
-      <mass value="4.79318"/>
-      <inertia ixx="0.0669306" ixy="0.00289597" ixz="-0.000212908" iyy="0.00864211" iyz="0.00251221" izz="0.0697499"/>
-    </inertial>
-    <!-- Part m6_threaded_bar_300mm -->
-    <visual>
-      <origin xyz="0.08085 -0.287625 0.0729994" rpy="-1.51492 0.191373 -0.0274192"/>
-      <geometry>
-        <mesh filename="package://dual_arm_description/meshes/visual/m6_threaded_bar_300mm.stl"/>
-      </geometry>
-      <material name="m6_threaded_bar_300mm_material">
-        <color rgba="0.141176 0.0352941 0.396078 1"/>
-      </material>
-    </visual>
-    <collision>
-      <origin xyz="0.08085 -0.287625 0.0729994" rpy="-1.51492 0.191373 -0.0274192"/>
-      <geometry>
-        <mesh filename="package://dual_arm_description/meshes/visual/m6_threaded_bar_300mm.stl"/>
-      </geometry>
-    </collision>
-    <!-- Part m6_threaded_bar_225mm -->
-    <visual>
-      <origin xyz="0.08085 -0.325171 0.0360012" rpy="1.63833 -0.167879 3.07635"/>
-      <geometry>
-        <mesh filename="package://dual_arm_description/meshes/visual/m6_threaded_bar_225mm.stl"/>
-      </geometry>
-      <material name="m6_threaded_bar_225mm_material">
-        <color rgba="0.27451 0.0117647 0.317647 1"/>
-      </material>
-    </visual>
-    <collision>
-      <origin xyz="0.08085 -0.325171 0.0360012" rpy="1.63833 -0.167879 3.07635"/>
-      <geometry>
-        <mesh filename="package://dual_arm_description/meshes/visual/m6_threaded_bar_225mm.stl"/>
-      </geometry>
-    </collision>
-    <!-- Part shoe -->
-    <visual>
-      <origin xyz="0.0302829 -0.44863 0.054" rpy="-1.5708 -1.5708 0"/>
-      <geometry>
-        <mesh filename="package://dual_arm_description/meshes/visual/shoe.stl"/>
-      </geometry>
-      <material name="shoe_material">
-        <color rgba="0.0941176 0.580392 0.545098 1"/>
-      </material>
-    </visual>
-    <collision>
-      <origin xyz="0.0302829 -0.44863 0.054" rpy="-1.5708 -1.5708 0"/>
-      <geometry>
-        <mesh filename="package://dual_arm_description/meshes/visual/shoe.stl"/>
-      </geometry>
-    </collision>
-    <!-- Part lower_fixation_leg_lontrol -->
-    <visual>
-      <origin xyz="0.0565 -0.424448 0.054" rpy="-1.5708 -1.5708 0"/>
-      <geometry>
-        <mesh filename="package://dual_arm_description/meshes/visual/lower_fixation_leg_lontrol.stl"/>
-      </geometry>
-      <material name="lower_fixation_leg_lontrol_material">
-        <color rgba="0.615686 0.811765 0.929412 1"/>
-      </material>
-    </visual>
-    <collision>
-      <origin xyz="0.0565 -0.424448 0.054" rpy="-1.5708 -1.5708 0"/>
-      <geometry>
-        <mesh filename="package://dual_arm_description/meshes/visual/lower_fixation_leg_lontrol.stl"/>
-      </geometry>
-    </collision>
-    <!-- Part foot -->
-    <visual>
-      <origin xyz="0.030138 -0.444982 0.054" rpy="-1.5708 -1.5708 0"/>
-      <geometry>
-        <mesh filename="package://dual_arm_description/meshes/visual/foot.stl"/>
-      </geometry>
-      <material name="foot_material">
-        <color rgba="0.615686 0.811765 0.929412 1"/>
-      </material>
-    </visual>
-    <collision>
-      <origin xyz="0.030138 -0.444982 0.054" rpy="-1.5708 -1.5708 0"/>
-      <geometry>
-        <mesh filename="package://dual_arm_description/meshes/visual/foot.stl"/>
-      </geometry>
-    </collision>
-    <!-- Part spacer_bottom_tibia -->
-    <visual>
-      <origin xyz="5.55112e-17 -0.3755 0.055" rpy="-1.5708 -1.5708 0"/>
-      <geometry>
-        <mesh filename="package://dual_arm_description/meshes/visual/spacer_bottom_tibia.stl"/>
-      </geometry>
-      <material name="spacer_bottom_tibia_material">
-        <color rgba="0.615686 0.811765 0.929412 1"/>
-      </material>
-    </visual>
-    <collision>
-      <origin xyz="5.55112e-17 -0.3755 0.055" rpy="-1.5708 -1.5708 0"/>
-      <geometry>
-        <mesh filename="package://dual_arm_description/meshes/visual/spacer_bottom_tibia.stl"/>
-      </geometry>
-    </collision>
-    <!-- Part l_tibia -->
-    <visual>
-      <origin xyz="0.000700098 -0.182556 0.042918" rpy="-1.5708 -1.5708 0"/>
-      <geometry>
-        <mesh filename="package://dual_arm_description/meshes/visual/l_tibia.stl"/>
-      </geometry>
-      <material name="l_tibia_material">
-        <color rgba="0.615686 0.811765 0.929412 1"/>
-      </material>
-    </visual>
-    <collision>
-      <origin xyz="0.000700098 -0.182556 0.042918" rpy="-1.5708 -1.5708 0"/>
-      <geometry>
-        <mesh filename="package://dual_arm_description/meshes/visual/l_tibia.stl"/>
-      </geometry>
-    </collision>
-    <!-- Part m6_threaded_eye -->
-    <visual>
-      <origin xyz="0.076 -0.415 0.042" rpy="-3.14159 -1.5708 0"/>
-      <geometry>
-        <mesh filename="package://dual_arm_description/meshes/visual/m6_threaded_eye.stl"/>
-      </geometry>
-      <material name="m6_threaded_eye_material">
-        <color rgba="0.615686 0.811765 0.929412 1"/>
-      </material>
-    </visual>
-    <collision>
-      <origin xyz="0.076 -0.415 0.042" rpy="-3.14159 -1.5708 0"/>
-      <geometry>
-        <mesh filename="package://dual_arm_description/meshes/visual/m6_threaded_eye.stl"/>
-      </geometry>
-    </collision>
-    <!-- Part 12_7mm_ball_with_6mm_hole -->
-    <visual>
-      <origin xyz="0.076 -0.415 0.042" rpy="2.76264 -1.38996 0.319398"/>
-      <geometry>
-        <mesh filename="package://dual_arm_description/meshes/visual/12_7mm_ball_with_6mm_hole.stl"/>
-      </geometry>
-      <material name="12_7mm_ball_with_6mm_hole_material">
-        <color rgba="0.647059 0.647059 0.647059 1"/>
-      </material>
-    </visual>
-    <collision>
-      <origin xyz="0.076 -0.415 0.042" rpy="2.76264 -1.38996 0.319398"/>
-      <geometry>
-        <mesh filename="package://dual_arm_description/meshes/visual/12_7mm_ball_with_6mm_hole.stl"/>
-      </geometry>
-    </collision>
-    <!-- Part rulment_d22_x_d8_x_t7 -->
-    <visual>
-      <origin xyz="0.0165 -0.423 0.054" rpy="1.5708 -1.5708 0"/>
-      <geometry>
-        <mesh filename="package://dual_arm_description/meshes/visual/rulment_d22_x_d8_x_t7.stl"/>
-      </geometry>
-      <material name="rulment_d22_x_d8_x_t7_material">
-        <color rgba="0.901961 0.901961 0.901961 1"/>
-      </material>
-    </visual>
-    <collision>
-      <origin xyz="0.0165 -0.423 0.054" rpy="1.5708 -1.5708 0"/>
-      <geometry>
-        <mesh filename="package://dual_arm_description/meshes/visual/rulment_d22_x_d8_x_t7.stl"/>
-      </geometry>
-    </collision>
-    <!-- Part ankle_bearing_house -->
-    <visual>
-      <origin xyz="0.0191799 -0.428357 0.054" rpy="-1.5708 -1.5708 0"/>
-      <geometry>
-        <mesh filename="package://dual_arm_description/meshes/visual/ankle_bearing_house.stl"/>
-      </geometry>
-      <material name="ankle_bearing_house_material">
-        <color rgba="0.615686 0.811765 0.929412 1"/>
-      </material>
-    </visual>
-    <collision>
-      <origin xyz="0.0191799 -0.428357 0.054" rpy="-1.5708 -1.5708 0"/>
-      <geometry>
-        <mesh filename="package://dual_arm_description/meshes/visual/ankle_bearing_house.stl"/>
-      </geometry>
-    </collision>
-    <!-- Part m6_threaded_eye_2 -->
-    <visual>
-      <origin xyz="0.076 -0.415 0.066" rpy="-3.14159 -1.5708 0"/>
-      <geometry>
-        <mesh filename="package://dual_arm_description/meshes/visual/m6_threaded_eye.stl"/>
-      </geometry>
-      <material name="m6_threaded_eye_2_material">
-        <color rgba="0.615686 0.811765 0.929412 1"/>
-      </material>
-    </visual>
-    <collision>
-      <origin xyz="0.076 -0.415 0.066" rpy="-3.14159 -1.5708 0"/>
-      <geometry>
-        <mesh filename="package://dual_arm_description/meshes/visual/m6_threaded_eye.stl"/>
-      </geometry>
-    </collision>
-    <!-- Part 12_7mm_ball_with_6mm_hole_2 -->
-    <visual>
-      <origin xyz="0.076 -0.415 0.066" rpy="-3.08572 0.191373 -0.0274192"/>
-      <geometry>
-        <mesh filename="package://dual_arm_description/meshes/visual/12_7mm_ball_with_6mm_hole.stl"/>
-      </geometry>
-      <material name="12_7mm_ball_with_6mm_hole_2_material">
-        <color rgba="0.647059 0.647059 0.647059 1"/>
-      </material>
-    </visual>
-    <collision>
-      <origin xyz="0.076 -0.415 0.066" rpy="-3.08572 0.191373 -0.0274192"/>
-      <geometry>
-        <mesh filename="package://dual_arm_description/meshes/visual/12_7mm_ball_with_6mm_hole.stl"/>
-      </geometry>
-    </collision>
-    <!-- Part rulment_d22_x_d8_x_t7_2 -->
-    <visual>
-      <origin xyz="-0.0165 -0.423 0.054" rpy="1.5708 1.5708 0"/>
-      <geometry>
-        <mesh filename="package://dual_arm_description/meshes/visual/rulment_d22_x_d8_x_t7.stl"/>
-      </geometry>
-      <material name="rulment_d22_x_d8_x_t7_2_material">
-        <color rgba="0.901961 0.901961 0.901961 1"/>
-      </material>
-    </visual>
-    <collision>
-      <origin xyz="-0.0165 -0.423 0.054" rpy="1.5708 1.5708 0"/>
-      <geometry>
-        <mesh filename="package://dual_arm_description/meshes/visual/rulment_d22_x_d8_x_t7.stl"/>
-      </geometry>
-    </collision>
-    <!-- Part ankle_bearing_house_2 -->
-    <visual>
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