Commit message: review moveit config dual arm

File: src/robot_description/dual_arm_description/urdf/joints/dual_arm_joints.xacro (robot description, xacro)
@@ -6,5 +6,6 @@
     <child link="urdf_l_wrist_assembly"/>
     <axis xyz="0 0 1"/>
-    <limit effort="10" velocity="10" lower="-1.74533" upper="1.39626"/>
+    <limit effort="40.0" velocity="10" lower="-1.74533" upper="1.39626"/>
+    <dynamics damping="0.5" friction="0.1"/>
   </joint>
   <joint name="left_wrist_yaw_joint_X4" type="revolute">
@@ -13,5 +14,6 @@
     <child link="urdf_l_lower_forearm_assembly"/>
     <axis xyz="0 0 1"/>
-    <limit effort="10" velocity="10" lower="-2.35619" upper="2.35619"/>
+    <limit effort="40.0" velocity="10" lower="-2.35619" upper="2.35619"/>
+    <dynamics damping="0.5" friction="0.1"/>
   </joint>
   <joint name="left_elbow_pitch_joint_X6" type="revolute">
@@ -20,5 +22,6 @@
     <child link="urdf_l_upper_forearm_assembly"/>
     <axis xyz="0 0 1"/>
-    <limit effort="10" velocity="10" lower="-1.5708" upper="1.5708"/>
+    <limit effort="40.0" velocity="10" lower="-1.5708" upper="1.5708"/>
+    <dynamics damping="0.5" friction="0.1"/>
   </joint>
   <joint name="left_shoulder_yaw_joint_X4" type="revolute">
@@ -27,5 +30,6 @@
     <child link="urdf_l_elbow_assembly"/>
     <axis xyz="0 0 1"/>
-    <limit effort="10" velocity="10" lower="-2.35619" upper="2.35619"/>
+    <limit effort="40.0" velocity="10" lower="-2.35619" upper="2.35619"/>
+    <dynamics damping="0.5" friction="0.1"/>
   </joint>
   <joint name="left_shoulder_roll_joint_X6" type="revolute">
@@ -34,5 +38,6 @@
     <child link="urdf_l_upper_arm_assembly"/>
     <axis xyz="0 0 1"/>
-    <limit effort="10" velocity="10" lower="-1.39626" upper="1.74533"/>
+    <limit effort="40.0" velocity="10" lower="-1.39626" upper="1.74533"/>
+    <dynamics damping="0.5" friction="0.1"/>
   </joint>
   <joint name="left_shoulder_pitch_joint_X6" type="revolute">
@@ -41,5 +46,6 @@
     <child link="urdf_l_shoulder_assembly"/>
     <axis xyz="0 0 1"/>
-    <limit effort="10" velocity="10" lower="-1.5708" upper="3.14159"/>
+    <limit effort="40.0" velocity="10" lower="-1.5708" upper="3.14159"/>
+    <dynamics damping="0.5" friction="0.1"/>
   </joint>
   <joint name="right_wrist_roll_joint_X4" type="revolute">
@@ -48,5 +54,6 @@
     <child link="urdf_r_wrist_assembly"/>
     <axis xyz="0 0 1"/>
-    <limit effort="10" velocity="10" lower="-1.39626" upper="1.74533"/>
+    <limit effort="40.0" velocity="10" lower="-1.39626" upper="1.74533"/>
+    <dynamics damping="0.5" friction="0.1"/>
   </joint>
   <joint name="right_wrist_yaw_joint_X4" type="revolute">
@@ -55,5 +62,6 @@
     <child link="urdf_r_lower_forearm_assembly"/>
     <axis xyz="0 0 1"/>
-    <limit effort="10" velocity="10" lower="-2.35619" upper="2.35619"/>
+    <limit effort="40.0" velocity="10" lower="-2.35619" upper="2.35619"/>
+    <dynamics damping="0.5" friction="0.1"/>
   </joint>
   <joint name="right_elbow_pitch_joint_X6" type="revolute">
@@ -62,5 +70,6 @@
     <child link="urdf_r_upper_forearm_assembly"/>
     <axis xyz="0 0 1"/>
-    <limit effort="10" velocity="10" lower="-1.5708" upper="1.5708"/>
+    <limit effort="40.0" velocity="10" lower="-1.5708" upper="1.5708"/>
+    <dynamics damping="0.5" friction="0.1"/>
   </joint>
   <joint name="right_shoulder_yaw_joint_X4" type="revolute">
@@ -69,5 +78,6 @@
     <child link="urdf_r_elbow_assembly"/>
     <axis xyz="0 0 1"/>
-    <limit effort="10" velocity="10" lower="-2.35619" upper="2.35619"/>
+    <limit effort="40.0" velocity="10" lower="-2.35619" upper="2.35619"/>
+    <dynamics damping="0.5" friction="0.1"/>
   </joint>
   <joint name="right_shoulder_roll_joint_X6" type="revolute">
@@ -76,5 +86,6 @@
     <child link="urdf_r_upper_arm_assembly"/>
     <axis xyz="0 0 1"/>
-    <limit effort="10" velocity="10" lower="-1.74533" upper="1.39626"/>
+    <limit effort="40.0" velocity="10" lower="-1.74533" upper="1.39626"/>
+    <dynamics damping="0.5" friction="0.1"/>
   </joint>
   <joint name="right_shoulder_pitch_joint_X6" type="revolute">
@@ -83,5 +94,6 @@
     <child link="urdf_r_shoulder_assembly"/>
     <axis xyz="0 0 1"/>
-    <limit effort="10" velocity="10" lower="-3.14159" upper="1.5708"/>
+    <limit effort="40.0" velocity="10" lower="-3.14159" upper="1.5708"/>
+    <dynamics damping="0.5" friction="0.1"/>
   </joint>
   <joint name="waist_yaw_joint" type="fixed">
@@ -90,5 +102,6 @@
     <child link="urdf_simplified_torso_sub_assembly"/>
     <axis xyz="0 0 1"/>
-    <limit effort="10" velocity="10" lower="-1.5708" upper="1.5708"/>
+    <limit effort="40.0" velocity="10" lower="-1.5708" upper="1.5708"/>
+    <dynamics damping="0.5" friction="0.1"/>
   </joint>
   <!-- Left leg: single box replacing 6 links + 12 joints -->

Commit message: left_kee_joint limits and comments

File: src/robot_description/dual_arm_description/urdf/joints/dual_arm_joints.xacro (robot description, xacro)
@@ -2,9 +2,9 @@
 <robot xmlns:xacro="http://www.ros.org/wiki/xacro">
   <!-- ================================================================== -->
-  <!-- Legs — set fixed_legs:=false for revolute leg joints               -->
+  <!-- Legs — set fixed_legs:=false for revolute leg joints              -->
   <!-- ================================================================== -->
   <xacro:property name="leg_joint_type" value="${'fixed' if '$(arg fixed_legs)' == 'true' else 'revolute'}"/>
   <!-- ================================================================== -->
-  <!-- Waist (revolute — connects base to torso)                          -->
+  <!-- Waist                                                             -->
   <!-- ================================================================== -->
   <joint name="waist_yaw_joint" type="${leg_joint_type}">
@@ -17,5 +17,5 @@
   </joint>
   <!-- ================================================================== -->
-  <!-- Left Arm                                                           -->
+  <!-- Left Arm                                                          -->
   <!-- ================================================================== -->
   <joint name="left_shoulder_pitch_joint_X6" type="revolute">
@@ -68,5 +68,5 @@
   </joint>
   <!-- ================================================================== -->
-  <!-- Right Arm                                                          -->
+  <!-- Right Arm                                                         -->
   <!-- ================================================================== -->
   <joint name="right_shoulder_pitch_joint_X6" type="revolute">
@@ -118,5 +118,7 @@
     <dynamics damping="0.5" friction="0.1"/>
   </joint>
-  <!-- Left Leg -->
+  <!-- ================================================================== -->
+  <!-- Left Leg                                                          -->
+  <!-- ================================================================== -->
   <joint name="left_hip_pitch_joint" type="${leg_joint_type}">
     <origin xyz="0.0333466 0.111301 -0.46826" rpy="0 0 0"/>
@@ -148,5 +150,5 @@
     <child link="urdf_l_tibia_assembly"/>
     <axis xyz="0 1 0"/>
-    <limit effort="100" velocity="100" lower="-2.33882" upper="0.191906"/>
+    <limit effort="100" velocity="100" lower="0.191906" upper="-2.33882"/>
     <dynamics damping="0.5" friction="0.1"/>
   </joint>
@@ -160,5 +162,5 @@
   </joint>
   <!-- ================================================================== -->
-  <!-- Right Leg                                                          -->
+  <!-- Right Leg                                                         -->
   <!-- ================================================================== -->
   <joint name="right_hip_pitch_joint" type="${leg_joint_type}">

File: src/robot_description/dual_arm_description/urdf/links/dual_arm_links.xacro (robot description, xacro)
@@ -2,5 +2,5 @@
 <robot xmlns:xacro="http://www.ros.org/wiki/xacro">
   <!-- ================================================================== -->
-  <!-- Base                                                                -->
+  <!-- Base                                                              -->
   <!-- ================================================================== -->
   <link name="urdf_base">
@@ -42,5 +42,5 @@
   </link>
   <!-- ================================================================== -->
-  <!-- Torso                                                               -->
+  <!-- Torso                                                             -->
   <!-- ================================================================== -->
   <link name="urdf_simplified_torso_sub_assembly">
@@ -112,5 +112,5 @@
   </link>
   <!-- ================================================================== -->
-  <!-- Left Arm                                                            -->
+  <!-- Left Arm                                                          -->
   <!-- ================================================================== -->
   <link name="urdf_l_shoulder_assembly">
@@ -247,5 +247,5 @@
   </link>
   <!-- ================================================================== -->
-  <!-- Right Arm                                                           -->
+  <!-- Right Arm                                                         -->
   <!-- ================================================================== -->
   <link name="urdf_r_shoulder_assembly">
@@ -382,5 +382,5 @@
   </link>
   <!-- ================================================================== -->
-  <!-- Left Leg                                                            -->
+  <!-- Left Leg                                                          -->
   <!-- ================================================================== -->
   <link name="urdf_hip_assembly">
@@ -510,5 +510,5 @@
   </link>
   <!-- ================================================================== -->
-  <!-- Right Leg                                                           -->
+  <!-- Right Leg                                                         -->
   <!-- ================================================================== -->
   <link name="urdf_hip_assembly_2">
