Commit message: review single arm to use full robot description

File: src/planning/arm_moveit_config/config/arm_description.ros2_control.xacro (robot description, xacro)
@@ -8,43 +8,43 @@
                 <plugin>mock_components/GenericSystem</plugin>
             </hardware>
-            <joint name="shoulder_pitch_joint">
+            <joint name="left_shoulder_pitch_joint_X6">
                 <command_interface name="position"/>
                 <state_interface name="position">
-                  <param name="initial_value">${initial_positions['shoulder_pitch_joint']}</param>
+                  <param name="initial_value">${initial_positions['left_shoulder_pitch_joint_X6']}</param>
                 </state_interface>
                 <state_interface name="velocity"/>
             </joint>
-            <joint name="shoulder_roll_joint">
+            <joint name="left_shoulder_roll_joint_X6">
                 <command_interface name="position"/>
                 <state_interface name="position">
-                  <param name="initial_value">${initial_positions['shoulder_roll_joint']}</param>
+                  <param name="initial_value">${initial_positions['left_shoulder_roll_joint_X6']}</param>
                 </state_interface>
                 <state_interface name="velocity"/>
             </joint>
-            <joint name="shoulder_yaw_joint">
+            <joint name="left_shoulder_yaw_joint_X4">
                 <command_interface name="position"/>
                 <state_interface name="position">
-                  <param name="initial_value">${initial_positions['shoulder_yaw_joint']}</param>
+                  <param name="initial_value">${initial_positions['left_shoulder_yaw_joint_X4']}</param>
                 </state_interface>
                 <state_interface name="velocity"/>
             </joint>
-            <joint name="elbow_pitch_joint">
+            <joint name="left_elbow_pitch_joint_X6">
                 <command_interface name="position"/>
                 <state_interface name="position">
-                  <param name="initial_value">${initial_positions['elbow_pitch_joint']}</param>
+                  <param name="initial_value">${initial_positions['left_elbow_pitch_joint_X6']}</param>
                 </state_interface>
                 <state_interface name="velocity"/>
             </joint>
-            <joint name="elbow_yaw_joint">
+            <joint name="left_wrist_yaw_joint_X4">
                 <command_interface name="position"/>
                 <state_interface name="position">
-                  <param name="initial_value">${initial_positions['elbow_yaw_joint']}</param>
+                  <param name="initial_value">${initial_positions['left_wrist_yaw_joint_X4']}</param>
                 </state_interface>
                 <state_interface name="velocity"/>
             </joint>
-            <joint name="wrist_roll_joint">
+            <joint name="left_wrist_roll_joint_X4">
                 <command_interface name="position"/>
                 <state_interface name="position">
-                  <param name="initial_value">${initial_positions['wrist_roll_joint']}</param>
+                  <param name="initial_value">${initial_positions['left_wrist_roll_joint_X4']}</param>
                 </state_interface>
                 <state_interface name="velocity"/>

File: src/robot_description/arm_description/urdf/arm.urdf.xacro (robot description, xacro)
@@ -9,6 +9,4 @@
     <xacro:arg name="use_sim"
         default="false" />
-    <xacro:arg name="hand_type"
-        default="inspire_hand" />
     <xacro:if value="$(arg use_sim)">
         <xacro:include filename="$(find arm_description)/urdf/arm_gazebo.xacro" />

File: src/robot_description/arm_description/urdf/arm_base.xacro (robot description, xacro)
@@ -3,21 +3,39 @@
     <!-- Include macros -->
     <xacro:include filename="$(find arm_description)/urdf/macros/materials.xacro" />
-    <!-- Base link -->
-    <!-- <xacro:include filename="$(find arm_description)/urdf/links/base_link.xacro" /> -->
-    <!-- Arm Links -->
-    <xacro:include filename="$(find arm_description)/urdf/links/arm_links.xacro" />
-    <!-- Arm Joints -->
-    <xacro:include filename="$(find arm_description)/urdf/joints/arm_joints.xacro" />
-    <!-- Hand/Gripper macros -->
-    <xacro:include filename="$(find arm_description)/urdf/hands/simple_gripper.xacro" />
+     <!-- Body (base + torso) -->
+    <xacro:include filename="$(find full_robot_description)/urdf/links/body_links.xacro" />
+     <xacro:include filename="$(find full_robot_description)/urdf/joints/body_joints.xacro" />
+    <!-- Left Arm -->
+    <xacro:include filename="$(find full_robot_description)/urdf/links/left_arm_links.xacro" />
+    <xacro:include filename="$(find full_robot_description)/urdf/joints/left_arm_joints.xacro" />
+    <!-- Right Arm -->
+    <xacro:include filename="$(find full_robot_description)/urdf/links/right_arm_links.xacro" />
+    <xacro:include filename="$(find full_robot_description)/urdf/joints/right_arm_joints.xacro" />
+    <!-- Left Foot -->
+    <xacro:include filename="$(find full_robot_description)/urdf/links/left_foot_links.xacro" />
+    <xacro:include filename="$(find full_robot_description)/urdf/joints/left_foot_joints.xacro" />
+    <!-- Right Foot -->
+    <xacro:include filename="$(find full_robot_description)/urdf/links/right_foot_links.xacro" />
+    <xacro:include filename="$(find full_robot_description)/urdf/joints/right_foot_joints.xacro" />
+    <!-- Hands -->
     <xacro:include filename="$(find hand_description)/urdf/hands/inspire_hand_left.xacro" />
-    <!-- Resolve hand_type arg into a property for conditional evaluation -->
-    <xacro:property name="hand_type" value="$(arg hand_type)"/>
-    <!-- Conditionally instantiate hand based on hand_type arg -->
-    <xacro:if value="${hand_type == 'simple_gripper'}">
-        <xacro:simple_gripper parent="end_effector_link"/>
-    </xacro:if>
-    <xacro:if value="${hand_type == 'inspire_hand'}">
-        <xacro:inspire_hand_left parent="end_effector_link"/>
-    </xacro:if>
+    <xacro:include filename="$(find hand_description)/urdf/hands/inspire_hand_right.xacro" />
+    <xacro:inspire_hand_left
+        parent="urdf_l_wrist_assembly"
+        prefix="left_"
+        mount_x="-0.0303429"
+        mount_y="4.52464e-07 "
+        mount_z="-0.06"
+        mount_roll="1.5708"
+        mount_pitch="0"
+        mount_yaw="1.5708"/>
+    <xacro:inspire_hand_right
+        parent="urdf_r_wrist_assembly"
+        prefix="right_"
+        mount_x="-0.0303429"
+        mount_y="4.52464e-07 "
+        mount_z="-0.06"
+        mount_roll="1.5708"
+        mount_pitch="0"
+        mount_yaw="-1.5708"/>
 </robot>

File: src/robot_description/arm_description/urdf/arm_gazebo.xacro (robot description, xacro)
@@ -8,7 +8,6 @@
     <xacro:include filename="$(find arm_description)/urdf/arm_base.xacro" />
     <!-- ros2_control interfaces for Gazebo simulation -->
-    <!-- Load ros2_control macro -->
     <xacro:include filename="$(find arm_description)/urdf/macros/ros2_control.xacro"/>
-    <xacro:arm_ros2_control hand_type="$(arg hand_type)"/>
+    <xacro:arm_ros2_control/>
     <!-- Depth Camera -->
     <xacro:include filename="$(find arm_description)/urdf/macros/depth_camera.xacro"/>
@@ -16,5 +15,5 @@
     <!-- The new robot has the table at z=0, arm starts at table level -->
     <!-- Position camera 0.5m behind and 0.8m above the robot base, looking down slightly -->
-    <xacro:depth_camera parent_link="base_link" xyz="-0.3 0.0 0.8" rpy="0 ${pi/6} 0" name="camera"/>
+    <xacro:depth_camera parent_link="urdf_base" xyz="-0.3 0.0 1.26" rpy="0 ${pi/6} 0" name="camera"/>
     <!-- Gazebo plugins -->
     <gazebo>

File: src/robot_description/arm_description/urdf/arm_real.xacro (robot description, xacro)
@@ -3,4 +3,4 @@
     <xacro:include filename="$(find arm_description)/urdf/arm_base.xacro" />
     <xacro:include filename="$(find arm_description)/urdf/macros/ros2_control.xacro" />
-    <xacro:arm_ros2_control hand_type="$(arg hand_type)"/>
+    <xacro:arm_ros2_control/>
 </robot>

File: src/robot_description/arm_description/urdf/macros/gazebo_extensions.xacro (robot description, xacro)
@@ -3,21 +3,21 @@
     <xacro:property name="damping" value="0.05" />
     <xacro:property name="friction" value="0.01" />
-    <gazebo reference="shoulder_pitch_joint">
+    <gazebo reference="left_shoulder_pitch_joint_X6">
         <damping>${damping}</damping>
         <friction>${friction}</friction>
     </gazebo>
-    <gazebo reference="shoulder_roll_joint">
+    <gazebo reference="left_shoulder_roll_joint_X6">
         <damping>${damping}</damping>
         <friction>${friction}</friction>
     </gazebo>
-    <gazebo reference="shoulder_yaw_joint">
+    <gazebo reference="left_shoulder_yaw_joint_X4">
         <damping>${damping}</damping>
         <friction>${friction}</friction>
     </gazebo>
-    <gazebo reference="elbow_pitch_joint">
+    <gazebo reference="left_elbow_pitch_joint_X6">
         <damping>${damping}</damping>
         <friction>${friction}</friction>
     </gazebo>
-    <gazebo reference="elbow_yaw_joint">
+    <gazebo reference="left_wrist_yaw_joint_X4">
         <damping>${damping}</damping>
         <friction>${friction}</friction>
