Commit message: review single arm to use full robot description

File: src/robot_description/arm_description/urdf/macros/ros2_control.xacro (robot description, xacro)
@@ -1,144 +1,256 @@
 <?xml version="1.0"?>
 <robot xmlns:xacro="http://ros.org/wiki/xacro">
-    <xacro:macro name="arm_ros2_control" params="hand_type:=simple_gripper">
+    <xacro:arg name="only_left" default="true" />
+    <xacro:property name="only_left" value="$(arg only_left)"/>
+    <xacro:macro name="arm_ros2_control">
         <ros2_control name="ArmSystem" type="system">
             <hardware>
                 <plugin>gz_ros2_control/GazeboSimSystem</plugin>
             </hardware>
-            <!-- Arm joints (6 DOF) -->
-            <joint name="shoulder_pitch_joint">
-                <command_interface name="position"/>
-                <state_interface name="position"/>
-                <state_interface name="velocity"/>
-                <state_interface name="effort"/>
-            </joint>
-            <joint name="shoulder_roll_joint">
-                <command_interface name="position"/>
-                <state_interface name="position"/>
-                <state_interface name="velocity"/>
-                <state_interface name="effort"/>
-            </joint>
-            <joint name="shoulder_yaw_joint">
-                <command_interface name="position"/>
-                <state_interface name="position"/>
-                <state_interface name="velocity"/>
-                <state_interface name="effort"/>
-            </joint>
-            <joint name="elbow_pitch_joint">
-                <command_interface name="position"/>
-                <state_interface name="position"/>
-                <state_interface name="velocity"/>
-                <state_interface name="effort"/>
-            </joint>
-            <joint name="elbow_yaw_joint">
-                <command_interface name="position"/>
-                <state_interface name="position"/>
-                <state_interface name="velocity"/>
-                <state_interface name="effort"/>
-            </joint>
-            <joint name="wrist_roll_joint">
-                <command_interface name="position"/>
-                <state_interface name="position"/>
-                <state_interface name="velocity"/>
-                <state_interface name="effort"/>
-            </joint>
+            <!-- Left arm (6 DOF) -->
+            <joint name="left_shoulder_pitch_joint_X6">
+                <command_interface name="position"/>
+                <state_interface name="position"/>
+                <state_interface name="velocity"/>
+                <state_interface name="effort"/>
+            </joint>
+            <joint name="left_shoulder_roll_joint_X6">
+                <command_interface name="position"/>
+                <state_interface name="position"/>
+                <state_interface name="velocity"/>
+                <state_interface name="effort"/>
+            </joint>
+            <joint name="left_shoulder_yaw_joint_X4">
+                <command_interface name="position"/>
+                <state_interface name="position"/>
+                <state_interface name="velocity"/>
+                <state_interface name="effort"/>
+            </joint>
+            <joint name="left_elbow_pitch_joint_X6">
+                <command_interface name="position"/>
+                <state_interface name="position"/>
+                <state_interface name="velocity"/>
+                <state_interface name="effort"/>
+            </joint>
+            <joint name="left_wrist_yaw_joint_X4">
+                <command_interface name="position"/>
+                <state_interface name="position"/>
+                <state_interface name="velocity"/>
+                <state_interface name="effort"/>
+            </joint>
+            <joint name="left_wrist_roll_joint_X4">
+                <command_interface name="position"/>
+                <state_interface name="position"/>
+                <state_interface name="velocity"/>
+                <state_interface name="effort"/>
+            </joint>
+            <!-- Right arm (6 DOF) — only when not only_left -->
+            <xacro:unless value="${only_left == 'true'}">
+                <joint name="right_shoulder_pitch_joint_X6">
+                    <command_interface name="position"/>
+                    <state_interface name="position"/>
+                    <state_interface name="velocity"/>
+                    <state_interface name="effort"/>
+                </joint>
+                <joint name="right_shoulder_roll_joint_X6">
+                    <command_interface name="position"/>
+                    <state_interface name="position"/>
+                    <state_interface name="velocity"/>
+                    <state_interface name="effort"/>
+                </joint>
+                <joint name="right_shoulder_yaw_joint_X4">
+                    <command_interface name="position"/>
+                    <state_interface name="position"/>
+                    <state_interface name="velocity"/>
+                    <state_interface name="effort"/>
+                </joint>
+                <joint name="right_elbow_pitch_joint_X6">
+                    <command_interface name="position"/>
+                    <state_interface name="position"/>
+                    <state_interface name="velocity"/>
+                    <state_interface name="effort"/>
+                </joint>
+                <joint name="right_wrist_yaw_joint_X4">
+                    <command_interface name="position"/>
+                    <state_interface name="position"/>
+                    <state_interface name="velocity"/>
+                    <state_interface name="effort"/>
+                </joint>
+                <joint name="right_wrist_roll_joint_X4">
+                    <command_interface name="position"/>
+                    <state_interface name="position"/>
+                    <state_interface name="velocity"/>
+                    <state_interface name="effort"/>
+                </joint>
+            </xacro:unless>
         </ros2_control>
-        <!-- Simple gripper ros2_control joints -->
-        <xacro:if value="${hand_type == 'simple_gripper'}">
-            <ros2_control name="GripperSystem" type="system">
-                <hardware>
-                    <plugin>gz_ros2_control/GazeboSimSystem</plugin>
-                </hardware>
-                <!-- Gripper: right finger (controlled) -->
-                <joint name="left_palm_right_finger">
-                    <command_interface name="position"/>
-                    <state_interface name="position"/>
-                    <state_interface name="velocity"/>
-                    <state_interface name="effort"/>
-                </joint>
-                <!-- Gripper: left finger (mimic - state only) -->
-                <joint name="left_palm_left_finger">
-                    <state_interface name="position"/>
-                    <state_interface name="velocity"/>
-                    <state_interface name="effort"/>
-                </joint>
-            </ros2_control>
-        </xacro:if>
-        <!-- Inspire hand ros2_control joints -->
-        <xacro:if value="${hand_type == 'inspire_hand'}">
-            <ros2_control name="HandSystem" type="system">
-                <hardware>
-                    <plugin>gz_ros2_control/GazeboSimSystem</plugin>
-                </hardware>
-                <!-- 6 actuated joints (command + state) -->
-                <joint name="left_thumb_proximal_yaw_joint">
-                    <command_interface name="position"/>
-                    <state_interface name="position"/>
-                    <state_interface name="velocity"/>
-                    <state_interface name="effort"/>
-                </joint>
-                <joint name="left_thumb_proximal_pitch_joint">
-                    <command_interface name="position"/>
-                    <state_interface name="position"/>
-                    <state_interface name="velocity"/>
-                    <state_interface name="effort"/>
-                </joint>
-                <joint name="left_index_proximal_joint">
-                    <command_interface name="position"/>
-                    <state_interface name="position"/>
-                    <state_interface name="velocity"/>
-                    <state_interface name="effort"/>
-                </joint>
-                <joint name="left_middle_proximal_joint">
-                    <command_interface name="position"/>
-                    <state_interface name="position"/>
-                    <state_interface name="velocity"/>
-                    <state_interface name="effort"/>
-                </joint>
-                <joint name="left_ring_proximal_joint">
-                    <command_interface name="position"/>
-                    <state_interface name="position"/>
-                    <state_interface name="velocity"/>
-                    <state_interface name="effort"/>
-                </joint>
-                <joint name="left_pinky_proximal_joint">
-                    <command_interface name="position"/>
-                    <state_interface name="position"/>
-                    <state_interface name="velocity"/>
-                    <state_interface name="effort"/>
-                </joint>
-                <!-- 6 mimic joints (state only) -->
-                <joint name="left_thumb_intermediate_joint">
-                    <state_interface name="position"/>
-                    <state_interface name="velocity"/>
-                    <state_interface name="effort"/>
-                </joint>
-                <joint name="left_thumb_distal_joint">
-                    <state_interface name="position"/>
-                    <state_interface name="velocity"/>
-                    <state_interface name="effort"/>
-                </joint>
-                <joint name="left_index_intermediate_joint">
-                    <state_interface name="position"/>
-                    <state_interface name="velocity"/>
-                    <state_interface name="effort"/>
-                </joint>
-                <joint name="left_middle_intermediate_joint">
-                    <state_interface name="position"/>
-                    <state_interface name="velocity"/>
-                    <state_interface name="effort"/>
-                </joint>
-                <joint name="left_ring_intermediate_joint">
-                    <state_interface name="position"/>
-                    <state_interface name="velocity"/>
-                    <state_interface name="effort"/>
-                </joint>
-                <joint name="left_pinky_intermediate_joint">
-                    <state_interface name="position"/>
-                    <state_interface name="velocity"/>
-                    <state_interface name="effort"/>
-                </joint>
-            </ros2_control>
-        </xacro:if>
+        <ros2_control name="HandSystem" type="system">
+            <hardware>
+                <plugin>gz_ros2_control/GazeboSimSystem</plugin>
+            </hardware>
+            <!-- Left hand actuated -->
+            <joint name="left_thumb_proximal_yaw_joint">
+                <command_interface name="position"/>
+                <state_interface name="position">
+                    <param name="initial_value">0.1</param>
+                </state_interface>
+                <state_interface name="velocity"/>
+                <state_interface name="effort"/>
+            </joint>
+            <joint name="left_thumb_proximal_pitch_joint">
+                <command_interface name="position"/>
+                <state_interface name="position">
+                    <param name="initial_value">0.1</param>
+                </state_interface>
+                <state_interface name="velocity"/>
+                <state_interface name="effort"/>
+            </joint>
+            <joint name="left_index_proximal_joint">
+                <command_interface name="position"/>
+                <state_interface name="position">
+                    <param name="initial_value">0.1</param>
+                </state_interface>
+                <state_interface name="velocity"/>
+                <state_interface name="effort"/>
+            </joint>
+            <joint name="left_middle_proximal_joint">
+                <command_interface name="position"/>
+                <state_interface name="position">
+                    <param name="initial_value">0.1</param>
+                </state_interface>
+                <state_interface name="velocity"/>
+                <state_interface name="effort"/>
+            </joint>
+            <joint name="left_ring_proximal_joint">
+                <command_interface name="position"/>
+                <state_interface name="position">
+                    <param name="initial_value">0.1</param>
+                </state_interface>
+                <state_interface name="velocity"/>
+                <state_interface name="effort"/>
+            </joint>
+            <joint name="left_pinky_proximal_joint">
+                <command_interface name="position"/>
+                <state_interface name="position">
+                    <param name="initial_value">0.1</param>
+                </state_interface>
+                <state_interface name="velocity"/>
+                <state_interface name="effort"/>
+            </joint>
+            <!-- Left hand mimic (state only) -->
+            <joint name="left_thumb_intermediate_joint">
+                <state_interface name="position"/>
+                <state_interface name="velocity"/>
+                <state_interface name="effort"/>
+            </joint>
+            <joint name="left_thumb_distal_joint">
+                <state_interface name="position"/>
+                <state_interface name="velocity"/>
+                <state_interface name="effort"/>
+            </joint>
+            <joint name="left_index_intermediate_joint">
+                <state_interface name="position"/>
+                <state_interface name="velocity"/>
+                <state_interface name="effort"/>
+            </joint>
+            <joint name="left_middle_intermediate_joint">
+                <state_interface name="position"/>
+                <state_interface name="velocity"/>
+                <state_interface name="effort"/>
+            </joint>
+            <joint name="left_ring_intermediate_joint">
+                <state_interface name="position"/>
+                <state_interface name="velocity"/>
+                <state_interface name="effort"/>
+            </joint>
+            <joint name="left_pinky_intermediate_joint">
+                <state_interface name="position"/>
+                <state_interface name="velocity"/>
+                <state_interface name="effort"/>
+            </joint>
+            <!-- Right hand — only when not only_left -->
+            <xacro:unless value="${only_left == 'true'}">
+                <!-- Right hand actuated -->
+                <joint name="right_thumb_proximal_yaw_joint">
+                    <command_interface name="position"/>
+                    <state_interface name="position">
+                        <param name="initial_value">0.1</param>
+                    </state_interface>
+                    <state_interface name="velocity"/>
+                    <state_interface name="effort"/>
+                </joint>
+                <joint name="right_thumb_proximal_pitch_joint">
+                    <command_interface name="position"/>
+                    <state_interface name="position">
+                        <param name="initial_value">0.1</param>
+                    </state_interface>
+                    <state_interface name="velocity"/>
+                    <state_interface name="effort"/>
+                </joint>
+                <joint name="right_index_proximal_joint">
+                    <command_interface name="position"/>
+                    <state_interface name="position">
+                        <param name="initial_value">0.1</param>
+                    </state_interface>
+                    <state_interface name="velocity"/>
+                    <state_interface name="effort"/>
+                </joint>
+                <joint name="right_middle_proximal_joint">
+                    <command_interface name="position"/>
+                    <state_interface name="position">
+                        <param name="initial_value">0.1</param>
+                    </state_interface>
+                    <state_interface name="velocity"/>
+                    <state_interface name="effort"/>
+                </joint>
+                <joint name="right_ring_proximal_joint">
+                    <command_interface name="position"/>
+                    <state_interface name="position">
+                        <param name="initial_value">0.1</param>
+                    </state_interface>
+                    <state_interface name="velocity"/>
+                    <state_interface name="effort"/>
+                </joint>
+                <joint name="right_pinky_proximal_joint">
+                    <command_interface name="position"/>
+                    <state_interface name="position">
+                        <param name="initial_value">0.1</param>
+                    </state_interface>
+                    <state_interface name="velocity"/>
+                    <state_interface name="effort"/>
+                </joint>
+                <!-- Right hand mimic (state only) -->
+                <joint name="right_thumb_intermediate_joint">
+                    <state_interface name="position"/>
+                    <state_interface name="velocity"/>
+                    <state_interface name="effort"/>
+                </joint>
+                <joint name="right_thumb_distal_joint">
+                    <state_interface name="position"/>
+                    <state_interface name="velocity"/>
+                    <state_interface name="effort"/>
+                </joint>
+                <joint name="right_index_intermediate_joint">
+                    <state_interface name="position"/>
+                    <state_interface name="velocity"/>
+                    <state_interface name="effort"/>
+                </joint>
+                <joint name="right_middle_intermediate_joint">
+                    <state_interface name="position"/>
+                    <state_interface name="velocity"/>
+                    <state_interface name="effort"/>
+                </joint>
+                <joint name="right_ring_intermediate_joint">
+                    <state_interface name="position"/>
+                    <state_interface name="velocity"/>
+                    <state_interface name="effort"/>
+                </joint>
+                <joint name="right_pinky_intermediate_joint">
+                    <state_interface name="position"/>
+                    <state_interface name="velocity"/>
+                    <state_interface name="effort"/>
+                </joint>
+            </xacro:unless>
+        </ros2_control>
     </xacro:macro>
 </robot>

File: src/robot_description/full_robot_description/urdf/joints/body_joints.xacro (robot description, xacro)
@@ -7,7 +7,12 @@
   <xacro:property name="leg_joint_type" value="${'fixed' if '$(arg fixed_legs)' == 'true' else 'revolute'}"/>
   <!-- ================================================================== -->
+  <!-- only_left — when true, also lock waist yaw joint                  -->
+  <!-- ================================================================== -->
+  <xacro:arg name="only_left" default="true" />
+  <xacro:property name="waist_joint_type" value="${'fixed' if '$(arg only_left)' == 'true' or '$(arg fixed_legs)' == 'true' else 'revolute'}"/>
+  <!-- ================================================================== -->
   <!-- Waist                                                             -->
   <!-- ================================================================== -->
-  <joint name="waist_yaw_joint" type="${leg_joint_type}">
+  <joint name="waist_yaw_joint" type="${waist_joint_type}">
     <origin xyz="0.0333466 -0.000699067 -0.29826" rpy="0 0 0"/>
     <parent link="urdf_base"/>
