Commit message: feat(arm_moveit_config): extend arm planning group to 7 DOF
Add waist yaw to the MoveIt model, controller mappings, joint limits,
initial positions, and named arm states for coordinated waist-arm planning.

File: src/planning/arm_moveit_config/config/arm_description.ros2_control.xacro (robot description, xacro)
@@ -8,4 +8,11 @@
                 <plugin>mock_components/GenericSystem</plugin>
             </hardware>
+            <joint name="waist_yaw_joint_X8">
+                <command_interface name="position"/>
+                <state_interface name="position">
+                  <param name="initial_value">${initial_positions['waist_yaw_joint_X8']}</param>
+                </state_interface>
+                <state_interface name="velocity"/>
+            </joint>
             <joint name="left_shoulder_pitch_joint_X6">
                 <command_interface name="position"/>
