Commit message: delete mockup hands

File: src/robot_description/full_robot_description/urdf/links/left_arm_links.xacro (robot description, xacro)
@@ -270,19 +270,4 @@
       </geometry>
     </collision>
-    <visual>
-      <origin xyz="-0.0303429 2.67e-09 -0.135203" rpy="0 0 0"/>
-      <geometry>
-        <mesh filename="package://full_robot_description/meshes/l_hand.stl"/>
-      </geometry>
-      <material name="l_hand_material">
-        <color rgba="1 1 1 1"/>
-      </material>
-    </visual>
-    <collision>
-      <origin xyz="-0.0303429 2.67e-09 -0.135203" rpy="0 0 0"/>
-      <geometry>
-        <mesh filename="package://full_robot_description/meshes/l_hand.stl"/>
-      </geometry>
-    </collision>
   </link>
 </robot>

File: src/robot_description/full_robot_description/urdf/links/right_arm_links.xacro (robot description, xacro)
@@ -196,19 +196,4 @@
     </inertial>
     <visual>
-      <origin xyz="-0.0303429 -2.67e-09 -0.135003" rpy="0 0 3.14159"/>
-      <geometry>
-        <mesh filename="package://full_robot_description/meshes/r_hand.stl"/>
-      </geometry>
-      <material name="r_hand_material">
-        <color rgba="1 1 1 1"/>
-      </material>
-    </visual>
-    <collision>
-      <origin xyz="-0.0303429 -2.67e-09 -0.135003" rpy="0 0 3.14159"/>
-      <geometry>
-        <mesh filename="package://full_robot_description/meshes/r_hand.stl"/>
-      </geometry>
-    </collision>
-    <visual>
       <origin xyz="-0.0219316 -4.44584e-06 -0.0434653" rpy="0 0 -1.5708"/>
       <geometry>
