Commit message: add gemini camer to dual arm configurationa

File: src/robot_description/dual_arm_description/urdf/dual_arm_gazebo.xacro (robot description, xacro)
@@ -15,12 +15,12 @@
     <xacro:dual_arm_ros2_control/>
     <!-- Orbbec Gemini 335L/336L Depth Camera -->
-    <!--xacro:include filename="$(find camera_description)/urdf/gemini335L_336L.urdf.xacro"/-->
-    <!--xacro:include filename="$(find camera_description)/urdf/gemini335L_336L_gazebo.xacro"/-->
+    <xacro:include filename="$(find camera_description)/urdf/gemini335L_336L.urdf.xacro"/>
+    <xacro:include filename="$(find camera_description)/urdf/gemini335L_336L_gazebo.xacro"/>
     <!-- Mount camera on urdf_base, positioned to view the workspace -->
-    <!--joint name="camera_mount_joint" type="fixed">
+    <joint name="camera_mount_joint" type="fixed">
         <parent link="urdf_base"/>
         <child link="camera_link"/>
-        <origin xyz="0.13 0.0455 0.429" rpy="0 ${pi/12} 0"/>
-    </joint-->
+        <origin xyz="0.08 0.0455 0.829" rpy="0 ${pi/12} 0"/>
+    </joint>
     <!-- Gazebo plugins -->
     <gazebo>
