Commit message: orbec camera in isaac

File: src/robot_description/dual_arm_description/urdf/dual_arm_isaac.xacro (robot description, xacro)
@@ -14,7 +14,10 @@
     <xacro:include filename="$(find dual_arm_description)/urdf/macros/ros2_control_isaac.xacro"/>
     <xacro:dual_arm_ros2_control_isaac/>
-    <!-- Depth Camera -->
-    <xacro:include filename="$(find arm_description)/urdf/macros/depth_camera.xacro"/>
+    <xacro:include filename="$(find camera_description)/urdf/gemini335L_336L.urdf.xacro"/>
     <!-- Mount camera on urdf_base, positioned to view the workspace -->
-    <xacro:depth_camera parent_link="urdf_base" xyz="-0.3 0.0 0.8" rpy="0 ${pi/6} 0" name="camera"/>
+    <joint name="camera_mount_joint" type="fixed">
+        <parent link="urdf_base"/>
+        <child link="camera_link"/>
+        <origin xyz="0.13 0.0455 0.429" rpy="0 ${pi/12} 0"/>
+    </joint>
 </robot>
