Commit message: working moveit planner

File: src/robot_description/dual_arm_description/urdf/dual_arm_real.xacro (robot description, xacro)
@@ -3,4 +3,5 @@
     <!-- Public args so launches can change them -->
     <xacro:arg name="robot_name" default="dual_arm_description"/>
+    <xacro:arg name="readonly" default="false"/>
     <!-- Bring in base structure (links, joints, hands) -->
     <xacro:include filename="$(find dual_arm_description)/urdf/dual_arm_base.xacro" />

File: src/robot_description/dual_arm_description/urdf/macros/ros2_control_real.xacro (robot description, xacro)
@@ -6,5 +6,5 @@
         <!-- Select config directory and frequency based on readonly mode -->
         <xacro:property name="config_dir" value="ethercat"/>
-        <xacro:property name="ctrl_freq" value="1000"/>
+        <xacro:property name="ctrl_freq" value="100"/>
         <xacro:if value="$(arg readonly)">
             <xacro:property name="config_dir" value="ethercat_readonly"/>
@@ -23,4 +23,5 @@
                 <state_interface name="velocity"/>
                 <state_interface name="effort"/>
+                <state_interface name="status_word"/>
                 <ec_module name="LeftShoulderPitch">
                     <plugin>ethercat_generic_plugins/EcCiA402Drive</plugin>
@@ -35,4 +36,5 @@
                 <state_interface name="velocity"/>
                 <state_interface name="effort"/>
+                <state_interface name="status_word"/>
                 <ec_module name="LeftShoulderRoll">
                     <plugin>ethercat_generic_plugins/EcCiA402Drive</plugin>
@@ -47,4 +49,5 @@
                 <state_interface name="velocity"/>
                 <state_interface name="effort"/>
+                <state_interface name="status_word"/>
                 <ec_module name="LeftShoulderYaw">
                     <plugin>ethercat_generic_plugins/EcCiA402Drive</plugin>
@@ -59,4 +62,5 @@
                 <state_interface name="velocity"/>
                 <state_interface name="effort"/>
+                <state_interface name="status_word"/>
                 <ec_module name="LeftElbowPitch">
                     <plugin>ethercat_generic_plugins/EcCiA402Drive</plugin>
@@ -71,4 +75,5 @@
                 <state_interface name="velocity"/>
                 <state_interface name="effort"/>
+                <state_interface name="status_word"/>
                 <ec_module name="LeftWristYaw">
                     <plugin>ethercat_generic_plugins/EcCiA402Drive</plugin>
@@ -83,4 +88,5 @@
                 <state_interface name="velocity"/>
                 <state_interface name="effort"/>
+                <state_interface name="status_word"/>
                 <ec_module name="LeftWristRoll">
                     <plugin>ethercat_generic_plugins/EcCiA402Drive</plugin>

File: src/robot_description/full_robot_description/urdf/robot_harambe_v03_proccessed.urdf (robot description, URDF)
Before this commit: robot robot_harambe_v0.3, 26 links, 25 joints
Links:
- link urdf_ankle_assembly: geometry collision mesh filename=package://full_robot_description/meshes/collision/urdf_ankl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; visual mesh filename=package://full_robot_description/meshes/visual/urdf_ankle_a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
- link urdf_ankle_assembly_2: geometry collision mesh filename=package://full_robot_description/meshes/collision/urdf_ankl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; visual mesh filename=package://full_robot_description/meshes/visual/urdf_ankle_a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
- link urdf_base: geometry collision mesh filename=package://full_robot_description/meshes/collision/b_base.stl; collision mesh filename=package://full_robot_description/meshes/collision/f_base.stl
- link urdf_foot_assembly: geometry collision mesh filename=package://full_robot_description/meshes/collision/urdf_foot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; visual mesh filename=package://full_robot_description/meshes/visual/urdf_foot_as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
- link urdf_foot_assembly_2: geometry collision mesh filename=package://full_robot_description/meshes/collision/urdf_foot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; visual mesh filename=package://full_robot_description/meshes/visual/urdf_foot_as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
- link urdf_hip_assembly: geometry collision mesh filename=package://full_robot_description/meshes/collision/hip.stl; visual mesh filename=package://full_robot_description/meshes/visual/hip.stl
- link urdf_hip_assembly_2: geometry collision mesh filename=package://full_robot_description/meshes/collision/hip.stl; visual mesh filename=package://full_robot_description/meshes/visual/hip.stl
- link urdf_l_elbow_assembly: geometry collision mesh filename=package://full_robot_description/meshes/collision/urdf_l_el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; visual mesh filename=package://full_robot_description/meshes/visual/stator_x6_p2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
- link urdf_l_lower_forearm_assembly: geometry collision mesh filename=package://full_robot_description/meshes/collision/urdf_l_lo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; visual mesh filename=package://full_robot_description/meshes/visual/stator_x4_p3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
- link urdf_l_shoulder_assembly: geometry collision mesh filename=package://full_robot_description/meshes/collision/l_shoulde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; visual mesh filename=package://full_robot_description/meshes/visual/l_shoulder.s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
- link urdf_l_tibia_assembly: geometry collision mesh filename=package://full_robot_description/meshes/collision/urdf_l_ti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; visual mesh filename=package://full_robot_description/meshes/visual/m6_threaded_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
- link urdf_l_upper_arm_assembly: geometry collision mesh filename=package://full_robot_description/meshes/collision/urdf_l_up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; visual mesh filename=package://full_robot_description/meshes/visual/stator_x4_p3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
- link urdf_l_upper_femur_assembly: geometry collision mesh filename=package://full_robot_description/meshes/collision/l_upper_f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; visual mesh filename=package://full_robot_description/meshes/visual/l_upper_femu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
- link urdf_l_upper_forearm_assembly: geometry collision mesh filename=package://full_robot_description/meshes/collision/urdf_l_up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; visual mesh filename=package://full_robot_description/meshes/visual/stator_x4_p3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
- link urdf_l_wrist_assembly: geometry collision mesh filename=package://full_robot_description/meshes/collision/l_wrist.s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; visual mesh filename=package://full_robot_description/meshes/visual/l_wrist.stl
- link urdf_lower_femur_assembly: geometry collision mesh filename=package://full_robot_description/meshes/collision/lower_fem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; visual mesh filename=package://full_robot_description/meshes/visual/lower_femur.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
- link urdf_lower_femur_assembly_2: geometry collision mesh filename=package://full_robot_description/meshes/collision/lower_fem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; visual mesh filename=package://full_robot_description/meshes/visual/lower_femur.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
- link urdf_r_elbow_assembly: geometry collision mesh filename=package://full_robot_description/meshes/collision/r_elbow.s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; visual mesh filename=package://full_robot_description/meshes/visual/r_elbow.stl
- link urdf_r_lower_forearm_assembly: geometry collision mesh filename=package://full_robot_description/meshes/collision/r_lower_f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; visual mesh filename=package://full_robot_description/meshes/visual/r_lower_fore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
- link urdf_r_shoulder_assembly: geometry collision mesh filename=package://full_robot_description/meshes/collision/r_shoulde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; visual mesh filename=package://full_robot_description/meshes/visual/r_shoulder.s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
- link urdf_r_tibia_assembly: geometry collision mesh filename=package://full_robot_description/meshes/collision/urdf_r_ti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; visual mesh filename=package://full_robot_description/meshes/visual/m6_threaded_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
- link urdf_r_upper_arm_assembly: geometry collision mesh filename=package://full_robot_description/meshes/collision/r_upper_a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; visual mesh filename=package://full_robot_description/meshes/visual/r_upper_arm.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
- link urdf_r_upper_femur_assemby: geometry collision mesh filename=package://full_robot_description/meshes/collision/r_upper_f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; visual mesh filename=package://full_robot_description/meshes/visual/r_upper_femu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
- link urdf_r_upper_forearm_assembly: geometry collision mesh filename=package://full_robot_description/meshes/collision/r_upper_f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; visual mesh filename=package://full_robot_description/meshes/visual/r_upper_fore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
- link urdf_r_wrist_assembly: geometry collision mesh filename=package://full_robot_description/meshes/collision/r_wrist.s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; visual mesh filename=package://full_robot_description/meshes/visual/r_wrist.stl
- link urdf_simplified_torso: geometry collision mesh filename=package://full_robot_description/meshes/collision/head.stl; collision mesh filename=package://full_robot_description/meshes/collision/urdf_simp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
