Commit message: Fix dual arm Gazebo simulation: controllers now activate successfully
Root cause: the robot's urdf_base is at the waist, with all links
extending downward (arms to z=-0.83, legs to z=-0.6). Spawning at z=0
embedded all 208 collision bodies inside the ground plane, causing DART
physics to stall and controller switches to never complete.

Changes:
- Add world_joint (fixed) to pin robot base in Gazebo simulation
- Spawn robot at z=1.0 to keep all links above ground
- Create dual_arm_gazebo world file with 5ms physics step (vs 1ms)
- Fix headless_sim package refs (arm_gazebo → dual_arm_gazebo)
- Consolidate ros2_control from 4 to 2 hardware systems (ArmSystem + HandSystem)
- Tune controller spawner timeouts for heavier model

File: src/robot_description/dual_arm_description/urdf/dual_arm.urdf.xacro (robot description, xacro)
@@ -1,4 +1,11 @@
 <?xml version="1.0"?>
 <robot xmlns:xacro="http://ros.org/wiki/xacro" name="dual_arm_description">
-  <xacro:include filename="$(find dual_arm_description)/urdf/dual_arm_base.xacro" />
+    <!-- Select robot variant (base or gazebo) -->
+    <xacro:arg name="use_sim" default="false" />
+    <xacro:if value="$(arg use_sim)">
+        <xacro:include filename="$(find dual_arm_description)/urdf/dual_arm_gazebo.xacro" />
+    </xacro:if>
+    <xacro:unless value="$(arg use_sim)">
+        <xacro:include filename="$(find dual_arm_description)/urdf/dual_arm_base.xacro" />
+    </xacro:unless>
 </robot>

File: src/robot_description/dual_arm_description/urdf/dual_arm_base.xacro (robot description, xacro)
@@ -1,4 +1,4 @@
 <?xml version="1.0"?>
-<robot xmlns:xacro="http://ros.org/wiki/xacro">
+<robot xmlns:xacro="http://ros.org/wiki/xacro" name="dual_arm_base">
   <xacro:include filename="$(find dual_arm_description)/urdf/links/dual_arm_links.xacro" />
   <xacro:include filename="$(find dual_arm_description)/urdf/joints/dual_arm_joints.xacro" />

File: src/robot_description/hand_description/urdf/hands/inspire_hand_right.xacro (robot description, xacro)
@@ -1,4 +1,6 @@
 <?xml version="1.0"?>
 <robot xmlns:xacro="http://www.ros.org/wiki/xacro">
+  <!-- Inspire Hand Right - Dexterous 6-DOF hand
+       Collision geometry uses box primitives (OBJ meshes lack normals for DART) -->
   <xacro:macro name="inspire_hand_right" params="parent prefix:=right_ mount_x:=0.0 mount_y:=0.0 mount_z:=0.0 mount_roll:=0.0 mount_pitch:=0.0 mount_yaw:=0.0">
     <joint name="${prefix}hand_base_joint" type="fixed">
@@ -81,7 +83,7 @@
         </visual>
         <collision>
-          <origin xyz="0 0 0" rpy="0 0 0"/>
-          <geometry>
-            <mesh filename="package://hand_description/meshes/inspire_hand/collision/right_thumb_proximal_base.obj"/>
+          <origin xyz="0.005 0.001 -0.007" rpy="0 0 0"/>
+          <geometry>
+            <box size="0.015 0.012 0.014"/>
           </geometry>
         </collision>
@@ -107,7 +109,7 @@
         </visual>
         <collision>
-          <origin xyz="0 0 0" rpy="0 0 0"/>
-          <geometry>
-            <mesh filename="package://hand_description/meshes/inspire_hand/collision/right_thumb_proximal.obj"/>
+          <origin xyz="0.022 0.013 -0.008" rpy="0 0 0"/>
+          <geometry>
+            <box size="0.050 0.030 0.016"/>
           </geometry>
         </collision>
@@ -133,7 +135,7 @@
         </visual>
         <collision>
-          <origin xyz="0 0 0" rpy="0 0 0"/>
-          <geometry>
-            <mesh filename="package://hand_description/meshes/inspire_hand/collision/right_thumb_intermediate.obj"/>
+          <origin xyz="0.010 0.002 -0.007" rpy="0 0 0"/>
+          <geometry>
+            <box size="0.025 0.014 0.014"/>
           </geometry>
         </collision>
@@ -160,7 +162,7 @@
         </visual>
         <collision>
-          <origin xyz="0 0 0" rpy="0 0 0"/>
-          <geometry>
-            <mesh filename="package://hand_description/meshes/inspire_hand/collision/right_thumb_distal.obj"/>
+          <origin xyz="0.010 0.007 -0.006" rpy="0 0 0"/>
+          <geometry>
+            <box size="0.024 0.016 0.012"/>
           </geometry>
         </collision>
@@ -187,7 +189,7 @@
         </visual>
         <collision>
-          <origin xyz="0 0 0" rpy="0 0 0"/>
-          <geometry>
-            <mesh filename="package://hand_description/meshes/inspire_hand/collision/right_index_proximal.obj"/>
+          <origin xyz="0.001 0.014 -0.006" rpy="0 0 0"/>
+          <geometry>
+            <box size="0.014 0.032 0.012"/>
           </geometry>
         </collision>
@@ -213,7 +215,7 @@
         </visual>
         <collision>
-          <origin xyz="0 0 0" rpy="0 0 0"/>
-          <geometry>
-            <mesh filename="package://hand_description/meshes/inspire_hand/collision/right_index_intermediate.obj"/>
+          <origin xyz="0.001 0.020 -0.005" rpy="0 0 0"/>
+          <geometry>
+            <box size="0.014 0.042 0.010"/>
           </geometry>
         </collision>
@@ -240,7 +242,7 @@
         </visual>
         <collision>
-          <origin xyz="0 0 0" rpy="0 0 0"/>
-          <geometry>
-            <mesh filename="package://hand_description/meshes/inspire_hand/collision/right_index_proximal.obj"/>
+          <origin xyz="0.001 0.014 -0.006" rpy="0 0 0"/>
+          <geometry>
+            <box size="0.014 0.032 0.012"/>
           </geometry>
         </collision>
@@ -266,7 +268,7 @@
         </visual>
         <collision>
-          <origin xyz="0 0 0" rpy="0 0 0"/>
-          <geometry>
-            <mesh filename="package://hand_description/meshes/inspire_hand/collision/right_middle_intermediate.obj"/>
+          <origin xyz="0.001 0.022 -0.005" rpy="0 0 0"/>
+          <geometry>
+            <box size="0.014 0.046 0.010"/>
           </geometry>
         </collision>
@@ -293,7 +295,7 @@
         </visual>
         <collision>
-          <origin xyz="0 0 0" rpy="0 0 0"/>
-          <geometry>
-            <mesh filename="package://hand_description/meshes/inspire_hand/collision/right_index_proximal.obj"/>
+          <origin xyz="0.001 0.014 -0.006" rpy="0 0 0"/>
+          <geometry>
+            <box size="0.014 0.032 0.012"/>
           </geometry>
         </collision>
@@ -319,7 +321,7 @@
         </visual>
         <collision>
-          <origin xyz="0 0 0" rpy="0 0 0"/>
-          <geometry>
-            <mesh filename="package://hand_description/meshes/inspire_hand/collision/right_index_intermediate.obj"/>
+          <origin xyz="0.001 0.020 -0.005" rpy="0 0 0"/>
+          <geometry>
+            <box size="0.014 0.042 0.010"/>
           </geometry>
         </collision>
@@ -346,7 +348,7 @@
         </visual>
         <collision>
-          <origin xyz="0 0 0" rpy="0 0 0"/>
-          <geometry>
-            <mesh filename="package://hand_description/meshes/inspire_hand/collision/right_index_proximal.obj"/>
+          <origin xyz="0.001 0.014 -0.006" rpy="0 0 0"/>
+          <geometry>
+            <box size="0.014 0.032 0.012"/>
           </geometry>
         </collision>
@@ -372,7 +374,7 @@
         </visual>
         <collision>
-          <origin xyz="0 0 0" rpy="0 0 0"/>
-          <geometry>
-            <mesh filename="package://hand_description/meshes/inspire_hand/collision/right_pinky_intermediate.obj"/>
+          <origin xyz="0.002 0.016 -0.005" rpy="0 0 0"/>
+          <geometry>
+            <box size="0.014 0.034 0.010"/>
           </geometry>
         </collision>
