Commit message: update urdf

File: src/robot_description/dual_arm_description/urdf/links/dual_arm_links.xacro (robot description, xacro)
@@ -1,13 +1,15 @@
 <?xml version="1.0"?>
 <robot xmlns:xacro="http://www.ros.org/wiki/xacro">
+  <!-- ================================================================== -->
+  <!-- Base                                                                -->
+  <!-- ================================================================== -->
   <link name="urdf_base">
     <inertial>
-      <origin xyz="0.000699525 0.0334287 -0.43102" rpy="0 0 0"/>
+      <origin xyz="0.0334287 -0.000699525 -0.43102" rpy="0 0 0"/>
       <mass value="5.132"/>
-      <inertia ixx="0.022223" ixy="-1.07667e-07" ixz="4.86506e-08" iyy="0.0311091" iyz="-5.11204e-05" izz="0.0168242"/>
-    </inertial>
-    <!-- Part b_base -->
-    <visual>
-      <origin xyz="0.000698397 -0.00277529 -0.432554" rpy="1.41455e-17 -2.93952e-16 4.31931e-15"/>
+      <inertia ixx="0.0311091" ixy="1.07667e-07" ixz="-5.11204e-05" iyy="0.022223" iyz="-4.86506e-08" izz="0.0168242"/>
+    </inertial>
+    <visual>
+      <origin xyz="-0.00277529 -0.000698397 -0.432554" rpy="0 0 -1.5708"/>
       <geometry>
         <mesh filename="package://dual_arm_description/meshes/visual/b_base.stl"/>
@@ -18,12 +20,11 @@
     </visual>
     <collision>
-      <origin xyz="0.000698397 -0.00277529 -0.432554" rpy="1.41455e-17 -2.93952e-16 4.31931e-15"/>
+      <origin xyz="-0.00277529 -0.000698397 -0.432554" rpy="0 0 -1.5708"/>
       <geometry>
         <mesh filename="package://dual_arm_description/meshes/visual/b_base.stl"/>
       </geometry>
     </collision>
-    <!-- Part f_base -->
-    <visual>
-      <origin xyz="0.000705351 0.070373 -0.431099" rpy="1.41455e-17 -2.93952e-16 4.31931e-15"/>
+    <visual>
+      <origin xyz="0.070373 -0.000705351 -0.431099" rpy="0 0 -1.5708"/>
       <geometry>
         <mesh filename="package://dual_arm_description/meshes/visual/f_base.stl"/>
@@ -34,307 +35,21 @@
     </visual>
     <collision>
-      <origin xyz="0.000705351 0.070373 -0.431099" rpy="1.41455e-17 -2.93952e-16 4.31931e-15"/>
+      <origin xyz="0.070373 -0.000705351 -0.431099" rpy="0 0 -1.5708"/>
       <geometry>
         <mesh filename="package://dual_arm_description/meshes/visual/f_base.stl"/>
       </geometry>
     </collision>
-    <!-- Part rotor_x8_p20_120 -->
-    <visual>
-      <origin xyz="0.0146991 0.0333466 -0.46826" rpy="-4.31931e-15 1.5708 0"/>
-      <geometry>
-        <mesh filename="package://dual_arm_description/meshes/visual/rotor_x8_p20_120.stl"/>
-      </geometry>
-      <material name="rotor_x8_p20_120_material">
-        <color rgba="0.596078 0.176471 0.0509804 1"/>
-      </material>
-    </visual>
-    <collision>
-      <origin xyz="0.0146991 0.0333466 -0.46826" rpy="-4.31931e-15 1.5708 0"/>
-      <geometry>
-        <mesh filename="package://dual_arm_description/meshes/visual/rotor_x8_p20_120.stl"/>
-      </geometry>
-    </collision>
-    <!-- Part stator_x8_p20_120 -->
-    <visual>
-      <origin xyz="0.0146991 0.0333466 -0.46826" rpy="1.5708 -0.785398 1.5708"/>
-      <geometry>
-        <mesh filename="package://dual_arm_description/meshes/visual/stator_x8_p20_120.stl"/>
-      </geometry>
-      <material name="stator_x8_p20_120_material">
-        <color rgba="0.882353 0.572549 0.478431 1"/>
-      </material>
-    </visual>
-    <collision>
-      <origin xyz="0.0146991 0.0333466 -0.46826" rpy="1.5708 -0.785398 1.5708"/>
-      <geometry>
-        <mesh filename="package://dual_arm_description/meshes/visual/stator_x8_p20_120.stl"/>
-      </geometry>
-    </collision>
-    <!-- Part rotor_x8_p20_120_2 -->
-    <visual>
-      <origin xyz="-0.0133009 0.0333466 -0.46826" rpy="4.31931e-15 -1.5708 0"/>
-      <geometry>
-        <mesh filename="package://dual_arm_description/meshes/visual/rotor_x8_p20_120.stl"/>
-      </geometry>
-      <material name="rotor_x8_p20_120_2_material">
-        <color rgba="0.596078 0.176471 0.0509804 1"/>
-      </material>
-    </visual>
-    <collision>
-      <origin xyz="-0.0133009 0.0333466 -0.46826" rpy="4.31931e-15 -1.5708 0"/>
-      <geometry>
-        <mesh filename="package://dual_arm_description/meshes/visual/rotor_x8_p20_120.stl"/>
-      </geometry>
-    </collision>
-    <!-- Part stator_x8_p20_120_2 -->
-    <visual>
-      <origin xyz="-0.0133009 0.0333466 -0.46826" rpy="1.5708 0.785398 -1.5708"/>
-      <geometry>
-        <mesh filename="package://dual_arm_description/meshes/visual/stator_x8_p20_120.stl"/>
-      </geometry>
-      <material name="stator_x8_p20_120_2_material">
-        <color rgba="0.882353 0.572549 0.478431 1"/>
-      </material>
-    </visual>
-    <collision>
-      <origin xyz="-0.0133009 0.0333466 -0.46826" rpy="1.5708 0.785398 -1.5708"/>
-      <geometry>
-        <mesh filename="package://dual_arm_description/meshes/visual/stator_x8_p20_120.stl"/>
-      </geometry>
-    </collision>
-    <!-- Part rotor_x8_p20_120_3 -->
-    <visual>
-      <origin xyz="0.000699067 0.0333466 -0.39426" rpy="1.41455e-17 -2.93952e-16 4.31931e-15"/>
-      <geometry>
-        <mesh filename="package://dual_arm_description/meshes/visual/rotor_x8_p20_120.stl"/>
-      </geometry>
-      <material name="rotor_x8_p20_120_3_material">
-        <color rgba="0.596078 0.176471 0.0509804 1"/>
-      </material>
-    </visual>
-    <collision>
-      <origin xyz="0.000699067 0.0333466 -0.39426" rpy="1.41455e-17 -2.93952e-16 4.31931e-15"/>
-      <geometry>
-        <mesh filename="package://dual_arm_description/meshes/visual/rotor_x8_p20_120.stl"/>
-      </geometry>
-    </collision>
-    <!-- Part stator_x8_p20_120_3 -->
-    <visual>
-      <origin xyz="0.000699067 0.0333466 -0.39426" rpy="-1.41455e-17 2.93952e-16 -3.14159"/>
-      <geometry>
-        <mesh filename="package://dual_arm_description/meshes/visual/stator_x8_p20_120.stl"/>
-      </geometry>
-      <material name="stator_x8_p20_120_3_material">
-        <color rgba="0.882353 0.572549 0.478431 1"/>
-      </material>
-    </visual>
-    <collision>
-      <origin xyz="0.000699067 0.0333466 -0.39426" rpy="-1.41455e-17 2.93952e-16 -3.14159"/>
-      <geometry>
-        <mesh filename="package://dual_arm_description/meshes/visual/stator_x8_p20_120.stl"/>
-      </geometry>
-    </collision>
-  </link>
+  </link>
+  <!-- ================================================================== -->
+  <!-- Torso                                                               -->
+  <!-- ================================================================== -->
   <link name="urdf_simplified_torso_sub_assembly">
     <inertial>
-      <origin xyz="1.31908e-06 -0.00281871 -0.293935" rpy="0 0 0"/>
+      <origin xyz="0.00281871 -1.31908e-06 0.293935" rpy="0 0 0"/>
       <mass value="12.1543"/>
-      <inertia ixx="0.748255" ixy="-1.60096e-07" ixz="-1.32781e-06" iyy="0.865047" iyz="0.000814956" izz="0.171754"/>
-    </inertial>
-    <!-- Part urdf_btu_263 -->
-    <visual>
-      <origin xyz="1.69581e-06 0.069996 -0.481" rpy="3.14159 1.67633e-30 3.05311e-16"/>
-      <geometry>
-        <mesh filename="package://dual_arm_description/meshes/visual/urdf_btu_263.stl"/>
-      </geometry>
-      <material name="urdf_btu_263_material">
-        <color rgba="0.231373 0.380392 0.705882 1"/>
-      </material>
-    </visual>
-    <collision>
-      <origin xyz="1.69581e-06 0.069996 -0.481" rpy="3.14159 1.67633e-30 3.05311e-16"/>
-      <geometry>
-        <mesh filename="package://dual_arm_description/meshes/visual/urdf_btu_263.stl"/>
-      </geometry>
-    </collision>
-    <!-- Part urdf_rbm_120 -->
-    <visual>
-      <origin xyz="0.0700017 -3.95689e-06 -0.014" rpy="-3.14159 1.67633e-30 3.05311e-16"/>
-      <geometry>
-        <mesh filename="package://dual_arm_description/meshes/visual/urdf_rbm_120.stl"/>
-      </geometry>
-      <material name="urdf_rbm_120_material">
-        <color rgba="0.615686 0.811765 0.929412 1"/>
-      </material>
-    </visual>
-    <collision>
-      <origin xyz="0.0700017 -3.95689e-06 -0.014" rpy="-3.14159 1.67633e-30 3.05311e-16"/>
-      <geometry>
-        <mesh filename="package://dual_arm_description/meshes/visual/urdf_rbm_120.stl"/>
-      </geometry>
-    </collision>
-    <!-- Part urdf_ftl_263 -->
-    <visual>
-      <origin xyz="1.69581e-06 -0.070004 -0.361" rpy="3.14159 1.67633e-30 3.05311e-16"/>
-      <geometry>
-        <mesh filename="package://dual_arm_description/meshes/visual/urdf_ftl_263.stl"/>
-      </geometry>
-      <material name="urdf_ftl_263_material">
-        <color rgba="0.917647 0.917647 0.917647 1"/>
-      </material>
-    </visual>
-    <collision>
-      <origin xyz="1.69581e-06 -0.070004 -0.361" rpy="3.14159 1.67633e-30 3.05311e-16"/>
-      <geometry>
-        <mesh filename="package://dual_arm_description/meshes/visual/urdf_ftl_263.stl"/>
-      </geometry>
-    </collision>
-    <!-- Part urdf_br_467 -->
-    <visual>
-      <origin xyz="0.141502 0.069996 -0.2575" rpy="-3.14159 1.87354e-30 3.05311e-16"/>
-      <geometry>
-        <mesh filename="package://dual_arm_description/meshes/visual/urdf_br_467.stl"/>
-      </geometry>
-      <material name="urdf_br_467_material">
-        <color rgba="0.768627 0.886275 0.952941 1"/>
-      </material>
-    </visual>
-    <collision>
-      <origin xyz="0.141502 0.069996 -0.2575" rpy="-3.14159 1.87354e-30 3.05311e-16"/>
-      <geometry>
-        <mesh filename="package://dual_arm_description/meshes/visual/urdf_br_467.stl"/>
-      </geometry>
-    </collision>
-    <!-- Part urdf_ftu_263 -->
-    <visual>
-      <origin xyz="1.69581e-06 -0.070004 -0.481" rpy="3.14159 1.57772e-30 3.05311e-16"/>
-      <geometry>
-        <mesh filename="package://dual_arm_description/meshes/visual/urdf_ftu_263.stl"/>
-      </geometry>
-      <material name="urdf_ftu_263_material">
-        <color rgba="0.917647 0.917647 0.917647 1"/>
-      </material>
-    </visual>
-    <collision>
-      <origin xyz="1.69581e-06 -0.070004 -0.481" rpy="3.14159 1.57772e-30 3.05311e-16"/>
-      <geometry>
-        <mesh filename="package://dual_arm_description/meshes/visual/urdf_ftu_263.stl"/>
-      </geometry>
-    </collision>
-    <!-- Part urdf_bb_303 -->
-    <visual>
-      <origin xyz="1.69581e-06 0.069996 -0.014" rpy="-3.14159 1.87354e-30 2.77556e-16"/>
-      <geometry>
-        <mesh filename="package://dual_arm_description/meshes/visual/urdf_bb_303.stl"/>
-      </geometry>
-      <material name="urdf_bb_303_material">
-        <color rgba="0.231373 0.380392 0.705882 1"/>
-      </material>
-    </visual>
-    <collision>
-      <origin xyz="1.69581e-06 0.069996 -0.014" rpy="-3.14159 1.87354e-30 2.77556e-16"/>
-      <geometry>
-        <mesh filename="package://dual_arm_description/meshes/visual/urdf_bb_303.stl"/>
-      </geometry>
-    </collision>
-    <!-- Part urdf_bl_467 -->
-    <visual>
-      <origin xyz="-0.141498 0.069996 -0.2575" rpy="-3.14159 1.87354e-30 3.05311e-16"/>
-      <geometry>
-        <mesh filename="package://dual_arm_description/meshes/visual/urdf_bl_467.stl"/>
-      </geometry>
-      <material name="urdf_bl_467_material">
-        <color rgba="0.768627 0.886275 0.952941 1"/>
-      </material>
-    </visual>
-    <collision>
-      <origin xyz="-0.141498 0.069996 -0.2575" rpy="-3.14159 1.87354e-30 3.05311e-16"/>
-      <geometry>
-        <mesh filename="package://dual_arm_description/meshes/visual/urdf_bl_467.stl"/>
-      </geometry>
-    </collision>
-    <!-- Part urdf_fb_303 -->
-    <visual>
-      <origin xyz="1.69581e-06 -0.070004 -0.014" rpy="-3.14159 1.87354e-30 3.05311e-16"/>
-      <geometry>
-        <mesh filename="package://dual_arm_description/meshes/visual/urdf_fb_303.stl"/>
-      </geometry>
-      <material name="urdf_fb_303_material">
-        <color rgba="0.917647 0.917647 0.917647 1"/>
-      </material>
-    </visual>
-    <collision>
-      <origin xyz="1.69581e-06 -0.070004 -0.014" rpy="-3.14159 1.87354e-30 3.05311e-16"/>
-      <geometry>
-        <mesh filename="package://dual_arm_description/meshes/visual/urdf_fb_303.stl"/>
-      </geometry>
-    </collision>
-    <!-- Part urdf_lbm_120 -->
-    <visual>
-      <origin xyz="-0.0699983 -3.95689e-06 -0.014" rpy="-3.14159 1.77494e-30 3.05311e-16"/>
-      <geometry>
-        <mesh filename="package://dual_arm_description/meshes/visual/urdf_lbm_120.stl"/>
-      </geometry>
-      <material name="urdf_lbm_120_material">
-        <color rgba="0.615686 0.811765 0.929412 1"/>
-      </material>
-    </visual>
-    <collision>
-      <origin xyz="-0.0699983 -3.95689e-06 -0.014" rpy="-3.14159 1.77494e-30 3.05311e-16"/>
-      <geometry>
-        <mesh filename="package://dual_arm_description/meshes/visual/urdf_lbm_120.stl"/>
-      </geometry>
-    </collision>
-    <!-- Part urdf_lm_120 -->
-    <visual>
-      <origin xyz="-0.141498 -3.95689e-06 -0.211" rpy="3.14159 1.62703e-30 3.05311e-16"/>
-      <geometry>
-        <mesh filename="package://dual_arm_description/meshes/visual/urdf_lm_120.stl"/>
-      </geometry>
-      <material name="urdf_lm_120_material">
-        <color rgba="0.647059 0.647059 0.647059 1"/>
-      </material>
-    </visual>
-    <collision>
-      <origin xyz="-0.141498 -3.95689e-06 -0.211" rpy="3.14159 1.62703e-30 3.05311e-16"/>
-      <geometry>
-        <mesh filename="package://dual_arm_description/meshes/visual/urdf_lm_120.stl"/>
-      </geometry>
-    </collision>
-    <!-- Part urdf_ltu_120 -->
-    <visual>
-      <origin xyz="-0.141498 -3.95689e-06 -0.481" rpy="3.14159 1.67633e-30 3.05311e-16"/>
-      <geometry>
-        <mesh filename="package://dual_arm_description/meshes/visual/urdf_ltu_120.stl"/>
-      </geometry>
-      <material name="urdf_ltu_120_material">
-        <color rgba="0.647059 0.647059 0.647059 1"/>
-      </material>
-    </visual>
-    <collision>
-      <origin xyz="-0.141498 -3.95689e-06 -0.481" rpy="3.14159 1.67633e-30 3.05311e-16"/>
-      <geometry>
-        <mesh filename="package://dual_arm_description/meshes/visual/urdf_ltu_120.stl"/>
-      </geometry>
-    </collision>
-    <!-- Part urdf_rm_120 -->
-    <visual>
-      <origin xyz="0.141502 -3.95689e-06 -0.211" rpy="3.14159 1.77494e-30 3.05311e-16"/>
-      <geometry>
-        <mesh filename="package://dual_arm_description/meshes/visual/urdf_rm_120.stl"/>
-      </geometry>
-      <material name="urdf_rm_120_material">
-        <color rgba="0.647059 0.647059 0.647059 1"/>
-      </material>
-    </visual>
-    <collision>
-      <origin xyz="0.141502 -3.95689e-06 -0.211" rpy="3.14159 1.77494e-30 3.05311e-16"/>
-      <geometry>
-        <mesh filename="package://dual_arm_description/meshes/visual/urdf_rm_120.stl"/>
-      </geometry>
-    </collision>
-    <!-- Part urdf_r_shoulder_plate -->
-    <visual>
-      <origin xyz="0.151502 -3.95689e-06 -0.42041" rpy="-3.14159 3.64232e-22 4.51671e-32"/>
+      <inertia ixx="0.865047" ixy="-1.60096e-07" ixz="0.000814956" iyy="0.748255" iyz="-1.32781e-06" izz="0.171754"/>
+    </inertial>
+    <visual>
+      <origin xyz="3.95689e-06 -0.151502 0.42041" rpy="0 0 -1.5708"/>
       <geometry>
         <mesh filename="package://dual_arm_description/meshes/visual/urdf_r_shoulder_plate.stl"/>
@@ -345,28 +60,11 @@
     </visual>
     <collision>
-      <origin xyz="0.151502 -3.95689e-06 -0.42041" rpy="-3.14159 3.64232e-22 4.51671e-32"/>
+      <origin xyz="3.95689e-06 -0.151502 0.42041" rpy="0 0 -1.5708"/>
       <geometry>
         <mesh filename="package://dual_arm_description/meshes/visual/urdf_r_shoulder_plate.stl"/>
       </geometry>
     </collision>
-    <!-- Part urdf_rb_120 -->
-    <visual>
-      <origin xyz="0.141502 -3.95689e-06 -0.014" rpy="-3.14159 1.77494e-30 3.05311e-16"/>
-      <geometry>
-        <mesh filename="package://dual_arm_description/meshes/visual/urdf_rb_120.stl"/>
-      </geometry>
-      <material name="urdf_rb_120_material">
-        <color rgba="0.647059 0.647059 0.647059 1"/>
-      </material>
-    </visual>
-    <collision>
-      <origin xyz="0.141502 -3.95689e-06 -0.014" rpy="-3.14159 1.77494e-30 3.05311e-16"/>
-      <geometry>
-        <mesh filename="package://dual_arm_description/meshes/visual/urdf_rb_120.stl"/>
-      </geometry>
-    </collision>
-    <!-- Part urdf_l_shoulder_plate -->
-    <visual>
-      <origin xyz="-0.153498 -3.95689e-06 -0.42041" rpy="3.14159 1.77494e-30 3.05311e-16"/>
+    <visual>
+      <origin xyz="3.95689e-06 0.153498 0.42041" rpy="0 0 -1.5708"/>
       <geometry>
         <mesh filename="package://dual_arm_description/meshes/visual/urdf_l_shoulder_plate.stl"/>
@@ -377,108 +75,11 @@
     </visual>
     <collision>
-      <origin xyz="-0.153498 -3.95689e-06 -0.42041" rpy="3.14159 1.77494e-30 3.05311e-16"/>
+      <origin xyz="3.95689e-06 0.153498 0.42041" rpy="0 0 -1.5708"/>
       <geometry>
         <mesh filename="package://dual_arm_description/meshes/visual/urdf_l_shoulder_plate.stl"/>
       </geometry>
     </collision>
-    <!-- Part urdf_btl_263 -->
-    <visual>
-      <origin xyz="1.69581e-06 0.069996 -0.361" rpy="3.14159 1.87354e-30 3.05311e-16"/>
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