Commit message: functional ethercat monitor, calibration tools, icube transition

File: src/robot_description/dual_arm_description/urdf/dual_arm.urdf.xacro (robot description, xacro)
@@ -5,4 +5,5 @@
     <xacro:arg name="use_isaac" default="false" />
     <xacro:arg name="fixed_legs" default="true" />
+    <xacro:arg name="readonly" default="false" />
     <xacro:if value="$(arg use_isaac)">
         <xacro:include filename="$(find dual_arm_description)/urdf/dual_arm_isaac.xacro" />

File: src/robot_description/dual_arm_description/urdf/macros/ros2_control_real.xacro (robot description, xacro)
@@ -2,74 +2,91 @@
 <robot xmlns:xacro="http://ros.org/wiki/xacro">
     <!-- ros2_control interface for real EtherCAT hardware -->
-    <!-- Mirrors ros2_control.xacro but uses MyActuator EtherCAT plugin -->
+    <!-- Uses ethercat_driver_ros2 (ICube-Robotics) with EcCiA402Drive per joint -->
     <xacro:macro name="dual_arm_ros2_control_real">
+        <!-- Select config directory and frequency based on readonly mode -->
+        <xacro:property name="config_dir" value="ethercat"/>
+        <xacro:property name="ctrl_freq" value="1000"/>
+        <xacro:if value="$(arg readonly)">
+            <xacro:property name="config_dir" value="ethercat_readonly"/>
+            <xacro:property name="ctrl_freq" value="100"/>
+        </xacro:if>
         <!-- Left arm — 6 DOF EtherCAT actuators (MyActuator RMD X V4) -->
         <ros2_control name="LeftArmSystem" type="system">
             <hardware>
-                <plugin>myactuator_hardware/MyActuatorSystem</plugin>
-                <param name="ethercat_master_index">0</param>
-                <param name="network_interface">eth0</param>
-                <param name="cycle_time_us">1000</param>
-                <param name="dc_sync">true</param>
+                <plugin>ethercat_driver/EthercatDriver</plugin>
+                <param name="master_id">0</param>
+                <param name="control_frequency">${ctrl_freq}</param>
             </hardware>
             <joint name="left_shoulder_pitch_joint_X6">
-                <param name="slave_position">0</param>
-                <param name="motor_type">X6</param>
-                <param name="direction">1</param>
-                <param name="offset_raw">0</param>
                 <command_interface name="position"/>
                 <state_interface name="position"/>
                 <state_interface name="velocity"/>
                 <state_interface name="effort"/>
+                <ec_module name="LeftShoulderPitch">
+                    <plugin>ethercat_generic_plugins/EcCiA402Drive</plugin>
+                    <param name="alias">0</param>
+                    <param name="position">0</param>
+                    <param name="slave_config">$(find arm_real_bringup)/config/${config_dir}/left_shoulder_pitch_X6.yaml</param>
+                </ec_module>
             </joint>
             <joint name="left_shoulder_roll_joint_X6">
-                <param name="slave_position">1</param>
-                <param name="motor_type">X6</param>
-                <param name="direction">1</param>
-                <param name="offset_raw">0</param>
                 <command_interface name="position"/>
                 <state_interface name="position"/>
                 <state_interface name="velocity"/>
                 <state_interface name="effort"/>
+                <ec_module name="LeftShoulderRoll">
+                    <plugin>ethercat_generic_plugins/EcCiA402Drive</plugin>
+                    <param name="alias">0</param>
+                    <param name="position">1</param>
+                    <param name="slave_config">$(find arm_real_bringup)/config/${config_dir}/left_shoulder_roll_X6.yaml</param>
+                </ec_module>
             </joint>
             <joint name="left_shoulder_yaw_joint_X4">
-                <param name="slave_position">2</param>
-                <param name="motor_type">X4</param>
-                <param name="direction">-1</param>
-                <param name="offset_raw">0</param>
                 <command_interface name="position"/>
                 <state_interface name="position"/>
                 <state_interface name="velocity"/>
                 <state_interface name="effort"/>
+                <ec_module name="LeftShoulderYaw">
+                    <plugin>ethercat_generic_plugins/EcCiA402Drive</plugin>
+                    <param name="alias">0</param>
+                    <param name="position">2</param>
+                    <param name="slave_config">$(find arm_real_bringup)/config/${config_dir}/left_shoulder_yaw_X4.yaml</param>
+                </ec_module>
             </joint>
             <joint name="left_elbow_pitch_joint_X6">
-                <param name="slave_position">3</param>
-                <param name="motor_type">X6</param>
-                <param name="direction">1</param>
-                <param name="offset_raw">0</param>
                 <command_interface name="position"/>
                 <state_interface name="position"/>
                 <state_interface name="velocity"/>
                 <state_interface name="effort"/>
+                <ec_module name="LeftElbowPitch">
+                    <plugin>ethercat_generic_plugins/EcCiA402Drive</plugin>
+                    <param name="alias">0</param>
+                    <param name="position">3</param>
+                    <param name="slave_config">$(find arm_real_bringup)/config/${config_dir}/left_elbow_pitch_X6.yaml</param>
+                </ec_module>
             </joint>
             <joint name="left_wrist_yaw_joint_X4">
-                <param name="slave_position">4</param>
-                <param name="motor_type">X4</param>
-                <param name="direction">-1</param>
-                <param name="offset_raw">0</param>
                 <command_interface name="position"/>
                 <state_interface name="position"/>
                 <state_interface name="velocity"/>
                 <state_interface name="effort"/>
+                <ec_module name="LeftWristYaw">
+                    <plugin>ethercat_generic_plugins/EcCiA402Drive</plugin>
+                    <param name="alias">0</param>
+                    <param name="position">4</param>
+                    <param name="slave_config">$(find arm_real_bringup)/config/${config_dir}/left_wrist_yaw_X4.yaml</param>
+                </ec_module>
             </joint>
             <joint name="left_wrist_roll_joint_X4">
-                <param name="slave_position">5</param>
-                <param name="motor_type">X4</param>
-                <param name="direction">-1</param>
-                <param name="offset_raw">0</param>
                 <command_interface name="position"/>
                 <state_interface name="position"/>
                 <state_interface name="velocity"/>
                 <state_interface name="effort"/>
+                <ec_module name="LeftWristRoll">
+                    <plugin>ethercat_generic_plugins/EcCiA402Drive</plugin>
+                    <param name="alias">0</param>
+                    <param name="position">5</param>
+                    <param name="slave_config">$(find arm_real_bringup)/config/${config_dir}/left_wrist_roll_X4.yaml</param>
+                </ec_module>
             </joint>
         </ros2_control>
@@ -79,9 +96,7 @@
         <ros2_control name="RightArmSystem" type="system">
             <hardware>
-                <plugin>myactuator_hardware/MyActuatorSystem</plugin>
-                <param name="ethercat_master_index">0</param>
-                <param name="network_interface">eth0</param>
-                <param name="cycle_time_us">1000</param>
-                <param name="dc_sync">true</param>
+                <plugin>ethercat_driver/EthercatDriver</plugin>
+                <param name="master_id">0</param>
+                <param name="control_frequency">1000</param>
             </hardware>
             ... right arm joints (positions 6-11) ...

Commit message: working record and play motion left arm

File: src/robot_description/dual_arm_description/urdf/dual_arm.urdf.xacro (robot description, xacro)
@@ -6,4 +6,5 @@
     <xacro:arg name="fixed_legs" default="true" />
     <xacro:arg name="readonly" default="false" />
+    <xacro:arg name="gravcomp" default="false" />
     <xacro:if value="$(arg use_isaac)">
         <xacro:include filename="$(find dual_arm_description)/urdf/dual_arm_isaac.xacro" />

File: src/robot_description/dual_arm_description/urdf/dual_arm_real.xacro (robot description, xacro)
@@ -4,4 +4,5 @@
     <xacro:arg name="robot_name" default="dual_arm_description"/>
     <xacro:arg name="readonly" default="false"/>
+    <xacro:arg name="gravcomp" default="false"/>
     <!-- Bring in base structure (links, joints, hands) -->
     <xacro:include filename="$(find dual_arm_description)/urdf/dual_arm_base.xacro" />

File: src/robot_description/dual_arm_description/urdf/macros/ros2_control_real.xacro (robot description, xacro)
@@ -4,10 +4,12 @@
     <!-- Uses ethercat_driver_ros2 (ICube-Robotics) with EcCiA402Drive per joint -->
     <xacro:macro name="dual_arm_ros2_control_real">
-        <!-- Select config directory and frequency based on readonly mode -->
+        <!-- Select config directory based on operating mode -->
         <xacro:property name="config_dir" value="ethercat"/>
         <xacro:property name="ctrl_freq" value="100"/>
         <xacro:if value="$(arg readonly)">
             <xacro:property name="config_dir" value="ethercat_readonly"/>
-            <xacro:property name="ctrl_freq" value="100"/>
+        </xacro:if>
+        <xacro:if value="$(arg gravcomp)">
+            <xacro:property name="config_dir" value="ethercat_gravcomp"/>
         </xacro:if>
         <!-- Left arm — 6 DOF EtherCAT actuators (MyActuator RMD X V4) -->
@@ -20,4 +22,6 @@
             <joint name="left_shoulder_pitch_joint_X6">
                 <command_interface name="position"/>
+                <command_interface name="effort"/>
+                <command_interface name="mode_of_operation"/>
                 <state_interface name="position"/>
                 <state_interface name="velocity"/>
@@ -33,4 +37,6 @@
             <joint name="left_shoulder_roll_joint_X6">
                 <command_interface name="position"/>
+                <command_interface name="effort"/>
+                <command_interface name="mode_of_operation"/>
                 <state_interface name="position"/>
                 <state_interface name="velocity"/>
@@ -46,4 +52,6 @@
             <joint name="left_shoulder_yaw_joint_X4">
                 <command_interface name="position"/>
+                <command_interface name="effort"/>
+                <command_interface name="mode_of_operation"/>
                 <state_interface name="position"/>
                 <state_interface name="velocity"/>
@@ -59,4 +67,6 @@
             <joint name="left_elbow_pitch_joint_X6">
                 <command_interface name="position"/>
+                <command_interface name="effort"/>
+                <command_interface name="mode_of_operation"/>
                 <state_interface name="position"/>
                 <state_interface name="velocity"/>
@@ -72,4 +82,6 @@
             <joint name="left_wrist_yaw_joint_X4">
                 <command_interface name="position"/>
+                <command_interface name="effort"/>
+                <command_interface name="mode_of_operation"/>
                 <state_interface name="position"/>
                 <state_interface name="velocity"/>
@@ -85,4 +97,6 @@
             <joint name="left_wrist_roll_joint_X4">
                 <command_interface name="position"/>
+                <command_interface name="effort"/>
+                <command_interface name="mode_of_operation"/>
                 <state_interface name="position"/>
                 <state_interface name="velocity"/>
