Commit message: review

File: src/robot_description/dual_arm_description/urdf/dual_arm_base.xacro (robot description, xacro)
@@ -13,6 +13,5 @@
     mount_roll="1.5708"
     mount_pitch="0"
-    mount_yaw="1.5708"/>
-     <origin xyz="-0.0303429 -4.52461e-07 -0.135203" rpy="0 0 3.14159"/>
+    mount_yaw="1.5708"/>s
   <xacro:inspire_hand_right
     parent="urdf_r_wrist_assembly"

Commit message: 25 actuators callibration

File: src/robot_description/dual_arm_description/urdf/dual_arm_base.xacro (robot description, xacro)
@@ -21,21 +21,21 @@
   <xacro:include filename="$(find hand_description)/urdf/hands/inspire_hand_left.xacro" />
   <xacro:include filename="$(find hand_description)/urdf/hands/inspire_hand_right.xacro" />
-  <xacro:inspire_hand_left
-    parent="urdf_l_wrist_assembly"
-    prefix="left_"
-    mount_x="-0.034"
-    mount_y="0.015"
-    mount_z="-0.06"
-    mount_roll="1.424576"
-    mount_pitch="-0.201364"
-    mount_yaw="2.205507" />
-  <xacro:inspire_hand_right
-    parent="urdf_r_wrist_assembly"
-    prefix="right_"
-    mount_x="-0.029"
-    mount_y="-0.011"
-    mount_z="-0.06"
-    mount_roll="1.717027"
-    mount_pitch="-0.201373"
-    mount_yaw="-2.205496" />
+<xacro:inspire_hand_left
+        parent="urdf_l_wrist_assembly"
+        prefix="left_"
+        mount_x="-0.034"
+        mount_y="0.015"
+        mount_z="-0.06"
+        mount_roll="1.544576"
+        mount_pitch="-0.201364"
+        mount_yaw="1.6"/>
+    <xacro:inspire_hand_right
+        parent="urdf_r_wrist_assembly"
+        prefix="right_"
+        mount_x="-0.033"
+        mount_y="-0.011"
+        mount_z="-0.06"
+        mount_roll="1.617027"
+        mount_pitch="-0.301373"
+        mount_yaw="-1.605496"/>
 </robot>

File: src/robot_description/dual_arm_description/urdf/macros/ros2_control_real.xacro (robot description, xacro)
@@ -324,6 +324,5 @@
             </joint>
             <!-- ════════════════════════════════════════════════════════════════ -->
-            <!-- RIGHT LEG — 5 joints (bus 19-23)                               -->
-            <!-- NOTE: right_ankle_pitch (bus 24) not connected yet              -->
+            <!-- RIGHT LEG — 6 joints (bus 19-24)                               -->
             <!-- ════════════════════════════════════════════════════════════════ -->
             <joint name="right_hip_pitch_joint_X8">
@@ -402,5 +401,19 @@
                 </ec_module>
             </joint>
-            <!-- TODO: Add right_ankle_pitch_joint_X4 (bus 24) when actuator arrives -->
+            <joint name="right_ankle_pitch_joint_X4">
+                <command_interface name="position"/>
+                <command_interface name="effort"/>
+                <command_interface name="mode_of_operation"/>
+                <state_interface name="position"/>
+                <state_interface name="velocity"/>
+                <state_interface name="effort"/>
+                <state_interface name="status_word"/>
+                <ec_module name="RightAnklePitch">
+                    <plugin>ethercat_generic_plugins/EcCiA402Drive</plugin>
+                    <param name="alias">0</param>
+                    <param name="position">24</param>
+                    <param name="slave_config">$(find arm_real_bringup)/config/${config_dir}/right_ankle_pitch_X4.yaml</param>
+                </ec_module>
+            </joint>
             </xacro:unless>  <!-- only_arms -->
         </ros2_control>

File: src/robot_description/full_robot_description/urdf/macros/ros2_control_position.xacro (robot description, xacro)
@@ -9,6 +9,6 @@
       <joint name="waist_yaw_joint_X8">
         <command_interface name="position">
-          <param name="min">-1.57</param>
-          <param name="max">1.57</param>
+          <param name="min">-2.60054</param>
+          <param name="max">2.60054</param>
         </command_interface>
         <state_interface name="position" />
@@ -19,6 +19,6 @@
       <joint name="left_shoulder_pitch_joint_X6">
         <command_interface name="position">
-          <param name="min">-3.02</param>
-          <param name="max">1.69</param>
+          <param name="min">-3.01942</param>
+          <param name="max">1.69297</param>
         </command_interface>
         <state_interface name="position" />
@@ -28,6 +28,6 @@
       <joint name="left_shoulder_roll_joint_X6">
         <command_interface name="position">
-          <param name="min">-0.21</param>
-          <param name="max">2.93</param>
+          <param name="min">-0.20944</param>
+          <param name="max">2.93215</param>
         </command_interface>
         <state_interface name="position" />
@@ -37,6 +37,6 @@
       <joint name="left_shoulder_yaw_joint_X4">
         <command_interface name="position">
-          <param name="min">-1.75</param>
-          <param name="max">2.97</param>
+          <param name="min">-1.74533</param>
+          <param name="max">2.96706</param>
         </command_interface>
         <state_interface name="position" />
@@ -46,6 +46,6 @@
       <joint name="left_elbow_pitch_joint_X6">
         <command_interface name="position">
-          <param name="min">-1.31</param>
-          <param name="max">1.83</param>
+          <param name="min">-1.309</param>
+          <param name="max">1.8326</param>
         </command_interface>
         <state_interface name="position" />
@@ -55,6 +55,6 @@
       <joint name="left_wrist_yaw_joint_X4">
         <command_interface name="position">
-          <param name="min">-2.36</param>
-          <param name="max">2.36</param>
+          <param name="min">-2.35619</param>
+          <param name="max">2.35619</param>
         </command_interface>
         <state_interface name="position" />
@@ -64,6 +64,6 @@
       <joint name="left_wrist_roll_joint_X4">
         <command_interface name="position">
-          <param name="min">-1.57</param>
-          <param name="max">1.57</param>
+          <param name="min">-1.5708</param>
+          <param name="max">1.5708</param>
         </command_interface>
         <state_interface name="position" />
@@ -74,6 +74,6 @@
       <joint name="right_shoulder_pitch_joint_X6">
         <command_interface name="position">
-          <param name="min">-3.02</param>
-          <param name="max">1.69</param>
+          <param name="min">-3.01942</param>
+          <param name="max">1.69297</param>
         </command_interface>
         <state_interface name="position" />
@@ -83,6 +83,6 @@
       <joint name="right_shoulder_roll_joint_X6">
         <command_interface name="position">
-          <param name="min">-2.93</param>
-          <param name="max">0.21</param>
+          <param name="min">-2.93215</param>
+          <param name="max">0.20944</param>
         </command_interface>
         <state_interface name="position" />
@@ -92,6 +92,6 @@
       <joint name="right_shoulder_yaw_joint_X4">
         <command_interface name="position">
-          <param name="min">-2.97</param>
-          <param name="max">1.75</param>
+          <param name="min">-2.96706</param>
+          <param name="max">1.74533</param>
         </command_interface>
         <state_interface name="position" />
@@ -101,6 +101,6 @@
       <joint name="right_elbow_pitch_joint_X6">
         <command_interface name="position">
-          <param name="min">-1.31</param>
-          <param name="max">1.83</param>
+          <param name="min">-1.309</param>
+          <param name="max">1.8326</param>
         </command_interface>
         <state_interface name="position" />
@@ -110,6 +110,6 @@
       <joint name="right_wrist_yaw_joint_X4">
         <command_interface name="position">
-          <param name="min">-2.36</param>
-          <param name="max">2.36</param>
+          <param name="min">-2.35619</param>
+          <param name="max">2.35619</param>
         </command_interface>
         <state_interface name="position" />
@@ -119,6 +119,6 @@
       <joint name="right_wrist_roll_joint_X4">
         <command_interface name="position">
-          <param name="min">-1.57</param>
-          <param name="max">1.57</param>
+          <param name="min">-1.65806</param>
+          <param name="max">1.65806</param>
         </command_interface>
         <state_interface name="position" />
@@ -227,6 +227,6 @@
       <joint name="left_hip_pitch_joint_X8">
         <command_interface name="position">
-          <param name="min">-2.53</param>
-          <param name="max">1.57</param>
+          <param name="min">-2.61799</param>
+          <param name="max">2.61799</param>
         </command_interface>
         <state_interface name="position" />
@@ -236,6 +236,6 @@
       <joint name="left_hip_roll_joint_X8">
         <command_interface name="position">
-          <param name="min">-0.35</param>
-          <param name="max">3.14</param>
+          <param name="min">-0.383972</param>
+          <param name="max">3.22886</param>
         </command_interface>
         <state_interface name="position" />
@@ -245,6 +245,6 @@
       <joint name="left_hip_yaw_joint_X8">
         <command_interface name="position">
-          <param name="min">-1.57</param>
-          <param name="max">1.57</param>
+          <param name="min">-2.15199</param>
+          <param name="max">2.09003</param>
         </command_interface>
         <state_interface name="position" />
@@ -254,6 +254,6 @@
       <joint name="left_knee_joint_X8">
         <command_interface name="position">
-          <param name="min">-0.17</param>
-          <param name="max">1.57</param>
+          <param name="min">-1.52716</param>
+          <param name="max">1.52716</param>
         </command_interface>
         <state_interface name="position" />
@@ -263,6 +263,6 @@
       <joint name="left_ankle_roll_joint_X4">
         <command_interface name="position">
-          <param name="min">-0.79</param>
-          <param name="max">0.79</param>
+          <param name="min">-0.785398</param>
+          <param name="max">0.785398</param>
         </command_interface>
         <state_interface name="position" />
@@ -272,6 +272,6 @@
       <joint name="left_ankle_pitch_joint_X4">
         <command_interface name="position">
-          <param name="min">-0.79</param>
-          <param name="max">0.79</param>
+          <param name="min">-0.785398</param>
+          <param name="max">0.785398</param>
         </command_interface>
         <state_interface name="position" />
@@ -282,6 +282,6 @@
       <joint name="right_hip_pitch_joint_X8">
         <command_interface name="position">
-          <param name="min">-2.53</param>
-          <param name="max">1.57</param>
+          <param name="min">-2.61799</param>
+          <param name="max">2.61799</param>
         </command_interface>
         <state_interface name="position" />
@@ -291,6 +291,6 @@
       <joint name="right_hip_roll_joint_X8">
         <command_interface name="position">
-          <param name="min">-3.14</param>
-          <param name="max">0.35</param>
+          <param name="min">-3.22886</param>
+          <param name="max">0.383972</param>
         </command_interface>
         <state_interface name="position" />
@@ -300,6 +300,6 @@
       <joint name="right_hip_yaw_joint_X8">
         <command_interface name="position">
-          <param name="min">-1.57</param>
-          <param name="max">1.57</param>
+          <param name="min">-1.5708</param>
+          <param name="max">1.5708</param>
         </command_interface>
         <state_interface name="position" />
@@ -309,6 +309,6 @@
       <joint name="right_knee_joint_X8">
         <command_interface name="position">
-          <param name="min">-0.17</param>
-          <param name="max">1.57</param>
+          <param name="min">-1.52716</param>
+          <param name="max">1.52716</param>
         </command_interface>
         <state_interface name="position" />
@@ -318,6 +318,6 @@
       <joint name="right_ankle_roll_joint_X4">
         <command_interface name="position">
-          <param name="min">-0.79</param>
-          <param name="max">0.79</param>
+          <param name="min">-0.785398</param>
+          <param name="max">0.785398</param>
         </command_interface>
         <state_interface name="position" />
@@ -327,6 +327,6 @@
       <joint name="right_ankle_pitch_joint_X4">
         <command_interface name="position">
-          <param name="min">-0.79</param>
-          <param name="max">0.79</param>
+          <param name="min">-0.785398</param>
+          <param name="max">0.785398</param>
         </command_interface>
         <state_interface name="position" />

Commit message: update dual_arm_description with newest urdf

File: src/robot_description/dual_arm_description/urdf/dual_arm_base.xacro (robot description, xacro)
@@ -19,7 +19,7 @@
   <xacro:include filename="$(find full_robot_description)/urdf/joints/right_foot_joints.xacro" />
   <!-- Hands -->
-  <xacro:include filename="$(find hand_description)/urdf/hands/inspire_hand_left.xacro" />
-  <xacro:include filename="$(find hand_description)/urdf/hands/inspire_hand_right.xacro" />
-<xacro:inspire_hand_left
+  <!--xacro:include filename="$(find hand_description)/urdf/hands/inspire_hand_left.xacro" /-->
+  <!--xacro:include filename="$(find hand_description)/urdf/hands/inspire_hand_right.xacro" /-->
+<!--xacro:inspire_hand_left
         parent="urdf_l_wrist_assembly"
         prefix="left_"
@@ -29,6 +29,6 @@
         mount_roll="1.544576"
         mount_pitch="-0.201364"
-        mount_yaw="1.6"/>
-    <xacro:inspire_hand_right
+        mount_yaw="1.6"/-->
+    <!--xacro:inspire_hand_right
         parent="urdf_r_wrist_assembly"
         prefix="right_"
@@ -38,4 +38,4 @@
         mount_roll="1.617027"
         mount_pitch="-0.301373"
-        mount_yaw="-1.605496"/>
+        mount_yaw="-1.605496"/-->
 </robot>

File: src/robot_description/dual_arm_description/urdf/dual_arm_gazebo.xacro (robot description, xacro)
@@ -15,12 +15,12 @@
     <xacro:dual_arm_ros2_control/>
     <!-- Orbbec Gemini 335L/336L Depth Camera -->
-    <xacro:include filename="$(find camera_description)/urdf/gemini335L_336L.urdf.xacro"/>
-    <xacro:include filename="$(find camera_description)/urdf/gemini335L_336L_gazebo.xacro"/>
+    <!--xacro:include filename="$(find camera_description)/urdf/gemini335L_336L.urdf.xacro"/-->
+    <!--xacro:include filename="$(find camera_description)/urdf/gemini335L_336L_gazebo.xacro"/-->
     <!-- Mount camera on urdf_base, positioned to view the workspace -->
-    <joint name="camera_mount_joint" type="fixed">
+    <!--joint name="camera_mount_joint" type="fixed">
         <parent link="urdf_base"/>
         <child link="camera_link"/>
         <origin xyz="0.13 0.0455 0.429" rpy="0 ${pi/12} 0"/>
-    </joint>
+    </joint-->
     <!-- Gazebo plugins -->
     <gazebo>
@@ -30,7 +30,7 @@
         </plugin>
         <!-- Sensors plugin (required for cameras, depth sensors, etc.) -->
-        <plugin filename="gz-sim-sensors-system" name="gz::sim::systems::Sensors">
+        <!--plugin filename="gz-sim-sensors-system" name="gz::sim::systems::Sensors">
             <render_engine>ogre2</render_engine>
-        </plugin>
+        </plugin-->
     </gazebo>
 </robot>

File: src/robot_description/dual_arm_description/urdf/dual_arm_real.xacro (robot description, xacro)
@@ -26,6 +26,6 @@
     </xacro:unless>
     <!-- Depth Camera (if connected to real robot) -->
-    <xacro:include filename="$(find arm_description)/urdf/macros/depth_camera.xacro"/>
-    <xacro:depth_camera parent_link="urdf_base" xyz="-0.3 0.0 0.8" rpy="0 ${pi/6} 0" name="camera"/>
+    <!--xacro:include filename="$(find arm_description)/urdf/macros/depth_camera.xacro"/-->
+    <!--xacro:depth_camera parent_link="urdf_base" xyz="-0.3 0.0 0.8" rpy="0 ${pi/6} 0" name="camera"/-->
     <!-- No Gazebo plugins for real hardware -->
 </robot>

File: src/robot_description/dual_arm_description/urdf/macros/ros2_control.xacro (robot description, xacro)
@@ -83,9 +83,8 @@
         </ros2_control>
         <!-- Both hands in one system (like single arm's HandSystem) -->
-        <ros2_control name="HandSystem" type="system">
+        <!--ros2_control name="HandSystem" type="system">
             <hardware>
                 <plugin>gz_ros2_control/GazeboSimSystem</plugin>
             </hardware>
-            <!-- Left hand actuated -->
             <joint name="left_thumb_proximal_yaw_joint">
                 <command_interface name="position"/>
@@ -136,5 +135,4 @@
                 <state_interface name="effort"/>
             </joint>
-            <!-- Left hand mimic (state only) -->
             <joint name="left_thumb_intermediate_joint">
                 <state_interface name="position"/>
@@ -167,5 +165,4 @@
                 <state_interface name="effort"/>
             </joint>
-            <!-- Right hand actuated -->
             <joint name="right_thumb_proximal_yaw_joint">
                 <command_interface name="position"/>
@@ -216,5 +213,4 @@
                 <state_interface name="effort"/>
             </joint>
-            <!-- Right hand mimic (state only) -->
             <joint name="right_thumb_intermediate_joint">
                 <state_interface name="position"/>
@@ -247,5 +243,5 @@
                 <state_interface name="effort"/>
             </joint>
-        </ros2_control>
+        </ros2_control-->
     </xacro:macro>
 </robot>
