Commit message: correction for camera position

File: src/robot_description/arm_description/urdf/arm_gazebo.xacro (robot description, xacro)
@@ -10,10 +10,13 @@
     <xacro:include filename="$(find arm_description)/urdf/macros/ros2_control.xacro"/>
     <xacro:arm_ros2_control/>
-    <!-- Depth Camera -->
-    <xacro:include filename="$(find arm_description)/urdf/macros/depth_camera.xacro"/>
-    <!-- Mount camera on base_link, positioned to view the workspace -->
-    <!-- The new robot has the table at z=0, arm starts at table level -->
-    <!-- Position camera 0.5m behind and 0.8m above the robot base, looking down slightly -->
-    <xacro:depth_camera parent_link="urdf_base" xyz="-0.3 0.0 1.26" rpy="0 ${pi/6} 0" name="camera"/>
+    <!-- Orbbec Gemini 335L/336L Depth Camera -->
+    <xacro:include filename="$(find camera_description)/urdf/gemini335L_336L.urdf.xacro"/>
+    <xacro:include filename="$(find camera_description)/urdf/gemini335L_336L_gazebo.xacro"/>
+    <!-- Mount camera on urdf_base, positioned to view the workspace -->
+    <joint name="camera_mount_joint" type="fixed">
+        <parent link="urdf_base"/>
+        <child link="camera_link"/>
+        <origin xyz="0.13 0.0455 0.429" rpy="0 ${pi/12} 0"/>
+    </joint>
     <!-- Gazebo plugins -->
     <gazebo>

File: src/robot_description/dual_arm_description/urdf/dual_arm_gazebo.xacro (robot description, xacro)
@@ -21,5 +21,5 @@
         <parent link="urdf_base"/>
         <child link="camera_link"/>
-        <origin xyz="-0.3 0.0 0.8" rpy="0 ${pi/6} 0"/>
+        <origin xyz="0.13 0.0455 0.429" rpy="0 ${pi/12} 0"/>
     </joint>
     <!-- Gazebo plugins -->
