Commit message: camera joint correction

File: src/robot_description/arm_description/urdf/arm_gazebo.xacro (robot description, xacro)
@@ -15,7 +15,7 @@
     <!-- Mount camera on urdf_base, positioned to view the workspace -->
     <joint name="camera_mount_joint" type="fixed">
-        <parent link="urdf_base"/>
+        <parent link="urdf_simplified_torso"/>
         <child link="camera_link"/>
-        <origin xyz="0.08 0.0455 0.829" rpy="0 ${pi/12} 0"/>
+        <origin xyz="0.08 0.0455 0.75" rpy="0 ${pi/12} 0"/>
     </joint>
     <!-- Gazebo plugins -->

File: src/robot_description/dual_arm_description/urdf/dual_arm_gazebo.xacro (robot description, xacro)
@@ -19,7 +19,7 @@
     <!-- Mount camera on urdf_base, positioned to view the workspace -->
     <joint name="camera_mount_joint" type="fixed">
-        <parent link="urdf_base"/>
+        <parent link="urdf_simplified_torso"/>
         <child link="camera_link"/>
-        <origin xyz="0.08 0.0455 0.829" rpy="0 ${pi/12} 0"/>
+        <origin xyz="0.08 0.0455 0.75" rpy="0 ${pi/12} 0"/>
     </joint>
     <!-- Gazebo plugins -->

File: src/robot_description/full_robot_description/urdf/full_robot_gazebo.xacro (robot description, xacro)
@@ -60,7 +60,7 @@
   <!-- Mount camera on urdf_base, positioned to view the workspace -->
   <joint name="camera_mount_joint" type="fixed">
-      <parent link="urdf_base"/>
+      <parent link="urdf_simplified_torso"/>
       <child link="camera_link"/>
-      <origin xyz="0.08 0.0455 0.829" rpy="0 ${pi/12} 0"/>
+      <origin xyz="0.08 0.0455 0.75" rpy="0 ${pi/12} 0"/>
   </joint>
   <!-- IMU sensors (BNO055) -->
