Commit message: review : arm sim bring-up for MTC
- launch: repair broken includes (full_system→headless, moveit_gazebo→arm_world),
  default world lab-ldr, add full_robot_description to GZ_SIM_RESOURCE_PATH
- ros2_control: mirrored right-arm spawn, drop duplicate position state_interface
- srdf: disable leg-leg collisions, fix lower_femur link names
- moveit: disable depth-camera octomap (sensors_3d)
- world: move lab-mtc tables+lever to x=+0.45, make tables static
- arm_base: hand mount tuning

File: src/robot_description/arm_description/urdf/arm_base.xacro (robot description, xacro)
@@ -1,4 +1,6 @@
 <?xml version="1.0"?>
 <robot xmlns:xacro="http://ros.org/wiki/xacro">
+    <!-- Actuator properties (effort, velocity, damping, friction) -->
+    <xacro:include filename="$(find full_robot_description)/urdf/macros/actuator_properties.xacro" />
     <!-- Include macros -->
     <xacro:include filename="$(find arm_description)/urdf/macros/materials.xacro" />
@@ -24,18 +26,18 @@
         parent="urdf_l_wrist_assembly"
         prefix="left_"
-        mount_x="-0.034"
-        mount_y="0.015"
+        mount_x="-0.0303429"
+        mount_y="4.99302e-07"
         mount_z="-0.06"
-        mount_roll="1.424576"
-        mount_pitch="-0.201364"
-        mount_yaw="2.205507"/>
+        mount_roll="${pi/2}"
+        mount_pitch="0.0"
+        mount_yaw="${pi/2}"/>
     <xacro:inspire_hand_right
         parent="urdf_r_wrist_assembly"
         prefix="right_"
-        mount_x="-0.029"
-        mount_y="-0.011"
+        mount_x="-0.0327429 "
+        mount_y="0.008"
         mount_z="-0.06"
-        mount_roll="1.717027"
-        mount_pitch="-0.201373"
-        mount_yaw="-2.205496"/>
+        mount_roll="${pi/2}"
+        mount_pitch="0.0"
+        mount_yaw="-${pi/2}"/>
 </robot>

File: src/robot_description/arm_description/urdf/arm_gazebo.xacro (robot description, xacro)
@@ -17,5 +17,5 @@
         <parent link="urdf_base"/>
         <child link="camera_link"/>
-        <origin xyz="0.13 0.0455 0.429" rpy="0 ${pi/12} 0"/>
+        <origin xyz="0.08 0.0455 0.829" rpy="0 ${pi/12} 0"/>
     </joint>
     <!-- Gazebo plugins -->

File: src/robot_description/arm_description/urdf/macros/ros2_control.xacro (robot description, xacro)
@@ -12,7 +12,6 @@
                 <command_interface name="position"/>
                 <state_interface name="position">
-                    <param name="initial_value">0.1</param>
-                </state_interface>
-                <state_interface name="position"/>
+                    <param name="initial_value">0.0</param>
+                </state_interface>
                 <state_interface name="velocity"/>
                 <state_interface name="effort"/>
@@ -37,7 +36,6 @@
                 <command_interface name="position"/>
                 <state_interface name="position">
-                    <param name="initial_value">0.3</param>
-                </state_interface>
-                <state_interface name="position"/>
+                    <param name="initial_value">-0.1</param>
+                </state_interface>
                 <state_interface name="velocity"/>
                 <state_interface name="effort"/>
@@ -63,5 +61,7 @@
                 <joint name="right_shoulder_pitch_joint_X6">
                     <command_interface name="position"/>
-                    <state_interface name="position"/>
+                    <state_interface name="position">
+                        <param name="initial_value">0.0</param>
+                    </state_interface>
                     <state_interface name="velocity"/>
                     <state_interface name="effort"/>
@@ -69,5 +69,7 @@
                 <joint name="right_shoulder_roll_joint_X6">
                     <command_interface name="position"/>
-                    <state_interface name="position"/>
+                    <state_interface name="position">
+                        <param name="initial_value">-0.1</param>
+                    </state_interface>
                     <state_interface name="velocity"/>
                     <state_interface name="effort"/>
@@ -75,5 +77,7 @@
                 <joint name="right_shoulder_yaw_joint_X4">
                     <command_interface name="position"/>
-                    <state_interface name="position"/>
+                    <state_interface name="position">
+                        <param name="initial_value">0.0</param>
+                    </state_interface>
                     <state_interface name="velocity"/>
                     <state_interface name="effort"/>
@@ -81,5 +85,7 @@
                 <joint name="right_elbow_pitch_joint_X6">
                     <command_interface name="position"/>
-                    <state_interface name="position"/>
+                    <state_interface name="position">
+                        <param name="initial_value">-0.1</param>
+                    </state_interface>
                     <state_interface name="velocity"/>
                     <state_interface name="effort"/>
@@ -87,5 +93,7 @@
                 <joint name="right_wrist_yaw_joint_X4">
                     <command_interface name="position"/>
-                    <state_interface name="position"/>
+                    <state_interface name="position">
+                        <param name="initial_value">0.0</param>
+                    </state_interface>
                     <state_interface name="velocity"/>
                     <state_interface name="effort"/>
@@ -93,5 +101,7 @@
                 <joint name="right_wrist_roll_joint_X4">
                     <command_interface name="position"/>
-                    <state_interface name="position"/>
+                    <state_interface name="position">
+                        <param name="initial_value">0.0</param>
+                    </state_interface>
                     <state_interface name="velocity"/>
                     <state_interface name="effort"/>

File: src/robot_description/full_robot_description/urdf/links/left_arm_links.xacro (robot description, xacro)
@@ -165,4 +165,5 @@
       <inertia ixx="0.00213609" ixy="-7.00887e-09" ixz="-3.51538e-05" iyy="0.00236601" iyz="-1.94664e-08" izz="0.000415509"/>
     </inertial>
+    <!-- START OF Disable fake hands
     <visual>
       <origin xyz="-0.0303429 4.99302e-07 -0.135203" rpy="0 0 0"/>
@@ -180,4 +181,5 @@
       </geometry>
     </collision>
+    END OF Disable fake hands -->
     <visual>
       <origin xyz="-0.01 0 0" rpy="0 0 -1.5708"/>

File: src/robot_description/full_robot_description/urdf/links/right_arm_links.xacro (robot description, xacro)
@@ -165,4 +165,5 @@
       <inertia ixx="0.00248005" ixy="1.0712e-08" ixz="-7.96759e-05" iyy="0.00272432" iyz="3.9857e-08" izz="0.00046834"/>
     </inertial>
+     <!-- START OF Disable fake hands
     <visual>
       <origin xyz="-0.0303429 -2.67e-09 -0.135203" rpy="0 0 3.14159"/>
@@ -180,4 +181,5 @@
       </geometry>
     </collision>
+    ENB OF Disable fake hands -->
     <visual>
       <origin xyz="-0.01 0 0" rpy="0 0 -1.5708"/>
