Commit message: feat(robot_description): make waist locking independently configurable
Add a dedicated fixed_waist Xacro argument and decouple the waist joint
type from the arm and leg configurations. Preserve the existing defaults
for the arm, dual-arm, and full-robot models.
Fixes #3

File: src/robot_description/arm_description/urdf/arm.urdf.xacro (robot description, xacro)
@@ -11,4 +11,6 @@
     <xacro:arg name="fixed_legs"
         default="true" />
+    <xacro:arg name="fixed_waist"
+        default="true" />
     <xacro:arg name="only_left"
         default="true" />

File: src/robot_description/dual_arm_description/urdf/dual_arm.urdf.xacro (robot description, xacro)
@@ -5,4 +5,5 @@
     <xacro:arg name="use_isaac" default="false" />
     <xacro:arg name="fixed_legs" default="true" />
+    <xacro:arg name="fixed_waist" default="true" />
     <xacro:arg name="only_left" default="false" />
     <xacro:arg name="only_arms" default="false" />

File: src/robot_description/full_robot_description/urdf/full_robot_gazebo.xacro (robot description, xacro)
@@ -12,4 +12,5 @@
   <!-- Full robot: all joints active (not fixed) -->
   <xacro:arg name="fixed_legs" default="false" />
+  <xacro:arg name="fixed_waist" default="false" />
   <xacro:arg name="only_left" default="false" />
   <!-- Actuator properties macros -->

File: src/robot_description/full_robot_description/urdf/joints/body_joints.xacro (robot description, xacro)
@@ -7,8 +7,8 @@
   <xacro:property name="leg_joint_type" value="${'fixed' if '$(arg fixed_legs)' == 'true' else 'revolute'}"/>
   <!-- ================================================================== -->
-  <!-- only_left — when true, also lock waist yaw joint                  -->
+  <!-- Waist joint type — independent from the arm and leg configuration -->
   <!-- ================================================================== -->
-  <xacro:arg name="only_left" default="true"/>
-  <xacro:property name="waist_joint_type" value="${'fixed' if '$(arg only_left)' == 'true' or '$(arg fixed_legs)' == 'true' else 'revolute'}"/>
+  <xacro:arg name="fixed_waist" default="true"/>
+  <xacro:property name="waist_joint_type" value="${'fixed' if '$(arg fixed_waist)' == 'true' else 'revolute'}"/>
   <!-- ================================================================== -->
   <!-- Body                                                              -->

Commit message: feat(arm_control): expose and command waist yaw joint
Enable the waist by default in the arm model, add its ros2_control
interfaces, and extend the arm trajectory controllers to seven joints.

File: src/robot_description/arm_description/urdf/arm.urdf.xacro (robot description, xacro)
@@ -12,5 +12,5 @@
         default="true" />
     <xacro:arg name="fixed_waist"
-        default="true" />
+        default="false" />
     <xacro:arg name="only_left"
         default="true" />

File: src/robot_description/arm_description/urdf/macros/ros2_control.xacro (robot description, xacro)
@@ -8,5 +8,13 @@
                 <plugin>gz_ros2_control/GazeboSimSystem</plugin>
             </hardware>
-            <!-- Left arm (6 DOF) -->
+            <!-- Waist + left arm (7 DOF) -->
+            <joint name="waist_yaw_joint_X8">
+                <command_interface name="position"/>
+                <state_interface name="position">
+                    <param name="initial_value">0.0</param>
+                </state_interface>
+                <state_interface name="velocity"/>
+                <state_interface name="effort"/>
+            </joint>
             <joint name="left_shoulder_pitch_joint_X6">
                 <command_interface name="position"/>
