Commit message: first move in moveit

File: src/robot_description/full_robot_description/urdf/joints/left_arm_joints.xacro (robot description, xacro)
@@ -9,5 +9,5 @@
     <child link="urdf_l_shoulder_assembly"/>
     <axis xyz="0 1 0"/>
-    <limit effort="100" velocity="100" lower="-3.02" upper="1.69"/>
+    <limit effort="8" velocity="2" lower="-3.02" upper="1.69"/>
     <dynamics damping="0.5" friction="0.1"/>
   </joint>
@@ -17,5 +17,5 @@
     <child link="urdf_l_upper_arm_assembly"/>
     <axis xyz="1 0 0"/>
-    <limit effort="100" velocity="100" lower="-0.21" upper="2.93"/>
+    <limit effort="8" velocity="2" lower="-0.21" upper="2.93"/>
     <dynamics damping="0.5" friction="0.1"/>
   </joint>
@@ -25,5 +25,5 @@
     <child link="urdf_l_elbow_assembly"/>
     <axis xyz="0 0 1"/>
-    <limit effort="100" velocity="100" lower="-1.75" upper="2.97"/>
+    <limit effort="8" velocity="2" lower="-1.75" upper="2.97"/>
     <dynamics damping="0.5" friction="0.1"/>
   </joint>
@@ -33,5 +33,5 @@
     <child link="urdf_l_upper_forearm_assembly"/>
     <axis xyz="0 1 0"/>
-    <limit effort="100" velocity="100" lower="-1.31" upper="1.83"/>
+    <limit effort="8" velocity="2" lower="-1.31" upper="1.83"/>
     <dynamics damping="0.5" friction="0.1"/>
   </joint>
@@ -41,5 +41,5 @@
     <child link="urdf_l_lower_forearm_assembly"/>
     <axis xyz="0 0 1"/>
-    <limit effort="100" velocity="100" lower="-2.36" upper="2.36"/>
+    <limit effort="8" velocity="2" lower="-2.36" upper="2.36"/>
     <dynamics damping="0.5" friction="0.1"/>
   </joint>
@@ -49,5 +49,5 @@
     <child link="urdf_l_wrist_assembly"/>
     <axis xyz="1 0 0"/>
-    <limit effort="100" velocity="100" lower="-1.57" upper="1.57"/>
+    <limit effort="8" velocity="2" lower="-1.57" upper="1.57"/>
     <dynamics damping="0.5" friction="0.1"/>
   </joint>

File: src/robot_description/full_robot_description/urdf/joints/right_arm_joints.xacro (robot description, xacro)
@@ -9,5 +9,5 @@
     <child link="urdf_r_shoulder_assembly"/>
     <axis xyz="0 1 0"/>
-    <limit effort="100" velocity="100" lower="-3.02" upper="1.69"/>
+    <limit effort="8" velocity="2" lower="-3.02" upper="1.69"/>
     <dynamics damping="0.5" friction="0.1"/>
   </joint>
@@ -17,5 +17,5 @@
     <child link="urdf_r_upper_arm_assembly"/>
     <axis xyz="1 0 0"/>
-    <limit effort="100" velocity="100" lower="-2.93" upper="0.21"/>
+    <limit effort="8" velocity="2" lower="-2.93" upper="0.21"/>
     <dynamics damping="0.5" friction="0.1"/>
   </joint>
@@ -25,5 +25,5 @@
     <child link="urdf_r_elbow_assembly"/>
     <axis xyz="0 0 1"/>
-    <limit effort="100" velocity="100" lower="-2.97" upper="1.75"/>
+    <limit effort="8" velocity="2" lower="-2.97" upper="1.75"/>
     <dynamics damping="0.5" friction="0.1"/>
   </joint>
@@ -33,5 +33,5 @@
     <child link="urdf_r_upper_forearm_assembly"/>
     <axis xyz="0 1 0"/>
-    <limit effort="100" velocity="100" lower="-1.31" upper="1.83"/>
+    <limit effort="8" velocity="2" lower="-1.31" upper="1.83"/>
     <dynamics damping="0.5" friction="0.1"/>
   </joint>
@@ -41,5 +41,5 @@
     <child link="urdf_r_lower_forearm_assembly"/>
     <axis xyz="0 0 1"/>
-    <limit effort="100" velocity="100" lower="-2.36" upper="2.36"/>
+    <limit effort="8" velocity="2" lower="-2.36" upper="2.36"/>
     <dynamics damping="0.5" friction="0.1"/>
   </joint>
@@ -49,5 +49,5 @@
     <child link="urdf_r_wrist_assembly"/>
     <axis xyz="1 0 0"/>
-    <limit effort="100" velocity="100" lower="-1.57" upper="1.57"/>
+    <limit effort="8" velocity="2" lower="-1.57" upper="1.57"/>
     <dynamics damping="0.5" friction="0.1"/>
   </joint>
