Commit message: update joint limits using actuator specs

File: src/robot_description/full_robot_description/urdf/joints/body_joints.xacro (robot description, xacro)
@@ -1,24 +1,15 @@
-<?xml version="1.0"?>
-<robot xmlns:xacro="http://www.ros.org/wiki/xacro">
-  <!-- ================================================================== -->
-  <!-- Leg joint type — set fixed_legs:=true to lock leg joints          -->
-  <!-- ================================================================== -->
-  <xacro:arg name="fixed_legs" default="false"/>
-  <xacro:property name="leg_joint_type" value="${'fixed' if '$(arg fixed_legs)' == 'true' else 'revolute'}"/>
-  <!-- ================================================================== -->
-  <!-- only_left — when true, also lock waist yaw joint                  -->
-  <!-- ================================================================== -->
-  <xacro:arg name="only_left" default="true"/>
-  <xacro:property name="waist_joint_type" value="${'fixed' if '$(arg only_left)' == 'true' or '$(arg fixed_legs)' == 'true' else 'revolute'}"/>
-  <!-- ================================================================== -->
-  <!-- Body                                                              -->
-  <!-- ================================================================== -->
+<?xml version='1.0' encoding='utf-8'?>
+<robot xmlns:ns0="http://www.ros.org/wiki/xacro">
+  <ns0:arg name="fixed_legs" default="false" />
+  <ns0:property name="leg_joint_type" value="${'fixed' if '$(arg fixed_legs)' == 'true' else 'revolute'}" />
+  <ns0:arg name="only_left" default="true" />
+  <ns0:property name="waist_joint_type" value="${'fixed' if '$(arg only_left)' == 'true' or '$(arg fixed_legs)' == 'true' else 'revolute'}" />
   <joint name="waist_yaw_joint" type="${waist_joint_type}">
-    <origin xyz="0.0333787 -0.000698852 -0.300748" rpy="0 0 0"/>
-    <parent link="urdf_base"/>
-    <child link="urdf_simplified_torso"/>
-    <axis xyz="0 0 1"/>
-    <limit effort="100" velocity="100" lower="-1.57" upper="1.57"/>
-    <dynamics damping="0.5" friction="0.1"/>
+    <origin xyz="0.0333787 -0.000698852 -0.300748" rpy="0 0 0" />
+    <parent link="urdf_base" />
+    <child link="urdf_simplified_torso" />
+    <axis xyz="0 0 1" />
+    <limit effort="43" velocity="13.3" lower="-1.57" upper="1.57" />
+    <dynamics damping="0.321" friction="3.21" />
   </joint>
 </robot>

File: src/robot_description/full_robot_description/urdf/joints/left_arm_joints.xacro (robot description, xacro)
@@ -1,54 +1,51 @@
-<?xml version="1.0"?>
-<robot xmlns:xacro="http://www.ros.org/wiki/xacro">
-  <!-- ================================================================== -->
-  <!-- Left Arm                                                          -->
-  <!-- ================================================================== -->
+<?xml version='1.0' encoding='utf-8'?>
+<robot>
   <joint name="left_shoulder_pitch_joint_X6" type="revolute">
-    <origin xyz="0 0.1755 0.423977" rpy="0 0 0"/>
-    <parent link="urdf_simplified_torso"/>
-    <child link="urdf_l_shoulder_assembly"/>
-    <axis xyz="0 1 0"/>
-    <limit effort="100" velocity="100" lower="-3.02" upper="1.69"/>
-    <dynamics damping="0.5" friction="0.1"/>
+    <origin xyz="0 0.1755 0.423977" rpy="0 0 0" />
+    <parent link="urdf_simplified_torso" />
+    <child link="urdf_l_shoulder_assembly" />
+    <axis xyz="0 1 0" />
+    <limit effort="20" velocity="16.02" lower="-3.02" upper="1.69" />
+    <dynamics damping="0.16" friction="1.6" />
   </joint>
   <joint name="left_shoulder_roll_joint_X6" type="revolute">
-    <origin xyz="0.0456571 0.07 0.00560599" rpy="0 -0.122173 0"/>
-    <parent link="urdf_l_shoulder_assembly"/>
-    <child link="urdf_l_upper_arm_assembly"/>
-    <axis xyz="1 0 0"/>
-    <limit effort="100" velocity="100" lower="-0.21" upper="2.93"/>
-    <dynamics damping="0.5" friction="0.1"/>
+    <origin xyz="0.0456571 0.07 0.00560599" rpy="0 -0.122173 0" />
+    <parent link="urdf_l_shoulder_assembly" />
+    <child link="urdf_l_upper_arm_assembly" />
+    <axis xyz="1 0 0" />
+    <limit effort="20" velocity="16.02" lower="-0.21" upper="2.93" />
+    <dynamics damping="0.16" friction="1.6" />
   </joint>
   <joint name="left_shoulder_yaw_joint_X4" type="revolute">
-    <origin xyz="-0.046 0.0343048 -0.161394" rpy="0.209376 0.00530409 -0.0249664"/>
-    <parent link="urdf_l_upper_arm_assembly"/>
-    <child link="urdf_l_elbow_assembly"/>
-    <axis xyz="0 0 1"/>
-    <limit effort="100" velocity="100" lower="-1.75" upper="2.97"/>
-    <dynamics damping="0.5" friction="0.1"/>
+    <origin xyz="-0.046 0.0343048 -0.161394" rpy="0.209376 0.00530409 -0.0249664" />
+    <parent link="urdf_l_upper_arm_assembly" />
+    <child link="urdf_l_elbow_assembly" />
+    <axis xyz="0 0 1" />
+    <limit effort="10.5" velocity="8.69" lower="-1.75" upper="2.97" />
+    <dynamics damping="0.114" friction="1.14" />
   </joint>
   <joint name="left_elbow_pitch_joint_X6" type="revolute">
-    <origin xyz="0.019337 0.0291733 -0.075" rpy="0 -0.0190902 -0.585348"/>
-    <parent link="urdf_l_elbow_assembly"/>
-    <child link="urdf_l_upper_forearm_assembly"/>
-    <axis xyz="0 1 0"/>
-    <limit effort="100" velocity="100" lower="-1.31" upper="1.83"/>
-    <dynamics damping="0.5" friction="0.1"/>
+    <origin xyz="0.019337 0.0291733 -0.075" rpy="0 -0.0190902 -0.585348" />
+    <parent link="urdf_l_elbow_assembly" />
+    <child link="urdf_l_upper_forearm_assembly" />
+    <axis xyz="0 1 0" />
+    <limit effort="20" velocity="16.02" lower="-1.31" upper="1.83" />
+    <dynamics damping="0.16" friction="1.6" />
   </joint>
   <joint name="left_wrist_yaw_joint_X4" type="revolute">
-    <origin xyz="0.0391738 -0.035 -0.158223" rpy="-0.142861 -0.19688 0.634041"/>
-    <parent link="urdf_l_upper_forearm_assembly"/>
-    <child link="urdf_l_lower_forearm_assembly"/>
-    <axis xyz="0 0 1"/>
-    <limit effort="100" velocity="100" lower="-2.36" upper="2.36"/>
-    <dynamics damping="0.5" friction="0.1"/>
+    <origin xyz="0.0391738 -0.035 -0.158223" rpy="-0.142861 -0.19688 0.634041" />
+    <parent link="urdf_l_upper_forearm_assembly" />
+    <child link="urdf_l_lower_forearm_assembly" />
+    <axis xyz="0 0 1" />
+    <limit effort="10.5" velocity="8.69" lower="-2.36" upper="2.36" />
+    <dynamics damping="0.114" friction="1.14" />
   </joint>
   <joint name="left_wrist_roll_joint_X4" type="revolute">
-    <origin xyz="0.0219762 -0.0156859 -0.0615" rpy="-0.248271 0 -0.619909"/>
-    <parent link="urdf_l_lower_forearm_assembly"/>
-    <child link="urdf_l_wrist_assembly"/>
-    <axis xyz="1 0 0"/>
-    <limit effort="100" velocity="100" lower="-1.57" upper="1.57"/>
-    <dynamics damping="0.5" friction="0.1"/>
+    <origin xyz="0.0219762 -0.0156859 -0.0615" rpy="-0.248271 0 -0.619909" />
+    <parent link="urdf_l_lower_forearm_assembly" />
+    <child link="urdf_l_wrist_assembly" />
+    <axis xyz="1 0 0" />
+    <limit effort="10.5" velocity="8.69" lower="-1.57" upper="1.57" />
+    <dynamics damping="0.114" friction="1.14" />
   </joint>
 </robot>

File: src/robot_description/full_robot_description/urdf/joints/left_foot_joints.xacro (robot description, xacro)
@@ -1,54 +1,51 @@
-<?xml version="1.0"?>
-<robot xmlns:xacro="http://www.ros.org/wiki/xacro">
-  <!-- ================================================================== -->
-  <!-- Left Foot                                                         -->
-  <!-- ================================================================== -->
+<?xml version='1.0' encoding='utf-8'?>
+<robot>
   <joint name="left_hip_pitch_joint" type="${leg_joint_type}">
-    <origin xyz="0.0333787 0.111301 -0.467748" rpy="0 0 0"/>
-    <parent link="urdf_base"/>
-    <child link="urdf_hip_assembly"/>
-    <axis xyz="0 1 0"/>
-    <limit effort="100" velocity="100" lower="-2.53" upper="1.57"/>
-    <dynamics damping="0.5" friction="0.1"/>
+    <origin xyz="0.0333787 0.111301 -0.467748" rpy="0 0 0" />
+    <parent link="urdf_base" />
+    <child link="urdf_hip_assembly" />
+    <axis xyz="0 1 0" />
+    <limit effort="43" velocity="13.3" lower="-2.53" upper="1.57" />
+    <dynamics damping="0.321" friction="3.21" />
   </joint>
   <joint name="left_hip_roll_joint" type="${leg_joint_type}">
-    <origin xyz="0.055 0.073 0" rpy="0 0 0"/>
-    <parent link="urdf_hip_assembly"/>
-    <child link="urdf_l_upper_femur_assembly"/>
-    <axis xyz="1 0 0"/>
-    <limit effort="100" velocity="100" lower="-0.35" upper="3.14"/>
-    <dynamics damping="0.5" friction="0.1"/>
+    <origin xyz="0.055 0.073 0" rpy="0 0 0" />
+    <parent link="urdf_hip_assembly" />
+    <child link="urdf_l_upper_femur_assembly" />
+    <axis xyz="1 0 0" />
+    <limit effort="43" velocity="13.3" lower="-0.35" upper="3.14" />
+    <dynamics damping="0.321" friction="3.21" />
   </joint>
   <joint name="left_hip_yaw_joint" type="${leg_joint_type}">
-    <origin xyz="-0.053 -7.97086e-07 -0.217" rpy="0 0 0"/>
-    <parent link="urdf_l_upper_femur_assembly"/>
-    <child link="urdf_lower_femur_assembly"/>
-    <axis xyz="0 0 1"/>
-    <limit effort="100" velocity="100" lower="-1.57" upper="1.57"/>
-    <dynamics damping="0.5" friction="0.1"/>
+    <origin xyz="-0.053 -7.97086e-07 -0.217" rpy="0 0 0" />
+    <parent link="urdf_l_upper_femur_assembly" />
+    <child link="urdf_lower_femur_assembly" />
+    <axis xyz="0 0 1" />
+    <limit effort="43" velocity="13.3" lower="-1.57" upper="1.57" />
+    <dynamics damping="0.321" friction="3.21" />
   </joint>
   <joint name="left_knee_joint" type="${leg_joint_type}">
-    <origin xyz="0 0.055 -0.113" rpy="0 0 0"/>
-    <parent link="urdf_lower_femur_assembly"/>
-    <child link="urdf_l_tibia_assembly"/>
-    <axis xyz="0 1 0"/>
-    <limit effort="100" velocity="100" lower="-0.17" upper="1.57"/>
-    <dynamics damping="0.5" friction="0.1"/>
+    <origin xyz="0 0.055 -0.113" rpy="0 0 0" />
+    <parent link="urdf_lower_femur_assembly" />
+    <child link="urdf_l_tibia_assembly" />
+    <axis xyz="0 1 0" />
+    <limit effort="43" velocity="13.3" lower="-0.17" upper="1.57" />
+    <dynamics damping="0.321" friction="3.21" />
   </joint>
   <joint name="left_ankle_pitch_joint" type="${leg_joint_type}">
-    <origin xyz="-1.45092e-06 -0.051 -0.395" rpy="0 0 0"/>
-    <parent link="urdf_l_tibia_assembly"/>
-    <child link="urdf_ankle_assembly"/>
-    <axis xyz="0 1 0"/>
-    <limit effort="100" velocity="100" lower="-0.79" upper="0.79"/>
-    <dynamics damping="0.5" friction="0.1"/>
+    <origin xyz="-1.45092e-06 -0.051 -0.395" rpy="0 0 0" />
+    <parent link="urdf_l_tibia_assembly" />
+    <child link="urdf_ankle_assembly" />
+    <axis xyz="0 1 0" />
+    <limit effort="43" velocity="13.3" lower="-0.79" upper="0.79" />
+    <dynamics damping="0.321" friction="3.21" />
   </joint>
   <joint name="left_ankle_roll_joint" type="${leg_joint_type}">
-    <origin xyz="-0.0120001 -0.004 -0.028" rpy="0 0 0"/>
-    <parent link="urdf_ankle_assembly"/>
-    <child link="urdf_foot_assembly"/>
-    <axis xyz="1 0 0"/>
-    <limit effort="100" velocity="100" lower="-0.79" upper="0.79"/>
-    <dynamics damping="0.5" friction="0.1"/>
+    <origin xyz="-0.0120001 -0.004 -0.028" rpy="0 0 0" />
+    <parent link="urdf_ankle_assembly" />
+    <child link="urdf_foot_assembly" />
+    <axis xyz="1 0 0" />
+    <limit effort="43" velocity="13.3" lower="-0.79" upper="0.79" />
+    <dynamics damping="0.321" friction="3.21" />
   </joint>
 </robot>

File: src/robot_description/full_robot_description/urdf/joints/right_arm_joints.xacro (robot description, xacro)
@@ -1,54 +1,51 @@
-<?xml version="1.0"?>
-<robot xmlns:xacro="http://www.ros.org/wiki/xacro">
-  <!-- ================================================================== -->
-  <!-- Right Arm                                                         -->
-  <!-- ================================================================== -->
+<?xml version='1.0' encoding='utf-8'?>
+<robot>
   <joint name="right_shoulder_pitch_joint_X6" type="revolute">
-    <origin xyz="0 -0.1755 0.423977" rpy="0 0 0"/>
-    <parent link="urdf_simplified_torso"/>
-    <child link="urdf_r_shoulder_assembly"/>
-    <axis xyz="0 1 0"/>
-    <limit effort="100" velocity="100" lower="-3.02" upper="1.69"/>
-    <dynamics damping="0.5" friction="0.1"/>
+    <origin xyz="0 -0.1755 0.423977" rpy="0 0 0" />
+    <parent link="urdf_simplified_torso" />
+    <child link="urdf_r_shoulder_assembly" />
+    <axis xyz="0 1 0" />
+    <limit effort="20" velocity="16.02" lower="-3.02" upper="1.69" />
+    <dynamics damping="0.16" friction="1.6" />
   </joint>
   <joint name="right_shoulder_roll_joint_X6" type="revolute">
-    <origin xyz="0.0456571 -0.07 0.00560599" rpy="0 -0.122173 0"/>
-    <parent link="urdf_r_shoulder_assembly"/>
-    <child link="urdf_r_upper_arm_assembly"/>
-    <axis xyz="1 0 0"/>
-    <limit effort="100" velocity="100" lower="-2.93" upper="0.21"/>
-    <dynamics damping="0.5" friction="0.1"/>
+    <origin xyz="0.0456571 -0.07 0.00560599" rpy="0 -0.122173 0" />
+    <parent link="urdf_r_shoulder_assembly" />
+    <child link="urdf_r_upper_arm_assembly" />
+    <axis xyz="1 0 0" />
+    <limit effort="20" velocity="16.02" lower="-2.93" upper="0.21" />
+    <dynamics damping="0.16" friction="1.6" />
   </joint>
   <joint name="right_shoulder_yaw_joint_X4" type="revolute">
-    <origin xyz="-0.046 -0.0353456 -0.166285" rpy="-0.209378 0.00530246 0.0249661"/>
-    <parent link="urdf_r_upper_arm_assembly"/>
-    <child link="urdf_r_elbow_assembly"/>
-    <axis xyz="0 0 1"/>
-    <limit effort="100" velocity="100" lower="-2.97" upper="1.75"/>
-    <dynamics damping="0.5" friction="0.1"/>
+    <origin xyz="-0.046 -0.0353456 -0.166285" rpy="-0.209378 0.00530246 0.0249661" />
+    <parent link="urdf_r_upper_arm_assembly" />
+    <child link="urdf_r_elbow_assembly" />
+    <axis xyz="0 0 1" />
+    <limit effort="10.5" velocity="8.69" lower="-2.97" upper="1.75" />
+    <dynamics damping="0.114" friction="1.14" />
   </joint>
   <joint name="right_elbow_pitch_joint_X6" type="revolute">
-    <origin xyz="0.0220994 -0.0333409 -0.065" rpy="0 -0.019088 0.585341"/>
-    <parent link="urdf_r_elbow_assembly"/>
-    <child link="urdf_r_upper_forearm_assembly"/>
-    <axis xyz="0 1 0"/>
-    <limit effort="100" velocity="100" lower="-1.31" upper="1.83"/>
-    <dynamics damping="0.5" friction="0.1"/>
+    <origin xyz="0.0220994 -0.0333409 -0.065" rpy="0 -0.019088 0.585341" />
+    <parent link="urdf_r_elbow_assembly" />
+    <child link="urdf_r_upper_forearm_assembly" />
+    <axis xyz="0 1 0" />
+    <limit effort="20" velocity="16.02" lower="-1.31" upper="1.83" />
+    <dynamics damping="0.16" friction="1.6" />
   </joint>
   <joint name="right_wrist_yaw_joint_X4" type="revolute">
-    <origin xyz="0.0403763 0.04 -0.163076" rpy="0.142857 -0.196885 -0.634033"/>
-    <parent link="urdf_r_upper_forearm_assembly"/>
-    <child link="urdf_r_lower_forearm_assembly"/>
-    <axis xyz="0 0 1"/>
-    <limit effort="100" velocity="100" lower="-2.36" upper="2.36"/>
-    <dynamics damping="0.5" friction="0.1"/>
+    <origin xyz="0.0403763 0.04 -0.163076" rpy="0.142857 -0.196885 -0.634033" />
+    <parent link="urdf_r_upper_forearm_assembly" />
+    <child link="urdf_r_lower_forearm_assembly" />
+    <axis xyz="0 0 1" />
+    <limit effort="10.5" velocity="8.69" lower="-2.36" upper="2.36" />
+    <dynamics damping="0.114" friction="1.14" />
   </joint>
   <joint name="right_wrist_roll_joint_X4" type="revolute">
-    <origin xyz="0.0219763 0.0156857 -0.0565" rpy="0.248281 0 0.619897"/>
-    <parent link="urdf_r_lower_forearm_assembly"/>
-    <child link="urdf_r_wrist_assembly"/>
-    <axis xyz="1 0 0"/>
-    <limit effort="100" velocity="100" lower="-1.57" upper="1.57"/>
-    <dynamics damping="0.5" friction="0.1"/>
+    <origin xyz="0.0219763 0.0156857 -0.0565" rpy="0.248281 0 0.619897" />
+    <parent link="urdf_r_lower_forearm_assembly" />
+    <child link="urdf_r_wrist_assembly" />
+    <axis xyz="1 0 0" />
+    <limit effort="10.5" velocity="8.69" lower="-1.57" upper="1.57" />
+    <dynamics damping="0.114" friction="1.14" />
   </joint>
 </robot>

File: src/robot_description/full_robot_description/urdf/joints/right_foot_joints.xacro (robot description, xacro)
@@ -1,54 +1,51 @@
-<?xml version="1.0"?>
-<robot xmlns:xacro="http://www.ros.org/wiki/xacro">
-  <!-- ================================================================== -->
-  <!-- Right Foot                                                        -->
-  <!-- ================================================================== -->
+<?xml version='1.0' encoding='utf-8'?>
+<robot>
   <joint name="right_hip_pitch_joint" type="${leg_joint_type}">
-    <origin xyz="0.0333787 -0.107699 -0.467748" rpy="0 0 0"/>
-    <parent link="urdf_base"/>
-    <child link="urdf_hip_assembly_2"/>
-    <axis xyz="0 1 0"/>
-    <limit effort="100" velocity="100" lower="-2.53" upper="1.57"/>
-    <dynamics damping="0.5" friction="0.1"/>
+    <origin xyz="0.0333787 -0.107699 -0.467748" rpy="0 0 0" />
+    <parent link="urdf_base" />
+    <child link="urdf_hip_assembly_2" />
+    <axis xyz="0 1 0" />
+    <limit effort="43" velocity="13.3" lower="-2.53" upper="1.57" />
+    <dynamics damping="0.321" friction="3.21" />
   </joint>
   <joint name="right_hip_roll_joint" type="${leg_joint_type}">
-    <origin xyz="0.055 -0.078 0" rpy="0 0 0"/>
-    <parent link="urdf_hip_assembly_2"/>
-    <child link="urdf_r_upper_femur_assemby"/>
-    <axis xyz="1 0 0"/>
-    <limit effort="100" velocity="100" lower="-3.14" upper="0.35"/>
-    <dynamics damping="0.5" friction="0.1"/>
+    <origin xyz="0.055 -0.078 0" rpy="0 0 0" />
+    <parent link="urdf_hip_assembly_2" />
+    <child link="urdf_r_upper_femur_assemby" />
+    <axis xyz="1 0 0" />
+    <limit effort="43" velocity="13.3" lower="-3.14" upper="0.35" />
+    <dynamics damping="0.321" friction="3.21" />
   </joint>
   <joint name="right_hip_yaw_joint" type="${leg_joint_type}">
-    <origin xyz="-0.053 7.97086e-07 -0.217" rpy="0 0 0"/>
-    <parent link="urdf_r_upper_femur_assemby"/>
-    <child link="urdf_lower_femur_assembly_2"/>
-    <axis xyz="0 0 1"/>
-    <limit effort="100" velocity="100" lower="-1.57" upper="1.57"/>
-    <dynamics damping="0.5" friction="0.1"/>
+    <origin xyz="-0.053 7.97086e-07 -0.217" rpy="0 0 0" />
+    <parent link="urdf_r_upper_femur_assemby" />
+    <child link="urdf_lower_femur_assembly_2" />
+    <axis xyz="0 0 1" />
+    <limit effort="43" velocity="13.3" lower="-1.57" upper="1.57" />
+    <dynamics damping="0.321" friction="3.21" />
   </joint>
   <joint name="right_knee_joint" type="${leg_joint_type}">
-    <origin xyz="0 -0.055 -0.113" rpy="0 0 0"/>
-    <parent link="urdf_lower_femur_assembly_2"/>
-    <child link="urdf_r_tibia_assembly"/>
-    <axis xyz="0 1 0"/>
-    <limit effort="100" velocity="100" lower="-0.17" upper="1.57"/>
-    <dynamics damping="0.5" friction="0.1"/>
+    <origin xyz="0 -0.055 -0.113" rpy="0 0 0" />
+    <parent link="urdf_lower_femur_assembly_2" />
+    <child link="urdf_r_tibia_assembly" />
+    <axis xyz="0 1 0" />
+    <limit effort="43" velocity="13.3" lower="-0.17" upper="1.57" />
+    <dynamics damping="0.321" friction="3.21" />
   </joint>
   <joint name="right_ankle_roll_joint" type="${leg_joint_type}">
-    <origin xyz="-4.02748e-07 0.059 -0.395" rpy="0 0 0"/>
-    <parent link="urdf_r_tibia_assembly"/>
-    <child link="urdf_ankle_assembly_2"/>
-    <axis xyz="0 1 0"/>
-    <limit effort="100" velocity="100" lower="-0.79" upper="0.79"/>
-    <dynamics damping="0.5" friction="0.1"/>
+    <origin xyz="-4.02748e-07 0.059 -0.395" rpy="0 0 0" />
+    <parent link="urdf_r_tibia_assembly" />
+    <child link="urdf_ankle_assembly_2" />
+    <axis xyz="0 1 0" />
+    <limit effort="43" velocity="13.3" lower="-0.79" upper="0.79" />
+    <dynamics damping="0.321" friction="3.21" />
   </joint>
   <joint name="right_ankle_pitch_joint" type="${leg_joint_type}">
-    <origin xyz="-0.012 -0.004 -0.028" rpy="0 0 0"/>
-    <parent link="urdf_ankle_assembly_2"/>
-    <child link="urdf_foot_assembly_2"/>
-    <axis xyz="1 0 0"/>
-    <limit effort="100" velocity="100" lower="-0.79" upper="0.79"/>
-    <dynamics damping="0.5" friction="0.1"/>
+    <origin xyz="-0.012 -0.004 -0.028" rpy="0 0 0" />
+    <parent link="urdf_ankle_assembly_2" />
+    <child link="urdf_foot_assembly_2" />
+    <axis xyz="1 0 0" />
+    <limit effort="43" velocity="13.3" lower="-0.79" upper="0.79" />
+    <dynamics damping="0.321" friction="3.21" />
   </joint>
 </robot>
