Commit message: update joint limits using actuator specs

File: src/robot_description/full_robot_description/urdf/robot_harambe_v03_proccessed.urdf (robot description, URDF)
Before this commit: robot robot_harambe_v0.3, 26 links, 25 joints
Joints:
- joint left_ankle_pitch_joint: limit lower=-0.79 upper=0.79 effort=100 velocity=100 -> lower=-0.79 upper=0.79 effort=43 velocity=13.3
- joint left_ankle_roll_joint: limit lower=-0.79 upper=0.79 effort=100 velocity=100 -> lower=-0.79 upper=0.79 effort=43 velocity=13.3
- joint left_elbow_pitch_joint_X6: limit lower=-1.31 upper=1.83 effort=100 velocity=100 -> lower=-1.31 upper=1.83 effort=20 velocity=16.02
- joint left_hip_pitch_joint: limit lower=-2.53 upper=1.57 effort=100 velocity=100 -> lower=-2.53 upper=1.57 effort=43 velocity=13.3
- joint left_hip_roll_joint: limit lower=-0.35 upper=3.14 effort=100 velocity=100 -> lower=-0.35 upper=3.14 effort=43 velocity=13.3
- joint left_hip_yaw_joint: limit lower=-1.57 upper=1.57 effort=100 velocity=100 -> lower=-1.57 upper=1.57 effort=43 velocity=13.3
- joint left_knee_joint: limit lower=-0.17 upper=1.57 effort=100 velocity=100 -> lower=-0.17 upper=1.57 effort=43 velocity=13.3
- joint left_shoulder_pitch_joint_X6: limit lower=-3.02 upper=1.69 effort=100 velocity=100 -> lower=-3.02 upper=1.69 effort=20 velocity=16.02
- joint left_shoulder_roll_joint_X6: limit lower=-0.21 upper=2.93 effort=100 velocity=100 -> lower=-0.21 upper=2.93 effort=20 velocity=16.02
- joint left_shoulder_yaw_joint_X4: limit lower=-1.75 upper=2.97 effort=100 velocity=100 -> lower=-1.75 upper=2.97 effort=10.5 velocity=8.69
- joint left_wrist_roll_joint_X4: limit lower=-1.57 upper=1.57 effort=100 velocity=100 -> lower=-1.57 upper=1.57 effort=10.5 velocity=8.69
- joint left_wrist_yaw_joint_X4: limit lower=-2.36 upper=2.36 effort=100 velocity=100 -> lower=-2.36 upper=2.36 effort=10.5 velocity=8.69
- joint right_ankle_pitch_joint: axis 1 0 0 -> 0 1 0; child urdf_foot_assembly_2 -> urdf_ankle_assembly_2; limit lower=-0.79 upper=0.79 effort=100 velocity=100 -> lower=-0.79 upper=0.79 effort=43 velocity=13.3; origin xyz=-0.012 -0.004 -0.028 rpy=0 0 0 -> xyz=-4.02748e-07 0.059 -0.395 rpy=0 0 0; parent urdf_ankle_assembly_2 -> urdf_r_tibia_assembly
- joint right_ankle_roll_joint: axis 0 1 0 -> 1 0 0; child urdf_ankle_assembly_2 -> urdf_foot_assembly_2; limit lower=-0.79 upper=0.79 effort=100 velocity=100 -> lower=-0.79 upper=0.79 effort=43 velocity=13.3; origin xyz=-4.02748e-07 0.059 -0.395 rpy=0 0 0 -> xyz=-0.012 -0.004 -0.028 rpy=0 0 0; parent urdf_r_tibia_assembly -> urdf_ankle_assembly_2
- joint right_elbow_pitch_joint_X6: limit lower=-1.31 upper=1.83 effort=100 velocity=100 -> lower=-1.31 upper=1.83 effort=20 velocity=16.02
- joint right_hip_pitch_joint: limit lower=-2.53 upper=1.57 effort=100 velocity=100 -> lower=-2.53 upper=1.57 effort=43 velocity=13.3
- joint right_hip_roll_joint: limit lower=-3.14 upper=0.35 effort=100 velocity=100 -> lower=-3.14 upper=0.35 effort=43 velocity=13.3
- joint right_hip_yaw_joint: limit lower=-1.57 upper=1.57 effort=100 velocity=100 -> lower=-1.57 upper=1.57 effort=43 velocity=13.3
- joint right_knee_joint: limit lower=-0.17 upper=1.57 effort=100 velocity=100 -> lower=-0.17 upper=1.57 effort=43 velocity=13.3
- joint right_shoulder_pitch_joint_X6: limit lower=-3.02 upper=1.69 effort=100 velocity=100 -> lower=-3.02 upper=1.69 effort=20 velocity=16.02
- joint right_shoulder_roll_joint_X6: limit lower=-2.93 upper=0.21 effort=100 velocity=100 -> lower=-2.93 upper=0.21 effort=20 velocity=16.02
- joint right_shoulder_yaw_joint_X4: limit lower=-2.97 upper=1.75 effort=100 velocity=100 -> lower=-2.97 upper=1.75 effort=10.5 velocity=8.69
- joint right_wrist_roll_joint_X4: limit lower=-1.57 upper=1.57 effort=100 velocity=100 -> lower=-1.57 upper=1.57 effort=10.5 velocity=8.69
- joint right_wrist_yaw_joint_X4: limit lower=-2.36 upper=2.36 effort=100 velocity=100 -> lower=-2.36 upper=2.36 effort=10.5 velocity=8.69
- joint waist_yaw_joint: limit lower=-1.57 upper=1.57 effort=100 velocity=100 -> lower=-1.57 upper=1.57 effort=43 velocity=13.3

Commit message: update joints names and limits

File: src/robot_description/full_robot_description/urdf/joints/body_joints.xacro (robot description, xacro)
@@ -5,5 +5,5 @@
   <ns0:arg name="only_left" default="true" />
   <ns0:property name="waist_joint_type" value="${'fixed' if '$(arg only_left)' == 'true' or '$(arg fixed_legs)' == 'true' else 'revolute'}" />
-  <joint name="waist_yaw_joint" type="${waist_joint_type}">
+  <joint name="waist_yaw_joint_X8" type="${waist_joint_type}">
     <origin xyz="0.0333787 -0.000698852 -0.300748" rpy="0 0 0" />
     <parent link="urdf_base" />

File: src/robot_description/full_robot_description/urdf/joints/left_foot_joints.xacro (robot description, xacro)
@@ -1,5 +1,5 @@
 <?xml version='1.0' encoding='utf-8'?>
 <robot>
-  <joint name="left_hip_pitch_joint" type="${leg_joint_type}">
+  <joint name="left_hip_pitch_joint_X8" type="${leg_joint_type}">
     <origin xyz="0.0333787 0.111301 -0.467748" rpy="0 0 0" />
     <parent link="urdf_base" />
@@ -9,5 +9,5 @@
     <dynamics damping="0.321" friction="3.21" />
   </joint>
-  <joint name="left_hip_roll_joint" type="${leg_joint_type}">
+  <joint name="left_hip_roll_joint_X8" type="${leg_joint_type}">
     <origin xyz="0.055 0.073 0" rpy="0 0 0" />
     <parent link="urdf_hip_assembly" />
@@ -17,5 +17,5 @@
     <dynamics damping="0.321" friction="3.21" />
   </joint>
-  <joint name="left_hip_yaw_joint" type="${leg_joint_type}">
+  <joint name="left_hip_yaw_joint_X8" type="${leg_joint_type}">
     <origin xyz="-0.053 -7.97086e-07 -0.217" rpy="0 0 0" />
     <parent link="urdf_l_upper_femur_assembly" />
@@ -25,5 +25,5 @@
     <dynamics damping="0.321" friction="3.21" />
   </joint>
-  <joint name="left_knee_joint" type="${leg_joint_type}">
+  <joint name="left_knee_joint_X8" type="${leg_joint_type}">
     <origin xyz="0 0.055 -0.113" rpy="0 0 0" />
     <parent link="urdf_lower_femur_assembly" />
@@ -33,19 +33,19 @@
     <dynamics damping="0.321" friction="3.21" />
   </joint>
-  <joint name="left_ankle_pitch_joint" type="${leg_joint_type}">
+  <joint name="left_ankle_pitch_joint_X4" type="${leg_joint_type}">
     <origin xyz="-1.45092e-06 -0.051 -0.395" rpy="0 0 0" />
     <parent link="urdf_l_tibia_assembly" />
     <child link="urdf_ankle_assembly" />
     <axis xyz="0 1 0" />
-    <limit effort="43" velocity="13.3" lower="-0.79" upper="0.79" />
-    <dynamics damping="0.321" friction="3.21" />
+    <limit effort="10.5" velocity="8.69" lower="-0.79" upper="0.79" />
+    <dynamics damping="0.114" friction="1.14" />
   </joint>
-  <joint name="left_ankle_roll_joint" type="${leg_joint_type}">
+  <joint name="left_ankle_roll_joint_X4" type="${leg_joint_type}">
     <origin xyz="-0.0120001 -0.004 -0.028" rpy="0 0 0" />
     <parent link="urdf_ankle_assembly" />
     <child link="urdf_foot_assembly" />
     <axis xyz="1 0 0" />
-    <limit effort="43" velocity="13.3" lower="-0.79" upper="0.79" />
-    <dynamics damping="0.321" friction="3.21" />
+    <limit effort="10.5" velocity="8.69" lower="-0.79" upper="0.79" />
+    <dynamics damping="0.114" friction="1.14" />
   </joint>
 </robot>

File: src/robot_description/full_robot_description/urdf/joints/right_foot_joints.xacro (robot description, xacro)
@@ -1,5 +1,5 @@
 <?xml version='1.0' encoding='utf-8'?>
 <robot>
-  <joint name="right_hip_pitch_joint" type="${leg_joint_type}">
+  <joint name="right_hip_pitch_joint_X8" type="${leg_joint_type}">
     <origin xyz="0.0333787 -0.107699 -0.467748" rpy="0 0 0" />
     <parent link="urdf_base" />
@@ -9,5 +9,5 @@
     <dynamics damping="0.321" friction="3.21" />
   </joint>
-  <joint name="right_hip_roll_joint" type="${leg_joint_type}">
+  <joint name="right_hip_roll_joint_X8" type="${leg_joint_type}">
     <origin xyz="0.055 -0.078 0" rpy="0 0 0" />
     <parent link="urdf_hip_assembly_2" />
@@ -17,5 +17,5 @@
     <dynamics damping="0.321" friction="3.21" />
   </joint>
-  <joint name="right_hip_yaw_joint" type="${leg_joint_type}">
+  <joint name="right_hip_yaw_joint_X8" type="${leg_joint_type}">
     <origin xyz="-0.053 7.97086e-07 -0.217" rpy="0 0 0" />
     <parent link="urdf_r_upper_femur_assemby" />
@@ -25,5 +25,5 @@
     <dynamics damping="0.321" friction="3.21" />
   </joint>
-  <joint name="right_knee_joint" type="${leg_joint_type}">
+  <joint name="right_knee_joint_X8" type="${leg_joint_type}">
     <origin xyz="0 -0.055 -0.113" rpy="0 0 0" />
     <parent link="urdf_lower_femur_assembly_2" />
@@ -33,19 +33,19 @@
     <dynamics damping="0.321" friction="3.21" />
   </joint>
-  <joint name="right_ankle_roll_joint" type="${leg_joint_type}">
+  <joint name="right_ankle_roll_joint_X4" type="${leg_joint_type}">
     <origin xyz="-4.02748e-07 0.059 -0.395" rpy="0 0 0" />
     <parent link="urdf_r_tibia_assembly" />
     <child link="urdf_ankle_assembly_2" />
     <axis xyz="0 1 0" />
-    <limit effort="43" velocity="13.3" lower="-0.79" upper="0.79" />
-    <dynamics damping="0.321" friction="3.21" />
+    <limit effort="10.5" velocity="8.69" lower="-0.79" upper="0.79" />
+    <dynamics damping="0.114" friction="1.14" />
   </joint>
-  <joint name="right_ankle_pitch_joint" type="${leg_joint_type}">
+  <joint name="right_ankle_pitch_joint_X4" type="${leg_joint_type}">
     <origin xyz="-0.012 -0.004 -0.028" rpy="0 0 0" />
     <parent link="urdf_ankle_assembly_2" />
     <child link="urdf_foot_assembly_2" />
     <axis xyz="1 0 0" />
-    <limit effort="43" velocity="13.3" lower="-0.79" upper="0.79" />
-    <dynamics damping="0.321" friction="3.21" />
+    <limit effort="10.5" velocity="8.69" lower="-0.79" upper="0.79" />
+    <dynamics damping="0.114" friction="1.14" />
   </joint>
 </robot>

File: src/robot_description/full_robot_description/urdf/robot_harambe_v03_proccessed.urdf (robot description, URDF)
Before this commit: robot robot_harambe_v0.3, 26 links, 25 joints
Joints:
- removed joint left_ankle_pitch_joint
- removed joint left_ankle_roll_joint
- removed joint left_hip_pitch_joint
- removed joint left_hip_roll_joint
- removed joint left_hip_yaw_joint
- removed joint left_knee_joint
- removed joint right_ankle_pitch_joint
- removed joint right_ankle_roll_joint
- removed joint right_hip_pitch_joint
- removed joint right_hip_roll_joint
- removed joint right_hip_yaw_joint
- removed joint right_knee_joint
- removed joint waist_yaw_joint
- added joint left_ankle_pitch_joint_X4: type revolute, parent urdf_l_tibia_assembly, child urdf_ankle_assembly, origin xyz=-1.45092e-06 -0.051 -0.395 rpy=0 0 0, axis 0 1 0, limit lower=-0.79 upper=0.79 effort=10.5 velocity=8.69
- added joint left_ankle_roll_joint_X4: type revolute, parent urdf_ankle_assembly, child urdf_foot_assembly, origin xyz=-0.0120001 -0.004 -0.028 rpy=0 0 0, axis 1 0 0, limit lower=-0.79 upper=0.79 effort=10.5 velocity=8.69
- added joint left_hip_pitch_joint_X8: type revolute, parent urdf_base, child urdf_hip_assembly, origin xyz=0.0333787 0.111301 -0.467748 rpy=0 0 0, axis 0 1 0, limit lower=-2.53 upper=1.57 effort=43 velocity=13.3
- added joint left_hip_roll_joint_X8: type revolute, parent urdf_hip_assembly, child urdf_l_upper_femur_assembly, origin xyz=0.055 0.073 0 rpy=0 0 0, axis 1 0 0, limit lower=-0.35 upper=3.14 effort=43 velocity=13.3
- added joint left_hip_yaw_joint_X8: type revolute, parent urdf_l_upper_femur_assembly, child urdf_lower_femur_assembly, origin xyz=-0.053 -7.97086e-07 -0.217 rpy=0 0 0, axis 0 0 1, limit lower=-1.57 upper=1.57 effort=43 velocity=13.3
- added joint left_knee_joint_X8: type revolute, parent urdf_lower_femur_assembly, child urdf_l_tibia_assembly, origin xyz=0 0.055 -0.113 rpy=0 0 0, axis 0 1 0, limit lower=-0.17 upper=1.57 effort=43 velocity=13.3
- added joint right_ankle_pitch_joint_X4: type revolute, parent urdf_r_tibia_assembly, child urdf_ankle_assembly_2, origin xyz=-4.02748e-07 0.059 -0.395 rpy=0 0 0, axis 0 1 0, limit lower=-0.79 upper=0.79 effort=10.5 velocity=8.69
- added joint right_ankle_roll_joint_X4: type revolute, parent urdf_ankle_assembly_2, child urdf_foot_assembly_2, origin xyz=-0.012 -0.004 -0.028 rpy=0 0 0, axis 1 0 0, limit lower=-0.79 upper=0.79 effort=10.5 velocity=8.69
- added joint right_hip_pitch_joint_X8: type revolute, parent urdf_base, child urdf_hip_assembly_2, origin xyz=0.0333787 -0.107699 -0.467748 rpy=0 0 0, axis 0 1 0, limit lower=-2.53 upper=1.57 effort=43 velocity=13.3
- added joint right_hip_roll_joint_X8: type revolute, parent urdf_hip_assembly_2, child urdf_r_upper_femur_assemby, origin xyz=0.055 -0.078 0 rpy=0 0 0, axis 1 0 0, limit lower=-3.14 upper=0.35 effort=43 velocity=13.3
- added joint right_hip_yaw_joint_X8: type revolute, parent urdf_r_upper_femur_assemby, child urdf_lower_femur_assembly_2, origin xyz=-0.053 7.97086e-07 -0.217 rpy=0 0 0, axis 0 0 1, limit lower=-1.57 upper=1.57 effort=43 velocity=13.3
- added joint right_knee_joint_X8: type revolute, parent urdf_lower_femur_assembly_2, child urdf_r_tibia_assembly, origin xyz=0 -0.055 -0.113 rpy=0 0 0, axis 0 1 0, limit lower=-0.17 upper=1.57 effort=43 velocity=13.3
- added joint waist_yaw_joint_X8: type revolute, parent urdf_base, child urdf_simplified_torso, origin xyz=0.0333787 -0.000698852 -0.300748 rpy=0 0 0, axis 0 0 1, limit lower=-1.57 upper=1.57 effort=43 velocity=13.3

Commit message: add full robot simulation

File: src/robot_description/full_robot_description/urdf/joints/body_joints.xacro (robot description, xacro)
@@ -1,8 +1,8 @@
 <?xml version='1.0' encoding='utf-8'?>
-<robot xmlns:ns0="http://www.ros.org/wiki/xacro">
-  <ns0:arg name="fixed_legs" default="false" />
-  <ns0:property name="leg_joint_type" value="${'fixed' if '$(arg fixed_legs)' == 'true' else 'revolute'}" />
-  <ns0:arg name="only_left" default="true" />
-  <ns0:property name="waist_joint_type" value="${'fixed' if '$(arg only_left)' == 'true' or '$(arg fixed_legs)' == 'true' else 'revolute'}" />
+<robot xmlns:xacro="http://www.ros.org/wiki/xacro">
+  <xacro:arg name="fixed_legs" default="false" />
+  <xacro:property name="leg_joint_type" value="${'fixed' if '$(arg fixed_legs)' == 'true' else 'revolute'}" />
+  <xacro:arg name="only_left" default="true" />
+  <xacro:property name="waist_joint_type" value="${'fixed' if '$(arg only_left)' == 'true' or '$(arg fixed_legs)' == 'true' else 'revolute'}" />
   <joint name="waist_yaw_joint_X8" type="${waist_joint_type}">
     <origin xyz="0.0333787 -0.000698852 -0.300748" rpy="0 0 0" />

Commit message: final callibration, 98% complete

File: src/robot_description/full_robot_description/urdf/joints/body_joints.xacro (robot description, xacro)
@@ -19,5 +19,5 @@
     <child link="urdf_simplified_torso"/>
     <axis xyz="0 0 1"/>
-    <limit effort="100" velocity="100" lower="-1.57" upper="1.57"/>
+    <limit effort="100" velocity="100" lower="-2.6005" upper="2.60054"/>
     <dynamics damping="0.5" friction="0.1"/>
   </joint>

File: src/robot_description/full_robot_description/urdf/joints/left_arm_joints.xacro (robot description, xacro)
@@ -9,5 +9,5 @@
     <child link="urdf_l_shoulder_assembly"/>
     <axis xyz="0 1 0"/>
-    <limit effort="8" velocity="2" lower="-3.02" upper="1.69"/>
+    <limit effort="8" velocity="2" lower="-3.0194" upper="1.69296"/>
     <dynamics damping="0.5" friction="0.1"/>
   </joint>
@@ -17,5 +17,5 @@
     <child link="urdf_l_upper_arm_assembly"/>
     <axis xyz="1 0 0"/>
-    <limit effort="8" velocity="2" lower="-0.21" upper="2.93"/>
+    <limit effort="8" velocity="2" lower="-0.2094" upper="2.93215"/>
     <dynamics damping="0.5" friction="0.1"/>
   </joint>
@@ -25,5 +25,5 @@
     <child link="urdf_l_elbow_assembly"/>
     <axis xyz="0 0 1"/>
-    <limit effort="8" velocity="2" lower="-1.75" upper="2.97"/>
+    <limit effort="8" velocity="2" lower="-1.7453" upper="2.96705"/>
     <dynamics damping="0.5" friction="0.1"/>
   </joint>
@@ -33,5 +33,5 @@
     <child link="urdf_l_upper_forearm_assembly"/>
     <axis xyz="0 1 0"/>
-    <limit effort="8" velocity="2" lower="-1.31" upper="1.83"/>
+    <limit effort="8" velocity="2" lower="-1.3089" upper="1.8326"/>
     <dynamics damping="0.5" friction="0.1"/>
   </joint>
@@ -41,5 +41,5 @@
     <child link="urdf_l_lower_forearm_assembly"/>
     <axis xyz="0 0 1"/>
-    <limit effort="8" velocity="2" lower="-2.36" upper="2.36"/>
+    <limit effort="8" velocity="2" lower="-2.3561" upper="2.35619"/>
     <dynamics damping="0.5" friction="0.1"/>
   </joint>
@@ -49,5 +49,5 @@
     <child link="urdf_l_wrist_assembly"/>
     <axis xyz="1 0 0"/>
-    <limit effort="8" velocity="2" lower="-1.57" upper="1.57"/>
+    <limit effort="8" velocity="2" lower="-1.5707" upper="1.57079"/>
     <dynamics damping="0.5" friction="0.1"/>
   </joint>

File: src/robot_description/full_robot_description/urdf/joints/left_foot_joints.xacro (robot description, xacro)
@@ -9,5 +9,5 @@
     <child link="urdf_hip_assembly"/>
     <axis xyz="0 1 0"/>
-    <limit effort="100" velocity="100" lower="-2.53" upper="1.57"/>
+    <limit effort="100" velocity="100" lower="-4.4680" upper="1.3265"/>
     <dynamics damping="0.5" friction="0.1"/>
   </joint>
@@ -17,5 +17,5 @@
     <child link="urdf_l_upper_femur_assembly"/>
     <axis xyz="1 0 0"/>
-    <limit effort="100" velocity="100" lower="-0.35" upper="3.14"/>
+    <limit effort="100" velocity="100" lower="-0.3490" upper="3.31612"/>
     <dynamics damping="0.5" friction="0.1"/>
   </joint>
@@ -25,5 +25,5 @@
     <child link="urdf_lower_femur_assembly"/>
     <axis xyz="0 0 1"/>
-    <limit effort="100" velocity="100" lower="-1.57" upper="1.57"/>
+    <limit effort="100" velocity="100" lower="-2.2689" upper="3.5256"/>
     <dynamics damping="0.5" friction="0.1"/>
   </joint>
@@ -33,5 +33,5 @@
     <child link="urdf_l_tibia_assembly"/>
     <axis xyz="0 1 0"/>
-    <limit effort="100" velocity="100" lower="-0.17" upper="1.57"/>
+    <limit effort="100" velocity="100" lower="-1.5271" upper="1.52716"/>
     <dynamics damping="0.5" friction="0.1"/>
   </joint>
@@ -41,5 +41,5 @@
     <child link="urdf_ankle_assembly"/>
     <axis xyz="0 1 0"/>
-    <limit effort="100" velocity="100" lower="-0.79" upper="0.79"/>
+    <limit effort="100" velocity="100" lower="-0.7853" upper="0.78539"/>
     <dynamics damping="0.5" friction="0.1"/>
   </joint>
@@ -49,5 +49,5 @@
     <child link="urdf_foot_assembly"/>
     <axis xyz="1 0 0"/>
-    <limit effort="100" velocity="100" lower="-0.79" upper="0.79"/>
+    <limit effort="100" velocity="100" lower="-0.7853" upper="0.78539"/>
     <dynamics damping="0.5" friction="0.1"/>
   </joint>

File: src/robot_description/full_robot_description/urdf/joints/right_arm_joints.xacro (robot description, xacro)
@@ -9,5 +9,5 @@
     <child link="urdf_r_shoulder_assembly"/>
     <axis xyz="0 1 0"/>
-    <limit effort="8" velocity="2" lower="-3.02" upper="1.69"/>
+    <limit effort="8" velocity="2" lower="-3.0194" upper="1.69296"/>
     <dynamics damping="0.5" friction="0.1"/>
   </joint>
@@ -17,5 +17,5 @@
     <child link="urdf_r_upper_arm_assembly"/>
     <axis xyz="1 0 0"/>
-    <limit effort="8" velocity="2" lower="-2.93" upper="0.21"/>
+    <limit effort="8" velocity="2" lower="-2.9321" upper="0.20943"/>
     <dynamics damping="0.5" friction="0.1"/>
   </joint>
@@ -25,5 +25,5 @@
     <child link="urdf_r_elbow_assembly"/>
     <axis xyz="0 0 1"/>
-    <limit effort="8" velocity="2" lower="-2.97" upper="1.75"/>
+    <limit effort="8" velocity="2" lower="-2.9670" upper="1.74532"/>
     <dynamics damping="0.5" friction="0.1"/>
   </joint>
@@ -33,5 +33,5 @@
     <child link="urdf_r_upper_forearm_assembly"/>
     <axis xyz="0 1 0"/>
-    <limit effort="8" velocity="2" lower="-1.31" upper="1.83"/>
+    <limit effort="8" velocity="2" lower="-1.3089" upper="1.8326"/>
     <dynamics damping="0.5" friction="0.1"/>
   </joint>
@@ -41,5 +41,5 @@
     <child link="urdf_r_lower_forearm_assembly"/>
     <axis xyz="0 0 1"/>
-    <limit effort="8" velocity="2" lower="-2.36" upper="2.36"/>
+    <limit effort="8" velocity="2" lower="-2.3561" upper="2.35619"/>
     <dynamics damping="0.5" friction="0.1"/>
   </joint>
@@ -49,5 +49,5 @@
     <child link="urdf_r_wrist_assembly"/>
     <axis xyz="1 0 0"/>
-    <limit effort="8" velocity="2" lower="-1.57" upper="1.57"/>
+    <limit effort="8" velocity="2" lower="-1.5707" upper="1.57079"/>
     <dynamics damping="0.5" friction="0.1"/>
   </joint>

File: src/robot_description/full_robot_description/urdf/joints/right_foot_joints.xacro (robot description, xacro)
@@ -9,5 +9,5 @@
     <child link="urdf_hip_assembly_2"/>
     <axis xyz="0 1 0"/>
-    <limit effort="100" velocity="100" lower="-2.53" upper="1.57"/>
+    <limit effort="100" velocity="100" lower="-2.7576" upper="2.75762"/>
     <dynamics damping="0.5" friction="0.1"/>
   </joint>
@@ -17,5 +17,5 @@
     <child link="urdf_r_upper_femur_assemby"/>
     <axis xyz="1 0 0"/>
-    <limit effort="100" velocity="100" lower="-3.14" upper="0.35"/>
+    <limit effort="100" velocity="100" lower="-3.3161" upper="0.34906"/>
     <dynamics damping="0.5" friction="0.1"/>
   </joint>
@@ -25,5 +25,5 @@
     <child link="urdf_lower_femur_assembly_2"/>
     <axis xyz="0 0 1"/>
-    <limit effort="100" velocity="100" lower="-1.57" upper="1.57"/>
+    <limit effort="100" velocity="100" lower="-2.7576" upper="2.75762"/>
     <dynamics damping="0.5" friction="0.1"/>
   </joint>
@@ -33,5 +33,5 @@
     <child link="urdf_r_tibia_assembly"/>
     <axis xyz="0 1 0"/>
-    <limit effort="100" velocity="100" lower="-0.17" upper="1.57"/>
+    <limit effort="100" velocity="100" lower="-1.5271" upper="1.52716"/>
     <dynamics damping="0.5" friction="0.1"/>
   </joint>
@@ -41,5 +41,5 @@
     <child link="urdf_ankle_assembly_2"/>
     <axis xyz="0 1 0"/>
-    <limit effort="100" velocity="100" lower="-0.79" upper="0.79"/>
+    <limit effort="100" velocity="100" lower="-0.7853" upper="0.78539"/>
     <dynamics damping="0.5" friction="0.1"/>
   </joint>
@@ -49,5 +49,5 @@
     <child link="urdf_foot_assembly_2"/>
     <axis xyz="1 0 0"/>
-    <limit effort="100" velocity="100" lower="-0.79" upper="0.79"/>
+    <limit effort="100" velocity="100" lower="-0.7853" upper="0.78539"/>
     <dynamics damping="0.5" friction="0.1"/>
   </joint>
