Commit message: harambe v0.4

File: src/robot_description/full_robot_description/urdf/joints/body_joints.xacro (robot description, xacro)
@@ -1,15 +1,24 @@
-<?xml version='1.0' encoding='utf-8'?>
+<?xml version="1.0"?>
 <robot xmlns:xacro="http://www.ros.org/wiki/xacro">
-  <xacro:arg name="fixed_legs" default="false" />
-  <xacro:property name="leg_joint_type" value="${'fixed' if '$(arg fixed_legs)' == 'true' else 'revolute'}" />
-  <xacro:arg name="only_left" default="true" />
-  <xacro:property name="waist_joint_type" value="${'fixed' if '$(arg only_left)' == 'true' or '$(arg fixed_legs)' == 'true' else 'revolute'}" />
+  <!-- ================================================================== -->
+  <!-- Leg joint type — set fixed_legs:=true to lock leg joints          -->
+  <!-- ================================================================== -->
+  <xacro:arg name="fixed_legs" default="false"/>
+  <xacro:property name="leg_joint_type" value="${'fixed' if '$(arg fixed_legs)' == 'true' else 'revolute'}"/>
+  <!-- ================================================================== -->
+  <!-- only_left — when true, also lock waist yaw joint                  -->
+  <!-- ================================================================== -->
+  <xacro:arg name="only_left" default="true"/>
+  <xacro:property name="waist_joint_type" value="${'fixed' if '$(arg only_left)' == 'true' or '$(arg fixed_legs)' == 'true' else 'revolute'}"/>
+  <!-- ================================================================== -->
+  <!-- Body                                                              -->
+  <!-- ================================================================== -->
   <joint name="waist_yaw_joint_X8" type="${waist_joint_type}">
-    <origin xyz="0.0333787 -0.000698852 -0.300748" rpy="0 0 0" />
-    <parent link="urdf_base" />
-    <child link="urdf_simplified_torso" />
-    <axis xyz="0 0 1" />
-    <limit effort="${X8_moderate_effort}" velocity="${X8_rated_velocity}" lower="-1.57" upper="1.57" />
-    <dynamics damping="${X8_damping}" friction="${X8_friction}" />
+    <origin xyz="0.070373 -0.000705351 -0.281099" rpy="0 0 0"/>
+    <parent link="urdf_base"/>
+    <child link="urdf_simplified_torso"/>
+    <axis xyz="0 0 1"/>
+    <limit effort="${X8_moderate_effort}" velocity="${X8_rated_velocity}" lower="-1.57" upper="1.57"/>
+    <dynamics friction="${X8_friction}" damping="${X8_damping}"/>
   </joint>
 </robot>

File: src/robot_description/full_robot_description/urdf/joints/left_arm_joints.xacro (robot description, xacro)
@@ -1,51 +1,54 @@
-<?xml version='1.0' encoding='utf-8'?>
-<robot>
+<?xml version="1.0"?>
+<robot xmlns:xacro="http://www.ros.org/wiki/xacro">
+  <!-- ================================================================== -->
+  <!-- Left Arm                                                          -->
+  <!-- ================================================================== -->
   <joint name="left_shoulder_pitch_joint_X6" type="revolute">
-    <origin xyz="0 0.1755 0.423977" rpy="0 0 0" />
-    <parent link="urdf_simplified_torso" />
-    <child link="urdf_l_shoulder_assembly" />
-    <axis xyz="0 1 0" />
-    <limit effort="${X6_moderate_effort}" velocity="${X6_rated_velocity}" lower="-3.02" upper="1.69" />
-    <dynamics damping="${X6_damping}" friction="${X6_friction}" />
+    <origin xyz="0 0.1695 0.423977" rpy="0 0 0"/>
+    <parent link="urdf_simplified_torso"/>
+    <child link="urdf_l_shoulder_assembly"/>
+    <axis xyz="0 1 0"/>
+    <limit effort="${X6_moderate_effort}" velocity="${X6_rated_velocity}" lower="-3.02" upper="1.69"/>
+    <dynamics friction="${X6_friction}" damping="${X6_damping}"/>
   </joint>
   <joint name="left_shoulder_roll_joint_X6" type="revolute">
-    <origin xyz="0.0456571 0.07 0.00560599" rpy="0 -0.122173 0" />
-    <parent link="urdf_l_shoulder_assembly" />
-    <child link="urdf_l_upper_arm_assembly" />
-    <axis xyz="1 0 0" />
-    <limit effort="${X6_moderate_effort}" velocity="${X6_rated_velocity}" lower="-0.21" upper="2.93" />
-    <dynamics damping="${X6_damping}" friction="${X6_friction}" />
+    <origin xyz="0.0456571 0.07 0.00560611" rpy="0 -0.122176 0"/>
+    <parent link="urdf_l_shoulder_assembly"/>
+    <child link="urdf_l_upper_arm_assembly"/>
+    <axis xyz="1 0 0"/>
+    <limit effort="${X6_moderate_effort}" velocity="${X6_rated_velocity}" lower="-0.21" upper="2.93"/>
+    <dynamics friction="${X6_friction}" damping="${X6_damping}"/>
   </joint>
   <joint name="left_shoulder_yaw_joint_X4" type="revolute">
-    <origin xyz="-0.046 0.0343048 -0.161394" rpy="0.209376 0.00530409 -0.0249664" />
-    <parent link="urdf_l_upper_arm_assembly" />
-    <child link="urdf_l_elbow_assembly" />
-    <axis xyz="0 0 1" />
-    <limit effort="${X4_moderate_effort}" velocity="${X4_rated_velocity}" lower="-1.75" upper="2.97" />
-    <dynamics damping="${X4_damping}" friction="${X4_friction}" />
+    <origin xyz="-0.046 0.034306 -0.161394" rpy="0.209383 0.00530439 -0.024967"/>
+    <parent link="urdf_l_upper_arm_assembly"/>
+    <child link="urdf_l_elbow_assembly"/>
+    <axis xyz="0 0 1"/>
+    <limit effort="${X4_moderate_effort}" velocity="${X4_rated_velocity}" lower="-1.75" upper="2.97"/>
+    <dynamics friction="${X4_friction}" damping="${X4_damping}"/>
   </joint>
   <joint name="left_elbow_pitch_joint_X6" type="revolute">
-    <origin xyz="0.019337 0.0291733 -0.075" rpy="0 -0.0190902 -0.585348" />
-    <parent link="urdf_l_elbow_assembly" />
-    <child link="urdf_l_upper_forearm_assembly" />
-    <axis xyz="0 1 0" />
-    <limit effort="${X6_moderate_effort}" velocity="${X6_rated_velocity}" lower="-1.31" upper="1.83" />
-    <dynamics damping="${X6_damping}" friction="${X6_friction}" />
+    <origin xyz="0.0193369 0.0291733 -0.075" rpy="0 -0.0190922 -0.585347"/>
+    <parent link="urdf_l_elbow_assembly"/>
+    <child link="urdf_l_upper_forearm_assembly"/>
+    <axis xyz="0 1 0"/>
+    <limit effort="${X6_moderate_effort}" velocity="${X6_rated_velocity}" lower="-1.31" upper="1.83"/>
+    <dynamics friction="${X6_friction}" damping="${X6_damping}"/>
   </joint>
   <joint name="left_wrist_yaw_joint_X4" type="revolute">
-    <origin xyz="0.0391738 -0.035 -0.158223" rpy="-0.142861 -0.19688 0.634041" />
-    <parent link="urdf_l_upper_forearm_assembly" />
-    <child link="urdf_l_lower_forearm_assembly" />
-    <axis xyz="0 0 1" />
-    <limit effort="${X4_moderate_effort}" velocity="${X4_rated_velocity}" lower="-2.36" upper="2.36" />
-    <dynamics damping="${X4_damping}" friction="${X4_friction}" />
+    <origin xyz="0.0391735 -0.035 -0.158223" rpy="-0.14286 -0.196878 0.634041"/>
+    <parent link="urdf_l_upper_forearm_assembly"/>
+    <child link="urdf_l_lower_forearm_assembly"/>
+    <axis xyz="0 0 1"/>
+    <limit effort="${X4_moderate_effort}" velocity="${X4_rated_velocity}" lower="-2.36" upper="2.36"/>
+    <dynamics friction="${X4_friction}" damping="${X4_damping}"/>
   </joint>
   <joint name="left_wrist_roll_joint_X4" type="revolute">
-    <origin xyz="0.0219762 -0.0156859 -0.0615" rpy="-0.248271 0 -0.619909" />
-    <parent link="urdf_l_lower_forearm_assembly" />
-    <child link="urdf_l_wrist_assembly" />
-    <axis xyz="1 0 0" />
-    <limit effort="${X4_moderate_effort}" velocity="${X4_rated_velocity}" lower="-1.57" upper="1.57" />
-    <dynamics damping="${X4_damping}" friction="${X4_friction}" />
+    <origin xyz="0.0219762 -0.0156859 -0.0615" rpy="-0.248279 0 -0.619909"/>
+    <parent link="urdf_l_lower_forearm_assembly"/>
+    <child link="urdf_l_wrist_assembly"/>
+    <axis xyz="1 0 0"/>
+    <limit effort="${X4_moderate_effort}" velocity="${X4_rated_velocity}" lower="-1.57" upper="1.57"/>
+    <dynamics friction="${X4_friction}" damping="${X4_damping}"/>
   </joint>
 </robot>

File: src/robot_description/full_robot_description/urdf/joints/left_foot_joints.xacro (robot description, xacro)
@@ -1,51 +1,54 @@
-<?xml version='1.0' encoding='utf-8'?>
-<robot>
+<?xml version="1.0"?>
+<robot xmlns:xacro="http://www.ros.org/wiki/xacro">
+  <!-- ================================================================== -->
+  <!-- Left Foot                                                         -->
+  <!-- ================================================================== -->
   <joint name="left_hip_pitch_joint_X8" type="${leg_joint_type}">
-    <origin xyz="0.0333787 0.072699 -0.467748" rpy="0 0 0" />
-    <parent link="urdf_base" />
-    <child link="urdf_hip_assembly" />
-    <axis xyz="0 1 0" />
-    <limit effort="${X8_moderate_effort}" velocity="${X8_rated_velocity}" lower="-2.53" upper="1.57" />
-    <dynamics damping="${X8_damping}" friction="${X8_friction}" />
+    <origin xyz="0.070373 0.0872946 -0.431099" rpy="0 0 0"/>
+    <parent link="urdf_base"/>
+    <child link="urdf_hip_assembly"/>
+    <axis xyz="0 1 0"/>
+    <limit effort="${X8_moderate_effort}" velocity="${X8_rated_velocity}" lower="-2.53" upper="1.57"/>
+    <dynamics friction="${X8_friction}" damping="${X8_damping}"/>
   </joint>
   <joint name="left_hip_roll_joint_X8" type="${leg_joint_type}">
-    <origin xyz="0.055 0.073 0" rpy="0 0 0" />
-    <parent link="urdf_hip_assembly" />
-    <child link="urdf_l_upper_femur_assembly" />
-    <axis xyz="1 0 0" />
-    <limit effort="${X8_moderate_effort}" velocity="${X8_rated_velocity}" lower="-0.35" upper="3.14" />
-    <dynamics damping="${X8_damping}" friction="${X8_friction}" />
+    <origin xyz="0.053 0.062 0" rpy="0 0 0"/>
+    <parent link="urdf_hip_assembly"/>
+    <child link="urdf_l_upper_femur_assembly"/>
+    <axis xyz="1 0 0"/>
+    <limit effort="${X8_moderate_effort}" velocity="${X8_rated_velocity}" lower="-0.35" upper="3.14"/>
+    <dynamics friction="${X8_friction}" damping="${X8_damping}"/>
   </joint>
   <joint name="left_hip_yaw_joint_X8" type="${leg_joint_type}">
-    <origin xyz="-0.053 -7.97086e-07 -0.217" rpy="0 0 0" />
-    <parent link="urdf_l_upper_femur_assembly" />
-    <child link="urdf_lower_femur_assembly" />
-    <axis xyz="0 0 1" />
-    <limit effort="${X8_moderate_effort}" velocity="${X8_rated_velocity}" lower="-1.57" upper="1.57" />
-    <dynamics damping="${X8_damping}" friction="${X8_friction}" />
+    <origin xyz="-0.053 0 -0.217" rpy="0 0 0"/>
+    <parent link="urdf_l_upper_femur_assembly"/>
+    <child link="urdf_lower_femur_assembly"/>
+    <axis xyz="0 0 1"/>
+    <limit effort="${X8_moderate_effort}" velocity="${X8_rated_velocity}" lower="-1.57" upper="1.57"/>
+    <dynamics friction="${X8_friction}" damping="${X8_damping}"/>
   </joint>
   <joint name="left_knee_joint_X8" type="${leg_joint_type}">
-    <origin xyz="0 0.055 -0.113" rpy="0 0 0" />
-    <parent link="urdf_lower_femur_assembly" />
-    <child link="urdf_l_tibia_assembly" />
-    <axis xyz="0 1 0" />
-    <limit effort="${X8_moderate_effort}" velocity="${X8_rated_velocity}" lower="-0.17" upper="1.57" />
-    <dynamics damping="${X8_damping}" friction="${X8_friction}" />
+    <origin xyz="-1.45947e-07 0.055 -0.111" rpy="0 0 0"/>
+    <parent link="urdf_lower_femur_assembly"/>
+    <child link="urdf_l_tibia_assembly"/>
+    <axis xyz="0 1 0"/>
+    <limit effort="${X8_moderate_effort}" velocity="${X8_rated_velocity}" lower="-0.17" upper="1.57"/>
+    <dynamics friction="${X8_friction}" damping="${X8_damping}"/>
   </joint>
   <joint name="left_ankle_pitch_joint_X4" type="${leg_joint_type}">
-    <origin xyz="-1.45092e-06 -0.051 -0.395" rpy="0 0 0" />
-    <parent link="urdf_l_tibia_assembly" />
-    <child link="urdf_ankle_assembly" />
-    <axis xyz="0 1 0" />
-    <limit effort="${ankle_pitch_moderate_effort}" velocity="${ankle_pitch_rated_velocity}" lower="-0.79" upper="0.79" />
-    <dynamics damping="${X4_damping}" friction="${X4_friction}" />
+    <origin xyz="0 -0.051 -0.395" rpy="0 0 0"/>
+    <parent link="urdf_l_tibia_assembly"/>
+    <child link="udrf_ankle_assembly"/>
+    <axis xyz="0 1 0"/>
+    <limit effort="${X4_moderate_effort}" velocity="${X4_rated_velocity}" lower="-0.79" upper="0.79"/>
+    <dynamics friction="${X4_friction}" damping="${X4_damping}"/>
   </joint>
   <joint name="left_ankle_roll_joint_X4" type="${leg_joint_type}">
-    <origin xyz="-0.0120001 -0.004 -0.028" rpy="0 0 0" />
-    <parent link="urdf_ankle_assembly" />
-    <child link="urdf_foot_assembly" />
-    <axis xyz="1 0 0" />
-    <limit effort="${ankle_roll_moderate_effort}" velocity="${ankle_roll_rated_velocity}" lower="-0.79" upper="0.79" />
-    <dynamics damping="${X4_damping}" friction="${X4_friction}" />
+    <origin xyz="-0.012 -0.004 -0.028" rpy="0 0 0"/>
+    <parent link="udrf_ankle_assembly"/>
+    <child link="urdf_foot_assembly"/>
+    <axis xyz="1 0 0"/>
+    <limit effort="${X4_moderate_effort}" velocity="${X4_rated_velocity}" lower="-0.79" upper="0.79"/>
+    <dynamics friction="${X4_friction}" damping="${X4_damping}"/>
   </joint>
 </robot>

File: src/robot_description/full_robot_description/urdf/joints/right_arm_joints.xacro (robot description, xacro)
@@ -1,51 +1,54 @@
-<?xml version='1.0' encoding='utf-8'?>
-<robot>
+<?xml version="1.0"?>
+<robot xmlns:xacro="http://www.ros.org/wiki/xacro">
+  <!-- ================================================================== -->
+  <!-- Right Arm                                                         -->
+  <!-- ================================================================== -->
   <joint name="right_shoulder_pitch_joint_X6" type="revolute">
-    <origin xyz="0 -0.1755 0.423977" rpy="0 0 0" />
-    <parent link="urdf_simplified_torso" />
-    <child link="urdf_r_shoulder_assembly" />
-    <axis xyz="0 1 0" />
-    <limit effort="${X6_moderate_effort}" velocity="${X6_rated_velocity}" lower="-3.02" upper="1.69" />
-    <dynamics damping="${X6_damping}" friction="${X6_friction}" />
+    <origin xyz="0 -0.1695 0.423977" rpy="0 0 0"/>
+    <parent link="urdf_simplified_torso"/>
+    <child link="urdf_r_shoulder_assembly"/>
+    <axis xyz="0 1 0"/>
+    <limit effort="${X6_moderate_effort}" velocity="${X6_rated_velocity}" lower="-3.02" upper="1.69"/>
+    <dynamics friction="${X6_friction}" damping="${X6_damping}"/>
   </joint>
   <joint name="right_shoulder_roll_joint_X6" type="revolute">
-    <origin xyz="0.0456571 -0.07 0.00560599" rpy="0 -0.122173 0" />
-    <parent link="urdf_r_shoulder_assembly" />
-    <child link="urdf_r_upper_arm_assembly" />
-    <axis xyz="1 0 0" />
-    <limit effort="${X6_moderate_effort}" velocity="${X6_rated_velocity}" lower="-2.93" upper="0.21" />
-    <dynamics damping="${X6_damping}" friction="${X6_friction}" />
+    <origin xyz="0.0456571 -0.07 0.00560611" rpy="0 -0.122176 0"/>
+    <parent link="urdf_r_shoulder_assembly"/>
+    <child link="urdf_r_upper_arm_assembly"/>
+    <axis xyz="1 0 0"/>
+    <limit effort="${X6_moderate_effort}" velocity="${X6_rated_velocity}" lower="-2.93" upper="0.21"/>
+    <dynamics friction="${X6_friction}" damping="${X6_damping}"/>
   </joint>
   <joint name="right_shoulder_yaw_joint_X4" type="revolute">
-    <origin xyz="-0.046 -0.0353456 -0.166285" rpy="-0.209378 0.00530246 0.0249661" />
-    <parent link="urdf_r_upper_arm_assembly" />
-    <child link="urdf_r_elbow_assembly" />
-    <axis xyz="0 0 1" />
-    <limit effort="${X4_moderate_effort}" velocity="${X4_rated_velocity}" lower="-2.97" upper="1.75" />
-    <dynamics damping="${X4_damping}" friction="${X4_friction}" />
+    <origin xyz="-0.046 -0.0353444 -0.166285" rpy="-0.20937 0.00530239 0.0249667"/>
+    <parent link="urdf_r_upper_arm_assembly"/>
+    <child link="urdf_r_elbow_assembly"/>
+    <axis xyz="0 0 1"/>
+    <limit effort="${X4_moderate_effort}" velocity="${X4_rated_velocity}" lower="-2.97" upper="1.75"/>
+    <dynamics friction="${X4_friction}" damping="${X4_damping}"/>
   </joint>
   <joint name="right_elbow_pitch_joint_X6" type="revolute">
-    <origin xyz="0.0220994 -0.0333409 -0.065" rpy="0 -0.019088 0.585341" />
-    <parent link="urdf_r_elbow_assembly" />
-    <child link="urdf_r_upper_forearm_assembly" />
-    <axis xyz="0 1 0" />
-    <limit effort="${X6_moderate_effort}" velocity="${X6_rated_velocity}" lower="-1.31" upper="1.83" />
-    <dynamics damping="${X6_damping}" friction="${X6_friction}" />
+    <origin xyz="0.0220994 -0.033341 -0.065" rpy="0 -0.0190815 0.58534"/>
+    <parent link="urdf_r_elbow_assembly"/>
+    <child link="urdf_r_upper_forearm_assembly"/>
+    <axis xyz="0 1 0"/>
+    <limit effort="${X6_moderate_effort}" velocity="${X6_rated_velocity}" lower="-1.31" upper="1.83"/>
+    <dynamics friction="${X6_friction}" damping="${X6_damping}"/>
   </joint>
   <joint name="right_wrist_yaw_joint_X4" type="revolute">
-    <origin xyz="0.0403763 0.04 -0.163076" rpy="0.142857 -0.196885 -0.634033" />
-    <parent link="urdf_r_upper_forearm_assembly" />
-    <child link="urdf_r_lower_forearm_assembly" />
-    <axis xyz="0 0 1" />
-    <limit effort="${X4_moderate_effort}" velocity="${X4_rated_velocity}" lower="-2.36" upper="2.36" />
-    <dynamics damping="${X4_damping}" friction="${X4_friction}" />
+    <origin xyz="0.0403774 0.04 -0.163076" rpy="0.142861 -0.196891 -0.634034"/>
+    <parent link="urdf_r_upper_forearm_assembly"/>
+    <child link="urdf_r_lower_forearm_assembly"/>
+    <axis xyz="0 0 1"/>
+    <limit effort="${X4_moderate_effort}" velocity="${X4_rated_velocity}" lower="-2.36" upper="2.36"/>
+    <dynamics friction="${X4_friction}" damping="${X4_damping}"/>
   </joint>
   <joint name="right_wrist_roll_joint_X4" type="revolute">
-    <origin xyz="0.0219763 0.0156857 -0.0565" rpy="0.248281 0 0.619897" />
-    <parent link="urdf_r_lower_forearm_assembly" />
-    <child link="urdf_r_wrist_assembly" />
-    <axis xyz="1 0 0" />
-    <limit effort="${X4_moderate_effort}" velocity="${X4_rated_velocity}" lower="-1.57" upper="1.57" />
-    <dynamics damping="${X4_damping}" friction="${X4_friction}" />
+    <origin xyz="0.0219763 0.0156857 -0.0565" rpy="0.248276 0 0.619896"/>
+    <parent link="urdf_r_lower_forearm_assembly"/>
+    <child link="urdf_r_wrist_assembly"/>
+    <axis xyz="1 0 0"/>
+    <limit effort="${X4_moderate_effort}" velocity="${X4_rated_velocity}" lower="-1.57" upper="1.57"/>
+    <dynamics friction="${X4_friction}" damping="${X4_damping}"/>
   </joint>
 </robot>
