Commit message: harambe v0.4

File: src/robot_description/full_robot_description/urdf/joints/right_foot_joints.xacro (robot description, xacro)
@@ -1,51 +1,54 @@
-<?xml version='1.0' encoding='utf-8'?>
-<robot>
+<?xml version="1.0"?>
+<robot xmlns:xacro="http://www.ros.org/wiki/xacro">
+  <!-- ================================================================== -->
+  <!-- Right Foot                                                        -->
+  <!-- ================================================================== -->
   <joint name="right_hip_pitch_joint_X8" type="${leg_joint_type}">
-    <origin xyz="0.0333787 -0.072699 -0.467748" rpy="0 0 0" />
-    <parent link="urdf_base" />
-    <child link="urdf_hip_assembly_2" />
-    <axis xyz="0 1 0" />
-    <limit effort="${X8_moderate_effort}" velocity="${X8_rated_velocity}" lower="-2.53" upper="1.57" />
-    <dynamics damping="${X8_damping}" friction="${X8_friction}" />
+    <origin xyz="0.070373 -0.0887054 -0.431099" rpy="0 0 0"/>
+    <parent link="urdf_base"/>
+    <child link="urdf_hip_assembly_2"/>
+    <axis xyz="0 1 0"/>
+    <limit effort="${X8_moderate_effort}" velocity="${X8_rated_velocity}" lower="-2.53" upper="1.57"/>
+    <dynamics friction="${X8_friction}" damping="${X8_damping}"/>
   </joint>
   <joint name="right_hip_roll_joint_X8" type="${leg_joint_type}">
-    <origin xyz="0.055 -0.073 0" rpy="0 0 0" />
-    <parent link="urdf_hip_assembly_2" />
-    <child link="urdf_r_upper_femur_assemby" />
-    <axis xyz="1 0 0" />
-    <limit effort="${X8_moderate_effort}" velocity="${X8_rated_velocity}" lower="-3.14" upper="0.35" />
-    <dynamics damping="${X8_damping}" friction="${X8_friction}" />
+    <origin xyz="0.053 -0.062 0" rpy="0 0 0"/>
+    <parent link="urdf_hip_assembly_2"/>
+    <child link="urdf_r_upper_femur_assemby"/>
+    <axis xyz="1 0 0"/>
+    <limit effort="${X8_moderate_effort}" velocity="${X8_rated_velocity}" lower="-3.14" upper="0.35"/>
+    <dynamics friction="${X8_friction}" damping="${X8_damping}"/>
   </joint>
   <joint name="right_hip_yaw_joint_X8" type="${leg_joint_type}">
-    <origin xyz="-0.053 7.97086e-07 -0.217" rpy="0 0 0" />
-    <parent link="urdf_r_upper_femur_assemby" />
-    <child link="urdf_lower_femur_assembly_2" />
-    <axis xyz="0 0 1" />
-    <limit effort="${X8_moderate_effort}" velocity="${X8_rated_velocity}" lower="-1.57" upper="1.57" />
-    <dynamics damping="${X8_damping}" friction="${X8_friction}" />
+    <origin xyz="-0.053 0 -0.217" rpy="0 0 0"/>
+    <parent link="urdf_r_upper_femur_assemby"/>
+    <child link="urdf_lower_femur_assembly_2"/>
+    <axis xyz="0 0 1"/>
+    <limit effort="${X8_moderate_effort}" velocity="${X8_rated_velocity}" lower="-1.57" upper="1.57"/>
+    <dynamics friction="${X8_friction}" damping="${X8_damping}"/>
   </joint>
   <joint name="right_knee_joint_X8" type="${leg_joint_type}">
-    <origin xyz="0 -0.055 -0.113" rpy="0 0 0" />
-    <parent link="urdf_lower_femur_assembly_2" />
-    <child link="urdf_r_tibia_assembly" />
-    <axis xyz="0 1 0" />
-    <limit effort="${X8_moderate_effort}" velocity="${X8_rated_velocity}" lower="-0.17" upper="1.57" />
-    <dynamics damping="${X8_damping}" friction="${X8_friction}" />
+    <origin xyz="1.45947e-07 -0.055 -0.111" rpy="0 0 0"/>
+    <parent link="urdf_lower_femur_assembly_2"/>
+    <child link="urdf_r_tibia_assembly"/>
+    <axis xyz="0 1 0"/>
+    <limit effort="${X8_moderate_effort}" velocity="${X8_rated_velocity}" lower="-0.17" upper="1.57"/>
+    <dynamics friction="${X8_friction}" damping="${X8_damping}"/>
+  </joint>
+  <joint name="right_ankle_roll_joint_X4" type="${leg_joint_type}">
+    <origin xyz="0 0.059 -0.395" rpy="0 0 0"/>
+    <parent link="urdf_r_tibia_assembly"/>
+    <child link="udrf_ankle_assembly_2"/>
+    <axis xyz="1 0 0"/>
+    <limit effort="${X4_moderate_effort}" velocity="${X4_rated_velocity}" lower="-0.79" upper="0.79"/>
+    <dynamics friction="${X4_friction}" damping="${X4_damping}"/>
   </joint>
   <joint name="right_ankle_pitch_joint_X4" type="${leg_joint_type}">
-    <origin xyz="-4.02748e-07 0.051 -0.395" rpy="0 0 0" />
-    <parent link="urdf_r_tibia_assembly" />
-    <child link="urdf_ankle_assembly_2" />
-    <axis xyz="0 1 0" />
-    <limit effort="${ankle_pitch_moderate_effort}" velocity="${ankle_pitch_rated_velocity}" lower="-0.79" upper="0.79" />
-    <dynamics damping="${X4_damping}" friction="${X4_friction}" />
-  </joint>
-  <joint name="right_ankle_roll_joint_X4" type="${leg_joint_type}">
-    <origin xyz="-0.012 -0.004 -0.028" rpy="0 0 0" />
-    <parent link="urdf_ankle_assembly_2" />
-    <child link="urdf_foot_assembly_2" />
-    <axis xyz="1 0 0" />
-    <limit effort="${ankle_roll_moderate_effort}" velocity="${ankle_roll_rated_velocity}" lower="-0.79" upper="0.79" />
-    <dynamics damping="${X4_damping}" friction="${X4_friction}" />
+    <origin xyz="-0.012 -0.004 -0.028" rpy="0 0 0"/>
+    <parent link="udrf_ankle_assembly_2"/>
+    <child link="urdf_foot_assembly_2"/>
+    <axis xyz="0 1 0"/>
+    <limit effort="${X4_moderate_effort}" velocity="${X4_rated_velocity}" lower="-0.79" upper="0.79"/>
+    <dynamics friction="${X4_friction}" damping="${X4_damping}"/>
   </joint>
 </robot>
