Commit message: limts correction

File: src/robot_description/full_robot_description/urdf/joints/left_foot_joints.xacro (robot description, xacro)
@@ -33,5 +33,5 @@
     <child link="urdf_l_tibia_assembly"/>
     <axis xyz="0 1 0"/>
-    <limit effort="100" velocity="100" lower="0.191906" upper="-2.33882"/>
+    <limit effort="100" velocity="100" lower="-0.191906" upper="2.33882"/>
     <dynamics damping="0.5" friction="0.1"/>
   </joint>

Commit message: typo correction for v03

File: src/robot_description/full_robot_description/urdf/joints/left_foot_joints.xacro (robot description, xacro)
@@ -39,5 +39,5 @@
     <origin xyz="-1.45092e-06 -0.051 -0.395" rpy="0 0 0"/>
     <parent link="urdf_l_tibia_assembly"/>
-    <child link="udrf_ankle_assembly"/>
+    <child link="urdf_ankle_assembly"/>
     <axis xyz="0 1 0"/>
     <limit effort="100" velocity="100" lower="-0.79" upper="0.79"/>
@@ -46,5 +46,5 @@
   <joint name="left_ankle_roll_joint" type="${leg_joint_type}">
     <origin xyz="-0.0120001 -0.004 -0.028" rpy="0 0 0"/>
-    <parent link="udrf_ankle_assembly"/>
+    <parent link="urdf_ankle_assembly"/>
     <child link="urdf_foot_assembly"/>
     <axis xyz="1 0 0"/>

File: src/robot_description/full_robot_description/urdf/joints/right_foot_joints.xacro (robot description, xacro)
@@ -39,5 +39,5 @@
     <origin xyz="-4.02748e-07 0.059 -0.395" rpy="0 0 0"/>
     <parent link="urdf_r_tibia_assembly"/>
-    <child link="udrf_ankle_assembly_2"/>
+    <child link="urdf_ankle_assembly_2"/>
     <axis xyz="0 1 0"/>
     <limit effort="100" velocity="100" lower="-0.79" upper="0.79"/>
@@ -46,5 +46,5 @@
   <joint name="right_ankle_pitch_joint" type="${leg_joint_type}">
     <origin xyz="-0.012 -0.004 -0.028" rpy="0 0 0"/>
-    <parent link="udrf_ankle_assembly_2"/>
+    <parent link="urdf_ankle_assembly_2"/>
     <child link="urdf_foot_assembly_2"/>
     <axis xyz="1 0 0"/>

File: src/robot_description/full_robot_description/urdf/links/left_foot_links.xacro (robot description, xacro)
@@ -173,5 +173,5 @@
     </visual>
   </link>
-  <link name="udrf_ankle_assembly">
+  <link name="urdf_ankle_assembly">
     <inertial>
       <origin xyz="-4.60715e-08 -0.004 -0.0125426" rpy="0 0 0"/>
@@ -182,7 +182,7 @@
       <origin xyz="-4.60715e-08 -0.004 -0.0125426" rpy="0 0 -1.5708"/>
       <geometry>
-        <mesh filename="package://full_robot_description/meshes/visual/udrf_ankle_assembly.stl"/>
-      </geometry>
-      <material name="udrf_ankle_assembly_material">
+        <mesh filename="package://full_robot_description/meshes/visual/urdf_ankle_assembly.stl"/>
+      </geometry>
+      <material name="urdf_ankle_assembly_material">
         <color rgba="0.615686 0.811765 0.929412 1"/>
       </material>
@@ -191,5 +191,5 @@
       <origin xyz="-4.60715e-08 -0.004 -0.0125426" rpy="0 0 -1.5708"/>
       <geometry>
-        <mesh filename="package://full_robot_description/meshes/collision/udrf_ankle_assembly.stl"/>
+        <mesh filename="package://full_robot_description/meshes/collision/urdf_ankle_assembly.stl"/>
       </geometry>
     </collision>

File: src/robot_description/full_robot_description/urdf/links/right_foot_links.xacro (robot description, xacro)
@@ -173,5 +173,5 @@
     </visual>
   </link>
-  <link name="udrf_ankle_assembly_2">
+  <link name="urdf_ankle_assembly_2">
     <inertial>
       <origin xyz="-1.27886e-08 -0.004 -0.0125426" rpy="0 0 0"/>
@@ -182,7 +182,7 @@
       <origin xyz="-1.27886e-08 -0.004 -0.0125426" rpy="0 0 -1.5708"/>
       <geometry>
-        <mesh filename="package://full_robot_description/meshes/visual/udrf_ankle_assembly.stl"/>
-      </geometry>
-      <material name="udrf_ankle_assembly_2_material">
+        <mesh filename="package://full_robot_description/meshes/visual/urdf_ankle_assembly.stl"/>
+      </geometry>
+      <material name="urdf_ankle_assembly_2_material">
         <color rgba="0.615686 0.811765 0.929412 1"/>
       </material>
@@ -191,5 +191,5 @@
       <origin xyz="-1.27886e-08 -0.004 -0.0125426" rpy="0 0 -1.5708"/>
       <geometry>
-        <mesh filename="package://full_robot_description/meshes/collision/udrf_ankle_assembly.stl"/>
+        <mesh filename="package://full_robot_description/meshes/collision/urdf_ankle_assembly.stl"/>
       </geometry>
     </collision>

File: src/robot_description/full_robot_description/urdf/robot_harambe_v03_proccessed.urdf (robot description, URDF)
Before this commit: robot robot_harambe_v0.3, 26 links, 25 joints
Links:
- removed link udrf_ankle_assembly
- removed link udrf_ankle_assembly_2
- added link urdf_ankle_assembly, mass 0.0818219; collision mesh filename=package://meshes/collision/urdf_ankle_assembly.stl; visual mesh filename=package://meshes/visual/urdf_ankle_assembly.stl
- added link urdf_ankle_assembly_2, mass 0.0818219; collision mesh filename=package://meshes/collision/urdf_ankle_assembly.stl; visual mesh filename=package://meshes/visual/urdf_ankle_assembly.stl
Joints:
- joint left_ankle_pitch_joint: child udrf_ankle_assembly -> urdf_ankle_assembly
- joint left_ankle_roll_joint: parent udrf_ankle_assembly -> urdf_ankle_assembly
- joint right_ankle_pitch_joint: parent udrf_ankle_assembly_2 -> urdf_ankle_assembly_2
- joint right_ankle_roll_joint: child udrf_ankle_assembly_2 -> urdf_ankle_assembly_2

Commit message: Fix left/right leg asymmetry using smaller absolute Y values
Corrected 6 asymmetric Y offsets in hip and ankle joints/links.
Right hip assembly was 5mm wider than left, right ankle pitch
8mm offset. Used smaller absolute values as reference for symmetry.

File: src/robot_description/full_robot_description/urdf/joints/left_foot_joints.xacro (robot description, xacro)
@@ -2,5 +2,5 @@
 <robot>
   <joint name="left_hip_pitch_joint_X8" type="${leg_joint_type}">
-    <origin xyz="0.0333787 0.076301 -0.467748" rpy="0 0 0" />
+    <origin xyz="0.0333787 0.072699 -0.467748" rpy="0 0 0" />
     <parent link="urdf_base" />
     <child link="urdf_hip_assembly" />

File: src/robot_description/full_robot_description/urdf/joints/right_foot_joints.xacro (robot description, xacro)
@@ -10,5 +10,5 @@
   </joint>
   <joint name="right_hip_roll_joint_X8" type="${leg_joint_type}">
-    <origin xyz="0.055 -0.078 0" rpy="0 0 0" />
+    <origin xyz="0.055 -0.073 0" rpy="0 0 0" />
     <parent link="urdf_hip_assembly_2" />
     <child link="urdf_r_upper_femur_assemby" />
@@ -34,5 +34,5 @@
   </joint>
   <joint name="right_ankle_pitch_joint_X4" type="${leg_joint_type}">
-    <origin xyz="-4.02748e-07 0.059 -0.395" rpy="0 0 0" />
+    <origin xyz="-4.02748e-07 0.051 -0.395" rpy="0 0 0" />
     <parent link="urdf_r_tibia_assembly" />
     <child link="urdf_ankle_assembly_2" />

File: src/robot_description/full_robot_description/urdf/links/right_foot_links.xacro (robot description, xacro)
@@ -6,10 +6,10 @@
   <link name="urdf_hip_assembly_2">
     <inertial>
-      <origin xyz="-0.00420762 -0.0739982 6.23945e-06" rpy="0 0 0"/>
+      <origin xyz="-0.00420762 -0.0689982 6.23945e-06" rpy="0 0 0"/>
       <mass value="1.73"/>
       <inertia ixx="0.00302301" ixy="-2.30858e-05" ixz="-4.5747e-08" iyy="0.00228746" iyz="-8.49179e-07" izz="0.00263533"/>
     </inertial>
     <visual>
-      <origin xyz="0.00253653 -0.0570203 3.27638e-05" rpy="-3.14159 0 1.5708"/>
+      <origin xyz="0.00253653 -0.0520203 3.27638e-05" rpy="-3.14159 0 1.5708"/>
       <geometry>
         <mesh filename="package://full_robot_description/meshes/visual/hip.stl"/>
@@ -20,5 +20,5 @@
     </visual>
     <collision>
-      <origin xyz="0.00253653 -0.0570203 3.27638e-05" rpy="-3.14159 0 1.5708"/>
+      <origin xyz="0.00253653 -0.0520203 3.27638e-05" rpy="-3.14159 0 1.5708"/>
       <geometry>
         <mesh filename="package://full_robot_description/meshes/collision/hip.stl"/>
@@ -26,5 +26,5 @@
     </collision>
     <visual>
-      <origin xyz="-0.043 -0.078 0" rpy="-1.57079 0 -1.5708"/>
+      <origin xyz="-0.043 -0.073 0" rpy="-1.57079 0 -1.5708"/>
       <geometry>
         <mesh filename="package://full_robot_description/meshes/visual/stator_x8_p20_120_unified.stl"/>

File: src/robot_description/full_robot_description/urdf/robot_harambe_v04_short_processeded.urdf (robot description, URDF)
Before this commit: robot robot_harambe_v0.3, 26 links, 25 joints
Joints:
- joint left_hip_pitch_joint: origin xyz=0.0333787 0.076301 -0.467748 rpy=0 0 0 -> xyz=0.0333787 0.072699 -0.467748 rpy=0 0 0
- joint right_ankle_pitch_joint: origin xyz=-4.02748e-07 0.059 -0.395 rpy=0 0 0 -> xyz=-4.02748e-07 0.051 -0.395 rpy=0 0 0
- joint right_hip_roll_joint: origin xyz=0.055 -0.078 0 rpy=0 0 0 -> xyz=0.055 -0.073 0 rpy=0 0 0

Commit message: review harambe v0.4

File: src/robot_description/full_robot_description/urdf/joints/left_foot_joints.xacro (robot description, xacro)
@@ -39,5 +39,5 @@
     <origin xyz="0 -0.051 -0.395" rpy="0 0 0"/>
     <parent link="urdf_l_tibia_assembly"/>
-    <child link="udrf_ankle_assembly"/>
+    <child link="urdf_ankle_assembly"/>
     <axis xyz="0 1 0"/>
     <limit effort="${X4_moderate_effort}" velocity="${X4_rated_velocity}" lower="-0.79" upper="0.79"/>
@@ -46,5 +46,5 @@
   <joint name="left_ankle_roll_joint_X4" type="${leg_joint_type}">
     <origin xyz="-0.012 -0.004 -0.028" rpy="0 0 0"/>
-    <parent link="udrf_ankle_assembly"/>
+    <parent link="urdf_ankle_assembly"/>
     <child link="urdf_foot_assembly"/>
     <axis xyz="1 0 0"/>

File: src/robot_description/full_robot_description/urdf/joints/right_foot_joints.xacro (robot description, xacro)
@@ -36,19 +36,19 @@
     <dynamics friction="${X8_friction}" damping="${X8_damping}"/>
   </joint>
-  <joint name="right_ankle_roll_joint_X4" type="${leg_joint_type}">
+  <joint name="right_ankle_pitch_joint_X4" type="${leg_joint_type}">
     <origin xyz="0 0.059 -0.395" rpy="0 0 0"/>
     <parent link="urdf_r_tibia_assembly"/>
-    <child link="udrf_ankle_assembly_2"/>
+    <child link="urdf_ankle_assembly_2"/>
+    <axis xyz="0 1 0"/>
+    <limit effort="${X4_moderate_effort}" velocity="${X4_rated_velocity}" lower="-0.79" upper="0.79"/>
+    <dynamics friction="${X4_friction}" damping="${X4_damping}"/>
+  </joint>
+  <joint name="right_ankle_roll_joint_X4" type="${leg_joint_type}">
+    <origin xyz="-0.012 -0.004 -0.028" rpy="0 0 0"/>
+    <parent link="urdf_ankle_assembly_2"/>
+    <child link="urdf_foot_assembly_2"/>
     <axis xyz="1 0 0"/>
     <limit effort="${X4_moderate_effort}" velocity="${X4_rated_velocity}" lower="-0.79" upper="0.79"/>
     <dynamics friction="${X4_friction}" damping="${X4_damping}"/>
   </joint>
-  <joint name="right_ankle_pitch_joint_X4" type="${leg_joint_type}">
-    <origin xyz="-0.012 -0.004 -0.028" rpy="0 0 0"/>
-    <parent link="udrf_ankle_assembly_2"/>
-    <child link="urdf_foot_assembly_2"/>
-    <axis xyz="0 1 0"/>
-    <limit effort="${X4_moderate_effort}" velocity="${X4_rated_velocity}" lower="-0.79" upper="0.79"/>
-    <dynamics friction="${X4_friction}" damping="${X4_damping}"/>
-  </joint>
 </robot>

File: src/robot_description/full_robot_description/urdf/robot_harambe_v04_fixed_axes_simplified_no_collision.urdf (robot description, URDF)
Before this commit: robot robot_harambe_v04, 26 links, 25 joints
Links:
- removed link udrf_ankle_assembly
- removed link udrf_ankle_assembly_2
- added link urdf_ankle_assembly, mass 0.0818219; collision mesh filename=package://meshes/collision/urdf_ankle_assembly.stl; visual mesh filename=package://meshes/visual/urdf_ankle_assembly.stl
- added link urdf_ankle_assembly_2, mass 0.0818219; collision mesh filename=package://meshes/collision/urdf_ankle_assembly.stl; visual mesh filename=package://meshes/visual/urdf_ankle_assembly.stl
Joints:
- joint left_ankle_pitch_joint_X4: child udrf_ankle_assembly -> urdf_ankle_assembly
- joint left_ankle_roll_joint_X4: parent udrf_ankle_assembly -> urdf_ankle_assembly
- joint right_ankle_pitch_joint_X4: parent udrf_ankle_assembly_2 -> urdf_ankle_assembly_2
- joint right_ankle_roll_joint_X4: child udrf_ankle_assembly_2 -> urdf_ankle_assembly_2
