Commit message: swap right ankle pitch and roll

File: src/robot_description/full_robot_description/urdf/joints/right_foot_joints.xacro (robot description, xacro)
@@ -36,5 +36,5 @@
     <dynamics damping="${X8_damping}" friction="${X8_friction}"/>
   </joint>
-  <joint name="right_ankle_roll_joint_X4" type="${leg_joint_type}">
+  <joint name="right_ankle_pitch_joint_X4" type="${leg_joint_type}">
     <origin xyz="0 0.059 -0.395" rpy="0 0 0"/>
     <parent link="urdf_r_tibia_assembly"/>
@@ -44,5 +44,5 @@
     <dynamics damping="${X4_damping}" friction="${X4_friction}"/>
   </joint>
-  <joint name="right_ankle_pitch_joint_X4" type="${leg_joint_type}">
+  <joint name="right_ankle_roll_joint_X4" type="${leg_joint_type}">
     <origin xyz="-0.012 -0.004 -0.028" rpy="0 0 0"/>
     <parent link="urdf_ankle_assembly_2"/>
