Commit message: Remove finger joints from mc_rtc, fix right ankle naming, tune standing pose
- Remove 24 finger/hand joints from mc_rtc config (harambe.json, HarambeCoMPosture.yaml, PDgains_sim.dat)
- Convert finger joints to fixed in generate_urdf.sh URDF processing
- Fix right_ankle_pitch/roll name swap in right_foot_joints.xacro (axes were mismatched)
- Add armature=0.01 and damping=0.1 to all hinge joints for numerical stability
- Improve MuJoCo solver settings (impratio=10, Newton solver, 50 iterations)
- Set crouched standing pose (hip=-0.15, knee=0.3, ankle=-0.15) for stable CoM
- Increase leg PD gains (ankle pitch Kp=500, hip/knee Kp=400)
- Organize joint order consistently across all config files (left arm→right arm→waist→left leg→right leg)

File: src/control/mc_rtc_controller/urdf/harambe_mc_rtc.urdf (robot description, URDF)
Before this commit: robot full_robot_description, 62 links, 61 joints
Links:
- added link pelvis_imu_link; visual sphere radius=0.002
- added link pelvis_imu_sensor, mass 0.0042339; collision mesh filename=/home/alex/Documents/GitHub/ldr-harambe-arms-sim2real/src/r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; visual mesh filename=/home/alex/Documents/GitHub/ldr-harambe-arms-sim2real/src/r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
- added link torso_imu_link; visual sphere radius=0.002
- added link torso_imu_sensor, mass 0.0042339; collision mesh filename=/home/alex/Documents/GitHub/ldr-harambe-arms-sim2real/src/r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; visual mesh filename=/home/alex/Documents/GitHub/ldr-harambe-arms-sim2real/src/r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
Joints:
- removed joint left_ankle_pitch_joint
- removed joint left_ankle_roll_joint
- removed joint left_hip_pitch_joint
- removed joint left_hip_roll_joint
- removed joint left_hip_yaw_joint
- removed joint left_knee_joint
- removed joint right_ankle_pitch_joint
- removed joint right_ankle_roll_joint
- removed joint right_hip_pitch_joint
- removed joint right_hip_roll_joint
- removed joint right_hip_yaw_joint
- removed joint right_knee_joint
- removed joint waist_yaw_joint
- added joint left_ankle_pitch_joint_X4: type revolute, parent urdf_l_tibia_assembly, child urdf_ankle_assembly, origin xyz=-1.45092e-06 -0.051 -0.395 rpy=0 0 0, axis 0 1 0, limit lower=-0.79 upper=0.79 effort=10.5 velocity=8.69
- added joint left_ankle_roll_joint_X4: type revolute, parent urdf_ankle_assembly, child urdf_foot_assembly, origin xyz=-0.0120001 -0.004 -0.028 rpy=0 0 0, axis 1 0 0, limit lower=-0.79 upper=0.79 effort=10.5 velocity=8.69
- added joint left_hip_pitch_joint_X8: type revolute, parent urdf_base, child urdf_hip_assembly, origin xyz=0.0333787 0.111301 -0.467748 rpy=0 0 0, axis 0 1 0, limit lower=-2.53 upper=1.57 effort=43 velocity=13.3
- added joint left_hip_roll_joint_X8: type revolute, parent urdf_hip_assembly, child urdf_l_upper_femur_assembly, origin xyz=0.055 0.073 0 rpy=0 0 0, axis 1 0 0, limit lower=-0.35 upper=3.14 effort=43 velocity=13.3
- added joint left_hip_yaw_joint_X8: type revolute, parent urdf_l_upper_femur_assembly, child urdf_lower_femur_assembly, origin xyz=-0.053 -7.97086e-07 -0.217 rpy=0 0 0, axis 0 0 1, limit lower=-1.57 upper=1.57 effort=43 velocity=13.3
- added joint left_knee_joint_X8: type revolute, parent urdf_lower_femur_assembly, child urdf_l_tibia_assembly, origin xyz=0 0.055 -0.113 rpy=0 0 0, axis 0 1 0, limit lower=-0.17 upper=1.57 effort=43 velocity=13.3
- added joint pelvis_imu_joint: type fixed, parent urdf_simplified_torso, child pelvis_imu_link, origin xyz=0.0735 0.0 -0.17 rpy=0 1.5707963267948966 3.141592653589793
- added joint pelvis_imu_sensor_joint: type fixed, parent pelvis_imu_link, child pelvis_imu_sensor, origin xyz=0 0 0.003 rpy=0 0 0
- added joint right_ankle_pitch_joint_X4: type revolute, parent urdf_r_tibia_assembly, child urdf_ankle_assembly_2, origin xyz=-4.02748e-07 0.059 -0.395 rpy=0 0 0, axis 0 1 0, limit lower=-0.79 upper=0.79 effort=10.5 velocity=8.69
- added joint right_ankle_roll_joint_X4: type revolute, parent urdf_ankle_assembly_2, child urdf_foot_assembly_2, origin xyz=-0.012 -0.004 -0.028 rpy=0 0 0, axis 1 0 0, limit lower=-0.79 upper=0.79 effort=10.5 velocity=8.69
- added joint right_hip_pitch_joint_X8: type revolute, parent urdf_base, child urdf_hip_assembly_2, origin xyz=0.0333787 -0.107699 -0.467748 rpy=0 0 0, axis 0 1 0, limit lower=-2.53 upper=1.57 effort=43 velocity=13.3
- added joint right_hip_roll_joint_X8: type revolute, parent urdf_hip_assembly_2, child urdf_r_upper_femur_assemby, origin xyz=0.055 -0.078 0 rpy=0 0 0, axis 1 0 0, limit lower=-3.14 upper=0.35 effort=43 velocity=13.3
- added joint right_hip_yaw_joint_X8: type revolute, parent urdf_r_upper_femur_assemby, child urdf_lower_femur_assembly_2, origin xyz=-0.053 7.97086e-07 -0.217 rpy=0 0 0, axis 0 0 1, limit lower=-1.57 upper=1.57 effort=43 velocity=13.3
- added joint right_knee_joint_X8: type revolute, parent urdf_lower_femur_assembly_2, child urdf_r_tibia_assembly, origin xyz=0 -0.055 -0.113 rpy=0 0 0, axis 0 1 0, limit lower=-0.17 upper=1.57 effort=43 velocity=13.3
- added joint torso_imu_joint: type fixed, parent urdf_simplified_torso, child torso_imu_link, origin xyz=0.0635 0.0 0.35 rpy=0 1.5707963267948966 0
- added joint torso_imu_sensor_joint: type fixed, parent torso_imu_link, child torso_imu_sensor, origin xyz=0 0 0.003 rpy=0 0 0
- added joint waist_yaw_joint_X8: type revolute, parent urdf_base, child urdf_simplified_torso, origin xyz=0.0333787 -0.000698852 -0.300748 rpy=0 0 0, axis 0 0 1, limit lower=-1.57 upper=1.57 effort=43 velocity=13.3
- joint left_elbow_pitch_joint_X6: limit lower=-1.31 upper=1.83 effort=100 velocity=100 -> lower=-1.31 upper=1.83 effort=20 velocity=16.02
- joint left_index_intermediate_joint: axis 0 0 -1 -> (none); limit lower=-0.04545 upper=1.56 effort=1 velocity=0.5 -> (none); mimic joint=left_index_proximal_joint multiplier=1.06399 offset=-0.04545 -> (none); type revolute -> fixed
- joint left_index_proximal_joint: axis 0 0 -1 -> (none); limit lower=0 upper=1.47 effort=1 velocity=0.5 -> (none); type revolute -> fixed
- joint left_middle_intermediate_joint: axis 0 0 -1 -> (none); limit lower=-0.04545 upper=1.56 effort=1 velocity=0.5 -> (none); mimic joint=left_middle_proximal_joint multiplier=1.06399 offset=-0.04545 -> (none); type revolute -> fixed
- joint left_middle_proximal_joint: axis 0 0 -1 -> (none); limit lower=0 upper=1.47 effort=1 velocity=0.5 -> (none); type revolute -> fixed
- joint left_pinky_intermediate_joint: axis 0 0 -1 -> (none); limit lower=-0.04545 upper=1.56 effort=1 velocity=0.5 -> (none); mimic joint=left_pinky_proximal_joint multiplier=1.06399 offset=-0.04545 -> (none); type revolute -> fixed
- joint left_pinky_proximal_joint: axis 0 0 -1 -> (none); limit lower=0 upper=1.47 effort=1 velocity=0.5 -> (none); type revolute -> fixed
- joint left_ring_intermediate_joint: axis 0 0 -1 -> (none); limit lower=-0.04545 upper=1.56 effort=1 velocity=0.5 -> (none); mimic joint=left_ring_proximal_joint multiplier=1.06399 offset=-0.04545 -> (none); type revolute -> fixed
- joint left_ring_proximal_joint: axis 0 0 -1 -> (none); limit lower=0 upper=1.47 effort=1 velocity=0.5 -> (none); type revolute -> fixed
- joint left_shoulder_pitch_joint_X6: limit lower=-3.02 upper=1.69 effort=100 velocity=100 -> lower=-3.02 upper=1.69 effort=20 velocity=16.02
- joint left_shoulder_roll_joint_X6: limit lower=-0.21 upper=2.93 effort=100 velocity=100 -> lower=-0.21 upper=2.93 effort=20 velocity=16.02
- joint left_shoulder_yaw_joint_X4: limit lower=-1.75 upper=2.97 effort=100 velocity=100 -> lower=-1.75 upper=2.97 effort=10.5 velocity=8.69
- joint left_thumb_distal_joint: axis 0 0 -1 -> (none); limit lower=0 upper=0.4 effort=1 velocity=0.5 -> (none); mimic joint=left_thumb_proximal_pitch_joint multiplier=0.667 offset=0 -> (none); type revolute -> fixed
- joint left_thumb_intermediate_joint: axis 0 0 -1 -> (none); limit lower=0 upper=0.8 effort=1 velocity=0.5 -> (none); mimic joint=left_thumb_proximal_pitch_joint multiplier=1.334 offset=0 -> (none); type revolute -> fixed
- joint left_thumb_proximal_pitch_joint: axis 0 0 -1 -> (none); limit lower=0 upper=0.61 effort=1 velocity=0.5 -> (none); type revolute -> fixed
- joint left_thumb_proximal_yaw_joint: axis 0 0 1 -> (none); limit lower=0 upper=1.31 effort=1 velocity=0.5 -> (none); type revolute -> fixed
- joint left_wrist_roll_joint_X4: limit lower=-1.57 upper=1.57 effort=100 velocity=100 -> lower=-1.57 upper=1.57 effort=10.5 velocity=8.69
- joint left_wrist_yaw_joint_X4: limit lower=-2.36 upper=2.36 effort=100 velocity=100 -> lower=-2.36 upper=2.36 effort=10.5 velocity=8.69
- joint right_elbow_pitch_joint_X6: limit lower=-1.31 upper=1.83 effort=100 velocity=100 -> lower=-1.31 upper=1.83 effort=20 velocity=16.02
- joint right_index_intermediate_joint: axis 0 0 1 -> (none); limit lower=-0.04545 upper=1.56 effort=1 velocity=0.5 -> (none); mimic joint=right_index_proximal_joint multiplier=1.06399 offset=-0.04545 -> (none); type revolute -> fixed
- joint right_index_proximal_joint: axis 0 0 1 -> (none); limit lower=0 upper=1.47 effort=1 velocity=0.5 -> (none); type revolute -> fixed
- joint right_middle_intermediate_joint: axis 0 0 1 -> (none); limit lower=-0.04545 upper=1.56 effort=1 velocity=0.5 -> (none); mimic joint=right_middle_proximal_joint multiplier=1.06399 offset=-0.04545 -> (none); type revolute -> fixed
- joint right_middle_proximal_joint: axis 0 0 1 -> (none); limit lower=0 upper=1.47 effort=1 velocity=0.5 -> (none); type revolute -> fixed
- joint right_pinky_intermediate_joint: axis 0 0 1 -> (none); limit lower=-0.04545 upper=1.56 effort=1 velocity=0.5 -> (none); mimic joint=right_pinky_proximal_joint multiplier=1.06399 offset=-0.04545 -> (none); type revolute -> fixed
- joint right_pinky_proximal_joint: axis 0 0 1 -> (none); limit lower=0 upper=1.47 effort=1 velocity=0.5 -> (none); type revolute -> fixed
- joint right_ring_intermediate_joint: axis 0 0 1 -> (none); limit lower=-0.04545 upper=1.56 effort=1 velocity=0.5 -> (none); mimic joint=right_ring_proximal_joint multiplier=1.06399 offset=-0.04545 -> (none); type revolute -> fixed
- joint right_ring_proximal_joint: axis 0 0 1 -> (none); limit lower=0 upper=1.47 effort=1 velocity=0.5 -> (none); type revolute -> fixed
- joint right_shoulder_pitch_joint_X6: limit lower=-3.02 upper=1.69 effort=100 velocity=100 -> lower=-3.02 upper=1.69 effort=20 velocity=16.02
- joint right_shoulder_roll_joint_X6: limit lower=-2.93 upper=0.21 effort=100 velocity=100 -> lower=-2.93 upper=0.21 effort=20 velocity=16.02
- joint right_shoulder_yaw_joint_X4: limit lower=-2.97 upper=1.75 effort=100 velocity=100 -> lower=-2.97 upper=1.75 effort=10.5 velocity=8.69
- joint right_thumb_distal_joint: axis 0 0 1 -> (none); limit lower=0 upper=0.4 effort=1 velocity=0.5 -> (none); mimic joint=right_thumb_proximal_pitch_joint multiplier=0.667 offset=0 -> (none); type revolute -> fixed
- joint right_thumb_intermediate_joint: axis 0 0 1 -> (none); limit lower=0 upper=0.8 effort=1 velocity=0.5 -> (none); mimic joint=right_thumb_proximal_pitch_joint multiplier=1.334 offset=0 -> (none); type revolute -> fixed
- joint right_thumb_proximal_pitch_joint: axis 0 0 1 -> (none); limit lower=0 upper=0.6 effort=1 velocity=0.5 -> (none); type revolute -> fixed
- joint right_thumb_proximal_yaw_joint: axis 0 0 -1 -> (none); limit lower=0.0 upper=1.308 effort=1 velocity=0.5 -> (none); type revolute -> fixed
- joint right_wrist_roll_joint_X4: limit lower=-1.57 upper=1.57 effort=100 velocity=100 -> lower=-1.57 upper=1.57 effort=10.5 velocity=8.69
- joint right_wrist_yaw_joint_X4: limit lower=-2.36 upper=2.36 effort=100 velocity=100 -> lower=-2.36 upper=2.36 effort=10.5 velocity=8.69

File: src/robot_description/full_robot_description/urdf/joints/right_foot_joints.xacro (robot description, xacro)
@@ -33,5 +33,5 @@
     <dynamics damping="0.321" friction="3.21" />
   </joint>
-  <joint name="right_ankle_roll_joint_X4" type="${leg_joint_type}">
+  <joint name="right_ankle_pitch_joint_X4" type="${leg_joint_type}">
     <origin xyz="-4.02748e-07 0.059 -0.395" rpy="0 0 0" />
     <parent link="urdf_r_tibia_assembly" />
@@ -41,5 +41,5 @@
     <dynamics damping="0.114" friction="1.14" />
   </joint>
-  <joint name="right_ankle_pitch_joint_X4" type="${leg_joint_type}">
+  <joint name="right_ankle_roll_joint_X4" type="${leg_joint_type}">
     <origin xyz="-0.012 -0.004 -0.028" rpy="0 0 0" />
     <parent link="urdf_ankle_assembly_2" />
