Commit message: correction ankel axis

File: src/robot_description/full_robot_description/urdf/robot_harambe_v04_short_processeded.urdf (robot description, URDF)
Before this commit: robot robot_harambe_v0.3, 26 links, 25 joints
Joints:
- joint right_ankle_pitch_joint: axis 1 0 0 -> 0 1 0; child urdf_foot_assembly_2 -> urdf_ankle_assembly_2; origin xyz=-0.012 -0.004 -0.028 rpy=0 0 0 -> xyz=-4.02748e-07 0.059 -0.395 rpy=0 0 0; parent urdf_ankle_assembly_2 -> urdf_r_tibia_assembly
- joint right_ankle_roll_joint: axis 0 1 0 -> 1 0 0; child urdf_ankle_assembly_2 -> urdf_foot_assembly_2; origin xyz=-4.02748e-07 0.059 -0.395 rpy=0 0 0 -> xyz=-0.012 -0.004 -0.028 rpy=0 0 0; parent urdf_r_tibia_assembly -> urdf_ankle_assembly_2

Commit message: corected tibia mass

File: src/robot_description/full_robot_description/urdf/robot_harambe_v04_short_processeded.urdf (robot description, URDF)
Before this commit: robot robot_harambe_v0.3, 26 links, 25 joints
Links:
- link urdf_l_tibia_assembly: mass 2.6 -> 2.4
- link urdf_r_tibia_assembly: mass 2.6 -> 2.4
