Commit message: Add actuator properties macros and update joint effort limits
Centralized motor specs (X4/X6/X8 rated/moderate/peak) in
actuator_properties.xacro with ankle linkage torque calculations
(2x X4 eccentric-pushrod: pitch 100mm lever, roll ±30mm lever).
Set all joints to moderate profile. X8 moderate at 60% peak (72Nm)
for sustained walking thermal budget. Narrowed hip pitch stance 35mm
per side.

File: src/robot_description/full_robot_description/urdf/full_robot.urdf.xacro (robot description, xacro)
@@ -1,4 +1,6 @@
 <?xml version="1.0"?>
 <robot xmlns:xacro="http://ros.org/wiki/xacro" name="full_robot_description">
+    <!-- Actuator properties macros -->
+    <xacro:include filename="$(find full_robot_description)/urdf/macros/actuator_properties.xacro" />
     <!-- Body (base + torso) -->
     <xacro:include filename="$(find full_robot_description)/urdf/links/body_links.xacro" />

File: src/robot_description/full_robot_description/urdf/full_robot_gazebo.xacro (robot description, xacro)
@@ -6,4 +6,6 @@
   <xacro:arg name="fixed_legs" default="false" />
   <xacro:arg name="only_left" default="false" />
+  <!-- Actuator properties macros -->
+  <xacro:include filename="$(find full_robot_description)/urdf/macros/actuator_properties.xacro" />
   <!-- Body (base + torso) -->
   <xacro:include filename="$(find full_robot_description)/urdf/links/body_links.xacro" />
@@ -44,7 +46,7 @@
   <!-- IMU sensors (BNO055) -->
   <xacro:include filename="$(find imu_description)/urdf/bno055_imu.xacro" />
-  <!-- Pelvis IMU — raw sensor axes: x+=up, y+=right, z+=forward -->
-  <xacro:bno055_imu name="pelvis_imu" parent="urdf_simplified_torso" topic="/pelvis_imu/data" update_rate="100">
-    <origin xyz="0.0735 0.0 -0.17" rpy="0 ${pi/2} ${pi}"/>
+  <!-- Pelvis IMU — attached to pelvis (urdf_base), same world position as before -->
+  <xacro:bno055_imu name="pelvis_imu" parent="urdf_base" topic="/pelvis_imu/data" update_rate="100">
+    <origin xyz="0.1069 -0.0007 -0.4707" rpy="0 ${pi/2} ${pi}"/>
   </xacro:bno055_imu>
   <!-- Torso IMU — raw sensor axes: x+=up, y+=left, z+=backward -->

File: src/robot_description/full_robot_description/urdf/joints/body_joints.xacro (robot description, xacro)
@@ -10,6 +10,6 @@
     <child link="urdf_simplified_torso" />
     <axis xyz="0 0 1" />
-    <limit effort="43" velocity="13.3" lower="-1.57" upper="1.57" />
-    <dynamics damping="0.321" friction="3.21" />
+    <limit effort="${X8_moderate_effort}" velocity="${X8_rated_velocity}" lower="-1.57" upper="1.57" />
+    <dynamics damping="${X8_damping}" friction="${X8_friction}" />
   </joint>
 </robot>

File: src/robot_description/full_robot_description/urdf/joints/left_arm_joints.xacro (robot description, xacro)
@@ -6,6 +6,6 @@
     <child link="urdf_l_shoulder_assembly" />
     <axis xyz="0 1 0" />
-    <limit effort="20" velocity="16.02" lower="-3.02" upper="1.69" />
-    <dynamics damping="0.16" friction="1.6" />
+    <limit effort="${X6_moderate_effort}" velocity="${X6_rated_velocity}" lower="-3.02" upper="1.69" />
+    <dynamics damping="${X6_damping}" friction="${X6_friction}" />
   </joint>
   <joint name="left_shoulder_roll_joint_X6" type="revolute">
@@ -14,6 +14,6 @@
     <child link="urdf_l_upper_arm_assembly" />
     <axis xyz="1 0 0" />
-    <limit effort="20" velocity="16.02" lower="-0.21" upper="2.93" />
-    <dynamics damping="0.16" friction="1.6" />
+    <limit effort="${X6_moderate_effort}" velocity="${X6_rated_velocity}" lower="-0.21" upper="2.93" />
+    <dynamics damping="${X6_damping}" friction="${X6_friction}" />
   </joint>
   <joint name="left_shoulder_yaw_joint_X4" type="revolute">
@@ -22,6 +22,6 @@
     <child link="urdf_l_elbow_assembly" />
     <axis xyz="0 0 1" />
-    <limit effort="10.5" velocity="8.69" lower="-1.75" upper="2.97" />
-    <dynamics damping="0.114" friction="1.14" />
+    <limit effort="${X4_moderate_effort}" velocity="${X4_rated_velocity}" lower="-1.75" upper="2.97" />
+    <dynamics damping="${X4_damping}" friction="${X4_friction}" />
   </joint>
   <joint name="left_elbow_pitch_joint_X6" type="revolute">
@@ -30,6 +30,6 @@
     <child link="urdf_l_upper_forearm_assembly" />
     <axis xyz="0 1 0" />
-    <limit effort="20" velocity="16.02" lower="-1.31" upper="1.83" />
-    <dynamics damping="0.16" friction="1.6" />
+    <limit effort="${X6_moderate_effort}" velocity="${X6_rated_velocity}" lower="-1.31" upper="1.83" />
+    <dynamics damping="${X6_damping}" friction="${X6_friction}" />
   </joint>
   <joint name="left_wrist_yaw_joint_X4" type="revolute">
@@ -38,6 +38,6 @@
     <child link="urdf_l_lower_forearm_assembly" />
     <axis xyz="0 0 1" />
-    <limit effort="10.5" velocity="8.69" lower="-2.36" upper="2.36" />
-    <dynamics damping="0.114" friction="1.14" />
+    <limit effort="${X4_moderate_effort}" velocity="${X4_rated_velocity}" lower="-2.36" upper="2.36" />
+    <dynamics damping="${X4_damping}" friction="${X4_friction}" />
   </joint>
   <joint name="left_wrist_roll_joint_X4" type="revolute">
@@ -46,6 +46,6 @@
     <child link="urdf_l_wrist_assembly" />
     <axis xyz="1 0 0" />
-    <limit effort="10.5" velocity="8.69" lower="-1.57" upper="1.57" />
-    <dynamics damping="0.114" friction="1.14" />
+    <limit effort="${X4_moderate_effort}" velocity="${X4_rated_velocity}" lower="-1.57" upper="1.57" />
+    <dynamics damping="${X4_damping}" friction="${X4_friction}" />
   </joint>
 </robot>

File: src/robot_description/full_robot_description/urdf/joints/left_foot_joints.xacro (robot description, xacro)
@@ -2,10 +2,10 @@
 <robot>
   <joint name="left_hip_pitch_joint_X8" type="${leg_joint_type}">
-    <origin xyz="0.0333787 0.111301 -0.467748" rpy="0 0 0" />
+    <origin xyz="0.0333787 0.076301 -0.467748" rpy="0 0 0" />
     <parent link="urdf_base" />
     <child link="urdf_hip_assembly" />
     <axis xyz="0 1 0" />
-    <limit effort="43" velocity="13.3" lower="-2.53" upper="1.57" />
-    <dynamics damping="0.321" friction="3.21" />
+    <limit effort="${X8_moderate_effort}" velocity="${X8_rated_velocity}" lower="-2.53" upper="1.57" />
+    <dynamics damping="${X8_damping}" friction="${X8_friction}" />
   </joint>
   <joint name="left_hip_roll_joint_X8" type="${leg_joint_type}">
@@ -14,6 +14,6 @@
     <child link="urdf_l_upper_femur_assembly" />
     <axis xyz="1 0 0" />
-    <limit effort="43" velocity="13.3" lower="-0.35" upper="3.14" />
-    <dynamics damping="0.321" friction="3.21" />
+    <limit effort="${X8_moderate_effort}" velocity="${X8_rated_velocity}" lower="-0.35" upper="3.14" />
+    <dynamics damping="${X8_damping}" friction="${X8_friction}" />
   </joint>
   <joint name="left_hip_yaw_joint_X8" type="${leg_joint_type}">
@@ -22,6 +22,6 @@
     <child link="urdf_lower_femur_assembly" />
     <axis xyz="0 0 1" />
-    <limit effort="43" velocity="13.3" lower="-1.57" upper="1.57" />
-    <dynamics damping="0.321" friction="3.21" />
+    <limit effort="${X8_moderate_effort}" velocity="${X8_rated_velocity}" lower="-1.57" upper="1.57" />
+    <dynamics damping="${X8_damping}" friction="${X8_friction}" />
   </joint>
   <joint name="left_knee_joint_X8" type="${leg_joint_type}">
@@ -30,6 +30,6 @@
     <child link="urdf_l_tibia_assembly" />
     <axis xyz="0 1 0" />
-    <limit effort="43" velocity="13.3" lower="-0.17" upper="1.57" />
-    <dynamics damping="0.321" friction="3.21" />
+    <limit effort="${X8_moderate_effort}" velocity="${X8_rated_velocity}" lower="-0.17" upper="1.57" />
+    <dynamics damping="${X8_damping}" friction="${X8_friction}" />
   </joint>
   <joint name="left_ankle_pitch_joint_X4" type="${leg_joint_type}">
@@ -38,6 +38,6 @@
     <child link="urdf_ankle_assembly" />
     <axis xyz="0 1 0" />
-    <limit effort="10.5" velocity="8.69" lower="-0.79" upper="0.79" />
-    <dynamics damping="0.114" friction="1.14" />
+    <limit effort="${ankle_pitch_moderate_effort}" velocity="${ankle_pitch_rated_velocity}" lower="-0.79" upper="0.79" />
+    <dynamics damping="${X4_damping}" friction="${X4_friction}" />
   </joint>
   <joint name="left_ankle_roll_joint_X4" type="${leg_joint_type}">
@@ -46,6 +46,6 @@
     <child link="urdf_foot_assembly" />
     <axis xyz="1 0 0" />
-    <limit effort="10.5" velocity="8.69" lower="-0.79" upper="0.79" />
-    <dynamics damping="0.114" friction="1.14" />
+    <limit effort="${ankle_roll_moderate_effort}" velocity="${ankle_roll_rated_velocity}" lower="-0.79" upper="0.79" />
+    <dynamics damping="${X4_damping}" friction="${X4_friction}" />
   </joint>
 </robot>

File: src/robot_description/full_robot_description/urdf/joints/right_arm_joints.xacro (robot description, xacro)
@@ -6,6 +6,6 @@
     <child link="urdf_r_shoulder_assembly" />
     <axis xyz="0 1 0" />
-    <limit effort="20" velocity="16.02" lower="-3.02" upper="1.69" />
-    <dynamics damping="0.16" friction="1.6" />
+    <limit effort="${X6_moderate_effort}" velocity="${X6_rated_velocity}" lower="-3.02" upper="1.69" />
+    <dynamics damping="${X6_damping}" friction="${X6_friction}" />
   </joint>
   <joint name="right_shoulder_roll_joint_X6" type="revolute">
@@ -14,6 +14,6 @@
     <child link="urdf_r_upper_arm_assembly" />
     <axis xyz="1 0 0" />
-    <limit effort="20" velocity="16.02" lower="-2.93" upper="0.21" />
-    <dynamics damping="0.16" friction="1.6" />
+    <limit effort="${X6_moderate_effort}" velocity="${X6_rated_velocity}" lower="-2.93" upper="0.21" />
+    <dynamics damping="${X6_damping}" friction="${X6_friction}" />
   </joint>
   <joint name="right_shoulder_yaw_joint_X4" type="revolute">
@@ -22,6 +22,6 @@
     <child link="urdf_r_elbow_assembly" />
     <axis xyz="0 0 1" />
-    <limit effort="10.5" velocity="8.69" lower="-2.97" upper="1.75" />
-    <dynamics damping="0.114" friction="1.14" />
+    <limit effort="${X4_moderate_effort}" velocity="${X4_rated_velocity}" lower="-2.97" upper="1.75" />
+    <dynamics damping="${X4_damping}" friction="${X4_friction}" />
   </joint>
   <joint name="right_elbow_pitch_joint_X6" type="revolute">
@@ -30,6 +30,6 @@
     <child link="urdf_r_upper_forearm_assembly" />
     <axis xyz="0 1 0" />
-    <limit effort="20" velocity="16.02" lower="-1.31" upper="1.83" />
-    <dynamics damping="0.16" friction="1.6" />
+    <limit effort="${X6_moderate_effort}" velocity="${X6_rated_velocity}" lower="-1.31" upper="1.83" />
+    <dynamics damping="${X6_damping}" friction="${X6_friction}" />
   </joint>
   <joint name="right_wrist_yaw_joint_X4" type="revolute">
@@ -38,6 +38,6 @@
     <child link="urdf_r_lower_forearm_assembly" />
     <axis xyz="0 0 1" />
-    <limit effort="10.5" velocity="8.69" lower="-2.36" upper="2.36" />
-    <dynamics damping="0.114" friction="1.14" />
+    <limit effort="${X4_moderate_effort}" velocity="${X4_rated_velocity}" lower="-2.36" upper="2.36" />
+    <dynamics damping="${X4_damping}" friction="${X4_friction}" />
   </joint>
   <joint name="right_wrist_roll_joint_X4" type="revolute">
@@ -46,6 +46,6 @@
     <child link="urdf_r_wrist_assembly" />
     <axis xyz="1 0 0" />
-    <limit effort="10.5" velocity="8.69" lower="-1.57" upper="1.57" />
-    <dynamics damping="0.114" friction="1.14" />
+    <limit effort="${X4_moderate_effort}" velocity="${X4_rated_velocity}" lower="-1.57" upper="1.57" />
+    <dynamics damping="${X4_damping}" friction="${X4_friction}" />
   </joint>
 </robot>

File: src/robot_description/full_robot_description/urdf/joints/right_foot_joints.xacro (robot description, xacro)
@@ -2,10 +2,10 @@
 <robot>
   <joint name="right_hip_pitch_joint_X8" type="${leg_joint_type}">
-    <origin xyz="0.0333787 -0.107699 -0.467748" rpy="0 0 0" />
+    <origin xyz="0.0333787 -0.072699 -0.467748" rpy="0 0 0" />
     <parent link="urdf_base" />
     <child link="urdf_hip_assembly_2" />
     <axis xyz="0 1 0" />
-    <limit effort="43" velocity="13.3" lower="-2.53" upper="1.57" />
-    <dynamics damping="0.321" friction="3.21" />
+    <limit effort="${X8_moderate_effort}" velocity="${X8_rated_velocity}" lower="-2.53" upper="1.57" />
+    <dynamics damping="${X8_damping}" friction="${X8_friction}" />
   </joint>
   <joint name="right_hip_roll_joint_X8" type="${leg_joint_type}">
@@ -14,6 +14,6 @@
     <child link="urdf_r_upper_femur_assemby" />
     <axis xyz="1 0 0" />
-    <limit effort="43" velocity="13.3" lower="-3.14" upper="0.35" />
-    <dynamics damping="0.321" friction="3.21" />
+    <limit effort="${X8_moderate_effort}" velocity="${X8_rated_velocity}" lower="-3.14" upper="0.35" />
+    <dynamics damping="${X8_damping}" friction="${X8_friction}" />
   </joint>
   <joint name="right_hip_yaw_joint_X8" type="${leg_joint_type}">
@@ -22,6 +22,6 @@
     <child link="urdf_lower_femur_assembly_2" />
     <axis xyz="0 0 1" />
-    <limit effort="43" velocity="13.3" lower="-1.57" upper="1.57" />
-    <dynamics damping="0.321" friction="3.21" />
+    <limit effort="${X8_moderate_effort}" velocity="${X8_rated_velocity}" lower="-1.57" upper="1.57" />
+    <dynamics damping="${X8_damping}" friction="${X8_friction}" />
   </joint>
   <joint name="right_knee_joint_X8" type="${leg_joint_type}">
@@ -30,6 +30,6 @@
     <child link="urdf_r_tibia_assembly" />
     <axis xyz="0 1 0" />
-    <limit effort="43" velocity="13.3" lower="-0.17" upper="1.57" />
-    <dynamics damping="0.321" friction="3.21" />
+    <limit effort="${X8_moderate_effort}" velocity="${X8_rated_velocity}" lower="-0.17" upper="1.57" />
+    <dynamics damping="${X8_damping}" friction="${X8_friction}" />
   </joint>
   <joint name="right_ankle_pitch_joint_X4" type="${leg_joint_type}">
@@ -38,6 +38,6 @@
     <child link="urdf_ankle_assembly_2" />
     <axis xyz="0 1 0" />
-    <limit effort="10.5" velocity="8.69" lower="-0.79" upper="0.79" />
-    <dynamics damping="0.114" friction="1.14" />
+    <limit effort="${ankle_pitch_moderate_effort}" velocity="${ankle_pitch_rated_velocity}" lower="-0.79" upper="0.79" />
+    <dynamics damping="${X4_damping}" friction="${X4_friction}" />
   </joint>
   <joint name="right_ankle_roll_joint_X4" type="${leg_joint_type}">
@@ -46,6 +46,6 @@
     <child link="urdf_foot_assembly_2" />
     <axis xyz="1 0 0" />
-    <limit effort="10.5" velocity="8.69" lower="-0.79" upper="0.79" />
-    <dynamics damping="0.114" friction="1.14" />
+    <limit effort="${ankle_roll_moderate_effort}" velocity="${ankle_roll_rated_velocity}" lower="-0.79" upper="0.79" />
+    <dynamics damping="${X4_damping}" friction="${X4_friction}" />
   </joint>
 </robot>

File: src/robot_description/full_robot_description/urdf/links/left_foot_links.xacro (robot description, xacro)
@@ -100,5 +100,5 @@
     <inertial>
       <origin xyz="0.00463897 -0.0449177 -0.190721" rpy="0 0 0"/>
-      <mass value="6.45981"/>
+      <mass value="2.4"/>
       <inertia ixx="0.0785879" ixy="0.000322141" ixz="0.00174711" iyy="0.0762229" iyz="-0.00887502" izz="0.0153456"/>
     </inertial>

File: src/robot_description/full_robot_description/urdf/links/right_foot_links.xacro (robot description, xacro)
@@ -100,5 +100,5 @@
     <inertial>
       <origin xyz="0.00463902 0.0449175 -0.190727" rpy="0 0 0"/>
-      <mass value="6.45984"/>
+      <mass value="2.4"/>
       <inertia ixx="0.0785959" ixy="-0.000322085" ixz="0.00175009" iyy="0.0762312" iyz="0.0088755" izz="0.0153456"/>
     </inertial>

Commit message: hands and robot urdf vizualizer settings, hands corected placement

File: src/robot_description/full_robot_description/urdf/full_robot.urdf.xacro (robot description, xacro)
@@ -27,16 +27,16 @@
         mount_y="0.015"
         mount_z="-0.06"
-        mount_roll="1.424576"
+        mount_roll="1.544576"
         mount_pitch="-0.201364"
-        mount_yaw="2.205507"/>
+        mount_yaw="1.6"/>
     <xacro:inspire_hand_right
         parent="urdf_r_wrist_assembly"
         prefix="right_"
-        mount_x="-0.029"
+        mount_x="-0.033"
         mount_y="-0.011"
         mount_z="-0.06"
-        mount_roll="1.717027"
-        mount_pitch="-0.201373"
-        mount_yaw="-2.205496"/>
+        mount_roll="1.617027"
+        mount_pitch="-0.301373"
+        mount_yaw="-1.605496"/>
     <!-- Fix robot base to world frame -->
     <link name="world"/>

File: src/robot_description/full_robot_description/urdf/joints/body_joints.xacro (robot description, xacro)
@@ -5,10 +5,19 @@
   <!-- ================================================================== -->
   <xacro:arg name="fixed_legs" default="false"/>
-  <xacro:property name="leg_joint_type" value="${'fixed' if '$(arg fixed_legs)' == 'true' else 'revolute'}"/>
+  <xacro:property name="leg_joint_type"  value="revolute"/>
+  <xacro:if value="$(arg fixed_legs)">
+    <xacro:property name="leg_joint_type" value="fixed"/>
+  </xacro:if>
   <!-- ================================================================== -->
   <!-- only_left — when true, also lock waist yaw joint                  -->
   <!-- ================================================================== -->
   <xacro:arg name="only_left" default="true"/>
-  <xacro:property name="waist_joint_type" value="${'fixed' if '$(arg only_left)' == 'true' or '$(arg fixed_legs)' == 'true' else 'revolute'}"/>
+  <xacro:property name="waist_joint_type" value="revolute"/>
+  <xacro:if value="$(arg only_left)">
+    <xacro:property name="waist_joint_type" value="fixed"/>
+  </xacro:if>
+  <xacro:if value="$(arg fixed_legs)">
+    <xacro:property name="waist_joint_type" value="fixed"/>
+  </xacro:if>
   <!-- ================================================================== -->
   <!-- Body                                                              -->

File: src/robot_description/hand_description/urdf/hands/inspire_hand_left.xacro (robot description, xacro)
@@ -6,5 +6,5 @@
        6 actuated joints + 6 mimic joints + 5 tip fixed joints
        Collision geometry uses box primitives (OBJ meshes lack normals for DART) -->
-  <xacro:macro name="inspire_hand_left" params="parent prefix:=left_ mount_x:=0.0 mount_y:=0.07 mount_z:=-0.03 mount_roll:=0.0 mount_pitch:=0.0 mount_yaw:=3.14159">
+  <xacro:macro name="inspire_hand_left" params="parent prefix:=left_ mount_x:=0.0 mount_y:=0.0 mount_z:=-0.0 mount_roll:=0.0 mount_pitch:=0.0 mount_yaw:=0">
     <!-- Attach hand_base_link directly to parent (replaces dummy base link) -->
     <joint name="${prefix}hand_base_joint" type="fixed">
