Commit message: replace inspire hands with boxes in isaac urdf

File: src/robot_description/full_robot_description/urdf/full_robot_isaaclab.urdf (robot description, URDF)
Before this commit: robot harambe_full_robot, 66 links, 65 joints
Links:
- removed link left_index_intermediate
- removed link left_index_proximal
- removed link left_index_tip
- removed link left_middle_intermediate
- removed link left_middle_proximal
- removed link left_middle_tip
- removed link left_pinky_intermediate
- removed link left_pinky_proximal
- removed link left_pinky_tip
- removed link left_ring_intermediate
- removed link left_ring_proximal
- removed link left_ring_tip
- removed link left_thumb_distal
- removed link left_thumb_intermediate
- removed link left_thumb_proximal
- removed link left_thumb_proximal_base
- removed link left_thumb_tip
- removed link right_index_intermediate
- removed link right_index_proximal
- removed link right_index_tip
- removed link right_middle_intermediate
- removed link right_middle_proximal
- removed link right_middle_tip
- removed link right_pinky_intermediate
- removed link right_pinky_proximal
- removed link right_pinky_tip
- removed link right_ring_intermediate
- removed link right_ring_proximal
- removed link right_ring_tip
- removed link right_thumb_distal
- removed link right_thumb_intermediate
- removed link right_thumb_proximal
- removed link right_thumb_proximal_base
- removed link right_thumb_tip
- link left_hand_base_link: mass 0.52560 -> 0.84; geometry collision box size=0.04 0.15 0.08; visual box size=0.04 0.15 0.08
- link right_hand_base_link: mass 0.52560 -> 0.84; geometry collision box size=0.04 0.15 0.08; visual box size=0.04 0.15 0.08
Joints:
- removed joint left_index_intermediate_joint
- removed joint left_index_proximal_joint
- removed joint left_index_tip_joint
- removed joint left_middle_intermediate_joint
- removed joint left_middle_proximal_joint
- removed joint left_middle_tip_joint
- removed joint left_pinky_intermediate_joint
- removed joint left_pinky_proximal_joint
- removed joint left_pinky_tip_joint
- removed joint left_ring_intermediate_joint
- removed joint left_ring_proximal_joint
- removed joint left_ring_tip_joint
- removed joint left_thumb_distal_joint
- removed joint left_thumb_intermediate_joint
- removed joint left_thumb_proximal_pitch_joint
- removed joint left_thumb_proximal_yaw_joint
- removed joint left_thumb_tip_joint
- removed joint right_index_intermediate_joint
- removed joint right_index_proximal_joint
- removed joint right_index_tip_joint
- removed joint right_middle_intermediate_joint
- removed joint right_middle_proximal_joint
- removed joint right_middle_tip_joint
- removed joint right_pinky_intermediate_joint
- removed joint right_pinky_proximal_joint
- removed joint right_pinky_tip_joint
- removed joint right_ring_intermediate_joint
- removed joint right_ring_proximal_joint
- removed joint right_ring_tip_joint
- removed joint right_thumb_distal_joint
- removed joint right_thumb_intermediate_joint
- removed joint right_thumb_proximal_pitch_joint
- removed joint right_thumb_proximal_yaw_joint
- removed joint right_thumb_tip_joint
