Commit message: add pelvis imu

File: src/robot_description/full_robot_description/urdf/full_robot_gazebo.xacro (robot description, xacro)
@@ -42,4 +42,9 @@
       mount_pitch="-0.201373"
       mount_yaw="-2.205496"/>
+  <!-- IMU sensor (BNO055) mounted on torso -->
+  <xacro:include filename="$(find imu_description)/urdf/bno055_imu.xacro" />
+  <xacro:bno055_imu name="torso_imu" parent="urdf_simplified_torso" topic="/imu/data" update_rate="100">
+    <origin xyz="0.0735 0.0 -0.17" rpy="0 ${pi/2} ${pi}"/>
+  </xacro:bno055_imu>
   <!-- Fix robot base to world frame -->
   <link name="world"/>

Commit message: add second imu (for tosrso)

File: src/robot_description/full_robot_description/urdf/full_robot_gazebo.xacro (robot description, xacro)
@@ -42,15 +42,20 @@
       mount_pitch="-0.201373"
       mount_yaw="-2.205496"/>
-  <!-- IMU sensor (BNO055) mounted on torso -->
+  <!-- IMU sensors (BNO055) -->
   <xacro:include filename="$(find imu_description)/urdf/bno055_imu.xacro" />
-  <xacro:bno055_imu name="torso_imu" parent="urdf_simplified_torso" topic="/imu/data" update_rate="100">
+  <!-- Pelvis IMU — raw sensor axes: x+=up, y+=right, z+=forward -->
+  <xacro:bno055_imu name="pelvis_imu" parent="urdf_simplified_torso" topic="/pelvis_imu/data" update_rate="100">
     <origin xyz="0.0735 0.0 -0.17" rpy="0 ${pi/2} ${pi}"/>
   </xacro:bno055_imu>
+  <!-- Torso IMU — raw sensor axes: x+=up, y+=left, z+=backward -->
+  <xacro:bno055_imu name="torso_imu" parent="urdf_simplified_torso" topic="/torso_imu/data" update_rate="100">
+    <origin xyz="0.0635 0.0 0.35" rpy="0 ${pi/2} 0"/>
+  </xacro:bno055_imu>
   <!-- Fix robot base to world frame -->
-  <link name="world"/>
+  <!-- <link name="world"/>
   <joint name="world_joint" type="fixed">
     <parent link="world"/>
     <child link="urdf_base"/>
-  </joint>
+  </joint> -->
   <!-- ros2_control: position mode -->
   <xacro:if value="${'$(arg control_mode)' == 'position'}">

Commit message: harambe policy plugin effort controller

File: src/robot_description/full_robot_description/urdf/full_robot_gazebo.xacro (robot description, xacro)
@@ -1,6 +1,7 @@
 <?xml version="1.0"?>
 <robot xmlns:xacro="http://www.ros.org/wiki/xacro" name="harambe_full_robot">
-  <!-- Control mode: "position" or "effort" -->
+  <!-- Control mode: "position", "effort", "gz_pid", or "gz_policy" -->
   <xacro:arg name="control_mode" default="position" />
+  <xacro:arg name="onnx_path" default="" />
   <!-- Full robot: all joints active (not fixed) -->
   <xacro:arg name="fixed_legs" default="false" />
@@ -59,5 +60,5 @@
     <parent link="world"/>
     <child link="urdf_base"/>
-  </joint> -->
+  </joint>  -->
   <!-- ros2_control: position mode -->
   <xacro:if value="${'$(arg control_mode)' == 'position'}">
@@ -70,10 +71,76 @@
     <xacro:full_robot_ros2_control_effort />
   </xacro:if>
-  <!-- Gazebo gz_ros2_control plugin -->
-  <gazebo>
-    <plugin filename="gz_ros2_control-system" name="gz_ros2_control::GazeboSimROS2ControlPlugin">
-      <parameters>$(find full_robot_gazebo)/config/controllers_$(arg control_mode).yaml</parameters>
-      <update_rate>100</update_rate>
-    </plugin>
-  </gazebo>
+  <!-- ros2_control: effort_implicit_actuators mode (PD handled by ImplicitActuatorAdapter node) -->
+  <xacro:if value="${'$(arg control_mode)' == 'effort_implicit_actuators'}">
+    <xacro:include filename="$(find full_robot_description)/urdf/macros/ros2_control_effort.xacro" />
+    <xacro:full_robot_ros2_control_effort />
+  </xacro:if>
+  <!-- gz_pid mode: Gazebo-native JointPositionController per joint (no ros2_control) -->
+  <xacro:if value="${'$(arg control_mode)' == 'gz_pid'}">
+    <xacro:include filename="$(find full_robot_description)/urdf/macros/gz_joint_position_controllers.xacro" />
+    <xacro:gz_all_joint_position_controllers />
+  </xacro:if>
+  <!-- gz_policy mode: ONNX policy plugin with PD + velocity limiting (no ros2_control) -->
+  <xacro:if value="${'$(arg control_mode)' == 'gz_policy'}">
+    <!-- Default positions set by plugin at Configure (joints spawn at 0, PD moves to default) -->
+    <gazebo>
+      <plugin filename="/home/alex/Documents/GitHub/ldr-harambe-arms-sim2real/install/harambe_gz_policy_plugin/lib/libharambe_gz_policy_plugin.so" name="harambe_gz::HarambePolicyPlugin">
+        <onnx_path>$(arg onnx_path)</onnx_path>
+        <decimation>4</decimation>
+        <action_scale>0.25</action_scale>
+        <clip_actions>5.0</clip_actions>
+        <warmup_steps>0</warmup_steps>
+        <cmd_vel_x>0.0</cmd_vel_x>
+        <imu_link>urdf_base</imu_link>
+        <!-- 25 joints in HARDWARE_JOINT_ORDER — default positions from mc_rtc CoM controller -->
+        <!-- PD gains ÷5 to match PhysX implicit actuator step response -->
+        <!-- Left arm -->
+        <joint name="left_shoulder_pitch_joint_X6" kp="6"   kd="2"    effort_limit="23"    vel_limit="16.02" default_pos="0" />
+        <joint name="left_shoulder_roll_joint_X6"  kp="6"   kd="2"    effort_limit="23"    vel_limit="16.02" default_pos="0" />
+        <joint name="left_shoulder_yaw_joint_X4"   kp="6"   kd="2"    effort_limit="12.075" vel_limit="8.69" default_pos="0" />
+        <joint name="left_elbow_pitch_joint_X6"    kp="6"   kd="2"    effort_limit="23"    vel_limit="16.02" default_pos="0" />
+        <joint name="left_wrist_yaw_joint_X4"      kp="6"   kd="2"    effort_limit="12.075" vel_limit="8.69" default_pos="0" />
+        <joint name="left_wrist_roll_joint_X4"     kp="6"   kd="2"    effort_limit="12.075" vel_limit="8.69" default_pos="0" />
+        <!-- Right arm -->
+        <joint name="right_shoulder_pitch_joint_X6" kp="6"   kd="2"    effort_limit="23"    vel_limit="16.02" default_pos="0" />
+        <joint name="right_shoulder_roll_joint_X6"  kp="6"   kd="2"    effort_limit="23"    vel_limit="16.02" default_pos="0" />
+        <joint name="right_shoulder_yaw_joint_X4"   kp="6"   kd="2"    effort_limit="12.075" vel_limit="8.69" default_pos="0" />
+        <joint name="right_elbow_pitch_joint_X6"    kp="6"   kd="2"    effort_limit="23"    vel_limit="16.02" default_pos="0" />
+        <joint name="right_wrist_yaw_joint_X4"      kp="6"   kd="2"    effort_limit="12.075" vel_limit="8.69" default_pos="0" />
+        <joint name="right_wrist_roll_joint_X4"     kp="6"   kd="2"    effort_limit="12.075" vel_limit="8.69" default_pos="0" />
+        <!-- Waist -->
+        <joint name="waist_yaw_joint_X8"            kp="30"  kd="2"    effort_limit="100"   vel_limit="13.3" default_pos="0" />
+        <!-- Left leg — with friction compensation (values from URDF dynamics) -->
+        <joint name="left_hip_pitch_joint_X8"       kp="100" kd="15"   effort_limit="100"   vel_limit="13.3" default_pos="-0.15" friction="3.21" />
+        <joint name="left_hip_roll_joint_X8"        kp="20"  kd="0.5"  effort_limit="100"   vel_limit="13.3" default_pos="0"    friction="1.6" />
+        <joint name="left_hip_yaw_joint_X8"         kp="9"   kd="0.5"  effort_limit="100"   vel_limit="13.3" default_pos="0"    friction="1.6" />
+        <joint name="left_knee_joint_X8"            kp="60"  kd="6"    effort_limit="100"   vel_limit="13.3" default_pos="0.30" friction="1.14" />
+        <joint name="left_ankle_pitch_joint_X4"     kp="60"  kd="6"  effort_limit="96.6"  vel_limit="2.17" default_pos="-0.15" friction="1.14" />
+        <joint name="left_ankle_roll_joint_X4"      kp="20"  kd="1"    effort_limit="28.98" vel_limit="7.24" default_pos="0"    friction="1.14" />
+        <!-- Right leg (mirror) -->
+        <joint name="right_hip_pitch_joint_X8"      kp="100" kd="15"   effort_limit="100"   vel_limit="13.3" default_pos="-0.15" friction="3.21" />
+        <joint name="right_hip_roll_joint_X8"       kp="20"  kd="0.5"  effort_limit="100"   vel_limit="13.3" default_pos="0"    friction="1.6" />
+        <joint name="right_hip_yaw_joint_X8"        kp="9"   kd="0.5"  effort_limit="100"   vel_limit="13.3" default_pos="0"    friction="1.6" />
+        <joint name="right_knee_joint_X8"           kp="60"  kd="6"    effort_limit="100"   vel_limit="13.3" default_pos="0.30" friction="1.14" />
+        <joint name="right_ankle_pitch_joint_X4"    kp="60"  kd="6"  effort_limit="96.6"  vel_limit="2.17" default_pos="-0.15" friction="1.14" />
+        <joint name="right_ankle_roll_joint_X4"     kp="20"  kd="1"    effort_limit="28.98" vel_limit="7.24" default_pos="0"    friction="1.14" />
+      </plugin>
+    </gazebo>
+    <!-- Joint state publisher for observation -->
+    <gazebo>
+      <plugin filename="gz-sim-joint-state-publisher-system" name="gz::sim::systems::JointStatePublisher">
+        <update_rate>200</update_rate>
+        <topic>/joint_states_gz</topic>
+      </plugin>
+    </gazebo>
+  </xacro:if>
+  <!-- Gazebo gz_ros2_control plugin (only for ros2_control modes) -->
+  <xacro:if value="${'$(arg control_mode)' != 'gz_pid' and '$(arg control_mode)' != 'gz_policy'}">
+    <gazebo>
+      <plugin filename="gz_ros2_control-system" name="gz_ros2_control::GazeboSimROS2ControlPlugin">
+        <parameters>$(find full_robot_gazebo)/config/controllers_$(arg control_mode).yaml</parameters>
+        <update_rate>100</update_rate>
+      </plugin>
+    </gazebo>
+  </xacro:if>
 </robot>
