Commit message: Isaac Lab sim2real: match Gazebo policy plugin dynamics to PhysX
- Remove target interpolation (use HOLD like Isaac Lab)
- Remove velocity limiting and acceleration clamping from PD control
- Add reflected rotor inertia per motor type to URDF links
  (X4=0.039, X6=0.025, X8=0.058 kg·m² from datasheet gear_ratio²)
- Define rotor inertia properties in actuator_properties.xacro
  with automatic calculation via ${XX_reflected_inertia}
- Set PD gains to Isaac Lab nominal (kp_scale=1.0, kd_scale=1.0)
- Set clip_actions=5.0 to match Isaac Lab
- Remove max_accel parameter (unused)
- Clean up debug/hardcoded test code from plugin

File: src/robot_description/full_robot_description/urdf/full_robot_gazebo.xacro (robot description, xacro)
@@ -5,4 +5,7 @@
   <xacro:arg name="onnx_path" default="" />
   <xacro:arg name="policy_debug" default="false" />
+  <!-- PD gain scaling for Gazebo policy plugin (1.0 = Isaac Lab nominal) -->
+  <xacro:property name="kp_scale" value="0.7" />
+  <xacro:property name="kd_scale" value="1.5" />
   <!-- Full robot: all joints active (not fixed) -->
   <xacro:arg name="fixed_legs" default="false" />
@@ -85,36 +88,36 @@
         <cmd_vel_x>0.0</cmd_vel_x>
         <imu_link>urdf_base</imu_link>
-        <!-- 25 joints in HARDWARE_JOINT_ORDER — default positions from mc_rtc CoM controller -->
-        <!-- PD gains ÷5 to match PhysX implicit actuator step response -->
+        <!-- 25 joints in HARDWARE_JOINT_ORDER -->
+        <!-- PD gains: Isaac Lab nominal (center of domain randomization) × kp_scale/kd_scale -->
         <!-- Left arm -->
-        <joint name="left_shoulder_pitch_joint_X6" kp="6"   kd="2"    effort_limit="23"    vel_limit="16.02" default_pos="0" />
-        <joint name="left_shoulder_roll_joint_X6"  kp="6"   kd="2"    effort_limit="23"    vel_limit="16.02" default_pos="0" />
-        <joint name="left_shoulder_yaw_joint_X4"   kp="6"   kd="2"    effort_limit="12.075" vel_limit="8.69" default_pos="0" />
-        <joint name="left_elbow_pitch_joint_X6"    kp="6"   kd="2"    effort_limit="23"    vel_limit="16.02" default_pos="0" />
-        <joint name="left_wrist_yaw_joint_X4"      kp="6"   kd="2"    effort_limit="12.075" vel_limit="8.69" default_pos="0" />
-        <joint name="left_wrist_roll_joint_X4"     kp="6"   kd="2"    effort_limit="12.075" vel_limit="8.69" default_pos="0" />
+        <joint name="left_shoulder_pitch_joint_X6" kp="${30*kp_scale}"  kd="${8*kd_scale}"  effort_limit="23"    vel_limit="16.02" default_pos="0" />
+        <joint name="left_shoulder_roll_joint_X6"  kp="${30*kp_scale}"  kd="${8*kd_scale}"  effort_limit="23"    vel_limit="16.02" default_pos="0" />
+        <joint name="left_shoulder_yaw_joint_X4"   kp="${30*kp_scale}"  kd="${8*kd_scale}"  effort_limit="12.075" vel_limit="8.69" default_pos="0" />
+        <joint name="left_elbow_pitch_joint_X6"    kp="${30*kp_scale}"  kd="${8*kd_scale}"  effort_limit="23"    vel_limit="16.02" default_pos="0" />
+        <joint name="left_wrist_yaw_joint_X4"      kp="${30*kp_scale}"  kd="${8*kd_scale}"  effort_limit="12.075" vel_limit="8.69" default_pos="0" />
+        <joint name="left_wrist_roll_joint_X4"     kp="${30*kp_scale}"  kd="${8*kd_scale}"  effort_limit="12.075" vel_limit="8.69" default_pos="0" />
         <!-- Right arm -->
-        <joint name="right_shoulder_pitch_joint_X6" kp="6"   kd="2"    effort_limit="23"    vel_limit="16.02" default_pos="0" />
-        <joint name="right_shoulder_roll_joint_X6"  kp="6"   kd="2"    effort_limit="23"    vel_limit="16.02" default_pos="0" />
-        <joint name="right_shoulder_yaw_joint_X4"   kp="6"   kd="2"    effort_limit="12.075" vel_limit="8.69" default_pos="0" />
-        <joint name="right_elbow_pitch_joint_X6"    kp="6"   kd="2"    effort_limit="23"    vel_limit="16.02" default_pos="0" />
-        <joint name="right_wrist_yaw_joint_X4"      kp="6"   kd="2"    effort_limit="12.075" vel_limit="8.69" default_pos="0" />
-        <joint name="right_wrist_roll_joint_X4"     kp="6"   kd="2"    effort_limit="12.075" vel_limit="8.69" default_pos="0" />
+        <joint name="right_shoulder_pitch_joint_X6" kp="${30*kp_scale}"  kd="${8*kd_scale}"  effort_limit="23"    vel_limit="16.02" default_pos="0" />
+        <joint name="right_shoulder_roll_joint_X6"  kp="${30*kp_scale}"  kd="${8*kd_scale}"  effort_limit="23"    vel_limit="16.02" default_pos="0" />
+        <joint name="right_shoulder_yaw_joint_X4"   kp="${30*kp_scale}"  kd="${8*kd_scale}"  effort_limit="12.075" vel_limit="8.69" default_pos="0" />
+        <joint name="right_elbow_pitch_joint_X6"    kp="${30*kp_scale}"  kd="${8*kd_scale}"  effort_limit="23"    vel_limit="16.02" default_pos="0" />
+        <joint name="right_wrist_yaw_joint_X4"      kp="${30*kp_scale}"  kd="${8*kd_scale}"  effort_limit="12.075" vel_limit="8.69" default_pos="0" />
+        <joint name="right_wrist_roll_joint_X4"     kp="${30*kp_scale}"  kd="${8*kd_scale}"  effort_limit="12.075" vel_limit="8.69" default_pos="0" />
         <!-- Waist -->
-        <joint name="waist_yaw_joint_X8"            kp="30"  kd="2"    effort_limit="100"   vel_limit="13.3" default_pos="0" />
+        <joint name="waist_yaw_joint_X8"            kp="${150*kp_scale}" kd="${8*kd_scale}"  effort_limit="100"   vel_limit="13.3" default_pos="0" />
         <!-- Left leg — with friction compensation (values from URDF dynamics) -->
-        <joint name="left_hip_pitch_joint_X8"       kp="100" kd="15"   effort_limit="100"   vel_limit="13.3" default_pos="-0.15" friction="3.21" />
-        <joint name="left_hip_roll_joint_X8"        kp="20"  kd="0.5"  effort_limit="100"   vel_limit="13.3" default_pos="0"    friction="1.6" />
-        <joint name="left_hip_yaw_joint_X8"         kp="9"   kd="0.5"  effort_limit="100"   vel_limit="13.3" default_pos="0"    friction="1.6" />
-        <joint name="left_knee_joint_X8"            kp="60"  kd="6"    effort_limit="100"   vel_limit="13.3" default_pos="0.30" friction="1.14" />
-        <joint name="left_ankle_pitch_joint_X4"     kp="60"  kd="6"  effort_limit="96.6"  vel_limit="2.17" default_pos="-0.15" friction="1.14" />
-        <joint name="left_ankle_roll_joint_X4"      kp="20"  kd="1"    effort_limit="28.98" vel_limit="7.24" default_pos="0"    friction="1.14" />
+        <joint name="left_hip_pitch_joint_X8"       kp="${200*kp_scale}" kd="${10*kd_scale}" effort_limit="100"   vel_limit="13.3" default_pos="-0.15" friction="3.21" />
+        <joint name="left_hip_roll_joint_X8"        kp="${150*kp_scale}" kd="${10*kd_scale}" effort_limit="100"   vel_limit="13.3" default_pos="0"    friction="1.6" />
+        <joint name="left_hip_yaw_joint_X8"         kp="${150*kp_scale}" kd="${10*kd_scale}" effort_limit="100"   vel_limit="13.3" default_pos="0"    friction="1.6" />
+        <joint name="left_knee_joint_X8"            kp="${200*kp_scale}" kd="${10*kd_scale}" effort_limit="100"   vel_limit="13.3" default_pos="0.30" friction="1.14" />
+        <joint name="left_ankle_pitch_joint_X4"     kp="${200*kp_scale}" kd="${10*kd_scale}" effort_limit="96.6"  vel_limit="2.17" default_pos="-0.15" friction="1.14" />
+        <joint name="left_ankle_roll_joint_X4"      kp="${150*kp_scale}" kd="${8*kd_scale}"  effort_limit="28.98" vel_limit="7.24" default_pos="0"    friction="1.14" />
         <!-- Right leg (mirror) -->
-        <joint name="right_hip_pitch_joint_X8"      kp="100" kd="15"   effort_limit="100"   vel_limit="13.3" default_pos="-0.15" friction="3.21" />
-        <joint name="right_hip_roll_joint_X8"       kp="20"  kd="0.5"  effort_limit="100"   vel_limit="13.3" default_pos="0"    friction="1.6" />
-        <joint name="right_hip_yaw_joint_X8"        kp="9"   kd="0.5"  effort_limit="100"   vel_limit="13.3" default_pos="0"    friction="1.6" />
-        <joint name="right_knee_joint_X8"           kp="60"  kd="6"    effort_limit="100"   vel_limit="13.3" default_pos="0.30" friction="1.14" />
-        <joint name="right_ankle_pitch_joint_X4"    kp="60"  kd="6"  effort_limit="96.6"  vel_limit="2.17" default_pos="-0.15" friction="1.14" />
-        <joint name="right_ankle_roll_joint_X4"     kp="20"  kd="1"    effort_limit="28.98" vel_limit="7.24" default_pos="0"    friction="1.14" />
+        <joint name="right_hip_pitch_joint_X8"      kp="${200*kp_scale}" kd="${10*kd_scale}" effort_limit="100"   vel_limit="13.3" default_pos="-0.15" friction="3.21" />
+        <joint name="right_hip_roll_joint_X8"       kp="${150*kp_scale}" kd="${10*kd_scale}" effort_limit="100"   vel_limit="13.3" default_pos="0"    friction="1.6" />
+        <joint name="right_hip_yaw_joint_X8"        kp="${150*kp_scale}" kd="${10*kd_scale}" effort_limit="100"   vel_limit="13.3" default_pos="0"    friction="1.6" />
+        <joint name="right_knee_joint_X8"           kp="${200*kp_scale}" kd="${10*kd_scale}" effort_limit="100"   vel_limit="13.3" default_pos="0.30" friction="1.14" />
+        <joint name="right_ankle_pitch_joint_X4"    kp="${200*kp_scale}" kd="${10*kd_scale}" effort_limit="96.6"  vel_limit="2.17" default_pos="-0.15" friction="1.14" />
+        <joint name="right_ankle_roll_joint_X4"     kp="${150*kp_scale}" kd="${8*kd_scale}"  effort_limit="28.98" vel_limit="7.24" default_pos="0"    friction="1.14" />
       </plugin>
     </gazebo>

File: src/robot_description/full_robot_description/urdf/full_robot_isaaclab.urdf (robot description, URDF)
Before this commit: robot harambe_full_robot, 64 links, 63 joints
Links:
- added link torso_imu_link; visual sphere radius=0.002
- added link torso_imu_sensor, mass 0.0042339; collision mesh filename=package://imu_description/meshes/low_res_bno055_imu.stl; visual mesh filename=package://imu_description/meshes/low_res_bno055_imu.stl
- link left_hand_base_link: mass 0.14143 -> 0.52560
- link right_hand_base_link: mass 0.14143 -> 0.52560
- link urdf_base: mass 5.132 -> 5.734; geometry collision mesh filename=package://full_robot_description/meshes/collision/b_base.stl; collision mesh filename=package://full_robot_description/meshes/collision/f_base.stl
- link urdf_foot_assembly: mass 0.504 -> 0.309
- link urdf_foot_assembly_2: mass 0.504 -> 0.309
- link urdf_hip_assembly: mass 1.73 -> 1.829
- link urdf_hip_assembly_2: mass 1.73 -> 1.829
- link urdf_l_tibia_assembly: mass 2.4 -> 2.216
- link urdf_l_upper_femur_assembly: mass 1.912 -> 1.93; geometry collision mesh filename=package://full_robot_description/meshes/collision/l_upper_f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; collision mesh filename=package://full_robot_description/meshes/collision/stopper_l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
- link urdf_lower_femur_assembly: mass 1.817 -> 1.832; geometry collision mesh filename=package://full_robot_description/meshes/collision/lower_fem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; collision mesh filename=package://full_robot_description/meshes/collision/stopper_l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
- link urdf_r_tibia_assembly: mass 2.4 -> 2.215
Joints:
- added joint torso_imu_joint: type fixed, parent urdf_simplified_torso, child torso_imu_link, origin xyz=0.0635 0.0 0.35 rpy=0 1.5707963267948966 0
- added joint torso_imu_sensor_joint: type fixed, parent torso_imu_link, child torso_imu_sensor, origin xyz=0 0 0.003 rpy=0 0 0
- joint left_ankle_pitch_joint_X4: limit lower=-0.79 upper=0.79 effort=96.6 velocity=2.17 -> lower=-0.79 upper=0.79 effort=12.075 velocity=8.69; origin xyz=-1.45092e-06 -0.051 -0.395 rpy=0 0 0 -> xyz=0 -0.051 -0.395 rpy=0 0 0
- joint left_ankle_roll_joint_X4: limit lower=-0.79 upper=0.79 effort=28.98 velocity=7.24 -> lower=-0.79 upper=0.79 effort=12.075 velocity=8.69; origin xyz=-0.0120001 -0.004 -0.028 rpy=0 0 0 -> xyz=-0.012 -0.004 -0.028 rpy=0 0 0
- joint left_elbow_pitch_joint_X6: origin xyz=0.019337 0.0291733 -0.075 rpy=0 -0.0190902 -0.585348 -> xyz=0.0193369 0.0291733 -0.075 rpy=0 -0.0190922 -0.585347
- joint left_hip_pitch_joint_X8: origin xyz=0.0333787 0.072699 -0.467748 rpy=0 0 0 -> xyz=0.070373 0.0872946 -0.431099 rpy=0 0 0
- joint left_hip_roll_joint_X8: origin xyz=0.055 0.073 0 rpy=0 0 0 -> xyz=0.053 0.062 0 rpy=0 0 0
- joint left_hip_yaw_joint_X8: origin xyz=-0.053 -7.97086e-07 -0.217 rpy=0 0 0 -> xyz=-0.053 0 -0.217 rpy=0 0 0
- joint left_knee_joint_X8: origin xyz=0 0.055 -0.113 rpy=0 0 0 -> xyz=-1.45947e-07 0.055 -0.111 rpy=0 0 0
- joint left_shoulder_pitch_joint_X6: origin xyz=0 0.1755 0.423977 rpy=0 0 0 -> xyz=0 0.1695 0.423977 rpy=0 0 0
- joint left_shoulder_roll_joint_X6: origin xyz=0.0456571 0.07 0.00560599 rpy=0 -0.122173 0 -> xyz=0.0456571 0.07 0.00560611 rpy=0 -0.122176 0
- joint left_shoulder_yaw_joint_X4: origin xyz=-0.046 0.0343048 -0.161394 rpy=0.209376 0.00530409 -0.0249664 -> xyz=-0.046 0.034306 -0.161394 rpy=0.209383 0.00530439 -0.024967
- joint left_wrist_roll_joint_X4: origin xyz=0.0219762 -0.0156859 -0.0615 rpy=-0.248271 0 -0.619909 -> xyz=0.0219762 -0.0156859 -0.0615 rpy=-0.248279 0 -0.619909
- joint left_wrist_yaw_joint_X4: origin xyz=0.0391738 -0.035 -0.158223 rpy=-0.142861 -0.19688 0.634041 -> xyz=0.0391735 -0.035 -0.158223 rpy=-0.14286 -0.196878 0.634041
- joint right_ankle_pitch_joint_X4: limit lower=-0.79 upper=0.79 effort=96.6 velocity=2.17 -> lower=-0.79 upper=0.79 effort=12.075 velocity=8.69; origin xyz=-4.02748e-07 0.051 -0.395 rpy=0 0 0 -> xyz=0 0.059 -0.395 rpy=0 0 0
- joint right_ankle_roll_joint_X4: limit lower=-0.79 upper=0.79 effort=28.98 velocity=7.24 -> lower=-0.79 upper=0.79 effort=12.075 velocity=8.69
- joint right_elbow_pitch_joint_X6: origin xyz=0.0220994 -0.0333409 -0.065 rpy=0 -0.019088 0.585341 -> xyz=0.0220994 -0.033341 -0.065 rpy=0 -0.0190815 0.58534
- joint right_hip_pitch_joint_X8: origin xyz=0.0333787 -0.072699 -0.467748 rpy=0 0 0 -> xyz=0.070373 -0.0887054 -0.431099 rpy=0 0 0
- joint right_hip_roll_joint_X8: origin xyz=0.055 -0.073 0 rpy=0 0 0 -> xyz=0.053 -0.062 0 rpy=0 0 0
- joint right_hip_yaw_joint_X8: origin xyz=-0.053 7.97086e-07 -0.217 rpy=0 0 0 -> xyz=-0.053 0 -0.217 rpy=0 0 0
- joint right_knee_joint_X8: origin xyz=0 -0.055 -0.113 rpy=0 0 0 -> xyz=1.45947e-07 -0.055 -0.111 rpy=0 0 0
- joint right_shoulder_pitch_joint_X6: origin xyz=0 -0.1755 0.423977 rpy=0 0 0 -> xyz=0 -0.1695 0.423977 rpy=0 0 0
- joint right_shoulder_roll_joint_X6: origin xyz=0.0456571 -0.07 0.00560599 rpy=0 -0.122173 0 -> xyz=0.0456571 -0.07 0.00560611 rpy=0 -0.122176 0
- joint right_shoulder_yaw_joint_X4: origin xyz=-0.046 -0.0353456 -0.166285 rpy=-0.209378 0.00530246 0.0249661 -> xyz=-0.046 -0.0353444 -0.166285 rpy=-0.20937 0.00530239 0.0249667
- joint right_wrist_roll_joint_X4: origin xyz=0.0219763 0.0156857 -0.0565 rpy=0.248281 0 0.619897 -> xyz=0.0219763 0.0156857 -0.0565 rpy=0.248276 0 0.619896
- joint right_wrist_yaw_joint_X4: origin xyz=0.0403763 0.04 -0.163076 rpy=0.142857 -0.196885 -0.634033 -> xyz=0.0403774 0.04 -0.163076 rpy=0.142861 -0.196891 -0.634034
- joint waist_yaw_joint_X8: origin xyz=0.0333787 -0.000698852 -0.300748 rpy=0 0 0 -> xyz=0.070373 -0.000705351 -0.281099 rpy=0 0 0

File: src/robot_description/full_robot_description/urdf/links/body_links.xacro (robot description, xacro)
@@ -141,5 +141,5 @@
       <origin xyz="0.00199132 -4.19393e-05 0.328473" rpy="0 0 0"/>
       <mass value="5.9"/>
-      <inertia ixx="0.318197" ixy="5.25211e-07" ixz="-0.00444278" iyy="0.294961" iyz="9.73773e-05" izz="0.0735035"/>
+      <inertia ixx="${0.318197 + X8_reflected_inertia}" ixy="5.25211e-07" ixz="-0.00444278" iyy="${0.294961 + X8_reflected_inertia}" iyz="9.73773e-05" izz="${0.0735035 + X8_reflected_inertia}"/>
     </inertial>
     <visual>

File: src/robot_description/full_robot_description/urdf/links/left_arm_links.xacro (robot description, xacro)
@@ -8,5 +8,5 @@
       <origin xyz="-0.00409836 0.0631966 -0.000544507" rpy="0 0 0"/>
       <mass value="1.246"/>
-      <inertia ixx="0.00205876" ixy="-3.48871e-05" ixz="4.1195e-05" iyy="0.00152408" iyz="-7.63845e-06" izz="0.00171602"/>
+      <inertia ixx="${0.00205876 + X6_reflected_inertia}" ixy="-3.48871e-05" ixz="4.1195e-05" iyy="${0.00152408 + X6_reflected_inertia}" iyz="-7.63845e-06" izz="${0.00171602 + X6_reflected_inertia}"/>
     </inertial>
     <visual>
@@ -39,5 +39,5 @@
       <origin xyz="-0.0354438 0.0213187 -0.103332" rpy="0 0 0"/>
       <mass value="0.802"/>
-      <inertia ixx="0.00190836" ixy="8.88428e-05" ixz="-0.000467525" iyy="0.00203106" iyz="0.000183116" izz="0.00107639"/>
+      <inertia ixx="${0.00190836 + X6_reflected_inertia}" ixy="8.88428e-05" ixz="-0.000467525" iyy="${0.00203106 + X6_reflected_inertia}" iyz="0.000183116" izz="${0.00107639 + X6_reflected_inertia}"/>
     </inertial>
     <visual>
@@ -70,5 +70,5 @@
       <origin xyz="-0.004748 -0.00662541 -0.0710681" rpy="0 0 0"/>
       <mass value="1.109"/>
-      <inertia ixx="0.00145153" ixy="5.51714e-05" ixz="-3.01713e-05" iyy="0.00147549" iyz="-7.59581e-05" izz="0.00114035"/>
+      <inertia ixx="${0.00145153 + X4_reflected_inertia}" ixy="5.51714e-05" ixz="-3.01713e-05" iyy="${0.00147549 + X4_reflected_inertia}" iyz="-7.59581e-05" izz="${0.00114035 + X4_reflected_inertia}"/>
     </inertial>
     <visual>
@@ -101,5 +101,5 @@
       <origin xyz="0.0267132 -0.0286559 -0.0999185" rpy="0 0 0"/>
       <mass value="0.707"/>
-      <inertia ixx="0.00162524" ixy="9.29307e-05" ixz="0.000226906" iyy="0.00146156" iyz="-0.000353662" izz="0.000776911"/>
+      <inertia ixx="${0.00162524 + X6_reflected_inertia}" ixy="9.29307e-05" ixz="0.000226906" iyy="${0.00146156 + X6_reflected_inertia}" iyz="-0.000353662" izz="${0.000776911 + X6_reflected_inertia}"/>
     </inertial>
     <visual>
@@ -132,5 +132,5 @@
       <origin xyz="-0.00311766 0.00307025 -0.0515634" rpy="0 0 0"/>
       <mass value="0.618"/>
-      <inertia ixx="0.000628386" ixy="-1.68351e-06" ixz="-2.8195e-05" iyy="0.000617293" iyz="-3.24981e-07" izz="0.000448744"/>
+      <inertia ixx="${0.000628386 + X4_reflected_inertia}" ixy="-1.68351e-06" ixz="-2.8195e-05" iyy="${0.000617293 + X4_reflected_inertia}" iyz="-3.24981e-07" izz="${0.000448744 + X4_reflected_inertia}"/>
     </inertial>
     <visual>
@@ -163,5 +163,5 @@
       <origin xyz="-0.0219307 0.0106852 -0.0421315" rpy="0 0 0"/>
       <mass value="0.098"/>
-      <inertia ixx="0.000100785" ixy="8.20205e-06" ixz="-3.2373e-05" iyy="0.000121426" iyz="6.79922e-06" izz="9.6353e-05"/>
+      <inertia ixx="${0.000100785 + X4_reflected_inertia}" ixy="8.20205e-06" ixz="-3.2373e-05" iyy="${0.000121426 + X4_reflected_inertia}" iyz="6.79922e-06" izz="${9.6353e-05 + X4_reflected_inertia}"/>
     </inertial>
     <visual>

File: src/robot_description/full_robot_description/urdf/links/left_foot_links.xacro (robot description, xacro)
@@ -8,5 +8,5 @@
       <origin xyz="-0.00387043 0.0602754 -3.33254e-05" rpy="0 0 0"/>
       <mass value="1.829"/>
-      <inertia ixx="0.00318486" ixy="-1.248e-05" ixz="2.39579e-07" iyy="0.00257781" iyz="-3.95097e-06" izz="0.00266816"/>
+      <inertia ixx="${0.00318486 + X8_reflected_inertia}" ixy="-1.248e-05" ixz="2.39579e-07" iyy="${0.00257781 + X8_reflected_inertia}" iyz="-3.95097e-06" izz="${0.00266816 + X8_reflected_inertia}"/>
     </inertial>
     <visual>
@@ -39,5 +39,5 @@
       <origin xyz="-0.0460989 0.000881037 -0.148514" rpy="0 0 0"/>
       <mass value="1.93"/>
-      <inertia ixx="0.00524838" ixy="2.68214e-05" ixz="-0.000973448" iyy="0.00568591" iyz="1.37224e-06" izz="0.00347712"/>
+      <inertia ixx="${0.00524838 + X8_reflected_inertia}" ixy="2.68214e-05" ixz="-0.000973448" iyy="${0.00568591 + X8_reflected_inertia}" iyz="1.37224e-06" izz="${0.00347712 + X8_reflected_inertia}"/>
     </inertial>
     <visual>
@@ -85,5 +85,5 @@
       <origin xyz="2.11243e-05 -0.00408754 -0.100571" rpy="0 0 0"/>
       <mass value="1.832"/>
-      <inertia ixx="0.00401519" ixy="1.60501e-06" ixz="-3.40991e-06" iyy="0.00435606" iyz="-0.000112967" izz="0.00266245"/>
+      <inertia ixx="${0.00401519 + X8_reflected_inertia}" ixy="1.60501e-06" ixz="-3.40991e-06" iyy="${0.00435606 + X8_reflected_inertia}" iyz="-0.000112967" izz="${0.00266245 + X8_reflected_inertia}"/>
     </inertial>
     <visual>
@@ -131,5 +131,5 @@
       <origin xyz="0.01449 -0.0488281 -0.199552" rpy="0 0 0"/>
       <mass value="2.216"/>
-      <inertia ixx="0.0205548" ixy="0.000222702" ixz="0.00143905" iyy="0.0209762" iyz="-0.00195792" izz="0.00480101"/>
+      <inertia ixx="${0.0205548 + X8_reflected_inertia}" ixy="0.000222702" ixz="0.00143905" iyy="${0.0209762 + X8_reflected_inertia}" iyz="-0.00195792" izz="${0.00480101 + X8_reflected_inertia}"/>
     </inertial>
     <visual>
@@ -207,5 +207,5 @@
       <origin xyz="0 -0.004 -0.0125426" rpy="0 0 0"/>
       <mass value="0.0818219"/>
-      <inertia ixx="1.69449e-05" ixy="-1.30849e-26" ixz="-4.29315e-17" iyy="2.15245e-05" iyz="-5.80972e-28" izz="1.25404e-05"/>
+      <inertia ixx="${1.69449e-05 + X4_reflected_inertia}" ixy="-1.30849e-26" ixz="-4.29315e-17" iyy="${2.15245e-05 + X4_reflected_inertia}" iyz="-5.80972e-28" izz="${1.25404e-05 + X4_reflected_inertia}"/>
     </inertial>
     <visual>
@@ -229,5 +229,5 @@
       <origin xyz="0.0436027 8.11114e-08 -0.0200314" rpy="0 0 0"/>
       <mass value="0.309"/>
-      <inertia ixx="0.000232433" ixy="-1.58776e-11" ixz="-9.83566e-06" iyy="0.00121361" iyz="-6.57666e-10" izz="0.00137693"/>
+      <inertia ixx="${0.000232433 + X4_reflected_inertia}" ixy="-1.58776e-11" ixz="-9.83566e-06" iyy="${0.00121361 + X4_reflected_inertia}" iyz="-6.57666e-10" izz="${0.00137693 + X4_reflected_inertia}"/>
     </inertial>
     <visual>
