Commit message: Isaac Lab sim2real: match Gazebo policy plugin dynamics to PhysX
- Remove target interpolation (use HOLD like Isaac Lab)
- Remove velocity limiting and acceleration clamping from PD control
- Add reflected rotor inertia per motor type to URDF links
  (X4=0.039, X6=0.025, X8=0.058 kg·m² from datasheet gear_ratio²)
- Define rotor inertia properties in actuator_properties.xacro
  with automatic calculation via ${XX_reflected_inertia}
- Set PD gains to Isaac Lab nominal (kp_scale=1.0, kd_scale=1.0)
- Set clip_actions=5.0 to match Isaac Lab
- Remove max_accel parameter (unused)
- Clean up debug/hardcoded test code from plugin

File: src/robot_description/full_robot_description/urdf/links/right_arm_links.xacro (robot description, xacro)
@@ -8,5 +8,5 @@
       <origin xyz="-0.0047018 -0.0660727 -0.000602826" rpy="0 0 0"/>
       <mass value="1.02"/>
-      <inertia ixx="0.0013257" ixy="1.37507e-05" ixz="2.16644e-05" iyy="0.00104972" iyz="3.46311e-06" izz="0.0011458"/>
+      <inertia ixx="${0.0013257 + X6_reflected_inertia}" ixy="1.37507e-05" ixz="2.16644e-05" iyy="${0.00104972 + X6_reflected_inertia}" iyz="3.46311e-06" izz="${0.0011458 + X6_reflected_inertia}"/>
     </inertial>
     <visual>
@@ -39,5 +39,5 @@
       <origin xyz="-0.0347331 -0.0216398 -0.101809" rpy="0 0 0"/>
       <mass value="0.802"/>
-      <inertia ixx="0.00188605" ixy="-9.73927e-05" ixz="-0.00045821" iyy="0.00200295" iyz="-0.000209822" izz="0.00106039"/>
+      <inertia ixx="${0.00188605 + X6_reflected_inertia}" ixy="-9.73927e-05" ixz="-0.00045821" iyy="${0.00200295 + X6_reflected_inertia}" iyz="-0.000209822" izz="${0.00106039 + X6_reflected_inertia}"/>
     </inertial>
     <visual>
@@ -70,5 +70,5 @@
       <origin xyz="-0.00464628 0.00706688 -0.0612736" rpy="0 0 0"/>
       <mass value="1.109"/>
-      <inertia ixx="0.00142737" ixy="-5.60371e-05" ixz="-3.53572e-05" iyy="0.00147543" iyz="4.92594e-05" izz="0.00111817"/>
+      <inertia ixx="${0.00142737 + X4_reflected_inertia}" ixy="-5.60371e-05" ixz="-3.53572e-05" iyy="${0.00147543 + X4_reflected_inertia}" iyz="4.92594e-05" izz="${0.00111817 + X4_reflected_inertia}"/>
     </inertial>
     <visual>
@@ -101,5 +101,5 @@
       <origin xyz="0.0266786 0.0327896 -0.0982602" rpy="0 0 0"/>
       <mass value="0.707"/>
-      <inertia ixx="0.00160609" ixy="-9.59596e-05" ixz="0.000238823" iyy="0.0014499" iyz="0.00033935" izz="0.000766591"/>
+      <inertia ixx="${0.00160609 + X6_reflected_inertia}" ixy="-9.59596e-05" ixz="0.000238823" iyy="${0.0014499 + X6_reflected_inertia}" iyz="0.00033935" izz="${0.000766591 + X6_reflected_inertia}"/>
     </inertial>
     <visual>
@@ -132,5 +132,5 @@
       <origin xyz="-0.00325453 -0.0023229 -0.046852" rpy="0 0 0"/>
       <mass value="0.618"/>
-      <inertia ixx="0.000617744" ixy="-6.12409e-07" ixz="-3.11927e-05" iyy="0.000618165" iyz="-2.22632e-05" izz="0.000437775"/>
+      <inertia ixx="${0.000617744 + X4_reflected_inertia}" ixy="-6.12409e-07" ixz="-3.11927e-05" iyy="${0.000618165 + X4_reflected_inertia}" iyz="-2.22632e-05" izz="${0.000437775 + X4_reflected_inertia}"/>
     </inertial>
     <visual>
@@ -163,5 +163,5 @@
       <origin xyz="-0.0219123 -0.0106789 -0.0421059" rpy="0 0 0"/>
       <mass value="0.15"/>
-      <inertia ixx="0.000154293" ixy="-1.25537e-05" ixz="-4.9547e-05" iyy="0.000185908" iyz="-1.03834e-05" izz="0.00014762"/>
+      <inertia ixx="${0.000154293 + X4_reflected_inertia}" ixy="-1.25537e-05" ixz="-4.9547e-05" iyy="${0.000185908 + X4_reflected_inertia}" iyz="-1.03834e-05" izz="${0.00014762 + X4_reflected_inertia}"/>
     </inertial>
     <visual>

File: src/robot_description/full_robot_description/urdf/links/right_foot_links.xacro (robot description, xacro)
@@ -8,5 +8,5 @@
       <origin xyz="-0.00387043 -0.0602754 3.33254e-05" rpy="0 0 0"/>
       <mass value="1.829"/>
-      <inertia ixx="0.00318486" ixy="1.248e-05" ixz="-2.39579e-07" iyy="0.00257781" iyz="-3.95097e-06" izz="0.00266816"/>
+      <inertia ixx="${0.00318486 + X8_reflected_inertia}" ixy="1.248e-05" ixz="-2.39579e-07" iyy="${0.00257781 + X8_reflected_inertia}" iyz="-3.95097e-06" izz="${0.00266816 + X8_reflected_inertia}"/>
     </inertial>
     <visual>
@@ -39,5 +39,5 @@
       <origin xyz="-0.0457109 -0.000406025 -0.147969" rpy="0 0 0"/>
       <mass value="1.912"/>
-      <inertia ixx="0.00512969" ixy="-1.22901e-06" ixz="-0.000930002" iyy="0.00557257" iyz="5.18759e-05" izz="0.00336728"/>
+      <inertia ixx="${0.00512969 + X8_reflected_inertia}" ixy="-1.22901e-06" ixz="-0.000930002" iyy="${0.00557257 + X8_reflected_inertia}" iyz="5.18759e-05" izz="${0.00336728 + X8_reflected_inertia}"/>
     </inertial>
     <visual>
@@ -70,5 +70,5 @@
       <origin xyz="9.05521e-10 0.00357383 -0.101307" rpy="0 0 0"/>
       <mass value="1.817"/>
-      <inertia ixx="0.00383469" ixy="-1.04286e-09" ixz="2.0768e-08" iyy="0.00421827" iyz="0.00019709" izz="0.00258541"/>
+      <inertia ixx="${0.00383469 + X8_reflected_inertia}" ixy="-1.04286e-09" ixz="2.0768e-08" iyy="${0.00421827 + X8_reflected_inertia}" iyz="0.00019709" izz="${0.00258541 + X8_reflected_inertia}"/>
     </inertial>
     <visual>
@@ -101,5 +101,5 @@
       <origin xyz="0.0144959 0.0488304 -0.199574" rpy="0 0 0"/>
       <mass value="2.215"/>
-      <inertia ixx="0.0205486" ixy="-0.000222584" ixz="0.00144134" iyy="0.0209705" iyz="0.00195651" izz="0.00479841"/>
+      <inertia ixx="${0.0205486 + X8_reflected_inertia}" ixy="-0.000222584" ixz="0.00144134" iyy="${0.0209705 + X8_reflected_inertia}" iyz="0.00195651" izz="${0.00479841 + X8_reflected_inertia}"/>
     </inertial>
     <visual>
@@ -177,5 +177,5 @@
       <origin xyz="0 -0.004 -0.0125426" rpy="0 0 0"/>
       <mass value="0.0818219"/>
-      <inertia ixx="1.69449e-05" ixy="-2.22156e-26" ixz="4.29315e-17" iyy="2.15245e-05" iyz="3.73894e-27" izz="1.25404e-05"/>
+      <inertia ixx="${1.69449e-05 + X4_reflected_inertia}" ixy="-2.22156e-26" ixz="4.29315e-17" iyy="${2.15245e-05 + X4_reflected_inertia}" iyz="3.73894e-27" izz="${1.25404e-05 + X4_reflected_inertia}"/>
     </inertial>
     <visual>
@@ -199,5 +199,5 @@
       <origin xyz="0.0436027 8.11114e-08 -0.0200314" rpy="0 0 0"/>
       <mass value="0.309"/>
-      <inertia ixx="0.000232433" ixy="-1.58776e-11" ixz="-9.83566e-06" iyy="0.00121361" iyz="-6.57666e-10" izz="0.00137693"/>
+      <inertia ixx="${0.000232433 + X4_reflected_inertia}" ixy="-1.58776e-11" ixz="-9.83566e-06" iyy="${0.00121361 + X4_reflected_inertia}" iyz="-6.57666e-10" izz="${0.00137693 + X4_reflected_inertia}"/>
     </inertial>
     <visual>

File: src/robot_description/full_robot_description/urdf/macros/actuator_properties.xacro (robot description, xacro)
@@ -17,4 +17,8 @@
   <xacro:property name="X4_friction"           value="1.14" />
   <xacro:property name="X4_damping"            value="0.114" />
+  <!-- Reflected rotor inertia: I_rotor × gear_ratio² = 0.00003 × 36² = 0.0389 kg·m² -->
+  <xacro:property name="X4_rotor_inertia"      value="0.00003" />
+  <xacro:property name="X4_gear_ratio"         value="36" />
+  <xacro:property name="X4_reflected_inertia"  value="${0.00003 * 36 * 36}" />
   <!-- ==================== X6-60 (direct) ==================== -->
   <xacro:property name="X6_rated_effort"       value="20" />
@@ -25,4 +29,8 @@
   <xacro:property name="X6_friction"           value="1.6" />
   <xacro:property name="X6_damping"            value="0.16" />
+  <!-- Reflected rotor inertia: I_rotor × gear_ratio² = 0.000066 × 19.612² = 0.0254 kg·m² -->
+  <xacro:property name="X6_rotor_inertia"      value="0.000066" />
+  <xacro:property name="X6_gear_ratio"         value="19.612" />
+  <xacro:property name="X6_reflected_inertia"  value="${0.000066 * 19.612 * 19.612}" />
   <!-- ==================== X8-120 (direct) ==================== -->
   <xacro:property name="X8_rated_effort"       value="43" />
@@ -36,4 +44,8 @@
   <xacro:property name="X8_friction"           value="3.21" />
   <xacro:property name="X8_damping"            value="0.321" />
+  <!-- Reflected rotor inertia: I_rotor × gear_ratio² = 0.00015 × 19.612² = 0.0577 kg·m² -->
+  <xacro:property name="X8_rotor_inertia"      value="0.00015" />
+  <xacro:property name="X8_gear_ratio"         value="19.612" />
+  <xacro:property name="X8_reflected_inertia"  value="${0.00015 * 19.612 * 19.612}" />
   <!-- ==================== Ankle Linkage =====================
        2x X4 motors with eccentric-pushrod mechanism

Commit message: review

File: src/robot_description/full_robot_description/urdf/full_robot_gazebo.xacro (robot description, xacro)
@@ -6,6 +6,6 @@
   <xacro:arg name="policy_debug" default="false" />
   <!-- PD gain scaling for Gazebo policy plugin (1.0 = Isaac Lab nominal) -->
-  <xacro:property name="kp_scale" value="0.7" />
-  <xacro:property name="kd_scale" value="1.5" />
+  <xacro:property name="kp_scale" value="1.0" />
+  <xacro:property name="kd_scale" value="1.3" />
   <!-- Full robot: all joints active (not fixed) -->
   <xacro:arg name="fixed_legs" default="false" />
@@ -82,5 +82,5 @@
         <onnx_path>$(arg onnx_path)</onnx_path>
         <decimation>4</decimation>
-        <action_scale>0.25</action_scale>
+        <action_scale>0.12</action_scale>
         <clip_actions>5.0</clip_actions>
         <warmup_steps>0</warmup_steps>
@@ -105,18 +105,18 @@
         <joint name="right_wrist_roll_joint_X4"     kp="${30*kp_scale}"  kd="${8*kd_scale}"  effort_limit="12.075" vel_limit="8.69" default_pos="0" />
         <!-- Waist -->
-        <joint name="waist_yaw_joint_X8"            kp="${150*kp_scale}" kd="${8*kd_scale}"  effort_limit="100"   vel_limit="13.3" default_pos="0" />
+        <joint name="waist_yaw_joint_X8"            kp="${150*kp_scale}" kd="${15*kd_scale}"  effort_limit="100"   vel_limit="13.3" default_pos="0" />
         <!-- Left leg — with friction compensation (values from URDF dynamics) -->
-        <joint name="left_hip_pitch_joint_X8"       kp="${200*kp_scale}" kd="${10*kd_scale}" effort_limit="100"   vel_limit="13.3" default_pos="-0.15" friction="3.21" />
-        <joint name="left_hip_roll_joint_X8"        kp="${150*kp_scale}" kd="${10*kd_scale}" effort_limit="100"   vel_limit="13.3" default_pos="0"    friction="1.6" />
-        <joint name="left_hip_yaw_joint_X8"         kp="${150*kp_scale}" kd="${10*kd_scale}" effort_limit="100"   vel_limit="13.3" default_pos="0"    friction="1.6" />
-        <joint name="left_knee_joint_X8"            kp="${200*kp_scale}" kd="${10*kd_scale}" effort_limit="100"   vel_limit="13.3" default_pos="0.30" friction="1.14" />
-        <joint name="left_ankle_pitch_joint_X4"     kp="${200*kp_scale}" kd="${10*kd_scale}" effort_limit="96.6"  vel_limit="2.17" default_pos="-0.15" friction="1.14" />
+        <joint name="left_hip_pitch_joint_X8"       kp="${140*kp_scale}" kd="${35*kd_scale}" effort_limit="100"   vel_limit="13.3" default_pos="-0.15" friction="3.21" />
+        <joint name="left_hip_roll_joint_X8"        kp="${150*kp_scale}" kd="${15*kd_scale}" effort_limit="100"   vel_limit="13.3" default_pos="0"    friction="1.6" />
+        <joint name="left_hip_yaw_joint_X8"         kp="${150*kp_scale}" kd="${18*kd_scale}" effort_limit="100"   vel_limit="13.3" default_pos="0"    friction="1.6" />
+        <joint name="left_knee_joint_X8"            kp="${220*kp_scale}" kd="${10*kd_scale}" effort_limit="100"   vel_limit="13.3" default_pos="0.30" friction="1.14" />
+        <joint name="left_ankle_pitch_joint_X4"     kp="${200*kp_scale}" kd="${18*kd_scale}" effort_limit="96.6"  vel_limit="2.17" default_pos="-0.15" friction="1.14" />
         <joint name="left_ankle_roll_joint_X4"      kp="${150*kp_scale}" kd="${8*kd_scale}"  effort_limit="28.98" vel_limit="7.24" default_pos="0"    friction="1.14" />
         <!-- Right leg (mirror) -->
-        <joint name="right_hip_pitch_joint_X8"      kp="${200*kp_scale}" kd="${10*kd_scale}" effort_limit="100"   vel_limit="13.3" default_pos="-0.15" friction="3.21" />
-        <joint name="right_hip_roll_joint_X8"       kp="${150*kp_scale}" kd="${10*kd_scale}" effort_limit="100"   vel_limit="13.3" default_pos="0"    friction="1.6" />
-        <joint name="right_hip_yaw_joint_X8"        kp="${150*kp_scale}" kd="${10*kd_scale}" effort_limit="100"   vel_limit="13.3" default_pos="0"    friction="1.6" />
-        <joint name="right_knee_joint_X8"           kp="${200*kp_scale}" kd="${10*kd_scale}" effort_limit="100"   vel_limit="13.3" default_pos="0.30" friction="1.14" />
-        <joint name="right_ankle_pitch_joint_X4"    kp="${200*kp_scale}" kd="${10*kd_scale}" effort_limit="96.6"  vel_limit="2.17" default_pos="-0.15" friction="1.14" />
+        <joint name="right_hip_pitch_joint_X8"      kp="${140*kp_scale}" kd="${35*kd_scale}" effort_limit="100"   vel_limit="13.3" default_pos="-0.15" friction="3.21" />
+        <joint name="right_hip_roll_joint_X8"       kp="${150*kp_scale}" kd="${15*kd_scale}" effort_limit="100"   vel_limit="13.3" default_pos="0"    friction="1.6" />
+        <joint name="right_hip_yaw_joint_X8"        kp="${150*kp_scale}" kd="${18*kd_scale}" effort_limit="100"   vel_limit="13.3" default_pos="0"    friction="1.6" />
+        <joint name="right_knee_joint_X8"           kp="${220*kp_scale}" kd="${10*kd_scale}" effort_limit="100"   vel_limit="13.3" default_pos="0.30" friction="1.14" />
+        <joint name="right_ankle_pitch_joint_X4"    kp="${200*kp_scale}" kd="${18*kd_scale}" effort_limit="96.6"  vel_limit="2.17" default_pos="-0.15" friction="1.14" />
         <joint name="right_ankle_roll_joint_X4"     kp="${150*kp_scale}" kd="${8*kd_scale}"  effort_limit="28.98" vel_limit="7.24" default_pos="0"    friction="1.14" />
       </plugin>

Commit message: jtc pid controller, robot_tools, gains calculations from kdl tree, new pd_effort controller for real_robot

File: src/robot_description/full_robot_description/urdf/full_robot_gazebo.xacro (robot description, xacro)
@@ -54,10 +54,13 @@
     <origin xyz="0.0635 0.0 0.35" rpy="0 ${pi/2} 0"/>
   </xacro:bno055_imu>
-  <!-- Fix robot base to world frame -->
-  <!-- <link name="world"/>
-  <joint name="world_joint" type="fixed">
-    <parent link="world"/>
-    <child link="urdf_base"/>
-  </joint> -->
+  <!-- Fix robot base to world frame (for arms-only testing) -->
+  <xacro:arg name="fixed_base" default="false"/>
+  <xacro:if value="$(arg fixed_base)">
+    <link name="world"/>
+    <joint name="world_joint" type="fixed">
+      <parent link="world"/>
+      <child link="urdf_base"/>
+    </joint>
+  </xacro:if>
   <!-- ros2_control: position mode -->
   <xacro:if value="${'$(arg control_mode)' == 'position'}">
@@ -65,6 +68,6 @@
     <xacro:full_robot_ros2_control_position />
   </xacro:if>
-  <!-- ros2_control: effort mode -->
-  <xacro:if value="${'$(arg control_mode)' == 'effort'}">
+  <!-- ros2_control: effort mode (matches any control_mode starting with "effort") -->
+  <xacro:if value="${'$(arg control_mode)'.startswith('effort')}">
     <xacro:include filename="$(find full_robot_description)/urdf/macros/ros2_control_effort.xacro" />
     <xacro:full_robot_ros2_control_effort />
