Commit message: training issac first commit

File: src/robot_description/full_robot_description/urdf/full_robot_gazebo.xacro (robot description, xacro)
@@ -74,5 +74,11 @@
     <plugin filename="gz_ros2_control-system" name="gz_ros2_control::GazeboSimROS2ControlPlugin">
       <parameters>$(find full_robot_gazebo)/config/controllers_$(arg control_mode).yaml</parameters>
-      <update_rate>100</update_rate>
+      <update_rate>1000</update_rate>
+    </plugin>
+  </gazebo>
+  <!-- Odometry publisher (needed for RL locomotion node) -->
+  <gazebo>
+    <plugin filename="gz-sim-odometry-publisher-system" name="gz::sim::systems::OdometryPublisher">
+      <odom_publish_frequency>50</odom_publish_frequency>
     </plugin>
   </gazebo>

File: src/robot_description/full_robot_description/urdf/joints/body_joints.xacro (robot description, xacro)
@@ -28,5 +28,5 @@
     <child link="urdf_simplified_torso"/>
     <axis xyz="0 0 1"/>
-    <limit effort="${X8_moderate_effort}" velocity="${X8_rated_velocity}" lower="-2.60054" upper="2.60054"/>
+    <limit effort="${X8_peak_effort}" velocity="${X8_rated_velocity}" lower="-2.60054" upper="2.60054"/>
     <dynamics damping="${X8_damping}" friction="${X8_friction}"/>
   </joint>

File: src/robot_description/full_robot_description/urdf/joints/left_arm_joints.xacro (robot description, xacro)
@@ -9,5 +9,5 @@
     <child link="urdf_l_shoulder_assembly"/>
     <axis xyz="0 1 0"/>
-    <limit effort="${X6_moderate_effort}" velocity="${X6_rated_velocity}" lower="-3.01942" upper="1.69297"/>
+    <limit effort="${X6_peak_effort}" velocity="${X6_rated_velocity}" lower="-3.01942" upper="1.69297"/>
     <dynamics damping="${X6_damping}" friction="${X6_friction}"/>
   </joint>
@@ -17,5 +17,5 @@
     <child link="urdf_l_upper_arm_assembly"/>
     <axis xyz="1 0 0"/>
-    <limit effort="${X6_moderate_effort}" velocity="${X6_rated_velocity}" lower="-0.20944" upper="2.93215"/>
+    <limit effort="${X6_peak_effort}" velocity="${X6_rated_velocity}" lower="-0.20944" upper="2.93215"/>
     <dynamics damping="${X6_damping}" friction="${X6_friction}"/>
   </joint>
@@ -25,5 +25,5 @@
     <child link="urdf_l_elbow_assembly"/>
     <axis xyz="0 0 1"/>
-    <limit effort="${X4_moderate_effort}" velocity="${X4_rated_velocity}" lower="-1.74533" upper="2.96706"/>
+    <limit effort="${X4_peak_effort}" velocity="${X4_rated_velocity}" lower="-1.74533" upper="2.96706"/>
     <dynamics damping="${X4_damping}" friction="${X4_friction}"/>
   </joint>
@@ -33,5 +33,5 @@
     <child link="urdf_l_upper_forearm_assembly"/>
     <axis xyz="0 1 0"/>
-    <limit effort="${X6_moderate_effort}" velocity="${X6_rated_velocity}" lower="-1.309" upper="1.8326"/>
+    <limit effort="${X6_peak_effort}" velocity="${X6_rated_velocity}" lower="-1.309" upper="1.8326"/>
     <dynamics damping="${X6_damping}" friction="${X6_friction}"/>
   </joint>
@@ -41,5 +41,5 @@
     <child link="urdf_l_lower_forearm_assembly"/>
     <axis xyz="0 0 1"/>
-    <limit effort="${X4_moderate_effort}" velocity="${X4_rated_velocity}" lower="-2.35619" upper="2.35619"/>
+    <limit effort="${X4_peak_effort}" velocity="${X4_rated_velocity}" lower="-2.35619" upper="2.35619"/>
     <dynamics damping="${X4_damping}" friction="${X4_friction}"/>
   </joint>
@@ -49,5 +49,5 @@
     <child link="urdf_l_wrist_assembly"/>
     <axis xyz="1 0 0"/>
-    <limit effort="${X4_moderate_effort}" velocity="${X4_rated_velocity}" lower="-1.5708" upper="1.5708"/>
+    <limit effort="${X4_peak_effort}" velocity="${X4_rated_velocity}" lower="-1.5708" upper="1.5708"/>
     <dynamics damping="${X4_damping}" friction="${X4_friction}"/>
   </joint>

File: src/robot_description/full_robot_description/urdf/joints/left_foot_joints.xacro (robot description, xacro)
@@ -9,5 +9,5 @@
     <child link="urdf_hip_assembly"/>
     <axis xyz="0 1 0"/>
-    <limit effort="${X8_moderate_effort}" velocity="${X8_rated_velocity}" lower="-2.61799" upper="2.61799"/>
+    <limit effort="${X8_peak_effort}" velocity="${X8_rated_velocity}" lower="-2.61799" upper="2.61799"/>
     <dynamics damping="${X8_damping}" friction="${X8_friction}"/>
   </joint>
@@ -17,5 +17,5 @@
     <child link="urdf_l_upper_femur_assembly"/>
     <axis xyz="1 0 0"/>
-    <limit effort="${X8_moderate_effort}" velocity="${X8_rated_velocity}" lower="-0.383972" upper="3.22886"/>
+    <limit effort="${X8_peak_effort}" velocity="${X8_rated_velocity}" lower="-0.383972" upper="3.22886"/>
     <dynamics damping="${X8_damping}" friction="${X8_friction}"/>
   </joint>
@@ -25,5 +25,5 @@
     <child link="urdf_lower_femur_assembly"/>
     <axis xyz="0 0 1"/>
-    <limit effort="${X8_moderate_effort}" velocity="${X8_rated_velocity}" lower="-2.15199" upper="2.09003"/>
+    <limit effort="${X8_peak_effort}" velocity="${X8_rated_velocity}" lower="-2.15199" upper="2.09003"/>
     <dynamics damping="${X8_damping}" friction="${X8_friction}"/>
   </joint>
@@ -33,5 +33,5 @@
     <child link="urdf_l_tibia_assembly"/>
     <axis xyz="0 1 0"/>
-    <limit effort="${X8_moderate_effort}" velocity="${X8_rated_velocity}" lower="-1.52716" upper="1.52716"/>
+    <limit effort="${X8_peak_effort}" velocity="${X8_rated_velocity}" lower="-1.52716" upper="1.52716"/>
     <dynamics damping="${X8_damping}" friction="${X8_friction}"/>
   </joint>
@@ -41,5 +41,5 @@
     <child link="udrf_ankle_assembly"/>
     <axis xyz="0 1 0"/>
-    <limit effort="${X4_moderate_effort}" velocity="${X4_rated_velocity}" lower="-0.785398" upper="0.785398"/>
+    <limit effort="${ankle_pitch_peak_effort}" velocity="${ankle_pitch_rated_velocity}" lower="-0.785398" upper="0.785398"/>
     <dynamics damping="${X4_damping}" friction="${X4_friction}"/>
   </joint>
@@ -49,5 +49,5 @@
     <child link="urdf_foot_assembly"/>
     <axis xyz="1 0 0"/>
-    <limit effort="${X4_moderate_effort}" velocity="${X4_rated_velocity}" lower="-0.785398" upper="0.785398"/>
+    <limit effort="${ankle_roll_peak_effort}" velocity="${ankle_roll_rated_velocity}" lower="-0.785398" upper="0.785398"/>
     <dynamics damping="${X4_damping}" friction="${X4_friction}"/>
   </joint>

File: src/robot_description/full_robot_description/urdf/joints/right_arm_joints.xacro (robot description, xacro)
@@ -9,5 +9,5 @@
     <child link="urdf_r_shoulder_assembly"/>
     <axis xyz="0 1 0"/>
-    <limit effort="${X6_moderate_effort}" velocity="${X6_rated_velocity}" lower="-3.01942" upper="1.69297"/>
+    <limit effort="${X6_peak_effort}" velocity="${X6_rated_velocity}" lower="-3.01942" upper="1.69297"/>
     <dynamics damping="${X6_damping}" friction="${X6_friction}"/>
   </joint>
@@ -17,5 +17,5 @@
     <child link="urdf_r_upper_arm_assembly"/>
     <axis xyz="1 0 0"/>
-    <limit effort="${X6_moderate_effort}" velocity="${X6_rated_velocity}" lower="-2.93215" upper="0.20944"/>
+    <limit effort="${X6_peak_effort}" velocity="${X6_rated_velocity}" lower="-2.93215" upper="0.20944"/>
     <dynamics damping="${X6_damping}" friction="${X6_friction}"/>
   </joint>
@@ -25,5 +25,5 @@
     <child link="urdf_r_elbow_assembly"/>
     <axis xyz="0 0 1"/>
-    <limit effort="${X4_moderate_effort}" velocity="${X4_rated_velocity}" lower="-2.96706" upper="1.74533"/>
+    <limit effort="${X4_peak_effort}" velocity="${X4_rated_velocity}" lower="-2.96706" upper="1.74533"/>
     <dynamics damping="${X4_damping}" friction="${X4_friction}"/>
   </joint>
@@ -33,5 +33,5 @@
     <child link="urdf_r_upper_forearm_assembly"/>
     <axis xyz="0 1 0"/>
-    <limit effort="${X6_moderate_effort}" velocity="${X6_rated_velocity}" lower="-1.309" upper="1.8326"/>
+    <limit effort="${X6_peak_effort}" velocity="${X6_rated_velocity}" lower="-1.309" upper="1.8326"/>
     <dynamics damping="${X6_damping}" friction="${X6_friction}"/>
   </joint>
@@ -41,5 +41,5 @@
     <child link="urdf_r_lower_forearm_assembly"/>
     <axis xyz="0 0 1"/>
-    <limit effort="${X4_moderate_effort}" velocity="${X4_rated_velocity}" lower="-2.35619" upper="2.35619"/>
+    <limit effort="${X4_peak_effort}" velocity="${X4_rated_velocity}" lower="-2.35619" upper="2.35619"/>
     <dynamics damping="${X4_damping}" friction="${X4_friction}"/>
   </joint>
@@ -49,5 +49,5 @@
     <child link="urdf_r_wrist_assembly"/>
     <axis xyz="1 0 0"/>
-    <limit effort="${X4_moderate_effort}" velocity="${X4_rated_velocity}" lower="-1.65806" upper="1.65806"/>
+    <limit effort="${X4_peak_effort}" velocity="${X4_rated_velocity}" lower="-1.65806" upper="1.65806"/>
     <dynamics damping="${X4_damping}" friction="${X4_friction}"/>
   </joint>

File: src/robot_description/full_robot_description/urdf/joints/right_foot_joints.xacro (robot description, xacro)
@@ -9,5 +9,5 @@
     <child link="urdf_hip_assembly_2"/>
     <axis xyz="0 1 0"/>
-    <limit effort="${X8_moderate_effort}" velocity="${X8_rated_velocity}" lower="-2.61799" upper="2.61799"/>
+    <limit effort="${X8_peak_effort}" velocity="${X8_rated_velocity}" lower="-2.61799" upper="2.61799"/>
     <dynamics damping="${X8_damping}" friction="${X8_friction}"/>
   </joint>
@@ -17,5 +17,5 @@
     <child link="urdf_r_upper_femur_assemby"/>
     <axis xyz="1 0 0"/>
-    <limit effort="${X8_moderate_effort}" velocity="${X8_rated_velocity}" lower="-3.22886" upper="0.383972"/>
+    <limit effort="${X8_peak_effort}" velocity="${X8_rated_velocity}" lower="-3.22886" upper="0.383972"/>
     <dynamics damping="${X8_damping}" friction="${X8_friction}"/>
   </joint>
@@ -25,5 +25,5 @@
     <child link="urdf_lower_femur_assembly_2"/>
     <axis xyz="0 0 1"/>
-    <limit effort="${X8_moderate_effort}" velocity="${X8_rated_velocity}" lower="-1.5708" upper="1.5708"/>
+    <limit effort="${X8_peak_effort}" velocity="${X8_rated_velocity}" lower="-1.5708" upper="1.5708"/>
     <dynamics damping="${X8_damping}" friction="${X8_friction}"/>
   </joint>
@@ -33,5 +33,5 @@
     <child link="urdf_r_tibia_assembly"/>
     <axis xyz="0 1 0"/>
-    <limit effort="${X8_moderate_effort}" velocity="${X8_rated_velocity}" lower="-1.52716" upper="1.52716"/>
+    <limit effort="${X8_peak_effort}" velocity="${X8_rated_velocity}" lower="-1.52716" upper="1.52716"/>
     <dynamics damping="${X8_damping}" friction="${X8_friction}"/>
   </joint>
@@ -41,5 +41,5 @@
     <child link="udrf_ankle_assembly_2"/>
     <axis xyz="1 0 0"/>
-    <limit effort="${X4_moderate_effort}" velocity="${X4_rated_velocity}" lower="-0.785398" upper="0.785398"/>
+    <limit effort="${ankle_roll_peak_effort}" velocity="${ankle_roll_rated_velocity}" lower="-0.785398" upper="0.785398"/>
     <dynamics damping="${X4_damping}" friction="${X4_friction}"/>
   </joint>
@@ -49,5 +49,5 @@
     <child link="urdf_foot_assembly_2"/>
     <axis xyz="0 1 0"/>
-    <limit effort="${X4_moderate_effort}" velocity="${X4_rated_velocity}" lower="-0.785398" upper="0.785398"/>
+    <limit effort="${ankle_pitch_peak_effort}" velocity="${ankle_pitch_rated_velocity}" lower="-0.785398" upper="0.785398"/>
     <dynamics damping="${X4_damping}" friction="${X4_friction}"/>
   </joint>

File: src/robot_description/full_robot_description/urdf/macros/actuator_properties.xacro (robot description, xacro)
@@ -17,4 +17,7 @@
   <xacro:property name="X4_friction"           value="1.14" />
   <xacro:property name="X4_damping"            value="0.114" />
+  <!-- Rotor inertia: 0.3 Kg·cm² = 3.0e-6 kg·m², gear ratio 36:1
+       Reflected inertia = I_rotor × N² = 3.0e-6 × 1296 = 0.00389 kg·m² -->
+  <xacro:property name="X4_rotor_inertia"      value="0.00389" />
   <!-- ==================== X6-60 (direct) ==================== -->
   <xacro:property name="X6_rated_effort"       value="20" />
@@ -25,4 +28,7 @@
   <xacro:property name="X6_friction"           value="1.6" />
   <xacro:property name="X6_damping"            value="0.16" />
+  <!-- Rotor inertia: 0.66 Kg·cm² = 6.6e-6 kg·m², gear ratio 19.612:1
+       Reflected inertia = I_rotor × N² = 6.6e-6 × 384.6 = 0.00254 kg·m² -->
+  <xacro:property name="X6_rotor_inertia"      value="0.00254" />
   <!-- ==================== X8-120 (direct) ==================== -->
   <xacro:property name="X8_rated_effort"       value="43" />
@@ -36,4 +42,7 @@
   <xacro:property name="X8_friction"           value="3.21" />
   <xacro:property name="X8_damping"            value="0.321" />
+  <!-- Rotor inertia: 1.5 Kg·cm² = 1.5e-5 kg·m², gear ratio 19.612:1
+       Reflected inertia = I_rotor × N² = 1.5e-5 × 384.6 = 0.00577 kg·m² -->
+  <xacro:property name="X8_rotor_inertia"      value="0.00577" />
   <!-- ==================== Ankle Linkage =====================
        2x X4 motors with eccentric-pushrod mechanism

Commit message: Update left arm controller in wave_hello_4.yaml to use trajectory controller, added trajectory action tool controller to monitor and controller each joint based on the selected controller. renamed joint controllers from group to trajectory

File: src/robot_description/full_robot_description/urdf/full_robot_gazebo.xacro (robot description, xacro)
@@ -3,4 +3,6 @@
   <!-- Control mode: "position" or "effort" -->
   <xacro:arg name="control_mode" default="position" />
+  <!-- Fix base to world (no floating, for upper body work) -->
+  <xacro:arg name="fixed_base" default="false" />
   <!-- Full robot: all joints active (not fixed) -->
   <xacro:arg name="fixed_legs" default="false" />
@@ -55,9 +57,11 @@
   </xacro:bno055_imu>
   <!-- Fix robot base to world frame -->
-  <!-- <link name="world"/>
-  <joint name="world_joint" type="fixed">
-    <parent link="world"/>
-    <child link="urdf_base"/>
-  </joint> -->
+  <xacro:if value="$(arg fixed_base)">
+    <link name="world"/>
+    <joint name="world_joint" type="fixed">
+      <parent link="world"/>
+      <child link="urdf_base"/>
+    </joint>
+  </xacro:if>
   <!-- ros2_control: position mode -->
   <xacro:if value="${'$(arg control_mode)' == 'position'}">
