Commit message: Add gemini camera in full robot configuration

File: src/robot_description/full_robot_description/urdf/full_robot_gazebo.xacro (robot description, xacro)
@@ -31,26 +31,37 @@
   <xacro:include filename="$(find full_robot_description)/urdf/links/right_foot_links.xacro" />
   <xacro:include filename="$(find full_robot_description)/urdf/joints/right_foot_joints.xacro" />
-  <!-- Temporarily disable inspire hands to speed up simulation and avoid issues with the hand meshes. Will be re-enabled once the hand meshes are optimized for simulation. -->
   <!-- Hands -->
-  <!--xacro:include filename="$(find hand_description)/urdf/hands/inspire_hand_left.xacro" /-->
-  <!--xacro:include filename="$(find hand_description)/urdf/hands/inspire_hand_right.xacro" /-->
-  <!--xacro:inspire_hand_left
-      parent="urdf_l_wrist_assembly"
-      prefix="left_"
-      mount_x="-0.034"
-      mount_y="0.015"
-      mount_z="-0.06"
-      mount_roll="1.424576"
-      mount_pitch="-0.201364"
-      mount_yaw="2.205507"/-->
-  <!--xacro:inspire_hand_right
-      parent="urdf_r_wrist_assembly"
-      prefix="right_"
-      mount_x="-0.029"
-      mount_y="-0.011"
-      mount_z="-0.06"
-      mount_roll="1.717027"
-      mount_pitch="-0.201373"
-      mount_yaw="-2.205496"/-->
+  <xacro:include filename="$(find hand_description)/urdf/hands/inspire_hand_left.xacro" />
+  <xacro:include filename="$(find hand_description)/urdf/hands/inspire_hand_right.xacro" />
+  <!-- Mount offsets differ from arm_description/urdf/arm_base.xacro, which uses
+       idealised pi/2 rotations. These are the dual-arm values as measured; do not
+       substitute one set for the other without re-checking against the hardware. -->
+  <xacro:inspire_hand_left
+        parent="urdf_l_wrist_assembly"
+        prefix="left_"
+        mount_x="-0.0303429"
+        mount_y="4.99302e-07"
+        mount_z="-0.06"
+        mount_roll="${pi/2}"
+        mount_pitch="0.0"
+        mount_yaw="${pi/2}"/>
+  <xacro:inspire_hand_right
+        parent="urdf_r_wrist_assembly"
+        prefix="right_"
+        mount_x="-0.0327429 "
+        mount_y="0.008"
+        mount_z="-0.06"
+        mount_roll="${pi/2}"
+        mount_pitch="0.0"
+        mount_yaw="-${pi/2}"/>
+  <!-- Orbbec Gemini 335L/336L Depth Camera -->
+  <xacro:include filename="$(find camera_description)/urdf/gemini335L_336L.urdf.xacro"/>
+  <xacro:include filename="$(find camera_description)/urdf/gemini335L_336L_gazebo.xacro"/>
+  <!-- Mount camera on urdf_base, positioned to view the workspace -->
+  <joint name="camera_mount_joint" type="fixed">
+      <parent link="urdf_base"/>
+      <child link="camera_link"/>
+      <origin xyz="0.08 0.0455 0.829" rpy="0 ${pi/12} 0"/>
+  </joint>
   <!-- IMU sensors (BNO055) -->
   <xacro:include filename="$(find imu_description)/urdf/bno055_imu.xacro" />

Commit message: feat(full_robot): enable the hands and give the arms a start pose
HandSystem ros2_control block (12 actuated + 12 mimic) plus unconditional
hand controller spawners — no body controller claims a hand joint. Arms and
waist get dual_arm's initial_value. The old blocks were commented out as
"hands disabled in URDF"; full_robot_gazebo.xacro includes them.

File: src/robot_description/full_robot_description/urdf/full_robot_gazebo.xacro (robot description, xacro)
@@ -84,4 +84,5 @@
     <xacro:include filename="$(find full_robot_description)/urdf/macros/ros2_control_position.xacro" />
     <xacro:full_robot_ros2_control_position />
+    <xacro:full_robot_ros2_control_hands />
   </xacro:if>
   <!-- ros2_control: effort mode -->

File: src/robot_description/full_robot_description/urdf/macros/ros2_control_position.xacro (robot description, xacro)
@@ -12,5 +12,7 @@
           <param name="max">2.60054</param>
         </command_interface>
-        <state_interface name="position" />
+        <state_interface name="position">
+          <param name="initial_value">0.0</param>
+        </state_interface>
         <state_interface name="velocity" />
         <state_interface name="effort" />
@@ -22,5 +24,7 @@
           <param name="max">1.69297</param>
         </command_interface>
-        <state_interface name="position" />
+        <state_interface name="position">
+          <param name="initial_value">0.0</param>
+        </state_interface>
         <state_interface name="velocity" />
         <state_interface name="effort" />
@@ -31,5 +35,7 @@
           <param name="max">2.93215</param>
         </command_interface>
-        <state_interface name="position" />
+        <state_interface name="position">
+          <param name="initial_value">0.1</param>
+        </state_interface>
         <state_interface name="velocity" />
         <state_interface name="effort" />
@@ -40,5 +46,7 @@
           <param name="max">2.96706</param>
         </command_interface>
-        <state_interface name="position" />
+        <state_interface name="position">
+          <param name="initial_value">0.0</param>
+        </state_interface>
         <state_interface name="velocity" />
         <state_interface name="effort" />
@@ -49,5 +57,7 @@
           <param name="max">1.8326</param>
         </command_interface>
-        <state_interface name="position" />
+        <state_interface name="position">
+          <param name="initial_value">-0.1</param>
+        </state_interface>
         <state_interface name="velocity" />
         <state_interface name="effort" />
@@ -58,5 +68,7 @@
           <param name="max">2.35619</param>
         </command_interface>
-        <state_interface name="position" />
+        <state_interface name="position">
+          <param name="initial_value">0.0</param>
+        </state_interface>
         <state_interface name="velocity" />
         <state_interface name="effort" />
@@ -67,5 +79,7 @@
           <param name="max">1.5708</param>
         </command_interface>
-        <state_interface name="position" />
+        <state_interface name="position">
+          <param name="initial_value">0.0</param>
+        </state_interface>
         <state_interface name="velocity" />
         <state_interface name="effort" />
@@ -77,5 +91,7 @@
           <param name="max">1.69297</param>
         </command_interface>
-        <state_interface name="position" />
+        <state_interface name="position">
+          <param name="initial_value">0.0</param>
+        </state_interface>
         <state_interface name="velocity" />
         <state_interface name="effort" />
@@ -86,5 +102,7 @@
           <param name="max">0.20944</param>
         </command_interface>
-        <state_interface name="position" />
+        <state_interface name="position">
+          <param name="initial_value">-0.1</param>
+        </state_interface>
         <state_interface name="velocity" />
         <state_interface name="effort" />
@@ -95,5 +113,7 @@
           <param name="max">1.74533</param>
         </command_interface>
-        <state_interface name="position" />
+        <state_interface name="position">
+          <param name="initial_value">0.0</param>
+        </state_interface>
         <state_interface name="velocity" />
         <state_interface name="effort" />
@@ -104,5 +124,7 @@
           <param name="max">1.8326</param>
         </command_interface>
-        <state_interface name="position" />
+        <state_interface name="position">
+          <param name="initial_value">-0.1</param>
+        </state_interface>
         <state_interface name="velocity" />
         <state_interface name="effort" />
@@ -113,5 +135,7 @@
           <param name="max">2.35619</param>
         </command_interface>
-        <state_interface name="position" />
+        <state_interface name="position">
+          <param name="initial_value">0.0</param>
+        </state_interface>
         <state_interface name="velocity" />
         <state_interface name="effort" />
@@ -122,110 +146,10 @@
           <param name="max">1.65806</param>
         </command_interface>
-        <state_interface name="position" />
-        <state_interface name="velocity" />
-        <state_interface name="effort" />
-      </joint>
-      <!-- === LEFT HAND (6 actuated) — DISABLED: inspire hands commented out in URDF === -->
-      <!-- DISABLED
-      <joint name="left_thumb_proximal_yaw_joint">
-        <command_interface name="position">
-          <param name="min">0</param>
-          <param name="max">1.31</param>
-        </command_interface>
-        <state_interface name="position" />
-        <state_interface name="velocity" />
-      </joint>
-      <joint name="left_thumb_proximal_pitch_joint">
-        <command_interface name="position">
-          <param name="min">0</param>
-          <param name="max">0.61</param>
-        </command_interface>
-        <state_interface name="position" />
-        <state_interface name="velocity" />
-      </joint>
-      <joint name="left_index_proximal_joint">
-        <command_interface name="position">
-          <param name="min">0</param>
-          <param name="max">1.47</param>
-        </command_interface>
-        <state_interface name="position" />
-        <state_interface name="velocity" />
-      </joint>
-      <joint name="left_middle_proximal_joint">
-        <command_interface name="position">
-          <param name="min">0</param>
-          <param name="max">1.47</param>
-        </command_interface>
-        <state_interface name="position" />
-        <state_interface name="velocity" />
-      </joint>
-      <joint name="left_ring_proximal_joint">
-        <command_interface name="position">
-          <param name="min">0</param>
-          <param name="max">1.47</param>
-        </command_interface>
-        <state_interface name="position" />
-        <state_interface name="velocity" />
-      </joint>
-      <joint name="left_pinky_proximal_joint">
-        <command_interface name="position">
-          <param name="min">0</param>
-          <param name="max">1.47</param>
-        </command_interface>
-        <state_interface name="position" />
-        <state_interface name="velocity" />
-      </joint>
-      -->
-      <!-- === RIGHT HAND (6 actuated) — DISABLED: inspire hands commented out in URDF === -->
-      <!-- DISABLED
-      <joint name="right_thumb_proximal_yaw_joint">
-        <command_interface name="position">
-          <param name="min">0</param>
-          <param name="max">1.31</param>
-        </command_interface>
-        <state_interface name="position" />
-        <state_interface name="velocity" />
-      </joint>
-      <joint name="right_thumb_proximal_pitch_joint">
-        <command_interface name="position">
-          <param name="min">0</param>
-          <param name="max">0.61</param>
-        </command_interface>
-        <state_interface name="position" />
-        <state_interface name="velocity" />
-      </joint>
-      <joint name="right_index_proximal_joint">
-        <command_interface name="position">
-          <param name="min">0</param>
-          <param name="max">1.47</param>
-        </command_interface>
-        <state_interface name="position" />
-        <state_interface name="velocity" />
-      </joint>
-      <joint name="right_middle_proximal_joint">
-        <command_interface name="position">
-          <param name="min">0</param>
-          <param name="max">1.47</param>
-        </command_interface>
-        <state_interface name="position" />
-        <state_interface name="velocity" />
-      </joint>
-      <joint name="right_ring_proximal_joint">
-        <command_interface name="position">
-          <param name="min">0</param>
-          <param name="max">1.47</param>
-        </command_interface>
-        <state_interface name="position" />
-        <state_interface name="velocity" />
-      </joint>
-      <joint name="right_pinky_proximal_joint">
-        <command_interface name="position">
-          <param name="min">0</param>
-          <param name="max">1.47</param>
-        </command_interface>
-        <state_interface name="position" />
-        <state_interface name="velocity" />
-      </joint>
-      -->
+        <state_interface name="position">
+          <param name="initial_value">0.0</param>
+        </state_interface>
+        <state_interface name="velocity" />
+        <state_interface name="effort" />
+      </joint>
       <!-- === LEFT LEG === -->
       <joint name="left_hip_pitch_joint_X8">
@@ -334,4 +258,208 @@
           <param name="max">0.785398</param>
         </command_interface>
+        <state_interface name="position" />
+        <state_interface name="velocity" />
+        <state_interface name="effort" />
+      </joint>
+    </ros2_control>
+  </xacro:macro>
+  <!-- The hands are a separate system, as in dual_arm_description. They are their own
+       hardware on the real robot, and the mimic joints below have no command interface,
+       which keeps that oddity out of the body block. -->
+  <xacro:macro name="full_robot_ros2_control_hands">
+    <ros2_control name="HandSystem" type="system">
+      <hardware>
+        <plugin>gz_ros2_control/GazeboSimSystem</plugin>
+      </hardware>
+      <!-- === ACTUATED (6 per hand) === -->
+      <joint name="left_thumb_proximal_yaw_joint">
+        <command_interface name="position">
+          <param name="min">0</param>
+          <param name="max">1.31</param>
+        </command_interface>
+        <state_interface name="position">
+          <param name="initial_value">0.1</param>
+        </state_interface>
+        <state_interface name="velocity" />
+        <state_interface name="effort" />
+      </joint>
+      <joint name="left_thumb_proximal_pitch_joint">
+        <command_interface name="position">
+          <param name="min">0</param>
+          <param name="max">0.61</param>
+        </command_interface>
+        <state_interface name="position">
+          <param name="initial_value">0.1</param>
+        </state_interface>
+        <state_interface name="velocity" />
+        <state_interface name="effort" />
+      </joint>
+      <joint name="left_index_proximal_joint">
+        <command_interface name="position">
+          <param name="min">0</param>
+          <param name="max">1.47</param>
+        </command_interface>
+        <state_interface name="position">
+          <param name="initial_value">0.1</param>
+        </state_interface>
+        <state_interface name="velocity" />
+        <state_interface name="effort" />
+      </joint>
+      <joint name="left_middle_proximal_joint">
+        <command_interface name="position">
+          <param name="min">0</param>
+          <param name="max">1.47</param>
+        </command_interface>
+        <state_interface name="position">
+          <param name="initial_value">0.1</param>
+        </state_interface>
+        <state_interface name="velocity" />
+        <state_interface name="effort" />
+      </joint>
+      <joint name="left_ring_proximal_joint">
+        <command_interface name="position">
+          <param name="min">0</param>
+          <param name="max">1.47</param>
+        </command_interface>
+        <state_interface name="position">
+          <param name="initial_value">0.1</param>
+        </state_interface>
+        <state_interface name="velocity" />
+        <state_interface name="effort" />
+      </joint>
+      <joint name="left_pinky_proximal_joint">
+        <command_interface name="position">
+          <param name="min">0</param>
+          <param name="max">1.47</param>
+        </command_interface>
+        <state_interface name="position">
+          <param name="initial_value">0.1</param>
+        </state_interface>
+        <state_interface name="velocity" />
+        <state_interface name="effort" />
+      </joint>
+      <joint name="right_thumb_proximal_yaw_joint">
+        <command_interface name="position">
+          <param name="min">0.0</param>
+          <param name="max">1.308</param>
+        </command_interface>
+        <state_interface name="position">
+          <param name="initial_value">0.1</param>
+        </state_interface>
+        <state_interface name="velocity" />
+        <state_interface name="effort" />
+      </joint>
+      <joint name="right_thumb_proximal_pitch_joint">
+        <command_interface name="position">
+          <param name="min">0</param>
+          <param name="max">0.6</param>
+        </command_interface>
+        <state_interface name="position">
+          <param name="initial_value">0.1</param>
+        </state_interface>
+        <state_interface name="velocity" />
+        <state_interface name="effort" />
+      </joint>
+      <joint name="right_index_proximal_joint">
+        <command_interface name="position">
+          <param name="min">0</param>
+          <param name="max">1.47</param>
+        </command_interface>
+        <state_interface name="position">
+          <param name="initial_value">0.1</param>
+        </state_interface>
+        <state_interface name="velocity" />
+        <state_interface name="effort" />
+      </joint>
+      <joint name="right_middle_proximal_joint">
+        <command_interface name="position">
+          <param name="min">0</param>
+          <param name="max">1.47</param>
+        </command_interface>
+        <state_interface name="position">
+          <param name="initial_value">0.1</param>
+        </state_interface>
+        <state_interface name="velocity" />
+        <state_interface name="effort" />
+      </joint>
+      <joint name="right_ring_proximal_joint">
+        <command_interface name="position">
+          <param name="min">0</param>
+          <param name="max">1.47</param>
+        </command_interface>
+        <state_interface name="position">
+          <param name="initial_value">0.1</param>
+        </state_interface>
+        <state_interface name="velocity" />
+        <state_interface name="effort" />
+      </joint>
+      <joint name="right_pinky_proximal_joint">
+        <command_interface name="position">
+          <param name="min">0</param>
+          <param name="max">1.47</param>
+        </command_interface>
+        <state_interface name="position">
+          <param name="initial_value">0.1</param>
+        </state_interface>
+        <state_interface name="velocity" />
+        <state_interface name="effort" />
+      </joint>
+      <!-- === MIMIC (driven by the proximal joints; state only, no command) === -->
+      <joint name="left_thumb_intermediate_joint">
+        <state_interface name="position" />
+        <state_interface name="velocity" />
+        <state_interface name="effort" />
+      </joint>
+      <joint name="left_thumb_distal_joint">
+        <state_interface name="position" />
+        <state_interface name="velocity" />
+        <state_interface name="effort" />
+      </joint>
+      <joint name="left_index_intermediate_joint">
+        <state_interface name="position" />
+        <state_interface name="velocity" />
+        <state_interface name="effort" />
+      </joint>
+      <joint name="left_middle_intermediate_joint">
+        <state_interface name="position" />
+        <state_interface name="velocity" />
+        <state_interface name="effort" />
+      </joint>
+      <joint name="left_ring_intermediate_joint">
+        <state_interface name="position" />
+        <state_interface name="velocity" />
+        <state_interface name="effort" />
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