Commit message: harambe walks full robot callibration, controller, demos

File: src/robot_description/dual_arm_description/urdf/macros/ros2_control_real.xacro (robot description, xacro)
@@ -215,5 +215,5 @@
             <!-- WAIST — 1 joint (bus 12)                                       -->
             <!-- ════════════════════════════════════════════════════════════════ -->
-            <joint name="waist_yaw_joint">
+            <joint name="waist_yaw_joint_X8">
                 <command_interface name="position"/>
                 <command_interface name="effort"/>
@@ -233,5 +233,5 @@
             <!-- LEFT LEG — 6 joints (bus 13-18)                                -->
             <!-- ════════════════════════════════════════════════════════════════ -->
-            <joint name="left_hip_pitch_joint">
+            <joint name="left_hip_pitch_joint_X8">
                 <command_interface name="position"/>
                 <command_interface name="effort"/>
@@ -248,5 +248,5 @@
                 </ec_module>
             </joint>
-            <joint name="left_hip_roll_joint">
+            <joint name="left_hip_roll_joint_X8">
                 <command_interface name="position"/>
                 <command_interface name="effort"/>
@@ -263,5 +263,5 @@
                 </ec_module>
             </joint>
-            <joint name="left_hip_yaw_joint">
+            <joint name="left_hip_yaw_joint_X8">
                 <command_interface name="position"/>
                 <command_interface name="effort"/>
@@ -278,5 +278,5 @@
                 </ec_module>
             </joint>
-            <joint name="left_knee_joint">
+            <joint name="left_knee_joint_X8">
                 <command_interface name="position"/>
                 <command_interface name="effort"/>
@@ -293,5 +293,5 @@
                 </ec_module>
             </joint>
-            <joint name="left_ankle_pitch_joint">
+            <joint name="left_ankle_pitch_joint_X4">
                 <command_interface name="position"/>
                 <command_interface name="effort"/>
@@ -308,5 +308,5 @@
                 </ec_module>
             </joint>
-            <joint name="left_ankle_roll_joint">
+            <joint name="left_ankle_roll_joint_X4">
                 <command_interface name="position"/>
                 <command_interface name="effort"/>
@@ -327,5 +327,5 @@
             <!-- NOTE: right_ankle_pitch (bus 24) not connected yet              -->
             <!-- ════════════════════════════════════════════════════════════════ -->
-            <joint name="right_hip_pitch_joint">
+            <joint name="right_hip_pitch_joint_X8">
                 <command_interface name="position"/>
                 <command_interface name="effort"/>
@@ -342,5 +342,5 @@
                 </ec_module>
             </joint>
-            <joint name="right_hip_roll_joint">
+            <joint name="right_hip_roll_joint_X8">
                 <command_interface name="position"/>
                 <command_interface name="effort"/>
@@ -357,5 +357,5 @@
                 </ec_module>
             </joint>
-            <joint name="right_hip_yaw_joint">
+            <joint name="right_hip_yaw_joint_X8">
                 <command_interface name="position"/>
                 <command_interface name="effort"/>
@@ -372,5 +372,5 @@
                 </ec_module>
             </joint>
-            <joint name="right_knee_joint">
+            <joint name="right_knee_joint_X8">
                 <command_interface name="position"/>
                 <command_interface name="effort"/>
@@ -387,5 +387,5 @@
                 </ec_module>
             </joint>
-            <joint name="right_ankle_roll_joint">
+            <joint name="right_ankle_roll_joint_X4">
                 <command_interface name="position"/>
                 <command_interface name="effort"/>
@@ -402,5 +402,5 @@
                 </ec_module>
             </joint>
-            <!-- TODO: Add right_ankle_pitch_joint (bus 24, X4) when actuator arrives -->
+            <!-- TODO: Add right_ankle_pitch_joint_X4 (bus 24) when actuator arrives -->
             </xacro:unless>  <!-- only_arms -->
         </ros2_control>

File: src/robot_description/full_robot_description/urdf/joints/body_joints.xacro (robot description, xacro)
@@ -10,5 +10,5 @@
     <child link="urdf_simplified_torso" />
     <axis xyz="0 0 1" />
-    <limit effort="${X8_moderate_effort}" velocity="${X8_rated_velocity}" lower="-1.57" upper="1.57" />
+    <limit effort="${X8_moderate_effort}" velocity="${X8_rated_velocity}" lower="-2.6005" upper="2.60054" />
     <dynamics damping="${X8_damping}" friction="${X8_friction}" />
   </joint>

File: src/robot_description/full_robot_description/urdf/joints/left_foot_joints.xacro (robot description, xacro)
@@ -6,5 +6,5 @@
     <child link="urdf_hip_assembly" />
     <axis xyz="0 1 0" />
-    <limit effort="${X8_moderate_effort}" velocity="${X8_rated_velocity}" lower="-2.53" upper="1.57" />
+    <limit effort="${X8_moderate_effort}" velocity="${X8_rated_velocity}" lower="-4.4680" upper="1.3265" />
     <dynamics damping="${X8_damping}" friction="${X8_friction}" />
   </joint>
@@ -14,5 +14,5 @@
     <child link="urdf_l_upper_femur_assembly" />
     <axis xyz="1 0 0" />
-    <limit effort="${X8_moderate_effort}" velocity="${X8_rated_velocity}" lower="-0.35" upper="3.14" />
+    <limit effort="${X8_moderate_effort}" velocity="${X8_rated_velocity}" lower="-0.3490" upper="3.31612" />
     <dynamics damping="${X8_damping}" friction="${X8_friction}" />
   </joint>
@@ -22,5 +22,5 @@
     <child link="urdf_lower_femur_assembly" />
     <axis xyz="0 0 1" />
-    <limit effort="${X8_moderate_effort}" velocity="${X8_rated_velocity}" lower="-1.57" upper="1.57" />
+    <limit effort="${X8_moderate_effort}" velocity="${X8_rated_velocity}" lower="-2.2689" upper="3.5256" />
     <dynamics damping="${X8_damping}" friction="${X8_friction}" />
   </joint>
@@ -30,5 +30,5 @@
     <child link="urdf_l_tibia_assembly" />
     <axis xyz="0 1 0" />
-    <limit effort="${X8_moderate_effort}" velocity="${X8_rated_velocity}" lower="-0.17" upper="1.57" />
+    <limit effort="${X8_moderate_effort}" velocity="${X8_rated_velocity}" lower="-1.5271" upper="1.52716" />
     <dynamics damping="${X8_damping}" friction="${X8_friction}" />
   </joint>
@@ -38,5 +38,5 @@
     <child link="urdf_ankle_assembly" />
     <axis xyz="0 1 0" />
-    <limit effort="${ankle_pitch_moderate_effort}" velocity="${ankle_pitch_rated_velocity}" lower="-0.79" upper="0.79" />
+    <limit effort="${ankle_pitch_moderate_effort}" velocity="${ankle_pitch_rated_velocity}" lower="-0.7853" upper="0.78539" />
     <dynamics damping="${X4_damping}" friction="${X4_friction}" />
   </joint>
@@ -46,5 +46,5 @@
     <child link="urdf_foot_assembly" />
     <axis xyz="1 0 0" />
-    <limit effort="${ankle_roll_moderate_effort}" velocity="${ankle_roll_rated_velocity}" lower="-0.79" upper="0.79" />
+    <limit effort="${ankle_roll_moderate_effort}" velocity="${ankle_roll_rated_velocity}" lower="-0.7853" upper="0.78539" />
     <dynamics damping="${X4_damping}" friction="${X4_friction}" />
   </joint>

File: src/robot_description/full_robot_description/urdf/joints/right_foot_joints.xacro (robot description, xacro)
@@ -6,5 +6,5 @@
     <child link="urdf_hip_assembly_2" />
     <axis xyz="0 1 0" />
-    <limit effort="${X8_moderate_effort}" velocity="${X8_rated_velocity}" lower="-2.53" upper="1.57" />
+    <limit effort="${X8_moderate_effort}" velocity="${X8_rated_velocity}" lower="-2.7576" upper="2.75762" />
     <dynamics damping="${X8_damping}" friction="${X8_friction}" />
   </joint>
@@ -14,5 +14,5 @@
     <child link="urdf_r_upper_femur_assemby" />
     <axis xyz="1 0 0" />
-    <limit effort="${X8_moderate_effort}" velocity="${X8_rated_velocity}" lower="-3.14" upper="0.35" />
+    <limit effort="${X8_moderate_effort}" velocity="${X8_rated_velocity}" lower="-3.3161" upper="0.34906" />
     <dynamics damping="${X8_damping}" friction="${X8_friction}" />
   </joint>
@@ -22,5 +22,5 @@
     <child link="urdf_lower_femur_assembly_2" />
     <axis xyz="0 0 1" />
-    <limit effort="${X8_moderate_effort}" velocity="${X8_rated_velocity}" lower="-1.57" upper="1.57" />
+    <limit effort="${X8_moderate_effort}" velocity="${X8_rated_velocity}" lower="-2.7576" upper="2.75762" />
     <dynamics damping="${X8_damping}" friction="${X8_friction}" />
   </joint>
@@ -30,5 +30,5 @@
     <child link="urdf_r_tibia_assembly" />
     <axis xyz="0 1 0" />
-    <limit effort="${X8_moderate_effort}" velocity="${X8_rated_velocity}" lower="-0.17" upper="1.57" />
+    <limit effort="${X8_moderate_effort}" velocity="${X8_rated_velocity}" lower="-1.5271" upper="1.52716" />
     <dynamics damping="${X8_damping}" friction="${X8_friction}" />
   </joint>
@@ -38,5 +38,5 @@
     <child link="urdf_ankle_assembly_2" />
     <axis xyz="0 1 0" />
-    <limit effort="${ankle_pitch_moderate_effort}" velocity="${ankle_pitch_rated_velocity}" lower="-0.79" upper="0.79" />
+    <limit effort="${ankle_pitch_moderate_effort}" velocity="${ankle_pitch_rated_velocity}" lower="-0.7853" upper="0.78539" />
     <dynamics damping="${X4_damping}" friction="${X4_friction}" />
   </joint>
@@ -46,5 +46,5 @@
     <child link="urdf_foot_assembly_2" />
     <axis xyz="1 0 0" />
-    <limit effort="${ankle_roll_moderate_effort}" velocity="${ankle_roll_rated_velocity}" lower="-0.79" upper="0.79" />
+    <limit effort="${ankle_roll_moderate_effort}" velocity="${ankle_roll_rated_velocity}" lower="-0.7853" upper="0.78539" />
     <dynamics damping="${X4_damping}" friction="${X4_friction}" />
   </joint>
