Commit message: pure cosmetic corrections

File: src/robot_description/full_robot_description/harambe_mujoco.urdf (robot description, URDF)
Before this commit: robot robot_harambe_v0.3, 26 links, 25 joints
Links:
- removed link urdf_r_upper_femur_assemby
- added link urdf_r_upper_femur_assembly, mass 1.912; collision mesh filename=meshes/collision/r_upper_femur.stl; visual mesh filename=meshes/visual/r_upper_femur.stl
Joints:
- joint left_knee_joint_X8: limit lower=-0.17 upper=1.57 effort=43 velocity=13.3 -> lower=0 upper=1.51844 effort=43 velocity=13.3
- joint right_hip_roll_joint_X8: child urdf_r_upper_femur_assemby -> urdf_r_upper_femur_assembly
- joint right_hip_yaw_joint_X8: parent urdf_r_upper_femur_assemby -> urdf_r_upper_femur_assembly
- joint right_knee_joint_X8: limit lower=-0.17 upper=1.57 effort=43 velocity=13.3 -> lower=0 upper=1.51844 effort=43 velocity=13.3

File: src/robot_description/full_robot_description/urdf/joints/right_foot_joints.xacro (robot description, xacro)
@@ -15,5 +15,5 @@
     <origin xyz="0.053 -0.062 0" rpy="0 0 0"/>
     <parent link="urdf_hip_assembly_2"/>
-    <child link="urdf_r_upper_femur_assemby"/>
+    <child link="urdf_r_upper_femur_assembly"/>
     <axis xyz="1 0 0"/>
     <limit effort="${X8_moderate_effort}" velocity="${X8_rated_velocity}" lower="-3.22886" upper="0.383972"/>
@@ -22,5 +22,5 @@
   <joint name="right_hip_yaw_joint_X8" type="${leg_joint_type}">
     <origin xyz="-0.053 0 -0.217" rpy="0 0 0"/>
-    <parent link="urdf_r_upper_femur_assemby"/>
+    <parent link="urdf_r_upper_femur_assembly"/>
     <child link="urdf_lower_femur_assembly_2"/>
     <axis xyz="0 0 1"/>
@@ -33,5 +33,5 @@
     <child link="urdf_r_tibia_assembly"/>
     <axis xyz="0 1 0"/>
-    <limit effort="${X8_moderate_effort}" velocity="${X8_rated_velocity}" lower="-1.52716" upper="1.52716"/>
+    <limit effort="${X8_moderate_effort}" velocity="${X8_rated_velocity}" lower="0" upper="1.51844"/>
     <dynamics damping="${X8_damping}" friction="${X8_friction}"/>
   </joint>
@@ -39,5 +39,5 @@
     <origin xyz="0 0.059 -0.395" rpy="0 0 0"/>
     <parent link="urdf_r_tibia_assembly"/>
-    <child link="udrf_ankle_assembly_2"/>
+    <child link="urdf_ankle_assembly_2"/>
     <axis xyz="0 1 0"/>
     <limit effort="${X4_moderate_effort}" velocity="${X4_rated_velocity}" lower="-0.785398" upper="0.785398"/>
@@ -46,5 +46,5 @@
   <joint name="right_ankle_pitch_joint_X4" type="${leg_joint_type}">
     <origin xyz="-0.012 -0.004 -0.028" rpy="0 0 0"/>
-    <parent link="udrf_ankle_assembly_2"/>
+    <parent link="urdf_ankle_assembly_2"/>
     <child link="urdf_foot_assembly_2"/>
     <axis xyz="1 0 0"/>

File: src/robot_description/full_robot_description/urdf/macros/ros2_control_position.xacro (robot description, xacro)
@@ -254,6 +254,6 @@
       <joint name="left_knee_joint_X8">
         <command_interface name="position">
-          <param name="min">-1.52716</param>
-          <param name="max">1.52716</param>
+          <param name="min">0</param>
+          <param name="max">1.51844</param>
         </command_interface>
         <state_interface name="position" />
@@ -309,6 +309,6 @@
       <joint name="right_knee_joint_X8">
         <command_interface name="position">
-          <param name="min">-1.52716</param>
-          <param name="max">1.52716</param>
+          <param name="min">0</param>
+          <param name="max">1.51844</param>
         </command_interface>
         <state_interface name="position" />

File: src/robot_description/full_robot_description/urdf/robot_harambe_v04_fixed_axes_simplified_no_collision.urdf (robot description, URDF)
Before this commit: robot robot_harambe_v04, 26 links, 25 joints
Links:
- removed link udrf_ankle_assembly
- removed link udrf_ankle_assembly_2
- removed link urdf_r_upper_femur_assemby
- added link urdf_ankle_assembly, mass 0.0818219; collision mesh filename=package://meshes/collision/urdf_ankle_assembly.stl; visual mesh filename=package://meshes/visual/urdf_ankle_assembly.stl
- added link urdf_ankle_assembly_2, mass 0.0818219; collision mesh filename=package://meshes/collision/urdf_ankle_assembly.stl; visual mesh filename=package://meshes/visual/urdf_ankle_assembly.stl
- added link urdf_r_upper_femur_assembly, mass 1.912; collision mesh filename=package://meshes/collision/r_upper_femur.stl; visual mesh filename=package://meshes/visual/r_upper_femur.stl
Joints:
- joint left_ankle_pitch_joint_X4: child udrf_ankle_assembly -> urdf_ankle_assembly
- joint left_ankle_roll_joint_X4: parent udrf_ankle_assembly -> urdf_ankle_assembly
- joint left_knee_joint_X8: limit lower=-1.52716 upper=1.52716 effort=10 velocity=10 -> lower=0 upper=1.51844 effort=10 velocity=10
- joint right_ankle_pitch_joint_X4: parent udrf_ankle_assembly_2 -> urdf_ankle_assembly_2
- joint right_ankle_roll_joint_X4: child udrf_ankle_assembly_2 -> urdf_ankle_assembly_2
- joint right_hip_roll_joint_X8: child urdf_r_upper_femur_assemby -> urdf_r_upper_femur_assembly
- joint right_hip_yaw_joint_X8: parent urdf_r_upper_femur_assemby -> urdf_r_upper_femur_assembly
- joint right_knee_joint_X8: limit lower=-1.52716 upper=1.52716 effort=10 velocity=10 -> lower=0 upper=1.51844 effort=10 velocity=10
