Commit message: Refactor EtherCAT configuration and launch files for PVT system - Callibrated joints - Updated YAML configurations for various joints (e.g., left wrist yaw, right ankle pitch) to include offsets for target positions and actual positions. - Modified launch files to improve the setup of the ros2_control node and joint state broadcasters, ensuring proper remapping of topics. - Introduced a new launch file for a read-only viewer of the PVT system, allowing for inspection of joint positions without enabling torque output. - Adjusted the robot description Xacro macro to support dynamic YAML directory paths for both live and read-only configurations. - Updated the PVT dashboard to subscribe to the filtered joint states topic instead of the raw joint states, enhancing data accuracy for monitoring.

File: src/robot_description/full_robot_description/urdf/macros/ros2_control_real_pvt.xacro (robot description, xacro)
@@ -7,7 +7,12 @@
     <!-- drive_temperature, bus_voltage, error_code, status_word). The mode_of_operation -->
     <!-- command interface is NOT exposed in PVT — the firmware locks the PDO to mode 5. -->
+    <!-- Launches override pvt_yaml_dir to point at a sibling directory
+         (e.g. ethercat_pvt_readonly/ generated at build time) so the same
+         xacro macro can drive both live PVT and the read-only viewer.
+         Default = canonical config used by robot_pvt.launch.py. -->
+    <xacro:arg name="pvt_yaml_dir" default="$(find robot_bringup)/config/ethercat_pvt"/>
     <xacro:macro name="dual_arm_ros2_control_real_pvt">
         <xacro:property name="ctrl_freq" value="1000"/>
-        <xacro:property name="pvt_yaml_dir" value="$(find robot_bringup)/config/ethercat_pvt"/>
+        <xacro:property name="pvt_yaml_dir" value="$(arg pvt_yaml_dir)"/>
         <xacro:macro name="ec_pvt_joint" params="name bus_pos slave_file ec_name">
             <joint name="${name}">
