Commit message: Add v2 ankle drivers and associated tests
- Implement HarambeEthercatDriver and HarambePvtDriver for the new cubic kinematics.
- Introduce tests for ankle grid calibration, kinematics, and recording validation against real data.
- Update URDF macros to support driver selection between v1 and v2.
- Add a script to republish joint states in degrees for easier logging and visualization.

File: src/robot_description/full_robot_description/urdf/macros/ros2_control_real.xacro (robot description, xacro)
@@ -14,4 +14,22 @@
             <xacro:property name="config_dir" value="ethercat_gravcomp"/>
         </xacro:if>
+        <!-- Ankle driver selector. v1 (default) = original serial-chain plugin,
+             unchanged. v2 = cubic-primary plugin (fit to the measured grid; the
+             serial-chain method is published on /ankle_method_compare for live
+             comparison only). Only the plugin name + the 4 corrected geometry
+             values differ; ankle_linkage_pairs/signs are shared. -->
+        <xacro:arg name="ankle_driver" default="v1"/>
+        <xacro:property name="ankle_plugin" value="harambe_ankle_ethercat_driver/HarambeEthercatDriver"/>
+        <xacro:property name="ankle_cam_foreaft_mm" value="78.0"/>
+        <xacro:property name="ankle_rod_a_mm" value="255.0"/>
+        <xacro:property name="ankle_rod_b_mm" value="180.0"/>
+        <xacro:property name="ankle_mount_drop_mm" value="0.0"/>
+        <xacro:if value="${'$(arg ankle_driver)' == 'v2'}">
+            <xacro:property name="ankle_plugin" value="harambe_ankle_ethercat_driver_v2/HarambeEthercatDriver"/>
+            <xacro:property name="ankle_cam_foreaft_mm" value="67.5"/>
+            <xacro:property name="ankle_rod_a_mm" value="250.090484"/>
+            <xacro:property name="ankle_rod_b_mm" value="175.129238"/>
+            <xacro:property name="ankle_mount_drop_mm" value="-10.5"/>
+        </xacro:if>
         <!-- EtherCAT actuators (MyActuator RMD X V4) -->
         <!-- only_left=true: 6 DOF left arm only (bus 0-5) -->
@@ -19,17 +37,19 @@
         <ros2_control name="EthercatSystem" type="system">
             <hardware>
-                <plugin>harambe_ankle_ethercat_driver/HarambeEthercatDriver</plugin>
+                <plugin>${ankle_plugin}</plugin>
                 <param name="master_id">0</param>
                 <param name="control_frequency">${ctrl_freq}</param>
-                <!-- Exact differential-ankle serial-chain geometry (mm; ASSUMED docs
-                     placeholders — confirm against the real hardware). -->
+                <!-- Differential-ankle geometry (mm). v1 uses ASSUMED placeholders;
+                     v2 uses the corrected measured values (cam_foreaft/rods/mount_drop
+                     switched by ankle_driver). For v2 these feed only the analytic
+                     comparison — the cubic control path is fit to the grid. -->
                 <param name="crank_throw_mm">25.0</param>
                 <param name="mount_foreaft_mm">63.0</param>
                 <param name="mount_separation_mm">60.0</param>
-                <param name="cam_foreaft_mm">78.0</param>
+                <param name="cam_foreaft_mm">${ankle_cam_foreaft_mm}</param>
                 <param name="hinge_spacing_mm">28.0</param>
-                <param name="rod_a_length_mm">255.0</param>
-                <param name="rod_b_length_mm">180.0</param>
-                <param name="mount_drop_mm">0.0</param>
+                <param name="rod_a_length_mm">${ankle_rod_a_mm}</param>
+                <param name="rod_b_length_mm">${ankle_rod_b_mm}</param>
+                <param name="mount_drop_mm">${ankle_mount_drop_mm}</param>
                 <param name="lock_heights_to_rods">true</param>
                 <param name="motor_limit_deg">80.0</param>  <!-- CONFIRMED real actuator limit -->
@@ -39,5 +59,5 @@
                 <!-- Ankle linkage pairs: pitchJoint,rollJoint — pitch output stored in first, roll in second -->
                 <!-- θA = raw from pitchJoint's motor, θB = raw from rollJoint's motor -->
-                <param name="ankle_linkage_pairs">left_ankle_pitch_joint_X4,left_ankle_roll_joint_X4;right_ankle_pitch_joint_X4,right_ankle_roll_joint_X4</param>
+                <param name="ankle_linkage_pairs">left_ankle_roll_joint_X4,left_ankle_pitch_joint_X4;right_ankle_roll_joint_X4,right_ankle_pitch_joint_X4</param>
             </hardware>
             <!-- ════════════════════════════════════════════════════════════════ -->

File: src/robot_description/full_robot_description/urdf/macros/ros2_control_real_pvt.xacro (robot description, xacro)
@@ -15,4 +15,21 @@
         <xacro:property name="ctrl_freq" value="1000"/>
         <xacro:property name="pvt_yaml_dir" value="$(arg pvt_yaml_dir)"/>
+        <!-- Ankle driver selector (see ros2_control_real.xacro). v1 default = the
+             original serial-chain plugin, unchanged. v2 = cubic-primary plugin with
+             the serial-chain published on /ankle_method_compare. Only the plugin +
+             4 corrected geometry values switch. -->
+        <xacro:arg name="ankle_driver" default="v1"/>
+        <xacro:property name="ankle_plugin" value="harambe_ankle_ethercat_driver/HarambePvtDriver"/>
+        <xacro:property name="ankle_cam_foreaft_mm" value="78.0"/>
+        <xacro:property name="ankle_rod_a_mm" value="255.0"/>
+        <xacro:property name="ankle_rod_b_mm" value="180.0"/>
+        <xacro:property name="ankle_mount_drop_mm" value="0.0"/>
+        <xacro:if value="${'$(arg ankle_driver)' == 'v2'}">
+            <xacro:property name="ankle_plugin" value="harambe_ankle_ethercat_driver_v2/HarambePvtDriver"/>
+            <xacro:property name="ankle_cam_foreaft_mm" value="67.5"/>
+            <xacro:property name="ankle_rod_a_mm" value="250.090484"/>
+            <xacro:property name="ankle_rod_b_mm" value="175.129238"/>
+            <xacro:property name="ankle_mount_drop_mm" value="-10.5"/>
+        </xacro:if>
         <xacro:macro name="ec_pvt_joint" params="name bus_pos slave_file ec_name">
             <joint name="${name}">
@@ -40,17 +57,18 @@
         <ros2_control name="EthercatSystem" type="system">
             <hardware>
-                <plugin>harambe_ankle_ethercat_driver/HarambePvtDriver</plugin>
+                <plugin>${ankle_plugin}</plugin>
                 <param name="master_id">0</param>
                 <param name="control_frequency">${ctrl_freq}</param>
-                <!-- Exact differential-ankle serial-chain geometry (mm; ASSUMED docs
-                     placeholders — confirm against the real hardware). -->
+                <!-- Differential-ankle geometry (mm). v1 = ASSUMED placeholders;
+                     v2 = corrected measured values (switched by ankle_driver; for v2
+                     they feed only the analytic comparison, not the cubic control path). -->
                 <param name="crank_throw_mm">25.0</param>
                 <param name="mount_foreaft_mm">63.0</param>
                 <param name="mount_separation_mm">60.0</param>
-                <param name="cam_foreaft_mm">78.0</param>
+                <param name="cam_foreaft_mm">${ankle_cam_foreaft_mm}</param>
                 <param name="hinge_spacing_mm">28.0</param>
-                <param name="rod_a_length_mm">255.0</param>
-                <param name="rod_b_length_mm">180.0</param>
-                <param name="mount_drop_mm">0.0</param>
+                <param name="rod_a_length_mm">${ankle_rod_a_mm}</param>
+                <param name="rod_b_length_mm">${ankle_rod_b_mm}</param>
+                <param name="mount_drop_mm">${ankle_mount_drop_mm}</param>
                 <param name="lock_heights_to_rods">true</param>
                 <param name="motor_limit_deg">80.0</param>  <!-- CONFIRMED real actuator limit -->
@@ -58,5 +76,5 @@
                 <param name="roll_sign">1</param>
                 <!-- Format is pitchJoint,rollJoint (pitch output stored in the first). -->
-                <param name="ankle_linkage_pairs">left_ankle_pitch_joint_X4,left_ankle_roll_joint_X4;right_ankle_pitch_joint_X4,right_ankle_roll_joint_X4</param>
+                <param name="ankle_linkage_pairs">left_ankle_roll_joint_X4,left_ankle_pitch_joint_X4;right_ankle_roll_joint_X4,right_ankle_pitch_joint_X4</param>
             </hardware>
             <!-- LEFT ARM (bus 0-5) -->

Commit message: feat: Update ankle driver configuration and linkage pairs for improved joint mapping in real and PVT modes

File: src/robot_description/full_robot_description/urdf/macros/ros2_control_real.xacro (robot description, xacro)
@@ -17,6 +17,7 @@
              unchanged. v2 = cubic-primary plugin (fit to the measured grid; the
              serial-chain method is published on /ankle_method_compare for live
-             comparison only). Only the plugin name + the 4 corrected geometry
-             values differ; ankle_linkage_pairs/signs are shared. -->
+             comparison only). v2 also lists the PITCH joint first in
+             ankle_linkage_pairs so the cubic pitch output (small range) lands on
+             the pitch joint and roll (large range) on the roll joint. -->
         <xacro:arg name="ankle_driver" default="v1"/>
         <xacro:property name="ankle_plugin" value="harambe_ankle_ethercat_driver/HarambeEthercatDriver"/>
@@ -25,4 +26,5 @@
         <xacro:property name="ankle_rod_b_mm" value="180.0"/>
         <xacro:property name="ankle_mount_drop_mm" value="0.0"/>
+        <xacro:property name="ankle_pairs" value="left_ankle_roll_joint_X4,left_ankle_pitch_joint_X4;right_ankle_roll_joint_X4,right_ankle_pitch_joint_X4"/>
         <xacro:if value="${'$(arg ankle_driver)' == 'v2'}">
             <xacro:property name="ankle_plugin" value="harambe_ankle_ethercat_driver_v2/HarambeEthercatDriver"/>
@@ -31,4 +33,5 @@
             <xacro:property name="ankle_rod_b_mm" value="175.129238"/>
             <xacro:property name="ankle_mount_drop_mm" value="-10.5"/>
+            <xacro:property name="ankle_pairs" value="left_ankle_pitch_joint_X4,left_ankle_roll_joint_X4;right_ankle_pitch_joint_X4,right_ankle_roll_joint_X4"/>
         </xacro:if>
         <!-- EtherCAT actuators (MyActuator RMD X V4) -->
@@ -58,6 +61,6 @@
                 <param name="roll_sign">1</param>
                 <!-- Ankle linkage pairs: pitchJoint,rollJoint — pitch output stored in first, roll in second -->
-                <!-- θA = raw from pitchJoint's motor, θB = raw from rollJoint's motor -->
-                <param name="ankle_linkage_pairs">left_ankle_roll_joint_X4,left_ankle_pitch_joint_X4;right_ankle_roll_joint_X4,right_ankle_pitch_joint_X4</param>
+                <!-- θA = raw from first joint's motor, θB = raw from second joint's motor -->
+                <param name="ankle_linkage_pairs">${ankle_pairs}</param>
             </hardware>
             <!-- ════════════════════════════════════════════════════════════════ -->

File: src/robot_description/full_robot_description/urdf/macros/ros2_control_real_pvt.xacro (robot description, xacro)
@@ -25,4 +25,5 @@
         <xacro:property name="ankle_rod_b_mm" value="180.0"/>
         <xacro:property name="ankle_mount_drop_mm" value="0.0"/>
+        <xacro:property name="ankle_pairs" value="left_ankle_roll_joint_X4,left_ankle_pitch_joint_X4;right_ankle_roll_joint_X4,right_ankle_pitch_joint_X4"/>
         <xacro:if value="${'$(arg ankle_driver)' == 'v2'}">
             <xacro:property name="ankle_plugin" value="harambe_ankle_ethercat_driver_v2/HarambePvtDriver"/>
@@ -31,4 +32,5 @@
             <xacro:property name="ankle_rod_b_mm" value="175.129238"/>
             <xacro:property name="ankle_mount_drop_mm" value="-10.5"/>
+            <xacro:property name="ankle_pairs" value="left_ankle_pitch_joint_X4,left_ankle_roll_joint_X4;right_ankle_pitch_joint_X4,right_ankle_roll_joint_X4"/>
         </xacro:if>
         <xacro:macro name="ec_pvt_joint" params="name bus_pos slave_file ec_name">
@@ -76,5 +78,5 @@
                 <param name="roll_sign">1</param>
                 <!-- Format is pitchJoint,rollJoint (pitch output stored in the first). -->
-                <param name="ankle_linkage_pairs">left_ankle_roll_joint_X4,left_ankle_pitch_joint_X4;right_ankle_roll_joint_X4,right_ankle_pitch_joint_X4</param>
+                <param name="ankle_linkage_pairs">${ankle_pairs}</param>
             </hardware>
             <!-- LEFT ARM (bus 0-5) -->

Commit message: feat: Update ankle kinematics and calibration for improved accuracy and performance

File: src/robot_description/full_robot_description/urdf/macros/ros2_control_real.xacro (robot description, xacro)
@@ -15,11 +15,15 @@
         </xacro:if>
         <!-- Ankle driver selector. v1 (default) = original serial-chain plugin,
-             unchanged. v2 = cubic-primary plugin (fit to the measured grid; the
-             serial-chain method is published on /ankle_method_compare for live
-             comparison only). v2 also lists the PITCH joint first in
-             ankle_linkage_pairs so the cubic pitch output (small range) lands on
-             the pitch joint and roll (large range) on the roll joint. -->
+             unchanged. v2 = corrected plugin whose PRIMARY control transform is the
+             analytic serial-chain with the MIRROR CRANK (motor B sweeps opposite),
+             calibrated to the measured grid (pitch 0.01 / roll 0.16 deg, exact IK);
+             the cubic fit is published on /ankle_method_compare as the cross-check.
+             v2 lists the PITCH joint first so the small-range pitch output lands on
+             the pitch joint and the large-range roll on the roll joint, and uses the
+             CALIBRATED geometry (differs from v1's hand-measured placeholders). -->
         <xacro:arg name="ankle_driver" default="v1"/>
         <xacro:property name="ankle_plugin" value="harambe_ankle_ethercat_driver/HarambeEthercatDriver"/>
+        <xacro:property name="ankle_mount_foreaft_mm" value="63.0"/>
+        <xacro:property name="ankle_mount_separation_mm" value="60.0"/>
         <xacro:property name="ankle_cam_foreaft_mm" value="78.0"/>
         <xacro:property name="ankle_rod_a_mm" value="255.0"/>
@@ -29,8 +33,10 @@
         <xacro:if value="${'$(arg ankle_driver)' == 'v2'}">
             <xacro:property name="ankle_plugin" value="harambe_ankle_ethercat_driver_v2/HarambeEthercatDriver"/>
-            <xacro:property name="ankle_cam_foreaft_mm" value="67.5"/>
-            <xacro:property name="ankle_rod_a_mm" value="250.090484"/>
-            <xacro:property name="ankle_rod_b_mm" value="175.129238"/>
-            <xacro:property name="ankle_mount_drop_mm" value="-10.5"/>
+            <xacro:property name="ankle_mount_foreaft_mm" value="73.2322"/>
+            <xacro:property name="ankle_mount_separation_mm" value="59.7839"/>
+            <xacro:property name="ankle_cam_foreaft_mm" value="79.9263"/>
+            <xacro:property name="ankle_rod_a_mm" value="229.0121"/>
+            <xacro:property name="ankle_rod_b_mm" value="166.6107"/>
+            <xacro:property name="ankle_mount_drop_mm" value="-10.2996"/>
             <xacro:property name="ankle_pairs" value="left_ankle_pitch_joint_X4,left_ankle_roll_joint_X4;right_ankle_pitch_joint_X4,right_ankle_roll_joint_X4"/>
         </xacro:if>
@@ -43,11 +49,11 @@
                 <param name="master_id">0</param>
                 <param name="control_frequency">${ctrl_freq}</param>
-                <!-- Differential-ankle geometry (mm). v1 uses ASSUMED placeholders;
-                     v2 uses the corrected measured values (cam_foreaft/rods/mount_drop
-                     switched by ankle_driver). For v2 these feed only the analytic
-                     comparison — the cubic control path is fit to the grid. -->
+                <!-- Differential-ankle geometry (mm). v1 = ASSUMED placeholders;
+                     v2 = CALIBRATED values that fit the analytic mirror-crank model
+                     to the grid (this is v2's PRIMARY control path). crank_throw and
+                     hinge_spacing are shared (held at measured during the fit). -->
                 <param name="crank_throw_mm">25.0</param>
-                <param name="mount_foreaft_mm">63.0</param>
-                <param name="mount_separation_mm">60.0</param>
+                <param name="mount_foreaft_mm">${ankle_mount_foreaft_mm}</param>
+                <param name="mount_separation_mm">${ankle_mount_separation_mm}</param>
                 <param name="cam_foreaft_mm">${ankle_cam_foreaft_mm}</param>
                 <param name="hinge_spacing_mm">28.0</param>

File: src/robot_description/full_robot_description/urdf/macros/ros2_control_real_pvt.xacro (robot description, xacro)
@@ -16,9 +16,12 @@
         <xacro:property name="pvt_yaml_dir" value="$(arg pvt_yaml_dir)"/>
         <!-- Ankle driver selector (see ros2_control_real.xacro). v1 default = the
-             original serial-chain plugin, unchanged. v2 = cubic-primary plugin with
-             the serial-chain published on /ankle_method_compare. Only the plugin +
-             4 corrected geometry values switch. -->
+             original serial-chain plugin, unchanged. v2 PRIMARY = analytic mirror-
+             crank model, calibrated to the grid (exact IK, physical Jacobian); the
+             cubic is published on /ankle_method_compare. Switches the plugin, the
+             pitch-first pairing, and the CALIBRATED geometry. -->
         <xacro:arg name="ankle_driver" default="v1"/>
         <xacro:property name="ankle_plugin" value="harambe_ankle_ethercat_driver/HarambePvtDriver"/>
+        <xacro:property name="ankle_mount_foreaft_mm" value="63.0"/>
+        <xacro:property name="ankle_mount_separation_mm" value="60.0"/>
         <xacro:property name="ankle_cam_foreaft_mm" value="78.0"/>
         <xacro:property name="ankle_rod_a_mm" value="255.0"/>
@@ -28,8 +31,10 @@
         <xacro:if value="${'$(arg ankle_driver)' == 'v2'}">
             <xacro:property name="ankle_plugin" value="harambe_ankle_ethercat_driver_v2/HarambePvtDriver"/>
-            <xacro:property name="ankle_cam_foreaft_mm" value="67.5"/>
-            <xacro:property name="ankle_rod_a_mm" value="250.090484"/>
-            <xacro:property name="ankle_rod_b_mm" value="175.129238"/>
-            <xacro:property name="ankle_mount_drop_mm" value="-10.5"/>
+            <xacro:property name="ankle_mount_foreaft_mm" value="73.2322"/>
+            <xacro:property name="ankle_mount_separation_mm" value="59.7839"/>
+            <xacro:property name="ankle_cam_foreaft_mm" value="79.9263"/>
+            <xacro:property name="ankle_rod_a_mm" value="229.0121"/>
+            <xacro:property name="ankle_rod_b_mm" value="166.6107"/>
+            <xacro:property name="ankle_mount_drop_mm" value="-10.2996"/>
             <xacro:property name="ankle_pairs" value="left_ankle_pitch_joint_X4,left_ankle_roll_joint_X4;right_ankle_pitch_joint_X4,right_ankle_roll_joint_X4"/>
         </xacro:if>
@@ -66,6 +71,6 @@
                      they feed only the analytic comparison, not the cubic control path). -->
                 <param name="crank_throw_mm">25.0</param>
-                <param name="mount_foreaft_mm">63.0</param>
-                <param name="mount_separation_mm">60.0</param>
+                <param name="mount_foreaft_mm">${ankle_mount_foreaft_mm}</param>
+                <param name="mount_separation_mm">${ankle_mount_separation_mm}</param>
                 <param name="cam_foreaft_mm">${ankle_cam_foreaft_mm}</param>
                 <param name="hinge_spacing_mm">28.0</param>
