Commit message: add friction for fingers

File: src/robot_description/hand_description/urdf/hands/inspire_hand_left.xacro (robot description, xacro)
@@ -155,4 +155,5 @@
       <axis xyz="0 0 -1"/>
       <limit lower="0" upper="0.8" effort="1" velocity="0.5"/>
+      <dynamics damping="0.05" friction="0.01"/>
       <mimic joint="${prefix}thumb_proximal_pitch_joint" multiplier="1.334" offset="0"/>
     </joint>
@@ -183,4 +184,5 @@
       <axis xyz="0 0 -1"/>
       <limit lower="0" upper="0.4" effort="1" velocity="0.5"/>
+      <dynamics damping="0.05" friction="0.01"/>
       <mimic joint="${prefix}thumb_proximal_pitch_joint" multiplier="0.667" offset="0"/>
     </joint>
@@ -239,4 +241,5 @@
       <axis xyz="0 0 -1"/>
       <limit lower="-0.04545" upper="1.56" effort="1" velocity="0.5"/>
+      <dynamics damping="0.05" friction="0.01"/>
       <mimic joint="${prefix}index_proximal_joint" multiplier="1.06399" offset="-0.04545"/>
     </joint>
@@ -295,4 +298,5 @@
       <axis xyz="0 0 -1"/>
       <limit lower="-0.04545" upper="1.56" effort="1" velocity="0.5"/>
+      <dynamics damping="0.05" friction="0.01"/>
       <mimic joint="${prefix}middle_proximal_joint" multiplier="1.06399" offset="-0.04545"/>
     </joint>
@@ -351,4 +355,5 @@
       <axis xyz="0 0 -1"/>
       <limit lower="-0.04545" upper="1.56" effort="1" velocity="0.5"/>
+      <dynamics damping="0.05" friction="0.01"/>
       <mimic joint="${prefix}ring_proximal_joint" multiplier="1.06399" offset="-0.04545"/>
     </joint>
@@ -407,4 +412,5 @@
       <axis xyz="0 0 -1"/>
       <limit lower="-0.04545" upper="1.56" effort="1" velocity="0.5"/>
+      <dynamics damping="0.05" friction="0.01"/>
       <mimic joint="${prefix}pinky_proximal_joint" multiplier="1.06399" offset="-0.04545"/>
     </joint>

File: src/robot_description/hand_description/urdf/hands/inspire_hand_right.xacro (robot description, xacro)
@@ -147,4 +147,5 @@
         <axis xyz="0 0 1"/>
         <limit lower="0" upper="0.8" effort="1" velocity="0.5"/>
+        <dynamics damping="0.05" friction="0.01"/>
         <mimic joint="${prefix}thumb_proximal_pitch_joint" multiplier="1.334" offset="0"/>
       </joint>
@@ -174,4 +175,5 @@
         <axis xyz="0 0 1"/>
         <limit lower="0" upper="0.4" effort="1" velocity="0.5"/>
+        <dynamics damping="0.05" friction="0.01"/>
         <mimic joint="${prefix}thumb_proximal_pitch_joint" multiplier="0.667" offset="0"/>
       </joint>
@@ -227,4 +229,5 @@
         <axis xyz="0 0 1"/>
         <limit lower="-0.04545" upper="1.56" effort="1" velocity="0.5"/>
+        <dynamics damping="0.05" friction="0.01"/>
         <mimic joint="${prefix}index_proximal_joint" multiplier="1.06399" offset="-0.04545"/>
       </joint>
@@ -280,4 +283,5 @@
         <axis xyz="0 0 1"/>
         <limit lower="-0.04545" upper="1.56" effort="1" velocity="0.5"/>
+        <dynamics damping="0.05" friction="0.01"/>
         <mimic joint="${prefix}middle_proximal_joint" multiplier="1.06399" offset="-0.04545"/>
       </joint>
@@ -333,4 +337,5 @@
         <axis xyz="0 0 1"/>
         <limit lower="-0.04545" upper="1.56" effort="1" velocity="0.5"/>
+        <dynamics damping="0.05" friction="0.01"/>
         <mimic joint="${prefix}ring_proximal_joint" multiplier="1.06399" offset="-0.04545"/>
       </joint>
@@ -386,4 +391,5 @@
         <axis xyz="0 0 1"/>
         <limit lower="-0.04545" upper="1.56" effort="1" velocity="0.5"/>
+        <dynamics damping="0.05" friction="0.01"/>
         <mimic joint="${prefix}pinky_proximal_joint" multiplier="1.06399" offset="-0.04545"/>
       </joint>

Commit message: damping for fingers

File: src/robot_description/hand_description/urdf/hands/inspire_hand_left.xacro (robot description, xacro)
@@ -101,4 +101,5 @@
       <axis xyz="0 0 1"/>
       <limit lower="0" upper="1.31" effort="1" velocity="0.5"/>
+      <dynamics damping="0.3" friction="0.05"/>
     </joint>
     <link name="${prefix}thumb_proximal">
@@ -128,4 +129,5 @@
       <axis xyz="0 0 -1"/>
       <limit lower="0" upper="0.61" effort="1" velocity="0.5"/>
+      <dynamics damping="0.3" friction="0.05"/>
     </joint>
     <link name="${prefix}thumb_intermediate">
@@ -155,5 +157,5 @@
       <axis xyz="0 0 -1"/>
       <limit lower="0" upper="0.8" effort="1" velocity="0.5"/>
-      <dynamics damping="0.05" friction="0.01"/>
+      <dynamics damping="0.3" friction="0.05"/>
       <mimic joint="${prefix}thumb_proximal_pitch_joint" multiplier="1.334" offset="0"/>
     </joint>
@@ -184,5 +186,5 @@
       <axis xyz="0 0 -1"/>
       <limit lower="0" upper="0.4" effort="1" velocity="0.5"/>
-      <dynamics damping="0.05" friction="0.01"/>
+      <dynamics damping="0.3" friction="0.05"/>
       <mimic joint="${prefix}thumb_proximal_pitch_joint" multiplier="0.667" offset="0"/>
     </joint>
@@ -214,4 +216,5 @@
       <axis xyz="0 0 -1"/>
       <limit lower="0" upper="1.47" effort="1" velocity="0.5"/>
+      <dynamics damping="0.3" friction="0.05"/>
     </joint>
     <link name="${prefix}index_intermediate">
@@ -241,5 +244,5 @@
       <axis xyz="0 0 -1"/>
       <limit lower="-0.04545" upper="1.56" effort="1" velocity="0.5"/>
-      <dynamics damping="0.05" friction="0.01"/>
+      <dynamics damping="0.3" friction="0.05"/>
       <mimic joint="${prefix}index_proximal_joint" multiplier="1.06399" offset="-0.04545"/>
     </joint>
@@ -271,4 +274,5 @@
       <axis xyz="0 0 -1"/>
       <limit lower="0" upper="1.47" effort="1" velocity="0.5"/>
+      <dynamics damping="0.3" friction="0.05"/>
     </joint>
     <link name="${prefix}middle_intermediate">
@@ -298,5 +302,5 @@
       <axis xyz="0 0 -1"/>
       <limit lower="-0.04545" upper="1.56" effort="1" velocity="0.5"/>
-      <dynamics damping="0.05" friction="0.01"/>
+      <dynamics damping="0.3" friction="0.05"/>
       <mimic joint="${prefix}middle_proximal_joint" multiplier="1.06399" offset="-0.04545"/>
     </joint>
@@ -328,4 +332,5 @@
       <axis xyz="0 0 -1"/>
       <limit lower="0" upper="1.47" effort="1" velocity="0.5"/>
+      <dynamics damping="0.3" friction="0.05"/>
     </joint>
     <link name="${prefix}ring_intermediate">
@@ -355,5 +360,5 @@
       <axis xyz="0 0 -1"/>
       <limit lower="-0.04545" upper="1.56" effort="1" velocity="0.5"/>
-      <dynamics damping="0.05" friction="0.01"/>
+      <dynamics damping="0.3" friction="0.05"/>
       <mimic joint="${prefix}ring_proximal_joint" multiplier="1.06399" offset="-0.04545"/>
     </joint>
@@ -385,4 +390,5 @@
       <axis xyz="0 0 -1"/>
       <limit lower="0" upper="1.47" effort="1" velocity="0.5"/>
+      <dynamics damping="0.3" friction="0.05"/>
     </joint>
     <link name="${prefix}pinky_intermediate">
@@ -412,5 +418,5 @@
       <axis xyz="0 0 -1"/>
       <limit lower="-0.04545" upper="1.56" effort="1" velocity="0.5"/>
-      <dynamics damping="0.05" friction="0.01"/>
+      <dynamics damping="0.3" friction="0.05"/>
       <mimic joint="${prefix}pinky_proximal_joint" multiplier="1.06399" offset="-0.04545"/>
     </joint>

File: src/robot_description/hand_description/urdf/hands/inspire_hand_right.xacro (robot description, xacro)
@@ -95,4 +95,5 @@
         <axis xyz="0 0 -1"/>
         <limit lower="0.0" upper="1.308" effort="1" velocity="0.5"/>
+        <dynamics damping="0.3" friction="0.05"/>
       </joint>
       <link name="${prefix}thumb_proximal">
@@ -121,4 +122,5 @@
         <axis xyz="0 0 1"/>
         <limit lower="0" upper="0.6" effort="1" velocity="0.5"/>
+        <dynamics damping="0.3" friction="0.05"/>
       </joint>
       <link name="${prefix}thumb_intermediate">
@@ -147,5 +149,5 @@
         <axis xyz="0 0 1"/>
         <limit lower="0" upper="0.8" effort="1" velocity="0.5"/>
-        <dynamics damping="0.05" friction="0.01"/>
+        <dynamics damping="0.3" friction="0.05"/>
         <mimic joint="${prefix}thumb_proximal_pitch_joint" multiplier="1.334" offset="0"/>
       </joint>
@@ -175,5 +177,5 @@
         <axis xyz="0 0 1"/>
         <limit lower="0" upper="0.4" effort="1" velocity="0.5"/>
-        <dynamics damping="0.05" friction="0.01"/>
+        <dynamics damping="0.3" friction="0.05"/>
         <mimic joint="${prefix}thumb_proximal_pitch_joint" multiplier="0.667" offset="0"/>
       </joint>
@@ -203,4 +205,5 @@
         <axis xyz="0 0 1"/>
         <limit lower="0" upper="1.47" effort="1" velocity="0.5"/>
+        <dynamics damping="0.3" friction="0.05"/>
       </joint>
       <link name="${prefix}index_intermediate">
@@ -229,5 +232,5 @@
         <axis xyz="0 0 1"/>
         <limit lower="-0.04545" upper="1.56" effort="1" velocity="0.5"/>
-        <dynamics damping="0.05" friction="0.01"/>
+        <dynamics damping="0.3" friction="0.05"/>
         <mimic joint="${prefix}index_proximal_joint" multiplier="1.06399" offset="-0.04545"/>
       </joint>
@@ -257,4 +260,5 @@
         <axis xyz="0 0 1"/>
         <limit lower="0" upper="1.47" effort="1" velocity="0.5"/>
+        <dynamics damping="0.3" friction="0.05"/>
       </joint>
       <link name="${prefix}middle_intermediate">
@@ -283,5 +287,5 @@
         <axis xyz="0 0 1"/>
         <limit lower="-0.04545" upper="1.56" effort="1" velocity="0.5"/>
-        <dynamics damping="0.05" friction="0.01"/>
+        <dynamics damping="0.3" friction="0.05"/>
         <mimic joint="${prefix}middle_proximal_joint" multiplier="1.06399" offset="-0.04545"/>
       </joint>
@@ -311,4 +315,5 @@
         <axis xyz="0 0 1"/>
         <limit lower="0" upper="1.47" effort="1" velocity="0.5"/>
+        <dynamics damping="0.3" friction="0.05"/>
       </joint>
       <link name="${prefix}ring_intermediate">
@@ -337,5 +342,5 @@
         <axis xyz="0 0 1"/>
         <limit lower="-0.04545" upper="1.56" effort="1" velocity="0.5"/>
-        <dynamics damping="0.05" friction="0.01"/>
+        <dynamics damping="0.3" friction="0.05"/>
         <mimic joint="${prefix}ring_proximal_joint" multiplier="1.06399" offset="-0.04545"/>
       </joint>
@@ -365,4 +370,5 @@
         <axis xyz="0 0 1"/>
         <limit lower="0" upper="1.47" effort="1" velocity="0.5"/>
+        <dynamics damping="0.3" friction="0.05"/>
       </joint>
       <link name="${prefix}pinky_intermediate">
@@ -391,5 +397,5 @@
         <axis xyz="0 0 1"/>
         <limit lower="-0.04545" upper="1.56" effort="1" velocity="0.5"/>
-        <dynamics damping="0.05" friction="0.01"/>
+        <dynamics damping="0.3" friction="0.05"/>
         <mimic joint="${prefix}pinky_proximal_joint" multiplier="1.06399" offset="-0.04545"/>
       </joint>

Commit message: recording and gravcomp changes for dual arms, hand mass correction, motions

File: src/robot_description/hand_description/urdf/hands/inspire_hand_left.xacro (robot description, xacro)
@@ -16,5 +16,5 @@
       <inertial>
         <origin xyz="-0.0025264 -0.066047 -0.0019598" rpy="0 0 0"/>
-        <mass value="0.14143"/>
+        <mass value="0.52560"/>
         <inertia ixx="0.00012281" ixy="2.1711E-06" ixz="1.7709E-06" iyy="8.3832E-05" iyz="-1.6551E-06" izz="7.6663E-05"/>
       </inertial>

File: src/robot_description/hand_description/urdf/hands/inspire_hand_right.xacro (robot description, xacro)
@@ -12,5 +12,5 @@
         <inertial>
           <origin xyz="-0.0025264 -0.066047 0.0019598" rpy="0 0 0"/>
-          <mass value="0.14143"/>
+          <mass value="0.52560"/>
           <inertia ixx="0.00012281" ixy="2.1711E-06" ixz="1.7709E-06" iyy="8.3832E-05" iyz="-1.6551E-06" izz="7.6663E-05"/>
         </inertial>

Commit message: feat(arm_mtc): pick-and-place plans and executes end-to-end (inspire hand)
Full MTC cylinder pipeline now plans (pick → lift → place → home) and
executes in sim. Grasp isn't perfectly aligned on the object yet, but the
whole sequence runs — intermediate milestone.

- Switch KDL → TRAC-IK; load robot_description_kinematics in all MTC launches
- Inspire hand as EEF with TCP frame (left/right_tcp_link); grasp/place use TCP
- Fix grasp/place orientation (RotY(pi)*RotX(pi - tilt)), shared tilt
- Place sweeps yaw angles like pick (Alternatives + exposeTo/configureInitFrom)
- Root-cause place fix: re-allow object↔table after attach (world allowance
  doesn't carry to the attached object); place IK monitors that stage
- allowed_start_tolerance=0.0 so MTC stitched trajectories aren't rejected

File: src/robot_description/hand_description/urdf/hands/inspire_hand_left.xacro (robot description, xacro)
@@ -452,4 +452,14 @@
       <child link="${prefix}pinky_tip"/>
     </joint>
+    <!-- ========== GRASP / TCP FRAME (fixed) ========== -->
+    <!-- Tool-center-point: MTC ik_frame / grasp frame.
+         +Y points toward the fingertips = approach/grasp direction.
+         Origin is a starting grasp point in the palm; tune depth (xyz) visually in RViz. -->
+    <link name="${prefix}tcp_link"/>
+    <joint name="${prefix}tcp_joint" type="fixed">
+      <origin xyz="-0.02 -0.11 0.0" rpy="0 0 3.14159"/>
+      <parent link="${prefix}hand_base_link"/>
+      <child link="${prefix}tcp_link"/>
+    </joint>
   </xacro:macro>
 </robot>

File: src/robot_description/hand_description/urdf/hands/inspire_hand_right.xacro (robot description, xacro)
@@ -430,4 +430,13 @@
         <child link="${prefix}pinky_tip"/>
       </joint>
+      <!-- ========== GRASP / TCP FRAME (fixed) ========== -->
+      <!-- Tool-center-point: MTC ik_frame / grasp frame.
+           +Y points toward the fingertips = approach/grasp direction. -->
+      <link name="${prefix}tcp_link"/>
+      <joint name="${prefix}tcp_joint" type="fixed">
+        <origin xyz="-0.02 -0.11 0.0" rpy="0 0 3.14159"/>
+        <parent link="${prefix}hand_base_link"/>
+        <child link="${prefix}tcp_link"/>
+      </joint>
   </xacro:macro>
 </robot>

Commit message: velocity hand review

File: src/robot_description/hand_description/urdf/hands/inspire_hand_left.xacro (robot description, xacro)
@@ -100,5 +100,5 @@
       <child link="${prefix}thumb_proximal_base"/>
       <axis xyz="0 0 1"/>
-      <limit lower="0" upper="1.31" effort="1" velocity="0.5"/>
+      <limit lower="0" upper="1.31" effort="8" velocity="2.0"/>
       <dynamics damping="0.3" friction="0.05"/>
     </joint>
@@ -128,5 +128,5 @@
       <child link="${prefix}thumb_proximal"/>
       <axis xyz="0 0 -1"/>
-      <limit lower="0" upper="0.61" effort="1" velocity="0.5"/>
+      <limit lower="0" upper="0.61" effort="8" velocity="2.0"/>
       <dynamics damping="0.3" friction="0.05"/>
     </joint>
@@ -156,5 +156,5 @@
       <child link="${prefix}thumb_intermediate"/>
       <axis xyz="0 0 -1"/>
-      <limit lower="0" upper="0.8" effort="1" velocity="0.5"/>
+      <limit lower="0" upper="0.8" effort="8" velocity="2.0"/>
       <dynamics damping="0.3" friction="0.05"/>
       <mimic joint="${prefix}thumb_proximal_pitch_joint" multiplier="1.334" offset="0"/>
@@ -185,5 +185,5 @@
       <child link="${prefix}thumb_distal"/>
       <axis xyz="0 0 -1"/>
-      <limit lower="0" upper="0.4" effort="1" velocity="0.5"/>
+      <limit lower="0" upper="0.4" effort="8" velocity="2.0"/>
       <dynamics damping="0.3" friction="0.05"/>
       <mimic joint="${prefix}thumb_proximal_pitch_joint" multiplier="0.667" offset="0"/>
@@ -215,5 +215,5 @@
       <child link="${prefix}index_proximal"/>
       <axis xyz="0 0 -1"/>
-      <limit lower="0" upper="1.47" effort="1" velocity="0.5"/>
+      <limit lower="0" upper="1.47" effort="8" velocity="2.0"/>
       <dynamics damping="0.3" friction="0.05"/>
     </joint>
@@ -243,5 +243,5 @@
       <child link="${prefix}index_intermediate"/>
       <axis xyz="0 0 -1"/>
-      <limit lower="-0.04545" upper="1.56" effort="1" velocity="0.5"/>
+      <limit lower="-0.04545" upper="1.56" effort="8" velocity="2.0"/>
       <dynamics damping="0.3" friction="0.05"/>
       <mimic joint="${prefix}index_proximal_joint" multiplier="1.06399" offset="-0.04545"/>
@@ -273,5 +273,5 @@
       <child link="${prefix}middle_proximal"/>
       <axis xyz="0 0 -1"/>
-      <limit lower="0" upper="1.47" effort="1" velocity="0.5"/>
+      <limit lower="0" upper="1.47" effort="8" velocity="2.0"/>
       <dynamics damping="0.3" friction="0.05"/>
     </joint>
@@ -301,5 +301,5 @@
       <child link="${prefix}middle_intermediate"/>
       <axis xyz="0 0 -1"/>
-      <limit lower="-0.04545" upper="1.56" effort="1" velocity="0.5"/>
+      <limit lower="-0.04545" upper="1.56" effort="8" velocity="2.0"/>
       <dynamics damping="0.3" friction="0.05"/>
       <mimic joint="${prefix}middle_proximal_joint" multiplier="1.06399" offset="-0.04545"/>
@@ -331,5 +331,5 @@
       <child link="${prefix}ring_proximal"/>
       <axis xyz="0 0 -1"/>
-      <limit lower="0" upper="1.47" effort="1" velocity="0.5"/>
+      <limit lower="0" upper="1.47" effort="8" velocity="2.0"/>
       <dynamics damping="0.3" friction="0.05"/>
     </joint>
@@ -359,5 +359,5 @@
       <child link="${prefix}ring_intermediate"/>
       <axis xyz="0 0 -1"/>
-      <limit lower="-0.04545" upper="1.56" effort="1" velocity="0.5"/>
+      <limit lower="-0.04545" upper="1.56" effort="8" velocity="2.0"/>
       <dynamics damping="0.3" friction="0.05"/>
       <mimic joint="${prefix}ring_proximal_joint" multiplier="1.06399" offset="-0.04545"/>
@@ -389,5 +389,5 @@
       <child link="${prefix}pinky_proximal"/>
       <axis xyz="0 0 -1"/>
-      <limit lower="0" upper="1.47" effort="1" velocity="0.5"/>
+      <limit lower="0" upper="1.47" effort="8" velocity="2.0"/>
       <dynamics damping="0.3" friction="0.05"/>
     </joint>
@@ -417,5 +417,5 @@
       <child link="${prefix}pinky_intermediate"/>
       <axis xyz="0 0 -1"/>
-      <limit lower="-0.04545" upper="1.56" effort="1" velocity="0.5"/>
+      <limit lower="-0.04545" upper="1.56" effort="8" velocity="2.0"/>
       <dynamics damping="0.3" friction="0.05"/>
       <mimic joint="${prefix}pinky_proximal_joint" multiplier="1.06399" offset="-0.04545"/>

File: src/robot_description/hand_description/urdf/hands/inspire_hand_right.xacro (robot description, xacro)
@@ -94,5 +94,5 @@
         <child link="${prefix}thumb_proximal_base"/>
         <axis xyz="0 0 -1"/>
-        <limit lower="0.0" upper="1.308" effort="1" velocity="0.5"/>
+        <limit lower="0.0" upper="1.308" effort="1" velocity="2.0"/>
         <dynamics damping="0.3" friction="0.05"/>
       </joint>
@@ -121,5 +121,5 @@
         <child link="${prefix}thumb_proximal"/>
         <axis xyz="0 0 1"/>
-        <limit lower="0" upper="0.6" effort="1" velocity="0.5"/>
+        <limit lower="0" upper="0.6" effort="1" velocity="2.0"/>
         <dynamics damping="0.3" friction="0.05"/>
       </joint>
@@ -148,5 +148,5 @@
         <child link="${prefix}thumb_intermediate"/>
         <axis xyz="0 0 1"/>
-        <limit lower="0" upper="0.8" effort="1" velocity="0.5"/>
+        <limit lower="0" upper="0.8" effort="1" velocity="2.0"/>
         <dynamics damping="0.3" friction="0.05"/>
         <mimic joint="${prefix}thumb_proximal_pitch_joint" multiplier="1.334" offset="0"/>
@@ -176,5 +176,5 @@
         <child link="${prefix}thumb_distal"/>
         <axis xyz="0 0 1"/>
-        <limit lower="0" upper="0.4" effort="1" velocity="0.5"/>
+        <limit lower="0" upper="0.4" effort="1" velocity="2.0"/>
         <dynamics damping="0.3" friction="0.05"/>
         <mimic joint="${prefix}thumb_proximal_pitch_joint" multiplier="0.667" offset="0"/>
@@ -204,5 +204,5 @@
         <child link="${prefix}index_proximal"/>
         <axis xyz="0 0 1"/>
-        <limit lower="0" upper="1.47" effort="1" velocity="0.5"/>
+        <limit lower="0" upper="1.47" effort="1" velocity="2.0"/>
         <dynamics damping="0.3" friction="0.05"/>
       </joint>
@@ -231,5 +231,5 @@
         <child link="${prefix}index_intermediate"/>
         <axis xyz="0 0 1"/>
-        <limit lower="-0.04545" upper="1.56" effort="1" velocity="0.5"/>
+        <limit lower="-0.04545" upper="1.56" effort="1" velocity="2.0"/>
         <dynamics damping="0.3" friction="0.05"/>
         <mimic joint="${prefix}index_proximal_joint" multiplier="1.06399" offset="-0.04545"/>
@@ -259,5 +259,5 @@
         <child link="${prefix}middle_proximal"/>
         <axis xyz="0 0 1"/>
-        <limit lower="0" upper="1.47" effort="1" velocity="0.5"/>
+        <limit lower="0" upper="1.47" effort="1" velocity="2.0"/>
         <dynamics damping="0.3" friction="0.05"/>
       </joint>
@@ -286,5 +286,5 @@
         <child link="${prefix}middle_intermediate"/>
         <axis xyz="0 0 1"/>
-        <limit lower="-0.04545" upper="1.56" effort="1" velocity="0.5"/>
+        <limit lower="-0.04545" upper="1.56" effort="1" velocity="2.0"/>
         <dynamics damping="0.3" friction="0.05"/>
         <mimic joint="${prefix}middle_proximal_joint" multiplier="1.06399" offset="-0.04545"/>
@@ -314,5 +314,5 @@
         <child link="${prefix}ring_proximal"/>
         <axis xyz="0 0 1"/>
-        <limit lower="0" upper="1.47" effort="1" velocity="0.5"/>
+        <limit lower="0" upper="1.47" effort="1" velocity="2.0"/>
         <dynamics damping="0.3" friction="0.05"/>
       </joint>
@@ -341,5 +341,5 @@
         <child link="${prefix}ring_intermediate"/>
         <axis xyz="0 0 1"/>
-        <limit lower="-0.04545" upper="1.56" effort="1" velocity="0.5"/>
+        <limit lower="-0.04545" upper="1.56" effort="1" velocity="2.0"/>
         <dynamics damping="0.3" friction="0.05"/>
         <mimic joint="${prefix}ring_proximal_joint" multiplier="1.06399" offset="-0.04545"/>
@@ -369,5 +369,5 @@
         <child link="${prefix}pinky_proximal"/>
         <axis xyz="0 0 1"/>
-        <limit lower="0" upper="1.47" effort="1" velocity="0.5"/>
+        <limit lower="0" upper="1.47" effort="1" velocity="2.0"/>
         <dynamics damping="0.3" friction="0.05"/>
       </joint>
@@ -396,5 +396,5 @@
         <child link="${prefix}pinky_intermediate"/>
         <axis xyz="0 0 1"/>
-        <limit lower="-0.04545" upper="1.56" effort="1" velocity="0.5"/>
+        <limit lower="-0.04545" upper="1.56" effort="1" velocity="2.0"/>
         <dynamics damping="0.3" friction="0.05"/>
         <mimic joint="${prefix}pinky_proximal_joint" multiplier="1.06399" offset="-0.04545"/>
