Commit message: fix(hand_description): tune joint damping and friction
Reduce damping and friction for active and mimic joints on both Inspire
hands to prevent delayed, uneven finger motion when the palms are tilted.

File: src/robot_description/hand_description/urdf/hands/inspire_hand_left.xacro (robot description, xacro)
@@ -101,5 +101,5 @@
       <axis xyz="0 0 1"/>
       <limit lower="0" upper="1.31" effort="8" velocity="2.0"/>
-      <dynamics damping="0.3" friction="0.05"/>
+      <dynamics damping="0.005" friction="0.0001"/>
     </joint>
     <link name="${prefix}thumb_proximal">
@@ -129,5 +129,5 @@
       <axis xyz="0 0 -1"/>
       <limit lower="0" upper="0.61" effort="8" velocity="2.0"/>
-      <dynamics damping="0.3" friction="0.05"/>
+      <dynamics damping="0.005" friction="0.0001"/>
     </joint>
     <link name="${prefix}thumb_intermediate">
@@ -157,5 +157,5 @@
       <axis xyz="0 0 -1"/>
       <limit lower="0" upper="0.8" effort="8" velocity="2.0"/>
-      <dynamics damping="0.3" friction="0.05"/>
+      <dynamics damping="0.002" friction="0.00005"/>
       <mimic joint="${prefix}thumb_proximal_pitch_joint" multiplier="1.334" offset="0"/>
     </joint>
@@ -186,5 +186,5 @@
       <axis xyz="0 0 -1"/>
       <limit lower="0" upper="0.4" effort="8" velocity="2.0"/>
-      <dynamics damping="0.3" friction="0.05"/>
+      <dynamics damping="0.002" friction="0.00005"/>
       <mimic joint="${prefix}thumb_proximal_pitch_joint" multiplier="0.667" offset="0"/>
     </joint>
@@ -216,5 +216,5 @@
       <axis xyz="0 0 -1"/>
       <limit lower="0" upper="1.47" effort="8" velocity="2.0"/>
-      <dynamics damping="0.3" friction="0.05"/>
+      <dynamics damping="0.005" friction="0.0001"/>
     </joint>
     <link name="${prefix}index_intermediate">
@@ -244,5 +244,5 @@
       <axis xyz="0 0 -1"/>
       <limit lower="-0.04545" upper="1.56" effort="8" velocity="2.0"/>
-      <dynamics damping="0.3" friction="0.05"/>
+      <dynamics damping="0.002" friction="0.00005"/>
       <mimic joint="${prefix}index_proximal_joint" multiplier="1.06399" offset="-0.04545"/>
     </joint>
@@ -274,5 +274,5 @@
       <axis xyz="0 0 -1"/>
       <limit lower="0" upper="1.47" effort="8" velocity="2.0"/>
-      <dynamics damping="0.3" friction="0.05"/>
+      <dynamics damping="0.005" friction="0.0001"/>
     </joint>
     <link name="${prefix}middle_intermediate">
@@ -302,5 +302,5 @@
       <axis xyz="0 0 -1"/>
       <limit lower="-0.04545" upper="1.56" effort="8" velocity="2.0"/>
-      <dynamics damping="0.3" friction="0.05"/>
+      <dynamics damping="0.002" friction="0.00005"/>
       <mimic joint="${prefix}middle_proximal_joint" multiplier="1.06399" offset="-0.04545"/>
     </joint>
@@ -332,5 +332,5 @@
       <axis xyz="0 0 -1"/>
       <limit lower="0" upper="1.47" effort="8" velocity="2.0"/>
-      <dynamics damping="0.3" friction="0.05"/>
+      <dynamics damping="0.005" friction="0.0001"/>
     </joint>
     <link name="${prefix}ring_intermediate">
@@ -360,5 +360,5 @@
       <axis xyz="0 0 -1"/>
       <limit lower="-0.04545" upper="1.56" effort="8" velocity="2.0"/>
-      <dynamics damping="0.3" friction="0.05"/>
+      <dynamics damping="0.002" friction="0.00005"/>
       <mimic joint="${prefix}ring_proximal_joint" multiplier="1.06399" offset="-0.04545"/>
     </joint>
@@ -390,5 +390,5 @@
       <axis xyz="0 0 -1"/>
       <limit lower="0" upper="1.47" effort="8" velocity="2.0"/>
-      <dynamics damping="0.3" friction="0.05"/>
+      <dynamics damping="0.005" friction="0.0001"/>
     </joint>
     <link name="${prefix}pinky_intermediate">
@@ -418,5 +418,5 @@
       <axis xyz="0 0 -1"/>
       <limit lower="-0.04545" upper="1.56" effort="8" velocity="2.0"/>
-      <dynamics damping="0.3" friction="0.05"/>
+      <dynamics damping="0.002" friction="0.00005"/>
       <mimic joint="${prefix}pinky_proximal_joint" multiplier="1.06399" offset="-0.04545"/>
     </joint>

File: src/robot_description/hand_description/urdf/hands/inspire_hand_right.xacro (robot description, xacro)
@@ -95,5 +95,5 @@
         <axis xyz="0 0 -1"/>
         <limit lower="0.0" upper="1.308" effort="1" velocity="2.0"/>
-        <dynamics damping="0.3" friction="0.05"/>
+        <dynamics damping="0.005" friction="0.0001"/>
       </joint>
       <link name="${prefix}thumb_proximal">
@@ -122,5 +122,5 @@
         <axis xyz="0 0 1"/>
         <limit lower="0" upper="0.6" effort="1" velocity="2.0"/>
-        <dynamics damping="0.3" friction="0.05"/>
+        <dynamics damping="0.005" friction="0.0001"/>
       </joint>
       <link name="${prefix}thumb_intermediate">
@@ -149,5 +149,5 @@
         <axis xyz="0 0 1"/>
         <limit lower="0" upper="0.8" effort="1" velocity="2.0"/>
-        <dynamics damping="0.3" friction="0.05"/>
+        <dynamics damping="0.002" friction="0.00005"/>
         <mimic joint="${prefix}thumb_proximal_pitch_joint" multiplier="1.334" offset="0"/>
       </joint>
@@ -177,5 +177,5 @@
         <axis xyz="0 0 1"/>
         <limit lower="0" upper="0.4" effort="1" velocity="2.0"/>
-        <dynamics damping="0.3" friction="0.05"/>
+        <dynamics damping="0.002" friction="0.00005"/>
         <mimic joint="${prefix}thumb_proximal_pitch_joint" multiplier="0.667" offset="0"/>
       </joint>
@@ -205,5 +205,5 @@
         <axis xyz="0 0 1"/>
         <limit lower="0" upper="1.47" effort="1" velocity="2.0"/>
-        <dynamics damping="0.3" friction="0.05"/>
+        <dynamics damping="0.005" friction="0.0001"/>
       </joint>
       <link name="${prefix}index_intermediate">
@@ -232,5 +232,5 @@
         <axis xyz="0 0 1"/>
         <limit lower="-0.04545" upper="1.56" effort="1" velocity="2.0"/>
-        <dynamics damping="0.3" friction="0.05"/>
+        <dynamics damping="0.002" friction="0.00005"/>
         <mimic joint="${prefix}index_proximal_joint" multiplier="1.06399" offset="-0.04545"/>
       </joint>
@@ -260,5 +260,5 @@
         <axis xyz="0 0 1"/>
         <limit lower="0" upper="1.47" effort="1" velocity="2.0"/>
-        <dynamics damping="0.3" friction="0.05"/>
+        <dynamics damping="0.005" friction="0.0001"/>
       </joint>
       <link name="${prefix}middle_intermediate">
@@ -287,5 +287,5 @@
         <axis xyz="0 0 1"/>
         <limit lower="-0.04545" upper="1.56" effort="1" velocity="2.0"/>
-        <dynamics damping="0.3" friction="0.05"/>
+        <dynamics damping="0.002" friction="0.00005"/>
         <mimic joint="${prefix}middle_proximal_joint" multiplier="1.06399" offset="-0.04545"/>
       </joint>
@@ -315,5 +315,5 @@
         <axis xyz="0 0 1"/>
         <limit lower="0" upper="1.47" effort="1" velocity="2.0"/>
-        <dynamics damping="0.3" friction="0.05"/>
+        <dynamics damping="0.005" friction="0.0001"/>
       </joint>
       <link name="${prefix}ring_intermediate">
@@ -342,5 +342,5 @@
         <axis xyz="0 0 1"/>
         <limit lower="-0.04545" upper="1.56" effort="1" velocity="2.0"/>
-        <dynamics damping="0.3" friction="0.05"/>
+        <dynamics damping="0.002" friction="0.00005"/>
         <mimic joint="${prefix}ring_proximal_joint" multiplier="1.06399" offset="-0.04545"/>
       </joint>
@@ -370,5 +370,5 @@
         <axis xyz="0 0 1"/>
         <limit lower="0" upper="1.47" effort="1" velocity="2.0"/>
-        <dynamics damping="0.3" friction="0.05"/>
+        <dynamics damping="0.005" friction="0.0001"/>
       </joint>
       <link name="${prefix}pinky_intermediate">
@@ -397,5 +397,5 @@
         <axis xyz="0 0 1"/>
         <limit lower="-0.04545" upper="1.56" effort="1" velocity="2.0"/>
-        <dynamics damping="0.3" friction="0.05"/>
+        <dynamics damping="0.002" friction="0.00005"/>
         <mimic joint="${prefix}pinky_proximal_joint" multiplier="1.06399" offset="-0.04545"/>
       </joint>
