Commit message: feat(dual_arm): activate the waist joint across both arm chains
fixed_waist flipped to false, making waist_yaw_joint_X8 revolute. It is the first
joint of both arm chains, so left_arm and right_arm become 7-DOF and share it —
neither arm controller can own it, hence a separate waist_controller. Two URDF
paths needed the change independently: dual_arm.urdf.xacro for Gazebo, and
dual_arm_moveit_config's wrapper, which bypasses it and includes dual_arm_base
directly with its own FakeSystem block.
Fixes #7

File: src/planning/dual_arm_moveit_config/config/dual_arm_description.ros2_control.xacro (robot description, xacro)
@@ -7,4 +7,12 @@
                 <plugin>mock_components/GenericSystem</plugin>
             </hardware>
+            <!-- Waist (first joint of both arm chains) -->
+            <joint name="waist_yaw_joint_X8">
+                <command_interface name="position"/>
+                <state_interface name="position">
+                  <param name="initial_value">${initial_positions['waist_yaw_joint_X8']}</param>
+                </state_interface>
+                <state_interface name="velocity"/>
+            </joint>
             <!-- Left arm -->
             <joint name="left_shoulder_pitch_joint_X6">

File: src/planning/dual_arm_moveit_config/config/dual_arm_description.urdf.xacro (robot description, xacro)
@@ -4,4 +4,7 @@
     <xacro:arg name="initial_positions_file" default="initial_positions.yaml" />
     <xacro:arg name="fixed_legs" default="true" />
+    <!-- Declared before the include so it wins over the default="true" in
+         full_robot_description/urdf/joints/body_joints.xacro. -->
+    <xacro:arg name="fixed_waist" default="false" />
     <xacro:include filename="$(find dual_arm_description)/urdf/dual_arm_base.xacro" />
     <xacro:include filename="dual_arm_description.ros2_control.xacro" />

File: src/robot_description/dual_arm_description/urdf/dual_arm.urdf.xacro (robot description, xacro)
@@ -5,5 +5,5 @@
     <xacro:arg name="use_isaac" default="false" />
     <xacro:arg name="fixed_legs" default="true" />
-    <xacro:arg name="fixed_waist" default="true" />
+    <xacro:arg name="fixed_waist" default="false" />
     <xacro:arg name="only_left" default="false" />
     <xacro:arg name="only_arms" default="false" />

File: src/robot_description/dual_arm_description/urdf/macros/ros2_control.xacro (robot description, xacro)
@@ -7,4 +7,13 @@
                 <plugin>gz_ros2_control/GazeboSimSystem</plugin>
             </hardware>
+            <!-- Waist (shared by both arm chains) -->
+            <joint name="waist_yaw_joint_X8">
+                <command_interface name="position"/>
+                <state_interface name="position">
+                    <param name="initial_value">0.0</param>
+                </state_interface>
+                <state_interface name="velocity"/>
+                <state_interface name="effort"/>
+            </joint>
             <!-- Left arm (6 DOF) -->
             <joint name="left_shoulder_pitch_joint_X6">
